File: dvk-dart-mx8m.sch (KiCad schematic (older format))
At the start: 3 parts

Commit message: Connect power symbols to the respective pins of the SoM
Parts:
- gave numbers to parts that had none: 1
Connections:
- net GND: now reaches J1.A18 (GND)
- net GND: now also J1.A21 (GND), J1.A30 (GND), J1.A33 (GND), J1.A49 (GND), J1.A52 (GND), J1.A55 (GND), J1.A58 (GND), J1.A64 (GND), J1.A67 (GND), J1.A70 (GND), J1.A76 (GND), J1.A85 (GND), J1.B18 (GND), J1.B23 (GND), J1.B47 (GND), J1.B53 (GND), J1.B75 (GND), J1.B84 (GND), J1.C10 (GND), J1.C15 (GND), J1.C21 (GND), J1.C24 (GND), J1.C27 (GND), J1.C33 (GND), J1.C34 (GND), J1.C39 (GND), J1.C45 (GND), J1.C51 (GND), J1.C57 (GND), J1.C63 (GND), J1.C68 (GND), J1.C74 (GND), J1.C9 (GND)
- net GNDA: now reaches J1.B12 (AGND)
- net SOM_VBAT_3V3: now reaches J1.C69 (VBAT_3V3)
- net SOM_VBAT: now reaches J1.C71 (VBAT)
- net SOM_VBAT: now also J1.C73 (VBAT), J1.C75 (VBAT), J1.C77 (VBAT), J1.C79 (VBAT), J1.C81 (VBAT), J1.C83 (VBAT), J1.C85 (VBAT), J1.C87 (VBAT), J1.C89 (VBAT)
- no-connect marks 0 -> 224
Other:
- moved on the sheet: J1A, J1B, J1C

Commit message: Add SGTL5000 audio CODEC and begin schematic around it
Connections:
- net SAI2_RXFS: now reaches J1.B48 (SAI2_RXFS/SAI5_TXFS/////GPIO4_IO21)
- net SAI2_RXC: now reaches J1.B50 (SAI2_RXC/SAI5_TXC/////GPIO4_IO22)
- net SAI2_TXFS: now reaches J1.B52 (SAI2_TXFS/SAI5_TXD1/////GPIO4_IO24)
- net SAI2_MCLK: now reaches J1.B54 (SAI2_MCLK/SAI5_MCLK/////GPIO4_IO27)
- net SAI2_TXC: now reaches J1.B56 (SAI2_TXC/SAI5_TXD2/////GPIO4_IO25)
- net SAI2_RXD: now reaches J1.B58 (SAI2_RXD0/SAI5_TXD0/////GPIO4_IO23)
- net SAI2_TXD: now reaches J1.B60 (SAI2_TXD0/SAI5_TXD3/////GPIO4_IO26)
- no-connect marks 224 -> 217
Changed lines of the file:
@@
 $Descr A2 23386 16535
 encoding utf-8
-Sheet 1 1
+Sheet 1 3
 Title ""
 Date ""
@@
 NoConn ~ 15250 8150
 NoConn ~ 15250 8250
-NoConn ~ 15250 8350
-NoConn ~ 15250 8450
-NoConn ~ 15250 8550
-NoConn ~ 15250 8650
-NoConn ~ 15250 8750
-NoConn ~ 15250 8850
-NoConn ~ 15250 8950
 NoConn ~ 15250 9050
 NoConn ~ 15250 9150
@@
 Wire Wire Line
 	8100 1950 8100 5400
+$Sheet
+S 700  650  500  150
+U 5ABE5061
+F0 "Battery" 60
+F1 "battery.sch" 60
+$EndSheet
+$Sheet
+S 2650 2400 1900 1400
+U 5ABE7AA4
+F0 "Audio" 60
+F1 "audio.sch" 60
+F2 "SAI2_TXFS" I L 2650 2750 60
+F3 "SAI2_TXC" I L 2650 2850 60
+F4 "SAI2_MCLK" I L 2650 2950 60
+F5 "SAI2_RXD" O L 2650 2500 60
+F6 "SAI2_TXD" I L 2650 2600 60
+$EndSheet
+Text Label 15800 8950 2    60   ~ 0
+SAI2_TXD
+Wire Wire Line
+	15800 8950 15250 8950
+Text Label 15800 8850 2    60   ~ 0
+SAI2_RXD
+Wire Wire Line
+	15800 8850 15250 8850
+Text Label 15800 8750 2    60   ~ 0
+SAI2_TXC
+Wire Wire Line
+	15800 8750 15250 8750
+Text Label 15800 8650 2    60   ~ 0
+SAI2_MCLK
+Text Label 15800 8550 2    60   ~ 0
+SAI2_TXFS
+Text Label 15800 8450 2    60   ~ 0
+SAI2_RXC
+Text Label 15800 8350 2    60   ~ 0
+SAI2_RXFS
+Wire Wire Line
+	15800 8350 15250 8350
+Wire Wire Line
+	15800 8450 15250 8450
+Wire Wire Line
+	15800 8550 15250 8550
+Wire Wire Line
+	15800 8650 15250 8650
+Text Label 2100 2600 0    60   ~ 0
+SAI2_TXD
+Wire Wire Line
+	2100 2600 2650 2600
+Text Label 2100 2500 0    60   ~ 0
+SAI2_RXD
+Wire Wire Line
+	2100 2500 2650 2500
+Text Label 2100 2850 0    60   ~ 0
+SAI2_TXC
+Wire Wire Line
+	2100 2850 2650 2850
+Text Label 2100 2950 0    60   ~ 0
+SAI2_MCLK
+Text Label 2100 2750 0    60   ~ 0
+SAI2_TXFS
+Text Label 1100 2500 0    60   ~ 0
+SAI2_RXC
+Text Label 1100 2300 0    60   ~ 0
+SAI2_RXFS
+Wire Wire Line
+	1650 2300 1100 2300
+Wire Wire Line
+	1650 2500 1100 2500
+Wire Wire Line
+	2650 2750 2100 2750
+Wire Wire Line
+	2100 2950 2650 2950
 $EndSCHEMATC

Commit message: Complete the SOM_VBAT regulator circuit, add RTC circuit and 3.3V regulator for BASE_PER_3V3
Passing ERC
Parts:
- added R1, R2: 10k, symbol R
Connections:
- net SOM_SNVS_3V3: now reaches J1.A15 (NVCC_SNVS_3V3)
- net PMIC_ON_REQ: now reaches J1.A22 (PMIC_ON_REQ)
- net PMIC_STBY_REQ: now reaches J1.A26 (PMIC_STBY_REQ)
- net SOM_NVCC_3V3: now reaches J1.A27 (NVCC_3V3)
- net I2C2_SDA: now reaches J1.B30 (I2C2_SDA/ENET1_1588_EVENT1_OUT/////GPIO5_IO17)
- net I2C2_SDA: now also R1.2
- net I2C2_SCL: now reaches J1.B32 (I2C2_SCL/ENET1_1588_EVENT1_IN/////GPIO5_IO16)
- net I2C2_SCL: now also R2.2
- net SAI2_RXC: no longer names the net of J1.B50 (SAI2_RXC/SAI5_TXC/////GPIO4_IO22)
- net SAI2_RXFS: no longer names the net of J1.B48 (SAI2_RXFS/SAI5_TXFS/////GPIO4_IO21)
- new net BASE_PER_3V3: R1.1, R2.1
- no-connect marks 217 -> 213
Other:
- note added: ""Variscite recommends using an\nexternal low power time keeping\ncircuitry which is [more] power\nefficient than the SOC RTC core""
- note added: "=3.0V"
- note added: "TODO!!!"
- note added: "power button!"

Commit message: Update pin types and names based on new DART-MX8M datasheet rev release
Rev 1.03 was just released with a date of Apr 1, 4 days late, pin changes were made on Feb 25th but not released (until now). Seems to more closely resemble the schematic, except for CLK1_* and CLK2_*.
Other:
- note added: "(A23 used to be CLK2_N)\n(A25 used to be CLK2_P)"
- note added: "(A29 used to be CLK1_N)\n(A31 used to be CLK1_P)"
- note added: "?"
- note added: "Internal SOM regulator 3.3V\noutput generated from VBAT\nused to be LICELL"
- note removed: "=3.0V"
Changed lines of the file:
@@
 $EndComp
 Wire Wire Line
-	8100 7150 8100 8350
-Wire Wire Line
-	8100 8350 8100 8650
-Wire Wire Line
-	8100 8650 8100 9750
-Wire Wire Line
-	8100 9750 8100 10500
+	8100 7150 8100 10500
 Wire Wire Line
 	8100 7150 8150 7150
@@
 Connection ~ 8100 9750
 Wire Wire Line
-	15300 1750 15300 2350
-Wire Wire Line
-	15300 2350 15300 3450
-Wire Wire Line
-	15300 3450 15300 3750
-Wire Wire Line
-	15300 3750 15300 4050
-Wire Wire Line
-	15300 4050 15300 4350
-Wire Wire Line
-	15300 4350 15300 4650
-Wire Wire Line
-	15300 4650 15300 5350
-Wire Wire Line
-	15300 5350 15300 5400
+	15300 1750 15300 5400
 Wire Wire Line
 	15300 1750 15250 1750
@@
 $EndComp
 Wire Wire Line
-	15300 6850 15300 10150
-Wire Wire Line
-	15300 10150 15300 10500
+	15300 6850 15300 10500
 Wire Wire Line
 	15300 6850 15250 6850
@@
 	15250 6550 15450 6550
 Wire Wire Line
-	15450 6500 15450 6550
-Wire Wire Line
-	15450 6550 15450 6600
+	15450 6500 15450 6600
 $Comp
 L GND #PWR06
@@
 $EndComp
 Wire Wire Line
-	8100 11550 8100 11850
-Wire Wire Line
-	8100 11850 8100 12150
-Wire Wire Line
-	8100 12150 8100 12450
-Wire Wire Line
-	8100 12450 8100 12750
-Wire Wire Line
-	8100 12750 8100 13050
-Wire Wire Line
-	8100 13050 8100 13350
-Wire Wire Line
-	8100 13350 8100 13650
-Wire Wire Line
-	8100 13650 8100 13950
-Wire Wire Line
-	8100 13950 8100 14250
-Wire Wire Line
-	8100 14250 8100 15600
+	8100 11550 8100 15600
 Wire Wire Line
 	8100 11550 8150 11550
@@
 $EndComp
 Wire Wire Line
-	15300 11550 15300 12250
-Wire Wire Line
-	15300 12250 15300 12750
-Wire Wire Line
-	15300 12750 15300 14450
-Wire Wire Line
-	15300 14450 15300 14750
-Wire Wire Line
-	15300 14750 15300 15600
+	15300 11550 15300 15600
 Wire Wire Line
 	15300 11550 15250 11550
@@
 $EndComp
 Wire Wire Line
-	6700 15550 8050 15550
-Wire Wire Line
-	8050 15550 8150 15550
+	6700 15550 8150 15550
 Wire Wire Line
 	6700 15550 6700 15500
 Wire Wire Line
-	8050 14650 8050 14750
-Wire Wire Line
-	8050 14750 8050 14850
-Wire Wire Line
-	8050 14850 8050 14950
-Wire Wire Line
-	8050 14950 8050 15050
-Wire Wire Line
-	8050 15050 8050 15150
-Wire Wire Line
-	8050 15150 8050 15250
-Wire Wire Line
-	8050 15250 8050 15350
-Wire Wire Line
-	8050 15350 8050 15450
-Wire Wire Line
-	8050 15450 8050 15550
+	8050 14650 8050 15550
 Wire Wire Line
 	8050 14650 8150 14650
@@
 $EndComp
 Wire Wire Line
-	6700 14550 7200 14550
-Wire Wire Line
-	7200 14550 8150 14550
+	6700 14550 8150 14550
 Wire Wire Line
 	6700 14550 6700 14500
 $Comp
 L PWR_FLAG #FLG010
-U 1 1 5ABB63DE
-P 7200 14500
-F 0 "#FLG010" H 7200 14575 50  0001 C CNN
-F 1 "PWR_FLAG" H 7200 14650 50  0000 C CNN
-F 2 "" H 7200 14500 50  0001 C CNN
-F 3 "" H 7200 14500 50  0001 C CNN
-	1    7200 14500
-	1    0    0    -1
-$EndComp
-Wire Wire Line
-	7200 14500 7200 14550
-Connection ~ 7200 14550
-$Comp
-L PWR_FLAG #FLG011
 U 1 1 5ABB67CD
 P 15500 5300
-F 0 "#FLG011" H 15500 5375 50  0001 C CNN
+F 0 "#FLG010" H 15500 5375 50  0001 C CNN
 F 1 "PWR_FLAG" H 15500 5450 50  0000 C CNN
 F 2 "" H 15500 5300 50  0001 C CNN
@@
 NoConn ~ 15250 15550
 $Comp
-L PWR_FLAG #FLG012
+L PWR_FLAG #FLG011
 U 1 1 5ABB7A07
 P 15450 6500
-F 0 "#FLG012" H 15450 6575 50  0001 C CNN
+F 0 "#FLG011" H 15450 6575 50  0001 C CNN
 F 1 "PWR_FLAG" H 15450 6650 50  0000 C CNN
 F 2 "" H 15450 6500 50  0001 C CNN
@@
 Connection ~ 15300 5350
 Wire Wire Line
-	8100 1950 8100 2550
-Wire Wire Line
-	8100 2550 8100 3350
-Wire Wire Line
-	8100 3350 8100 3650
-Wire Wire Line
-	8100 3650 8100 4250
-Wire Wire Line
-	8100 4250 8100 5150
-Wire Wire Line
-	8100 5150 8100 5400
+	8100 1950 8100 5400
 $Sheet
 S 600  600  850  200
@@
 $EndSheet
 $Comp
-L SOM_SNVS_3V3 #PWR013
+L SOM_SNVS_3V3 #PWR012
 U 1 1 5AC52F8D
-P 7400 1600
-F 0 "#PWR013" H 7400 1450 50  0001 C CNN
-F 1 "SOM_SNVS_3V3" H 7400 1740 50  0000 C CNN
-F 2 "" H 7400 1600 50  0001 C CNN
-F 3 "" H 7400 1600 50  0001 C CNN
-	1    7400 1600
-	1    0    0    -1
-$EndComp
-Wire Wire Line
-	8150 1650 7400 1650
-Wire Wire Line
-	7400 1650 7400 1600
+P 7200 1600
+F 0 "#PWR012" H 7200 1450 50  0001 C CNN
+F 1 "SOM_SNVS_3V3" H 7200 1740 50  0000 C CNN
+F 2 "" H 7200 1600 50  0001 C CNN
+F 3 "" H 7200 1600 50  0001 C CNN
+	1    7200 1600
+	1    0    0    -1
+$EndComp
+Wire Wire Line
+	7200 1650 8150 1650
+Wire Wire Line
+	7200 1650 7200 1600
 $Sheet
 S 600  1000 850  300
@@
 F3 "PMIC_STBY_REQ" I R 1450 1200 60
 $EndSheet
-Text Label 7750 14550 0    60   ~ 0
+Text Label 7750 1650 0    60   ~ 0
 LICELL
-Text Label 7550 1650 0    60   ~ 0
-VSNVS
-Text Notes 7850 1650 0    60   ~ 0
-=3.0V
-Text Notes 6450 14950 0    60   ~ 0
+Text Notes 5400 1750 0    60   ~ 0
 "Variscite recommends using an\nexternal low power time keeping\ncircuitry which is [more] power\nefficient than the SOC RTC core"
 Text Label 2200 1600 2    60   ~ 0
@@
 	16200 7550 16200 7400
 $Comp
-L BASE_PER_3V3 #PWR014
+L BASE_PER_3V3 #PWR013
 U 1 1 5AC65102
 P 16000 7000
-F 0 "#PWR014" H 16000 6850 50  0001 C CNN
+F 0 "#PWR013" H 16000 6850 50  0001 C CNN
 F 1 "BASE_PER_3V3" H 16000 7140 50  0000 C CNN
 F 2 "" H 16000 7000 50  0001 C CNN
@@
 	15800 7100 15800 7050
 Wire Wire Line
-	15800 7050 16000 7050
-Wire Wire Line
-	16000 7050 16200 7050
+	15800 7050 16200 7050
 Wire Wire Line
 	16200 7050 16200 7100
@@
 	2200 2550 1450 2550
 $Comp
-L SOM_NVCC_3V3 #PWR015
+L SOM_NVCC_3V3 #PWR014
 U 1 1 5AC989E1
-P 7400 2200
-F 0 "#PWR015" H 7400 2050 50  0001 C CNN
-F 1 "SOM_NVCC_3V3" H 7400 2340 50  0000 C CNN
-F 2 "" H 7400 2200 50  0001 C CNN
-F 3 "" H 7400 2200 50  0001 C CNN
-	1    7400 2200
-	1    0    0    -1
-$EndComp
-Wire Wire Line
-	7400 2200 7400 2250
-Wire Wire Line
-	7400 2250 7900 2250
-Wire Wire Line
-	7900 2250 8150 2250
+P 7200 2200
+F 0 "#PWR014" H 7200 2050 50  0001 C CNN
+F 1 "SOM_NVCC_3V3" H 7200 2340 50  0000 C CNN
+F 2 "" H 7200 2200 50  0001 C CNN
+F 3 "" H 7200 2200 50  0001 C CNN
+	1    7200 2200
+	1    0    0    -1
+$EndComp
+Wire Wire Line
+	7200 2200 7200 2250
+Wire Wire Line
+	7200 2250 8150 2250
+Text Notes 9000 2200 0    60   ~ 0
+(A23 used to be CLK2_N)\n(A25 used to be CLK2_P)
+Text Notes 9400 2500 0    60   ~ 0
+(A29 used to be CLK1_N)\n(A31 used to be CLK1_P)
+Text Notes 8050 1650 0    60   ~ 0
+?
+Text Notes 5100 14550 0    60   ~ 0
+Internal SOM regulator 3.3V\noutput generated from VBAT\nused to be LICELL
 $Comp
 L PWR_FLAG #FLG016
-U 1 1 5AC9915B
-P 7900 2200
-F 0 "#FLG016" H 7900 2275 50  0001 C CNN
-F 1 "PWR_FLAG" H 7900 2350 50  0000 C CNN
-F 2 "" H 7900 2200 50  0001 C CNN
-F 3 "" H 7900 2200 50  0001 C CNN
-	1    7900 2200
-	1    0    0    -1
-$EndComp
-Wire Wire Line
-	7900 2200 7900 2250
-Connection ~ 7900 2250
+U 1 1 5AC73A16
+P 7700 1600
+F 0 "#FLG016" H 7700 1675 50  0001 C CNN
+F 1 "PWR_FLAG" H 7700 1750 50  0000 C CNN
+F 2 "" H 7700 1600 50  0001 C CNN
+F 3 "" H 7700 1600 50  0001 C CNN
+	1    7700 1600
+	1    0    0    -1
+$EndComp
+Wire Wire Line
+	7700 1600 7700 1650
+Connection ~ 7700 1650
 $EndSCHEMATC

Commit message: Add the board ID EEPROM chip and move the 0Ohm resistor such that the coin cell battery would actually power SOM_SNVS_3V3 when removed and the NC resistor is populated
This re-arrengment of the resistor makes the reference schematic more clear knowing that SOM_VBAT_3V3 is not actually LICELL.
Other:
- note added: "Max 100mA"
Changed lines of the file:
@@
 L SOM_VBAT #PWR08
 U 1 1 5ABB586C
-P 6700 15500
-F 0 "#PWR08" H 6700 15350 50  0001 C CNN
-F 1 "SOM_VBAT" H 6700 15640 50  0000 C CNN
-F 2 "" H 6700 15500 50  0001 C CNN
-F 3 "" H 6700 15500 50  0001 C CNN
-	1    6700 15500
-	1    0    0    -1
-$EndComp
-Wire Wire Line
-	6700 15550 8150 15550
-Wire Wire Line
-	6700 15550 6700 15500
+P 7200 15500
+F 0 "#PWR08" H 7200 15350 50  0001 C CNN
+F 1 "SOM_VBAT" H 7200 15640 50  0000 C CNN
+F 2 "" H 7200 15500 50  0001 C CNN
+F 3 "" H 7200 15500 50  0001 C CNN
+	1    7200 15500
+	1    0    0    -1
+$EndComp
+Wire Wire Line
+	7200 15550 8150 15550
+Wire Wire Line
+	7200 15550 7200 15500
 Wire Wire Line
 	8050 14650 8050 15550
@@
 L SOM_VBAT_3V3 #PWR09
 U 1 1 5ABB5FA9
-P 6700 14500
-F 0 "#PWR09" H 6700 14350 50  0001 C CNN
-F 1 "SOM_VBAT_3V3" H 6700 14640 50  0000 C CNN
-F 2 "" H 6700 14500 50  0001 C CNN
-F 3 "" H 6700 14500 50  0001 C CNN
-	1    6700 14500
-	1    0    0    -1
-$EndComp
-Wire Wire Line
-	6700 14550 8150 14550
-Wire Wire Line
-	6700 14550 6700 14500
+P 7200 14500
+F 0 "#PWR09" H 7200 14350 50  0001 C CNN
+F 1 "SOM_VBAT_3V3" H 7200 14640 50  0000 C CNN
+F 2 "" H 7200 14500 50  0001 C CNN
+F 3 "" H 7200 14500 50  0001 C CNN
+	1    7200 14500
+	1    0    0    -1
+$EndComp
+Wire Wire Line
+	7200 14550 8150 14550
+Wire Wire Line
+	7200 14550 7200 14500
 $Comp
 L PWR_FLAG #FLG010
@@
 Text Notes 8050 1650 0    60   ~ 0
 ?
-Text Notes 5100 14550 0    60   ~ 0
+Text Notes 5600 14550 0    60   ~ 0
 Internal SOM regulator 3.3V\noutput generated from VBAT\nused to be LICELL
 $Comp
-L PWR_FLAG #FLG016
+L PWR_FLAG #FLG015
 U 1 1 5AC73A16
 P 7700 1600
-F 0 "#FLG016" H 7700 1675 50  0001 C CNN
+F 0 "#FLG015" H 7700 1675 50  0001 C CNN
 F 1 "PWR_FLAG" H 7700 1750 50  0000 C CNN
 F 2 "" H 7700 1600 50  0001 C CNN
@@
 	7700 1600 7700 1650
 Connection ~ 7700 1650
+Text Notes 7250 2250 0    60   ~ 0
+Max 100mA
+Text Notes 7250 14550 0    60   ~ 0
+Max 100mA
 $EndSCHEMATC
