File: dvk-dart-mx8m.sch (KiCad schematic (older format))
At the start: 3 parts, among them J1 DART-MX8M

Commit message: Add reset & watchdog, sd power, and BASE_PER_1V8 circuits
Connections:
- net POR_B: now reaches J1.A24 (POR_B)
- net ~CONN_SD2_RST: now reaches J1.A28 (SD2_RESET_B/////GPIO2_IO19)
- net NVCC_SD2_1V8_3V3: now reaches J1.A90 (NVCC_SD2_1V8_3V3)
- net GPIO1_IO02(nWDOG): now reaches J1.B28 (GPIO1_IO02/WDOG_B)
- no-connect marks 213 -> 209
Other:
- moved on the sheet: R1, R2
Changed lines of the file:
@@
 $Descr A2 23386 16535
 encoding utf-8
-Sheet 1 5
-Title ""
-Date ""
-Rev ""
-Comp ""
-Comment1 ""
-Comment2 ""
+Sheet 1 6
+Title "DVK-DART-MX8M"
+Date "2018-04-05"
+Rev "v0.1.0"
+Comp "Purism SPC"
+Comment1 "Copyright 2018"
+Comment2 "GNU GPLv3"
 Comment3 ""
 Comment4 ""
@@
 Wire Wire Line
 	7200 14550 7200 14500
-$Comp
-L PWR_FLAG #FLG010
-U 1 1 5ABB67CD
-P 15500 5300
-F 0 "#FLG010" H 15500 5375 50  0001 C CNN
-F 1 "PWR_FLAG" H 15500 5450 50  0000 C CNN
-F 2 "" H 15500 5300 50  0001 C CNN
-F 3 "" H 15500 5300 50  0001 C CNN
-	1    15500 5300
-	1    0    0    -1
-$EndComp
 NoConn ~ 8150 950
 NoConn ~ 8150 1050
@@
 NoConn ~ 15250 1650
 NoConn ~ 15250 1850
-NoConn ~ 15250 2050
-NoConn ~ 15250 2250
 NoConn ~ 15250 2450
 NoConn ~ 15250 2550
@@
 NoConn ~ 15250 5150
 NoConn ~ 15250 5250
-NoConn ~ 15250 5350
 NoConn ~ 8150 6050
 NoConn ~ 8150 6150
@@
 NoConn ~ 15250 7150
 NoConn ~ 15250 7250
-NoConn ~ 15250 7350
 NoConn ~ 15250 7650
 NoConn ~ 15250 7750
@@
 NoConn ~ 15250 15550
 $Comp
-L PWR_FLAG #FLG011
+L PWR_FLAG #FLG010
 U 1 1 5ABB7A07
 P 15450 6500
-F 0 "#FLG011" H 15450 6575 50  0001 C CNN
+F 0 "#FLG010" H 15450 6575 50  0001 C CNN
 F 1 "PWR_FLAG" H 15450 6650 50  0000 C CNN
 F 2 "" H 15450 6500 50  0001 C CNN
@@
 Connection ~ 15450 6550
 Wire Wire Line
-	15300 5350 15500 5350
-Wire Wire Line
-	15500 5350 15500 5300
-Connection ~ 15300 5350
-Wire Wire Line
 	8100 1950 8100 5400
 $Sheet
-S 600  600  850  200
+S 600  600  1050 200
 U 5ABE5061
 F0 "Battery" 60
 F1 "battery.sch" 60
-F2 "PWR_SAVE" I R 1450 700 60
+F2 "PWR_SAVE" I R 1650 700 60
 $EndSheet
 $Comp
-L SOM_SNVS_3V3 #PWR012
+L SOM_SNVS_3V3 #PWR011
 U 1 1 5AC52F8D
 P 7200 1600
-F 0 "#PWR012" H 7200 1450 50  0001 C CNN
+F 0 "#PWR011" H 7200 1450 50  0001 C CNN
 F 1 "SOM_SNVS_3V3" H 7200 1740 50  0000 C CNN
 F 2 "" H 7200 1600 50  0001 C CNN
@@
 	7200 1650 7200 1600
 $Sheet
-S 600  1000 850  300
+S 600  1000 1050 450
 U 5AC540E7
 F0 "Power" 60
 F1 "power.sch" 60
-F2 "PMIC_ON_REQ" I R 1450 1100 60
-F3 "PMIC_STBY_REQ" I R 1450 1200 60
+F2 "PMIC_ON_REQ" I R 1650 1100 60
+F3 "PMIC_STBY_REQ" I R 1650 1200 60
+F4 "~CONN_SD2_RST" I R 1650 1350 60
 $EndSheet
 Text Label 7750 1650 0    60   ~ 0
@@
 Text Notes 5400 1750 0    60   ~ 0
 "Variscite recommends using an\nexternal low power time keeping\ncircuitry which is [more] power\nefficient than the SOC RTC core"
-Text Label 2200 1600 2    60   ~ 0
+Text Label 2600 1750 2    60   ~ 0
 I2C2_SDA
-Text Label 2200 1700 2    60   ~ 0
+Text Label 2600 1850 2    60   ~ 0
 I2C2_SCL
 Wire Wire Line
-	1450 1600 2200 1600
-Wire Wire Line
-	1450 1700 2200 1700
-Wire Wire Line
-	15250 7450 15800 7450
-Wire Wire Line
-	15250 7550 16200 7550
-Text Label 15750 7450 2    60   ~ 0
+	1650 1750 2600 1750
+Wire Wire Line
+	1650 1850 2600 1850
+Wire Wire Line
+	15250 7450 16350 7450
+Wire Wire Line
+	15250 7550 16650 7550
+Text Label 16250 7450 2    60   ~ 0
 I2C2_SDA
-Text Label 15750 7550 2    60   ~ 0
+Text Label 16250 7550 2    60   ~ 0
 I2C2_SCL
 $Sheet
-S 600  1500 850  300
+S 600  1650 1050 300
 U 5AC56093
 F0 "RTC Battery" 60
 F1 "rtc.sch" 60
-F2 "I2C2_SDA" B R 1450 1600 60
-F3 "I2C2_SCL" I R 1450 1700 60
+F2 "I2C2_SDA" B R 1650 1750 60
+F3 "I2C2_SCL" I R 1650 1850 60
 $EndSheet
 $Comp
 L R R1
 U 1 1 5AC64F34
-P 15800 7250
-F 0 "R1" H 15900 7300 50  0000 C CNN
-F 1 "10k" H 15925 7200 50  0000 C CNN
-F 2 "" V 15730 7250 50  0001 C CNN
-F 3 "" H 15800 7250 50  0001 C CNN
-	1    15800 7250
+P 16350 7250
+F 0 "R1" H 16450 7300 50  0000 C CNN
+F 1 "10k" H 16475 7200 50  0000 C CNN
+F 2 "" V 16280 7250 50  0001 C CNN
+F 3 "" H 16350 7250 50  0001 C CNN
+	1    16350 7250
 	1    0    0    -1
 $EndComp
@@
 L R R2
 U 1 1 5AC64F91
-P 16200 7250
-F 0 "R2" H 16300 7300 50  0000 C CNN
-F 1 "10k" H 16325 7200 50  0000 C CNN
-F 2 "" V 16130 7250 50  0001 C CNN
-F 3 "" H 16200 7250 50  0001 C CNN
-	1    16200 7250
-	1    0    0    -1
-$EndComp
-Wire Wire Line
-	15800 7450 15800 7400
-Wire Wire Line
-	16200 7550 16200 7400
-$Comp
-L BASE_PER_3V3 #PWR013
+P 16650 7250
+F 0 "R2" H 16750 7300 50  0000 C CNN
+F 1 "10k" H 16775 7200 50  0000 C CNN
+F 2 "" V 16580 7250 50  0001 C CNN
+F 3 "" H 16650 7250 50  0001 C CNN
+	1    16650 7250
+	1    0    0    -1
+$EndComp
+Wire Wire Line
+	16350 7450 16350 7400
+Wire Wire Line
+	16650 7550 16650 7400
+$Comp
+L BASE_PER_3V3 #PWR012
 U 1 1 5AC65102
-P 16000 7000
-F 0 "#PWR013" H 16000 6850 50  0001 C CNN
-F 1 "BASE_PER_3V3" H 16000 7140 50  0000 C CNN
-F 2 "" H 16000 7000 50  0001 C CNN
-F 3 "" H 16000 7000 50  0001 C CNN
-	1    16000 7000
-	1    0    0    -1
-$EndComp
-Wire Wire Line
-	15800 7100 15800 7050
-Wire Wire Line
-	15800 7050 16200 7050
-Wire Wire Line
-	16200 7050 16200 7100
-Wire Wire Line
-	16000 7050 16000 7000
-Connection ~ 16000 7050
-Text Notes 15400 2050 0    60   ~ 0
+P 16500 7000
+F 0 "#PWR012" H 16500 6850 50  0001 C CNN
+F 1 "BASE_PER_3V3" H 16500 7140 50  0000 C CNN
+F 2 "" H 16500 7000 50  0001 C CNN
+F 3 "" H 16500 7000 50  0001 C CNN
+	1    16500 7000
+	1    0    0    -1
+$EndComp
+Wire Wire Line
+	16350 7100 16350 7050
+Wire Wire Line
+	16350 7050 16650 7050
+Wire Wire Line
+	16650 7050 16650 7100
+Wire Wire Line
+	16500 7050 16500 7000
+Connection ~ 16500 7050
+Text Notes 16050 2050 0    60   ~ 0
 power button!
 NoConn ~ 15250 8350
 NoConn ~ 15250 8450
 Wire Wire Line
-	1450 700  2200 700
-Text Label 2200 700  2    60   ~ 0
+	1650 700  2600 700
+Text Label 2600 700  2    60   ~ 0
 PWR_SAVE
-Text Notes 1850 600  0    60   ~ 0
+Text Notes 2250 600  0    60   ~ 0
 TODO!!!
-Text Label 2200 1100 2    60   ~ 0
+Text Label 2600 1100 2    60   ~ 0
 PMIC_ON_REQ
-Text Label 2200 1200 2    60   ~ 0
+Text Label 2600 1200 2    60   ~ 0
 PMIC_STBY_REQ
 Wire Wire Line
-	2200 1100 1450 1100
-Wire Wire Line
-	2200 1200 1450 1200
+	2600 1100 1650 1100
+Wire Wire Line
+	2600 1200 1650 1200
 Wire Wire Line
 	15250 1950 16000 1950
@@
 PMIC_STBY_REQ
 $Sheet
-S 600  2000 850  650
+S 600  2150 1050 650
 U 5ABE7AA4
 F0 "Audio" 60
 F1 "audio.sch" 60
-F2 "SAI2_TXFS" I R 1450 2350 60
-F3 "SAI2_TXC" I R 1450 2450 60
-F4 "SAI2_MCLK" I R 1450 2550 60
-F5 "SAI2_RXD" O R 1450 2100 60
-F6 "SAI2_TXD" I R 1450 2200 60
+F2 "SAI2_TXFS" I R 1650 2500 60
+F3 "SAI2_TXC" I R 1650 2600 60
+F4 "SAI2_MCLK" I R 1650 2700 60
+F5 "SAI2_RXD" O R 1650 2250 60
+F6 "SAI2_TXD" I R 1650 2350 60
 $EndSheet
 Text Label 15800 8950 2    60   ~ 0
@@
 Wire Wire Line
 	15800 8650 15250 8650
-Text Label 2200 2200 2    60   ~ 0
+Text Label 2600 2350 2    60   ~ 0
 SAI2_TXD
 Wire Wire Line
-	2200 2200 1450 2200
-Text Label 2200 2100 2    60   ~ 0
+	2600 2350 1650 2350
+Text Label 2600 2250 2    60   ~ 0
 SAI2_RXD
 Wire Wire Line
-	2200 2100 1450 2100
-Text Label 2200 2450 2    60   ~ 0
+	2600 2250 1650 2250
+Text Label 2600 2600 2    60   ~ 0
 SAI2_TXC
 Wire Wire Line
-	2200 2450 1450 2450
-Text Label 2200 2550 2    60   ~ 0
+	2600 2600 1650 2600
+Text Label 2600 2700 2    60   ~ 0
 SAI2_MCLK
-Text Label 2200 2350 2    60   ~ 0
+Text Label 2600 2500 2    60   ~ 0
 SAI2_TXFS
 Wire Wire Line
-	1450 2350 2200 2350
-Wire Wire Line
-	2200 2550 1450 2550
-$Comp
-L SOM_NVCC_3V3 #PWR014
+	1650 2500 2600 2500
+Wire Wire Line
+	2600 2700 1650 2700
+$Comp
+L SOM_NVCC_3V3 #PWR013
 U 1 1 5AC989E1
 P 7200 2200
-F 0 "#PWR014" H 7200 2050 50  0001 C CNN
+F 0 "#PWR013" H 7200 2050 50  0001 C CNN
 F 1 "SOM_NVCC_3V3" H 7200 2340 50  0000 C CNN
 F 2 "" H 7200 2200 50  0001 C CNN
@@
 Internal SOM regulator 3.3V\noutput generated from VBAT\nused to be LICELL
 $Comp
-L PWR_FLAG #FLG015
+L PWR_FLAG #FLG014
 U 1 1 5AC73A16
 P 7700 1600
-F 0 "#FLG015" H 7700 1675 50  0001 C CNN
+F 0 "#FLG014" H 7700 1675 50  0001 C CNN
 F 1 "PWR_FLAG" H 7700 1750 50  0000 C CNN
 F 2 "" H 7700 1600 50  0001 C CNN
@@
 Text Notes 7250 14550 0    60   ~ 0
 Max 100mA
+$Sheet
+S 600  3000 1050 450
+U 5AC89E64
+F0 "Reset & Watchdog" 60
+F1 "watchdog.sch" 60
+F2 "GPIO1_IO02(nWDOG)" I R 1650 3100 60
+F3 "POR_B" O R 1650 3250 60
+F4 "PMIC_ON_REQ" O R 1650 3350 60
+$EndSheet
+Wire Wire Line
+	1650 3100 2600 3100
+Wire Wire Line
+	1650 3250 2600 3250
+Wire Wire Line
+	1650 3350 2600 3350
+Text Label 2600 3100 2    60   ~ 0
+GPIO1_IO02(nWDOG)
+Text Label 2600 3250 2    60   ~ 0
+POR_B
+Text Label 2600 3350 2    60   ~ 0
+PMIC_ON_REQ
+Text Label 16250 7350 2    60   ~ 0
+GPIO1_IO02(nWDOG)
+Wire Wire Line
+	15250 7350 16250 7350
+Text Label 16000 2050 2    60   ~ 0
+POR_B
+Wire Wire Line
+	15250 2050 16000 2050
+$Comp
+L NVCC_SD2_1V8_3V3 #PWR015
+U 1 1 5ACBD5F9
+P 16050 5200
+F 0 "#PWR015" H 16050 5050 50  0001 C CNN
+F 1 "NVCC_SD2_1V8_3V3" H 16050 5340 50  0000 C CNN
+F 2 "" H 16050 5200 50  0001 C CNN
+F 3 "" H 16050 5200 50  0001 C CNN
+	1    16050 5200
+	1    0    0    -1
+$EndComp
+Wire Wire Line
+	15250 5350 16050 5350
+Wire Wire Line
+	16050 5350 16050 5200
+Wire Wire Line
+	1650 1350 2600 1350
+Text Label 2600 1350 2    60   ~ 0
+~CONN_SD2_RST
+Text Label 16000 2250 2    60   ~ 0
+~CONN_SD2_RST
+Wire Wire Line
+	15250 2250 16000 2250
 $EndSCHEMATC

Commit message: Add PTC Fuse, zener on VCC_PJ, USB PD current-limiting switch, 5V regulator, and make regulators' VINA=VIN (since VIH is 1.2V)
Equation for setting NX5P3090's current limit is included.
Connections:
- net GPIO1_IO02(nWDOG) renamed GPIO1_IO02(~WDOG~)
Other:
- note removed: "TODO!!!"
Changed lines of the file:
@@
 $Descr A2 23386 16535
 encoding utf-8
-Sheet 1 6
+Sheet 1 7
 Title "DVK-DART-MX8M"
 Date "2018-04-05"
@@
 Wire Wire Line
 	1650 700  2600 700
-Text Label 2600 700  2    60   ~ 0
-PWR_SAVE
-Text Notes 2250 600  0    60   ~ 0
-TODO!!!
 Text Label 2600 1100 2    60   ~ 0
 PMIC_ON_REQ
@@
 Text Notes 7250 14550 0    60   ~ 0
 Max 100mA
-$Sheet
-S 600  3000 1050 450
-U 5AC89E64
-F0 "Reset & Watchdog" 60
-F1 "watchdog.sch" 60
-F2 "GPIO1_IO02(nWDOG)" I R 1650 3100 60
-F3 "POR_B" O R 1650 3250 60
-F4 "PMIC_ON_REQ" O R 1650 3350 60
-$EndSheet
 Wire Wire Line
 	1650 3100 2600 3100
@@
 	1650 3350 2600 3350
 Text Label 2600 3100 2    60   ~ 0
-GPIO1_IO02(nWDOG)
+GPIO1_IO02(~WDOG~)
 Text Label 2600 3250 2    60   ~ 0
 POR_B
@@
 PMIC_ON_REQ
 Text Label 16250 7350 2    60   ~ 0
-GPIO1_IO02(nWDOG)
+GPIO1_IO02(~WDOG~)
 Wire Wire Line
 	15250 7350 16250 7350
@@
 Wire Wire Line
 	15250 2250 16000 2250
+Text Label 2600 700  2    60   ~ 0
+PMIC_STBY_REQ
+$Sheet
+S 600  3000 1050 450
+U 5AC89E64
+F0 "Reset & Watchdog" 60
+F1 "watchdog.sch" 60
+F2 "POR_B" O R 1650 3250 60
+F3 "PMIC_ON_REQ" O R 1650 3350 60
+F4 "GPIO1_IO02(~WDOG~)" I R 1650 3100 60
+$EndSheet
+$Sheet
+S 600  3650 1050 150
+U 5ACF2B88
+F0 "USB" 60
+F1 "usb.sch" 60
+$EndSheet
 $EndSCHEMATC
