File: dvk-dart-mx8m.sch (KiCad schematic (older format))
At the start: 6 parts, among them J1 DART-MX8M

Commit message: Add JTAG and buttons & LED schematics, reorder based on priority (especially for debugging/development)
Connections:
- net ONOFF: now reaches J1.A20 (ONOFF)
- net JTAG_TCK: now reaches J1.B1 (JTAG_TCK)
- net JTAG_TMS: now reaches J1.B3 (JTAG_TMS)
- net JTAG_~TRST: now reaches J1.B5 (JTAG_TRST_B)
- net JTAG_TDI: now reaches J1.B7 (JTAG_TDI)
- net JTAG_TDO: now reaches J1.B9 (JTAG_TDO)
- no-connect marks 182 -> 176
Other:
- note removed: "power button!"

Commit message: Add MIPI DSI, cap touch interface, and AMOLED display regulator circuits
TPS65632's components were selected based on the best match and price based on suggestions. The RT4720 does not seem to be sold by any distributors.
Connections:
- net DSI_TX0_P: now reaches J1.C12 (DSI_TX0_P/*/LVDS2_TX0_P)
- net DSI_TX0_N: now reaches J1.C14 (DSI_TX0_N/*/LVDS2_TX0_N)
- net DSI_TX1_P: now reaches J1.C16 (DSI_TX1_P/*/LVDS2_TX1_P)
- net DSI_TX1_N: now reaches J1.C18 (DSI_TX1_N/*/LVDS2_TX1_N)
- net DSI_TX3_P: now reaches J1.C20 (DSI_TX3_P/*/LVDS2_TX3_P)
- net DSI_TX3_N: now reaches J1.C22 (DSI_TX3_N/*/LVDS2_TX3_N)
- net DSI_TX2_P: now reaches J1.C23 (DSI_TX2_P/*/LVDS2_CLK_P)
- net DSI_TX2_N: now reaches J1.C25 (DSI_TX2_N/*/LVDS2_CLK_N)
- net DSI_CLK_N: now reaches J1.C29 (DSI_CLK_N/*/LVDS2_TX2_N)
- net DSI_CLK_P: now reaches J1.C31 (DSI_CLK_P/*/LVDS2_TX2_P)
- net CAPTOUCH_~INT: now reaches J1.C48 (GPIO1_IO14/USB2_OTG_PWR/////PWM3_OUT)
- net DSI_BL_PWM: now reaches J1.C64 (GPIO1_IO01/PWM1_OUT/////REF_CLK_24M//////EXT_CLK2)
- no-connect marks 176 -> 164

Commit message: Add 3.0V LDO for display's VCI and TP_VCC, include a 3~12ms rise time delay for the 1.8V rail to turn on before the 3.0V rail, begin the WWAN M.2 schematic (found a a low-profile key B connector)
Changed lines of the file:
@@
 $Descr A2 23386 16535
 encoding utf-8
-Sheet 1 13
+Sheet 1 14
 Title "DVK-DART-MX8M"
-Date "2018-04-09"
+Date "2018-04-10"
 Rev "v0.1.0"
 Comp "Purism SPC"
@@
 I2C2_SCL
 $Sheet
-S 550  1900 1350 1950
+S 550  1900 1400 1950
 U 5ACBD81C
 F0 "Boot Config" 60
 F1 "boot.sch" 60
-F2 "BOOT_CFG00" O R 1900 2000 60
-F3 "BOOT_CFG01" O R 1900 2100 60
-F4 "BOOT_CFG02" O R 1900 2200 60
-F5 "BOOT_CFG03" O R 1900 2300 60
-F6 "BOOT_CFG04" O R 1900 2400 60
-F7 "BOOT_CFG05" O R 1900 2500 60
-F8 "BOOT_CFG06" O R 1900 2600 60
-F9 "BOOT_CFG07" O R 1900 2700 60
-F10 "BOOT_CFG08" O R 1900 2800 60
-F11 "BOOT_CFG09" O R 1900 2900 60
-F12 "BOOT_CFG10" O R 1900 3000 60
-F13 "BOOT_CFG11" O R 1900 3100 60
-F14 "BOOT_CFG12" O R 1900 3200 60
-F15 "BOOT_CFG13" O R 1900 3300 60
-F16 "BOOT_CFG14" O R 1900 3400 60
-F17 "BOOT_CFG15" O R 1900 3500 60
-F18 "BOOT_MODE0" O R 1900 3650 60
-F19 "BOOT_MODE1" O R 1900 3750 60
+F2 "BOOT_CFG00" O R 1950 2000 60
+F3 "BOOT_CFG01" O R 1950 2100 60
+F4 "BOOT_CFG02" O R 1950 2200 60
+F5 "BOOT_CFG03" O R 1950 2300 60
+F6 "BOOT_CFG04" O R 1950 2400 60
+F7 "BOOT_CFG05" O R 1950 2500 60
+F8 "BOOT_CFG06" O R 1950 2600 60
+F9 "BOOT_CFG07" O R 1950 2700 60
+F10 "BOOT_CFG08" O R 1950 2800 60
+F11 "BOOT_CFG09" O R 1950 2900 60
+F12 "BOOT_CFG10" O R 1950 3000 60
+F13 "BOOT_CFG11" O R 1950 3100 60
+F14 "BOOT_CFG12" O R 1950 3200 60
+F15 "BOOT_CFG13" O R 1950 3300 60
+F16 "BOOT_CFG14" O R 1950 3400 60
+F17 "BOOT_CFG15" O R 1950 3500 60
+F18 "BOOT_MODE0" O R 1950 3650 60
+F19 "BOOT_MODE1" O R 1950 3750 60
 $EndSheet
 $Comp
@@
 $EndSheet
 $Sheet
-S 550  5200 1350 300
+S 550  5200 1400 300
 U 5ACD5BC1
 F0 "UART Debug" 60
 F1 "uart.sch" 60
-F2 "UART1_TXD" I R 1900 5300 60
-F3 "UART1_RXD" O R 1900 5400 60
+F2 "UART1_TXD" I R 1950 5300 60
+F3 "UART1_RXD" O R 1950 5400 60
 $EndSheet
 $Sheet
@@
 $EndSheet
 $Sheet
-S 550  6600 1350 800
+S 550  6600 1400 800
 U 5AC9B567
 F0 "uSD Card" 60
 F1 "sd.sch" 60
-F2 "CONN_SD2_DATA1" B R 1900 6700 60
-F3 "CONN_SD2_DATA0" B R 1900 6800 60
-F4 "CONN_SD2_CMD" I R 1900 6900 60
-F5 "CONN_SD2_DATA3" B R 1900 7000 60
-F6 "CONN_SD2_DATA2" B R 1900 7100 60
-F7 "CONN_SD2_CLK" I R 1900 7200 60
-F8 "CONN_SD2_CD_B" O R 1900 7300 60
+F2 "CONN_SD2_DATA1" B R 1950 6700 60
+F3 "CONN_SD2_DATA0" B R 1950 6800 60
+F4 "CONN_SD2_CMD" I R 1950 6900 60
+F5 "CONN_SD2_DATA3" B R 1950 7000 60
+F6 "CONN_SD2_DATA2" B R 1950 7100 60
+F7 "CONN_SD2_CLK" I R 1950 7200 60
+F8 "CONN_SD2_CD_B" O R 1950 7300 60
 $EndSheet
 $Sheet
@@
 $EndSheet
 $Sheet
-S 550  11150 1400 650
+S 550  11500 1400 650
 U 5ABE7AA4
 F0 "Audio" 60
 F1 "audio.sch" 60
-F2 "SAI2_TXFS" I R 1950 11500 60
-F3 "SAI2_TXC" I R 1950 11600 60
-F4 "SAI2_MCLK" I R 1950 11700 60
-F5 "SAI2_RXD" O R 1950 11250 60
-F6 "SAI2_TXD" I R 1950 11350 60
+F2 "SAI2_TXFS" I R 1950 11850 60
+F3 "SAI2_TXC" I R 1950 11950 60
+F4 "SAI2_MCLK" I R 1950 12050 60
+F5 "SAI2_RXD" O R 1950 11600 60
+F6 "SAI2_TXD" I R 1950 11700 60
 $EndSheet
 Text Label 16400 8950 2    60   ~ 0
@@
 Text Label 16400 8550 2    60   ~ 0
 SAI2_TXFS
-Text Label 3200 11350 2    60   ~ 0
+Text Label 3200 11700 2    60   ~ 0
 SAI2_TXD
-Text Label 3200 11250 2    60   ~ 0
+Text Label 3200 11600 2    60   ~ 0
 SAI2_RXD
-Text Label 3200 11600 2    60   ~ 0
+Text Label 3200 11950 2    60   ~ 0
 SAI2_TXC
-Text Label 3200 11700 2    60   ~ 0
+Text Label 3200 12050 2    60   ~ 0
 SAI2_MCLK
-Text Label 3200 11500 2    60   ~ 0
+Text Label 3200 11850 2    60   ~ 0
 SAI2_TXFS
 $Comp
@@
 Text Label 3200 7800 2    60   ~ 0
 USB1_ID
-Text Label 3200 6700 2    60   ~ 0
+Text Label 3250 6700 2    60   ~ 0
 CONN_SD2_DATA1
-Text Label 3200 6800 2    60   ~ 0
+Text Label 3250 6800 2    60   ~ 0
 CONN_SD2_DATA0
-Text Label 3200 6900 2    60   ~ 0
+Text Label 3250 6900 2    60   ~ 0
 CONN_SD2_CMD
-Text Label 3200 7000 2    60   ~ 0
+Text Label 3250 7000 2    60   ~ 0
 CONN_SD2_DATA3
-Text Label 3200 7100 2    60   ~ 0
+Text Label 3250 7100 2    60   ~ 0
 CONN_SD2_DATA2
-Text Label 3200 7200 2    60   ~ 0
+Text Label 3250 7200 2    60   ~ 0
 CONN_SD2_CLK
-Text Label 3200 7300 2    60   ~ 0
+Text Label 3250 7300 2    60   ~ 0
 CONN_SD2_CD_B
 Text Label 16400 4850 2    60   ~ 0
@@
 	16400 8650 15250 8650
 Wire Wire Line
-	3200 11350 1950 11350
-Wire Wire Line
-	3200 11250 1950 11250
+	3200 11700 1950 11700
 Wire Wire Line
 	3200 11600 1950 11600
 Wire Wire Line
-	1950 11500 3200 11500
-Wire Wire Line
-	3200 11700 1950 11700
+	3200 11950 1950 11950
+Wire Wire Line
+	1950 11850 3200 11850
+Wire Wire Line
+	3200 12050 1950 12050
 Wire Wire Line
 	7200 2200 7200 2250
@@
 	1950 7800 3200 7800
 Wire Wire Line
-	1900 6700 3200 6700
-Wire Wire Line
-	1900 6800 3200 6800
-Wire Wire Line
-	1900 6900 3200 6900
-Wire Wire Line
-	1900 7000 3200 7000
-Wire Wire Line
-	1900 7100 3200 7100
-Wire Wire Line
-	1900 7200 3200 7200
-Wire Wire Line
-	1900 7300 3200 7300
+	1950 6700 3250 6700
+Wire Wire Line
+	1950 6800 3250 6800
+Wire Wire Line
+	1950 6900 3250 6900
+Wire Wire Line
+	1950 7000 3250 7000
+Wire Wire Line
+	1950 7100 3250 7100
+Wire Wire Line
+	1950 7200 3250 7200
+Wire Wire Line
+	1950 7300 3250 7300
 Wire Wire Line
 	15250 4850 16400 4850
@@
 	15250 10450 16400 10450
 Wire Wire Line
-	1900 5300 3200 5300
-Wire Wire Line
-	1900 5400 3200 5400
-Wire Wire Line
-	1900 2000 3200 2000
-Wire Wire Line
-	1900 2100 3200 2100
-Wire Wire Line
-	1900 2200 3200 2200
-Wire Wire Line
-	1900 2300 3200 2300
-Wire Wire Line
-	1900 2400 3200 2400
-Wire Wire Line
-	1900 2500 3200 2500
-Wire Wire Line
-	1900 2600 3200 2600
-Wire Wire Line
-	1900 2700 3200 2700
-Wire Wire Line
-	1900 2800 3200 2800
-Wire Wire Line
-	1900 2900 3200 2900
-Wire Wire Line
-	1900 3000 3200 3000
-Wire Wire Line
-	1900 3100 3200 3100
-Wire Wire Line
-	1900 3200 3200 3200
-Wire Wire Line
-	1900 3300 3200 3300
-Wire Wire Line
-	1900 3400 3200 3400
-Wire Wire Line
-	1900 3500 3200 3500
+	1950 5300 3200 5300
+Wire Wire Line
+	1950 5400 3200 5400
+Wire Wire Line
+	1950 2000 3200 2000
+Wire Wire Line
+	1950 2100 3200 2100
+Wire Wire Line
+	1950 2200 3200 2200
+Wire Wire Line
+	1950 2300 3200 2300
+Wire Wire Line
+	1950 2400 3200 2400
+Wire Wire Line
+	1950 2500 3200 2500
+Wire Wire Line
+	1950 2600 3200 2600
+Wire Wire Line
+	1950 2700 3200 2700
+Wire Wire Line
+	1950 2800 3200 2800
+Wire Wire Line
+	1950 2900 3200 2900
+Wire Wire Line
+	1950 3000 3200 3000
+Wire Wire Line
+	1950 3100 3200 3100
+Wire Wire Line
+	1950 3200 3200 3200
+Wire Wire Line
+	1950 3300 3200 3300
+Wire Wire Line
+	1950 3400 3200 3400
+Wire Wire Line
+	1950 3500 3200 3500
 Wire Wire Line
 	15250 9050 16400 9050
@@
 	8150 9650 7000 9650
 Wire Wire Line
-	1900 3650 3200 3650
-Wire Wire Line
-	1900 3750 3200 3750
+	1950 3650 3200 3650
+Wire Wire Line
+	1950 3750 3200 3750
 Wire Wire Line
 	8150 6550 7000 6550
@@
 Wire Wire Line
 	15250 13450 16400 13450
+$Sheet
+S 550  11150 1400 150
+U 5ACD5EDE
+F0 "WWAN M.2" 60
+F1 "wwan_m2.sch" 60
+$EndSheet
 $EndSCHEMATC

Commit message: Route SIM card slot to M.2, add SIM2 slot, use null modem for the optional UART interface for modules such as the SIM7100 (no DCD, DTS, DTR, CTS)
Other:
- note added: "TODO!!!"
Changed lines of the file:
@@
 $EndSheet
 $Sheet
-S 550  11500 1400 650
+S 550  11550 1400 650
 U 5ABE7AA4
 F0 "Audio" 60
 F1 "audio.sch" 60
-F2 "SAI2_TXFS" I R 1950 11850 60
-F3 "SAI2_TXC" I R 1950 11950 60
-F4 "SAI2_MCLK" I R 1950 12050 60
-F5 "SAI2_RXD" O R 1950 11600 60
-F6 "SAI2_TXD" I R 1950 11700 60
+F2 "SAI2_TXFS" I R 1950 11900 60
+F3 "SAI2_TXC" I R 1950 12000 60
+F4 "SAI2_MCLK" I R 1950 12100 60
+F5 "SAI2_RXD" O R 1950 11650 60
+F6 "SAI2_TXD" I R 1950 11750 60
 $EndSheet
 Text Label 16400 8950 2    60   ~ 0
@@
 Text Label 16400 8550 2    60   ~ 0
 SAI2_TXFS
-Text Label 3200 11700 2    60   ~ 0
+Text Label 3200 11750 2    60   ~ 0
 SAI2_TXD
-Text Label 3200 11600 2    60   ~ 0
+Text Label 3200 11650 2    60   ~ 0
 SAI2_RXD
-Text Label 3200 11950 2    60   ~ 0
+Text Label 3200 12000 2    60   ~ 0
 SAI2_TXC
-Text Label 3200 12050 2    60   ~ 0
+Text Label 3200 12100 2    60   ~ 0
 SAI2_MCLK
-Text Label 3200 11850 2    60   ~ 0
+Text Label 3200 11900 2    60   ~ 0
 SAI2_TXFS
 $Comp
@@
 	16400 8650 15250 8650
 Wire Wire Line
-	3200 11700 1950 11700
-Wire Wire Line
-	3200 11600 1950 11600
-Wire Wire Line
-	3200 11950 1950 11950
-Wire Wire Line
-	1950 11850 3200 11850
-Wire Wire Line
-	3200 12050 1950 12050
+	3200 11750 1950 11750
+Wire Wire Line
+	3200 11650 1950 11650
+Wire Wire Line
+	3200 12000 1950 12000
+Wire Wire Line
+	1950 11900 3200 11900
+Wire Wire Line
+	3200 12100 1950 12100
 Wire Wire Line
 	7200 2200 7200 2250
@@
 	15250 13450 16400 13450
 $Sheet
-S 550  11150 1400 150
+S 550  11150 1400 200
 U 5ACD5EDE
 F0 "WWAN M.2" 60
 F1 "wwan_m2.sch" 60
+F2 "CONFIG" O R 1950 11250 60
 $EndSheet
+Wire Wire Line
+	1950 11250 3200 11250
+Text Label 3200 11250 2    60   ~ 0
+WWAN_CONFIG
+Text Notes 3250 11250 0    60   ~ 0
+TODO!!!
 $EndSCHEMATC

Commit message: Include HKS for baseband modem M.2 module
Low-pass filter included for switch ckt, rise and fall time should be nearly identical with the presence of a schottky diode. Since the M.2 spec calls out a >20Kohm resistor to GND on the ~FULL_CARD_POWER_OFF pin then then a voltage divider is formed between this resistor and the one to VBAT (min of ~2.2V, actually >2.4V).
Changed lines of the file:
@@
 $EndSheet
 $Sheet
-S 550  11550 1400 650
+S 550  12050 1400 650
 U 5ABE7AA4
 F0 "Audio" 60
 F1 "audio.sch" 60
-F2 "SAI2_TXFS" I R 1950 11900 60
-F3 "SAI2_TXC" I R 1950 12000 60
-F4 "SAI2_MCLK" I R 1950 12100 60
-F5 "SAI2_RXD" O R 1950 11650 60
-F6 "SAI2_TXD" I R 1950 11750 60
+F2 "SAI2_TXFS" I R 1950 12400 60
+F3 "SAI2_TXC" I R 1950 12500 60
+F4 "SAI2_MCLK" I R 1950 12600 60
+F5 "SAI2_RXD" O R 1950 12150 60
+F6 "SAI2_TXD" I R 1950 12250 60
 $EndSheet
 Text Label 16400 8950 2    60   ~ 0
@@
 Text Label 16400 8550 2    60   ~ 0
 SAI2_TXFS
-Text Label 3200 11750 2    60   ~ 0
+Text Label 3200 12250 2    60   ~ 0
 SAI2_TXD
-Text Label 3200 11650 2    60   ~ 0
+Text Label 3200 12150 2    60   ~ 0
 SAI2_RXD
-Text Label 3200 12000 2    60   ~ 0
+Text Label 3200 12500 2    60   ~ 0
 SAI2_TXC
-Text Label 3200 12100 2    60   ~ 0
+Text Label 3200 12600 2    60   ~ 0
 SAI2_MCLK
-Text Label 3200 11900 2    60   ~ 0
+Text Label 3200 12400 2    60   ~ 0
 SAI2_TXFS
 $Comp
@@
 	16400 8650 15250 8650
 Wire Wire Line
-	3200 11750 1950 11750
-Wire Wire Line
-	3200 11650 1950 11650
-Wire Wire Line
-	3200 12000 1950 12000
-Wire Wire Line
-	1950 11900 3200 11900
-Wire Wire Line
-	3200 12100 1950 12100
+	3200 12250 1950 12250
+Wire Wire Line
+	3200 12150 1950 12150
+Wire Wire Line
+	3200 12500 1950 12500
+Wire Wire Line
+	1950 12400 3200 12400
+Wire Wire Line
+	3200 12600 1950 12600
 Wire Wire Line
 	7200 2200 7200 2250
@@
 	15250 13450 16400 13450
 $Sheet
-S 550  11150 1400 200
+S 550  11150 1400 700
 U 5ACD5EDE
 F0 "WWAN M.2" 60

Commit message: Add 1.8V<->3.3V logic level shifter (NTS0102) for the WWAN M.2 slot and connect it to the i.MX8M's UART3
The NTS0102 explicitly lists UART as one of its applications, and contains internal 10k pull-up resistors for the outputs. Whereas NTB/TXB0102 are push-pull outputs but aren't intended for UART applications due to the following (needs testing):
"The subtlety here is that you need to be careful of the auto direction sense circuitry.  Works fine but there can be some gotchas."
"If there is a signal integrity concern which is generally not the case for UARTs, series ~32 Ohm resistors on TX output pins can help.  For the exact resistor value you need to look at the V/I curve of the transmitter and pick the resistor value that matches the driver to the 50 Ohm Transmission line.  Layout for 50Ohm T-Lines and cables.  This will also cut down the risk of the EMI/EMC issues since any residual ringing is cutdown by IR drop in the terminator."
Connections:
- net UART3_RX: now reaches J1.B87 (UART3_RXD/UART1_CTS_B/////GPIO5_IO26)
- net UART3_TX: now reaches J1.B89 (UART3_TXD/UART1_RTS_B/////GPIO5_IO27)
- no-connect marks 164 -> 162
Changed lines of the file:
@@
 NoConn ~ 8150 10150
 NoConn ~ 8150 10250
-NoConn ~ 8150 10350
-NoConn ~ 8150 10450
 NoConn ~ 8150 11150
 NoConn ~ 8150 11250
@@
 F1 "wwan_m2.sch" 60
 F2 "CONFIG" O R 1950 11250 60
+F3 "UART_TX/LED" O R 1950 11400 60
+F4 "UART_RX/DPR" I R 1950 11500 60
 $EndSheet
 Wire Wire Line
@@
 Text Notes 3250 11250 0    60   ~ 0
 TODO!!!
+Wire Wire Line
+	1950 11400 3200 11400
+Wire Wire Line
+	1950 11500 3200 11500
+Text Label 3200 11400 2    60   ~ 0
+UART3_RX
+Text Label 3200 11500 2    60   ~ 0
+UART3_TX
+Wire Wire Line
+	8150 10350 7000 10350
+Wire Wire Line
+	8150 10450 7000 10450
+Text Label 7000 10350 0    60   ~ 0
+UART3_RX
+Text Label 7000 10450 0    60   ~ 0
+UART3_TX
 $EndSCHEMATC

Commit message: Bring out M.2 signals to the main sheet and attach WoWWAN and RESET
Add notes regarding the WWAN M.2's USB interface. The Emcraft SoM has NAND_CE3_B available for the DISABLE pin. Still need to select which pin will be used for CONFIG_1.
Connections:
- net NAND_DATA03: now reaches J1.A46 (NAND_DATA03/QSPIA_DATA3/////GPIO3_IO09)
- net NAND_DATA02: now reaches J1.A50 (NAND_DATA02/QSPIA_DATA2/////GPIO3_IO08)
- no-connect marks 162 -> 168
Other:
- note added: "NAND_CE3_B"
Changed lines of the file:
@@
 Sheet 1 14
 Title "DVK-DART-MX8M"
-Date "2018-04-11"
+Date "2018-04-16"
 Rev "v0.1.0"
 Comp "Purism SPC"
@@
 NoConn ~ 15250 2950
 NoConn ~ 15250 3050
-NoConn ~ 15250 3150
 NoConn ~ 15250 3250
-NoConn ~ 15250 3350
 NoConn ~ 15250 3550
 NoConn ~ 15250 3650
@@
 F14 "CAPTOUCH_~INT" O R 1950 9800 60
 F15 "CAPTOUCH_~RST" I R 1950 9900 60
-F16 "DSI_BL_PWM" I R 1950 9250 60
-F17 "AVDD_EN" O R 1950 9350 60
-F18 "SWIRE" O R 1950 9450 60
+F16 "AVDD_EN" O R 1950 9350 60
+F17 "SWIRE" O R 1950 9450 60
+F18 "RESX" I R 1950 9250 60
 $EndSheet
 $Sheet
@@
 $EndSheet
 $Sheet
-S 550  12050 1400 650
+S 550  11150 1400 1600
+U 5ACD5EDE
+F0 "WWAN M.2" 60
+F1 "wwan_m2.sch" 60
+F2 "CONFIG" O R 1950 11250 60
+F3 "UART_TX/LED" O R 1950 11850 60
+F4 "UART_RX/DPR" I R 1950 11950 60
+F5 "~WoWWAN" O R 1950 11400 60
+F6 "USB_D+" B R 1950 12100 60
+F7 "USB_D-" B R 1950 12200 60
+F8 "PCM_SYNC/I2S_FSC" I R 1950 12650 60
+F9 "PCM_CLK/I2S_SCK" O R 1950 12350 60
+F10 "PCM_IN/I2S_IN" I R 1950 12550 60
+F11 "PCM_OUT/I2S_OUT" O R 1950 12450 60
+F12 "~W_DISABLE1" I R 1950 11550 60
+F13 "~RESET" I R 1950 11700 60
+$EndSheet
+$Sheet
+S 550  12950 1400 650
 U 5ABE7AA4
 F0 "Audio" 60
 F1 "audio.sch" 60
-F2 "SAI2_TXFS" I R 1950 12400 60
-F3 "SAI2_TXC" I R 1950 12500 60
-F4 "SAI2_MCLK" I R 1950 12600 60
-F5 "SAI2_RXD" O R 1950 12150 60
-F6 "SAI2_TXD" I R 1950 12250 60
+F2 "SAI2_TXFS" I R 1950 13300 60
+F3 "SAI2_TXC" I R 1950 13400 60
+F4 "SAI2_MCLK" I R 1950 13500 60
+F5 "SAI2_RXD" O R 1950 13050 60
+F6 "SAI2_TXD" I R 1950 13150 60
 $EndSheet
 Text Label 16400 8950 2    60   ~ 0
@@
 Text Label 16400 8550 2    60   ~ 0
 SAI2_TXFS
-Text Label 3200 12250 2    60   ~ 0
+Text Label 3200 13150 2    60   ~ 0
 SAI2_TXD
-Text Label 3200 12150 2    60   ~ 0
+Text Label 3200 13050 2    60   ~ 0
 SAI2_RXD
-Text Label 3200 12500 2    60   ~ 0
+Text Label 3200 13400 2    60   ~ 0
 SAI2_TXC
-Text Label 3200 12600 2    60   ~ 0
+Text Label 3200 13500 2    60   ~ 0
 SAI2_MCLK
-Text Label 3200 12400 2    60   ~ 0
+Text Label 3200 13300 2    60   ~ 0
 SAI2_TXFS
 $Comp
@@
 	16400 8650 15250 8650
 Wire Wire Line
-	3200 12250 1950 12250
-Wire Wire Line
-	3200 12150 1950 12150
-Wire Wire Line
-	3200 12500 1950 12500
-Wire Wire Line
-	1950 12400 3200 12400
-Wire Wire Line
-	3200 12600 1950 12600
+	3200 13150 1950 13150
+Wire Wire Line
+	3200 13050 1950 13050
+Wire Wire Line
+	3200 13400 1950 13400
+Wire Wire Line
+	1950 13300 3200 13300
+Wire Wire Line
+	3200 13500 1950 13500
 Wire Wire Line
 	7200 2200 7200 2250
@@
 Wire Wire Line
 	15250 13450 16400 13450
-$Sheet
-S 550  11150 1400 700
-U 5ACD5EDE
-F0 "WWAN M.2" 60
-F1 "wwan_m2.sch" 60
-F2 "CONFIG" O R 1950 11250 60
-F3 "UART_TX/LED" O R 1950 11400 60
-F4 "UART_RX/DPR" I R 1950 11500 60
-$EndSheet
 Wire Wire Line
 	1950 11250 3200 11250
@@
 TODO!!!
 Wire Wire Line
-	1950 11400 3200 11400
-Wire Wire Line
-	1950 11500 3200 11500
-Text Label 3200 11400 2    60   ~ 0
+	1950 11850 3200 11850
+Wire Wire Line
+	1950 11950 3200 11950
+Text Label 3200 11850 2    60   ~ 0
 UART3_RX
-Text Label 3200 11500 2    60   ~ 0
+Text Label 3200 11950 2    60   ~ 0
 UART3_TX
 Wire Wire Line
@@
 Text Label 7000 10450 0    60   ~ 0
 UART3_TX
+Wire Wire Line
+	1950 11400 3200 11400
+Wire Wire Line
+	1950 12100 3200 12100
+Wire Wire Line
+	1950 12200 3200 12200
+Text Label 3200 12100 2    60   ~ 0
+WWAN_USB_D+
+Text Label 3200 12200 2    60   ~ 0
+WWAN_USB_D-
+NoConn ~ 3200 12100
+NoConn ~ 3200 12200
+Wire Wire Line
+	1950 12350 3200 12350
+Wire Wire Line
+	1950 12450 3200 12450
+Wire Wire Line
+	1950 12550 3200 12550
+Wire Wire Line
+	1950 12650 3200 12650
+Text Label 3200 12350 2    60   ~ 0
+PCM_CLK/I2S_SCK
+Text Label 3200 12450 2    60   ~ 0
+PCM_OUT/I2S_OUT
+Text Label 3200 12550 2    60   ~ 0
+PCM_IN/I2S_IN
+Text Label 3200 12650 2    60   ~ 0
+PCM_SYNC/I2S_FSC
+Wire Wire Line
+	1950 11550 3200 11550
+Text Label 3200 11550 2    60   ~ 0
+~WWAN_DISABLE
+NoConn ~ 3200 12350
+NoConn ~ 3200 12450
+NoConn ~ 3200 12550
+NoConn ~ 3200 12650
+NoConn ~ 3200 11550
+Wire Wire Line
+	1950 11700 3200 11700
+Text Label 3200 11700 2    60   ~ 0
+NAND_DATA03
+Text Notes 3250 11550 0    60   ~ 0
+NAND_CE3_B
+Text Label 3200 11400 2    60   ~ 0
+NAND_DATA02
+Text Label 16400 3350 2    60   ~ 0
+NAND_DATA02
+Wire Wire Line
+	15250 3350 16400 3350
+Text Label 16400 3150 2    60   ~ 0
+NAND_DATA03
+Wire Wire Line
+	15250 3150 16400 3150
+NoConn ~ 3200 11250
 $EndSCHEMATC
