File: rtc.sch (KiCad schematic (older format))
At the start: 10 parts, among them U5 BR24G04NUX-3TTR, U6 RV-4162-C7

Commit message: Use a buck for the 1.8V rail for efficiency, include power line ferrite bead, change main buck-boost output caps to 0805 ones, move the main regulator's input caps to the VIN node, include USB power switch circuit's components
The 1.8V buck has a drop-in: "ST1S12G18R"
Parts:
- renumbered C22 to C24, C23 to C25, R22 to R23, R23 to R24, R24 to R25
Changed lines of the file:
@@
 $EndDescr
 $Comp
-L SOM_SNVS_3V3 #PWR055
+L SOM_SNVS_3V3 #PWR059
 U 1 1 5AC54E36
 P 5100 4300
-F 0 "#PWR055" H 5100 4150 50  0001 C CNN
+F 0 "#PWR059" H 5100 4150 50  0001 C CNN
 F 1 "SOM_SNVS_3V3" H 5100 4440 50  0000 C CNN
 F 2 "" H 5100 4300 50  0001 C CNN
@@
 $EndComp
 $Comp
-L R R22
+L R R23
 U 1 1 5AC54E4A
 P 4500 4350
-F 0 "R22" V 4580 4350 50  0000 C CNN
+F 0 "R23" V 4580 4350 50  0000 C CNN
 F 1 "0" V 4500 4350 50  0000 C CNN
 F 2 "" V 4430 4350 50  0001 C CNN
@@
 $EndComp
 $Comp
-L SOM_VBAT_3V3 #PWR056
+L SOM_VBAT_3V3 #PWR060
 U 1 1 5AC54E9B
 P 4300 4300
-F 0 "#PWR056" H 4300 4150 50  0001 C CNN
+F 0 "#PWR060" H 4300 4150 50  0001 C CNN
 F 1 "SOM_VBAT_3V3" H 4300 4440 50  0000 C CNN
 F 2 "" H 4300 4300 50  0001 C CNN
@@
 	4300 4300 4300 4350
 $Comp
-L R R23
+L R R24
 U 1 1 5AC553FE
 P 4700 3950
-F 0 "R23" H 4825 4000 50  0000 C CNN
+F 0 "R24" H 4825 4000 50  0000 C CNN
 F 1 "NC" H 4800 3900 50  0000 C CNN
 F 2 "" V 4630 3950 50  0001 C CNN
@@
 $EndComp
 $Comp
-L BASE_PER_3V3 #PWR057
+L BASE_PER_3V3 #PWR061
 U 1 1 5AC5AC58
 P 6700 3700
-F 0 "#PWR057" H 6700 3550 50  0001 C CNN
+F 0 "#PWR061" H 6700 3550 50  0001 C CNN
 F 1 "BASE_PER_3V3" H 6700 3840 50  0000 C CNN
 F 2 "" H 6700 3700 50  0001 C CNN
@@
 	6700 3700 6700 3800
 $Comp
-L R R24
+L R R25
 U 1 1 5AC5AF1B
 P 5850 3750
-F 0 "R24" V 5930 3750 50  0000 C CNN
+F 0 "R25" V 5930 3750 50  0000 C CNN
 F 1 "4.99k" V 5750 3750 50  0000 C CNN
 F 2 "" V 5780 3750 50  0001 C CNN
@@
 	6050 3750 6000 3750
 $Comp
-L C C23
+L C C25
 U 1 1 5AC5B61C
 P 6700 3950
-F 0 "C23" H 6725 4050 50  0000 L CNN
+F 0 "C25" H 6725 4050 50  0000 L CNN
 F 1 "0.1uF" H 6725 3850 50  0000 L CNN
 F 2 "" H 6738 3800 50  0001 C CNN
@@
 $EndComp
 $Comp
-L GND #PWR058
+L GND #PWR062
 U 1 1 5AC5B669
 P 6700 4150
-F 0 "#PWR058" H 6700 3900 50  0001 C CNN
+F 0 "#PWR062" H 6700 3900 50  0001 C CNN
 F 1 "GND" H 6700 4000 50  0000 C CNN
 F 2 "" H 6700 4150 50  0001 C CNN
@@
 	4700 3750 5700 3750
 $Comp
-L GND #PWR059
+L GND #PWR063
 U 1 1 5AC5D6B6
 P 5450 4150
-F 0 "#PWR059" H 5450 3900 50  0001 C CNN
+F 0 "#PWR063" H 5450 3900 50  0001 C CNN
 F 1 "GND" H 5450 4000 50  0000 C CNN
 F 2 "" H 5450 4150 50  0001 C CNN
@@
 	5900 3050 6000 3050
 $Comp
-L GND #PWR060
+L GND #PWR064
 U 1 1 5AC6302E
 P 5000 3300
-F 0 "#PWR060" H 5000 3050 50  0001 C CNN
+F 0 "#PWR064" H 5000 3050 50  0001 C CNN
 F 1 "GND" H 5000 3150 50  0000 C CNN
 F 2 "" H 5000 3300 50  0001 C CNN
@@
 NoConn ~ 5100 3150
 $Comp
-L BASE_PER_3V3 #PWR061
+L BASE_PER_3V3 #PWR065
 U 1 1 5AC84D25
 P 3750 2200
-F 0 "#PWR061" H 3750 2050 50  0001 C CNN
+F 0 "#PWR065" H 3750 2050 50  0001 C CNN
 F 1 "BASE_PER_3V3" H 3750 2340 50  0000 C CNN
 F 2 "" H 3750 2200 50  0001 C CNN
@@
 $EndComp
 $Comp
-L BASE_PER_3V3 #PWR062
+L BASE_PER_3V3 #PWR066
 U 1 1 5AC84D64
 P 4950 1850
-F 0 "#PWR062" H 4950 1700 50  0001 C CNN
+F 0 "#PWR066" H 4950 1700 50  0001 C CNN
 F 1 "BASE_PER_3V3" H 4950 1990 50  0000 C CNN
 F 2 "" H 4950 1850 50  0001 C CNN
@@
 Connection ~ 3800 2600
 $Comp
-L GND #PWR063
+L GND #PWR067
 U 1 1 5AC8586C
 P 4350 3000
-F 0 "#PWR063" H 4350 2750 50  0001 C CNN
+F 0 "#PWR067" H 4350 2750 50  0001 C CNN
 F 1 "GND" H 4350 2850 50  0000 C CNN
 F 2 "" H 4350 3000 50  0001 C CNN
@@
 Connection ~ 5950 3050
 $Comp
-L C C22
+L C C24
 U 1 1 5AC8752C
 P 5200 2100
-F 0 "C22" H 5225 2200 50  0000 L CNN
+F 0 "C24" H 5225 2200 50  0000 L CNN
 F 1 "100nF" H 5225 2000 50  0000 L CNN
 F 2 "" H 5238 1950 50  0001 C CNN
@@
 $EndComp
 $Comp
-L GND #PWR064
+L GND #PWR068
 U 1 1 5AC875D7
 P 5200 2300
-F 0 "#PWR064" H 5200 2050 50  0001 C CNN
+F 0 "#PWR068" H 5200 2050 50  0001 C CNN
 F 1 "GND" H 5200 2150 50  0000 C CNN
 F 2 "" H 5200 2300 50  0001 C CNN

Commit message: Include UART debug interface/header, using a 74LVC2G241 buffer which is 5V tolerant so that either 3.3V or 5V UART cables could be used
Six pin header used so that either 6-pin fixed, 4-pin, or 3-pin cables can be used. Only RX, TX, and GND are used since Vcc, RTS#, and CTS# is unneeded, the other three pins are NC.
Parts:
- renumbered C24 to C27, C25 to C28
Changed lines of the file:
@@
 $Descr A4 11693 8268
 encoding utf-8
-Sheet 4 8
+Sheet 4 9
 Title "RTC Battery"
 Date "2018-04-05"
@@
 $EndDescr
 $Comp
-L SOM_SNVS_3V3 #PWR059
+L SOM_SNVS_3V3 #PWR060
 U 1 1 5AC54E36
 P 5100 4300
-F 0 "#PWR059" H 5100 4150 50  0001 C CNN
+F 0 "#PWR060" H 5100 4150 50  0001 C CNN
 F 1 "SOM_SNVS_3V3" H 5100 4440 50  0000 C CNN
 F 2 "" H 5100 4300 50  0001 C CNN
@@
 $EndComp
 $Comp
-L SOM_VBAT_3V3 #PWR060
+L SOM_VBAT_3V3 #PWR061
 U 1 1 5AC54E9B
 P 4300 4300
-F 0 "#PWR060" H 4300 4150 50  0001 C CNN
+F 0 "#PWR061" H 4300 4150 50  0001 C CNN
 F 1 "SOM_VBAT_3V3" H 4300 4440 50  0000 C CNN
 F 2 "" H 4300 4300 50  0001 C CNN
@@
 $EndComp
 $Comp
-L BASE_PER_3V3 #PWR061
+L BASE_PER_3V3 #PWR062
 U 1 1 5AC5AC58
 P 6700 3700
-F 0 "#PWR061" H 6700 3550 50  0001 C CNN
+F 0 "#PWR062" H 6700 3550 50  0001 C CNN
 F 1 "BASE_PER_3V3" H 6700 3840 50  0000 C CNN
 F 2 "" H 6700 3700 50  0001 C CNN
@@
 	6050 3750 6000 3750
 $Comp
-L C C25
+L C C28
 U 1 1 5AC5B61C
 P 6700 3950
-F 0 "C25" H 6725 4050 50  0000 L CNN
+F 0 "C28" H 6725 4050 50  0000 L CNN
 F 1 "0.1uF" H 6725 3850 50  0000 L CNN
 F 2 "" H 6738 3800 50  0001 C CNN
@@
 $EndComp
 $Comp
-L GND #PWR062
+L GND #PWR063
 U 1 1 5AC5B669
 P 6700 4150
-F 0 "#PWR062" H 6700 3900 50  0001 C CNN
+F 0 "#PWR063" H 6700 3900 50  0001 C CNN
 F 1 "GND" H 6700 4000 50  0000 C CNN
 F 2 "" H 6700 4150 50  0001 C CNN
@@
 	4700 3750 5700 3750
 $Comp
-L GND #PWR063
+L GND #PWR064
 U 1 1 5AC5D6B6
 P 5450 4150
-F 0 "#PWR063" H 5450 3900 50  0001 C CNN
+F 0 "#PWR064" H 5450 3900 50  0001 C CNN
 F 1 "GND" H 5450 4000 50  0000 C CNN
 F 2 "" H 5450 4150 50  0001 C CNN
@@
 	5900 3050 6000 3050
 $Comp
-L GND #PWR064
+L GND #PWR065
 U 1 1 5AC6302E
 P 5000 3300
-F 0 "#PWR064" H 5000 3050 50  0001 C CNN
+F 0 "#PWR065" H 5000 3050 50  0001 C CNN
 F 1 "GND" H 5000 3150 50  0000 C CNN
 F 2 "" H 5000 3300 50  0001 C CNN
@@
 NoConn ~ 5100 3150
 $Comp
-L BASE_PER_3V3 #PWR065
+L BASE_PER_3V3 #PWR066
 U 1 1 5AC84D25
 P 3750 2200
-F 0 "#PWR065" H 3750 2050 50  0001 C CNN
+F 0 "#PWR066" H 3750 2050 50  0001 C CNN
 F 1 "BASE_PER_3V3" H 3750 2340 50  0000 C CNN
 F 2 "" H 3750 2200 50  0001 C CNN
@@
 $EndComp
 $Comp
-L BASE_PER_3V3 #PWR066
+L BASE_PER_3V3 #PWR067
 U 1 1 5AC84D64
 P 4950 1850
-F 0 "#PWR066" H 4950 1700 50  0001 C CNN
+F 0 "#PWR067" H 4950 1700 50  0001 C CNN
 F 1 "BASE_PER_3V3" H 4950 1990 50  0000 C CNN
 F 2 "" H 4950 1850 50  0001 C CNN
@@
 Connection ~ 3800 2600
 $Comp
-L GND #PWR067
+L GND #PWR068
 U 1 1 5AC8586C
 P 4350 3000
-F 0 "#PWR067" H 4350 2750 50  0001 C CNN
+F 0 "#PWR068" H 4350 2750 50  0001 C CNN
 F 1 "GND" H 4350 2850 50  0000 C CNN
 F 2 "" H 4350 3000 50  0001 C CNN
@@
 Connection ~ 5950 3050
 $Comp
-L C C24
+L C C27
 U 1 1 5AC8752C
 P 5200 2100
-F 0 "C24" H 5225 2200 50  0000 L CNN
+F 0 "C27" H 5225 2200 50  0000 L CNN
 F 1 "100nF" H 5225 2000 50  0000 L CNN
 F 2 "" H 5238 1950 50  0001 C CNN
@@
 $EndComp
 $Comp
-L GND #PWR068
+L GND #PWR069
 U 1 1 5AC875D7
 P 5200 2300
-F 0 "#PWR068" H 5200 2050 50  0001 C CNN
+F 0 "#PWR069" H 5200 2050 50  0001 C CNN
 F 1 "GND" H 5200 2150 50  0000 C CNN
 F 2 "" H 5200 2300 50  0001 C CNN
