File: rtc.sch (KiCad schematic (older format))
At the start: 7 parts, among them U601 RV-4162-C7

Commit message: Move the charge controller, USB-C TCPC, and RTC to I2C1
Since each of these ICs will be powered at the same time as the SoM regardless of the PWR_EN state, they should share the same I2C bus as the PMIC.
Connections:
- net labels added: I2C1_SCL, I2C1_SDA
- net labels removed: I2C3_SCL, I2C3_SDA
Changed lines of the file:
@@
 	6200 3850 6250 3850
 Text HLabel 4550 3100 0    60   BiDi ~ 0
-I2C3_SDA
+I2C1_SDA
 Text HLabel 5450 3100 2    60   Input ~ 0
-I2C3_SCL
+I2C1_SCL
 $Comp
-L GND #PWR0138
+L GND #PWR0139
 U 1 1 5AC6302E
 P 4500 3350
-F 0 "#PWR0138" H 4500 3100 50  0001 C CNN
+F 0 "#PWR0139" H 4500 3100 50  0001 C CNN
 F 1 "GND" H 4500 3200 50  0000 C CNN
 F 2 "" H 4500 3350 50  0001 C CNN
@@
 	7250 3800 7250 3900
 $Comp
-L GND #PWR0139
+L GND #PWR0140
 U 1 1 5AC5B669
 P 7250 4250
-F 0 "#PWR0139" H 7250 4000 50  0001 C CNN
+F 0 "#PWR0140" H 7250 4000 50  0001 C CNN
 F 1 "GND" H 7250 4100 50  0000 C CNN
 F 2 "" H 7250 4250 50  0001 C CNN
@@
 $EndComp
 $Comp
-L VBAT_REG #PWR0140
+L VBAT_REG #PWR0141
 U 1 1 5AE5DA7A
 P 7250 3800
-F 0 "#PWR0140" H 7250 3650 50  0001 C CNN
+F 0 "#PWR0141" H 7250 3650 50  0001 C CNN
 F 1 "VBAT_REG" H 7250 3940 50  0000 C CNN
 F 2 "" H 7250 3800 50  0001 C CNN
@@
 $EndComp
 $Comp
-L VBAT #PWR0141
+L VBAT #PWR0142
 U 1 1 5AE5DAE8
 P 6200 3800
-F 0 "#PWR0141" H 6200 3650 50  0001 C CNN
+F 0 "#PWR0142" H 6200 3650 50  0001 C CNN
 F 1 "VBAT" H 6200 3940 50  0000 C CNN
 F 2 "" H 6200 3800 50  0001 C CNN
@@
 Real-Time Clock
 $Comp
-L 3V3_OUT #PWR0142
+L 3V3_OUT #PWR0143
 U 1 1 5B6A7D4C
 P 6050 2900
-F 0 "#PWR0142" H 6050 2750 50  0001 C CNN
+F 0 "#PWR0143" H 6050 2750 50  0001 C CNN
 F 1 "3V3_OUT" H 6050 3040 50  0000 C CNN
 F 2 "" H 6050 2900 50  0001 C CNN

Commit message: Continue layout around the charge controller circuit
Other:
- note added: "VIH(min) not given, however\n assuming VIH(min)≅0.77647*VDD\n@VDD=4.25V then VIH(min)≅3.2999975V"
- note removed: "VIH(min) not given, however\n assuming VIH(min)≅VDD*0.7857\n@VDD=4.2 then VIH(min)≅3.3012V"
Changed lines of the file:
@@
 VBAT is PTC fused
 Text Notes 7050 3200 0    60   ~ 0
-   VIH(min) not given, however\n assuming VIH(min)≅VDD*0.7857\n@VDD=4.2 then VIH(min)≅3.3012V
+      VIH(min) not given, however\n    assuming VIH(min)≅0.77647*VDD\n@VDD=4.25V then VIH(min)≅3.2999975V
 Text Notes 7050 3575 0    60   ~ 0
 3.5~~4.25V

Commit message: Update project files to KiCad 5.0.0
Parts:
- C601: symbol C -> dvk-mx8m-bsb-rescue:C
- D601: symbol D_Schottky_ALT -> dvk-mx8m-bsb-rescue:D_Schottky_ALT
- D602: symbol D_Schottky_x2_KCom_AAK -> dvk-mx8m-bsb-rescue:D_Schottky_x2_KCom_AAK
- FB601: symbol Ferrite_Bead -> dvk-mx8m-bsb-rescue:Ferrite_Bead
- R601, R602: symbol R -> dvk-mx8m-bsb-rescue:R
- U601: symbol RV-4162-C7 -> dvk-mx8m-bsb:RV-4162-C7
Changed lines of the file:
@@
-EESchema Schematic File Version 2
-LIBS:power
-LIBS:device
-LIBS:switches
-LIBS:relays
-LIBS:motors
-LIBS:transistors
-LIBS:conn
-LIBS:linear
-LIBS:regul
-LIBS:74xx
-LIBS:cmos4000
-LIBS:adc-dac
-LIBS:memory
-LIBS:xilinx
-LIBS:microcontrollers
-LIBS:dsp
-LIBS:microchip
-LIBS:analog_switches
-LIBS:motorola
-LIBS:texas
-LIBS:intel
-LIBS:audio
-LIBS:interface
-LIBS:digital-audio
-LIBS:philips
-LIBS:display
-LIBS:cypress
-LIBS:siliconi
-LIBS:opto
-LIBS:atmel
-LIBS:contrib
-LIBS:valves
-LIBS:dvk-mx8m-bsb
+EESchema Schematic File Version 4
 LIBS:dvk-mx8m-bsb-cache
-EELAYER 25 0
+EELAYER 26 0
 EELAYER END
 $Descr A4 11693 8268
@@
 $EndDescr
 $Comp
-L R R602
+L dvk-mx8m-bsb-rescue:R R602
 U 1 1 5AC5AF1B
 P 6400 3850
@@
 	6600 3850 6550 3850
 $Comp
-L RV-4162-C7 U601
+L dvk-mx8m-bsb:RV-4162-C7 U601
 U 1 1 5AC5BD52
 P 5000 3250
@@
 I2C1_SCL
 $Comp
-L GND #PWR0139
+L power:GND #PWR0139
 U 1 1 5AC6302E
 P 4500 3350
@@
 NoConn ~ 4600 3200
 $Comp
-L D_Schottky_x2_KCom_AAK D602
+L dvk-mx8m-bsb-rescue:D_Schottky_x2_KCom_AAK D602
 U 1 1 5AC55F7F
 P 6900 3850
@@
 	7250 3800 7250 3900
 $Comp
-L GND #PWR0140
+L power:GND #PWR0140
 U 1 1 5AC5B669
 P 7250 4250
@@
 	7250 4250 7250 4200
 $Comp
-L C C601
+L dvk-mx8m-bsb-rescue:C C601
 U 1 1 5AC5B61C
 P 7250 4050
@@
 $EndComp
 $Comp
-L VBAT_REG #PWR0141
+L dvk-mx8m-bsb:VBAT_REG #PWR0141
 U 1 1 5AE5DA7A
 P 7250 3800
@@
 $EndComp
 $Comp
-L VBAT #PWR0142
+L dvk-mx8m-bsb:VBAT #PWR0142
 U 1 1 5AE5DAE8
 P 6200 3800
@@
 	4550 3100 4600 3100
 $Comp
-L D_Schottky_ALT D601
+L dvk-mx8m-bsb-rescue:D_Schottky_ALT D601
 U 1 1 5B6718B5
 P 5600 3300
@@
 $EndComp
 $Comp
-L R R601
+L dvk-mx8m-bsb-rescue:R R601
 U 1 1 5B68E84A
 P 6050 3100
@@
 Reference:\nhttps://github.com/HIO-Project/linux-imx6-nano-imx_3.10.17_1.0.1_ga/\nblob/8848e94b2f889fe44f6736e2d4c98851a2282275/arch/arm/boot/dts/\nimx6qdl-mtp.dtsi#L351
 $Comp
-L Ferrite_Bead FB601
+L dvk-mx8m-bsb-rescue:Ferrite_Bead FB601
 U 1 1 5B175E17
 P 6500 3400
@@
 Real-Time Clock
 $Comp
-L 3V3_OUT #PWR0143
+L dvk-mx8m-bsb:3V3_OUT #PWR0143
 U 1 1 5B6A7D4C
 P 6050 2900

Commit message: Update the schematic symbols and footprints after upgrading to KiCad 5.0.0, fix all ERC and DRC violations after the new update/upgrade
Parts:
- C601: footprint Capacitors_SMD:C_0603 -> Capacitor_SMD:C_0603_1608Metric; symbol dvk-mx8m-bsb-rescue:C -> Device:C
- D601: symbol dvk-mx8m-bsb-rescue:D_Schottky_ALT -> Device:D_Schottky_ALT
- D602: footprint TO_SOT_Packages_SMD:SOT-23 -> Package_TO_SOT_SMD:SOT-23; symbol dvk-mx8m-bsb-rescue:D_Schottky_x2_KCom_AAK -> Device:D_Schottky_x2_KCom_AAK
- FB601: symbol dvk-mx8m-bsb-rescue:Ferrite_Bead -> Device:Ferrite_Bead
- R601, R602: footprint Resistors_SMD:R_0603 -> Resistor_SMD:R_0603_1608Metric; symbol dvk-mx8m-bsb-rescue:R -> Device:R
Connections:
- wire segments 17 -> 19
Changed lines of the file:
@@
 Sheet 6 24
 Title "RTC"
-Date "2018-06-18"
+Date "2018-07-17"
 Rev "v0.1.0"
 Comp "Copyright 2018 GNU GPLv3"
@@
 $EndDescr
 $Comp
-L dvk-mx8m-bsb-rescue:R R602
+L Device:R R602
 U 1 1 5AC5AF1B
 P 6400 3850
 F 0 "R602" V 6480 3850 50  0000 C CNN
 F 1 "4.99k" V 6300 3850 50  0000 C CNN
-F 2 "Resistors_SMD:R_0603" V 6330 3850 50  0001 C CNN
+F 2 "Resistor_SMD:R_0603_1608Metric" V 6330 3850 50  0001 C CNN
 F 3 "" H 6400 3850 50  0001 C CNN
 	1    6400 3850
@@
 NoConn ~ 4600 3200
 $Comp
-L dvk-mx8m-bsb-rescue:D_Schottky_x2_KCom_AAK D602
+L Device:D_Schottky_x2_KCom_AAK D602
 U 1 1 5AC55F7F
 P 6900 3850
 F 0 "D602" H 6800 3750 50  0000 C CNN
 F 1 "BAT54C" H 6900 3950 50  0000 C CNN
-F 2 "TO_SOT_Packages_SMD:SOT-23" H 6900 3850 50  0001 C CNN
+F 2 "Package_TO_SOT_SMD:SOT-23" H 6900 3850 50  0001 C CNN
 F 3 "https://goodarksemi.com/docs/datasheets/schottky_diodes/BAT54-A-C-S.pdf" H 6900 3850 50  0001 C CNN
 F 4 "Good-Ark Semi" H 6900 3850 60  0001 C CNN "MFG Name"
@@
 Connection ~ 7250 3850
 Wire Wire Line
-	7250 3800 7250 3900
+	7250 3800 7250 3850
 $Comp
 L power:GND #PWR0140
@@
 	7250 4250 7250 4200
 $Comp
-L dvk-mx8m-bsb-rescue:C C601
+L Device:C C601
 U 1 1 5AC5B61C
 P 7250 4050
 F 0 "C601" H 7275 4150 50  0000 L CNN
 F 1 "100nF" H 7275 3950 50  0000 L CNN
-F 2 "Capacitors_SMD:C_0603" H 7288 3900 50  0001 C CNN
+F 2 "Capacitor_SMD:C_0603_1608Metric" H 7288 3900 50  0001 C CNN
 F 3 "" H 7250 4050 50  0001 C CNN
 	1    7250 4050
@@
 	4550 3100 4600 3100
 $Comp
-L dvk-mx8m-bsb-rescue:D_Schottky_ALT D601
+L Device:D_Schottky_ALT D601
 U 1 1 5B6718B5
 P 5600 3300
@@
 $EndComp
 $Comp
-L dvk-mx8m-bsb-rescue:R R601
+L Device:R R601
 U 1 1 5B68E84A
 P 6050 3100
 F 0 "R601" H 6200 3150 50  0000 C CNN
 F 1 "10k" H 6175 3050 50  0000 C CNN
-F 2 "Resistors_SMD:R_0603" V 5980 3100 50  0001 C CNN
+F 2 "Resistor_SMD:R_0603_1608Metric" V 5980 3100 50  0001 C CNN
 F 3 "https://www.seielect.com/Catalog/SEI-RMCF_RMCP.pdf" H 6050 3100 50  0001 C CNN
 F 4 "Stackpole" H 6050 3100 60  0001 C CNN "MFG Name"
@@
 ~IRQ
 Wire Wire Line
-	5750 3300 6100 3300
+	5750 3300 6050 3300
 Connection ~ 6050 3300
 Text Notes 4400 2650 0    60   ~ 0
@@
 Reference:\nhttps://github.com/HIO-Project/linux-imx6-nano-imx_3.10.17_1.0.1_ga/\nblob/8848e94b2f889fe44f6736e2d4c98851a2282275/arch/arm/boot/dts/\nimx6qdl-mtp.dtsi#L351
 $Comp
-L dvk-mx8m-bsb-rescue:Ferrite_Bead FB601
+L Device:Ferrite_Bead FB601
 U 1 1 5B175E17
 P 6500 3400
@@
 	1    0    0    -1
 $EndComp
+Wire Wire Line
+	7250 3850 7250 3900
+Wire Wire Line
+	6050 3300 6100 3300
 $EndSCHEMATC

Commit message: Reduce all 0603 resistor sizes to 0402
Parts:
- R601, R602: footprint Resistor_SMD:R_0603_1608Metric -> Resistor_SMD:R_0402_1005Metric
Changed lines of the file:
@@
 F 0 "R602" V 6480 3850 50  0000 C CNN
 F 1 "4.99k" V 6300 3850 50  0000 C CNN
-F 2 "Resistor_SMD:R_0603_1608Metric" V 6330 3850 50  0001 C CNN
+F 2 "Resistor_SMD:R_0402_1005Metric" V 6330 3850 50  0001 C CNN
 F 3 "" H 6400 3850 50  0001 C CNN
 	1    6400 3850
@@
 F 0 "R601" H 6200 3150 50  0000 C CNN
 F 1 "10k" H 6175 3050 50  0000 C CNN
-F 2 "Resistor_SMD:R_0603_1608Metric" V 5980 3100 50  0001 C CNN
+F 2 "Resistor_SMD:R_0402_1005Metric" V 5980 3100 50  0001 C CNN
 F 3 "https://www.seielect.com/Catalog/SEI-RMCF_RMCP.pdf" H 6050 3100 50  0001 C CNN
 F 4 "Stackpole" H 6050 3100 60  0001 C CNN "MFG Name"

Commit message: Change all 0603 capacitors _EXCEPT_ the 2.2uF, 4.7uF, 8.2uF, 10uF, and 22uF caps to 0402
Parts:
- C601: footprint Capacitor_SMD:C_0603_1608Metric -> Capacitor_SMD:C_0402_1005Metric
Changed lines of the file:
@@
 F 0 "C601" H 7275 4150 50  0000 L CNN
 F 1 "100nF" H 7275 3950 50  0000 L CNN
-F 2 "Capacitor_SMD:C_0603_1608Metric" H 7288 3900 50  0001 C CNN
+F 2 "Capacitor_SMD:C_0402_1005Metric" H 7288 3900 50  0001 C CNN
 F 3 "" H 7250 4050 50  0001 C CNN
 	1    7250 4050
