File: watchdog.sch (KiCad schematic (older format))
At the start: 17 parts, among them SW1 SW_Push, U8 TPS3808G30DBVT

Commit message: Add JTAG and buttons & LED schematics, reorder based on priority (especially for debugging/development)
Parts:
- renumbered C43 to C30, C44 to C31, C45 to C32, C46 to C33, D7 to D5, D8 to D6, D9 to D7, D10 to D8, R31 to R45, R32 to R46, R33 to R47, R34 to R48, R35 to R49, R36 to R50, R37 to R51, SW1 to SW2
Connections:
- net ~SW_RST renamed SW_~RST
Other:
- moved on the sheet: D5, SW2
Changed lines of the file:
@@
 $Descr A4 11693 8268
 encoding utf-8
-Sheet 6 10
+Sheet 5 12
 Title "Reset & Watchdog"
 Date "2018-04-09"
@@
 $EndDescr
 $Comp
-L SOM_SNVS_3V3 #PWR083
+L SOM_SNVS_3V3 #PWR075
 U 1 1 5AC8A151
 P 7200 3000
-F 0 "#PWR083" H 7200 2850 50  0001 C CNN
+F 0 "#PWR075" H 7200 2850 50  0001 C CNN
 F 1 "SOM_SNVS_3V3" H 7200 3140 50  0000 C CNN
 F 2 "" H 7200 3000 50  0001 C CNN
@@
 $EndComp
 $Comp
-L R R35
+L R R49
 U 1 1 5AC8A17C
 P 6600 3300
-F 0 "R35" H 6725 3350 50  0000 C CNN
+F 0 "R49" H 6725 3350 50  0000 C CNN
 F 1 "NC" H 6700 3250 50  0000 C CNN
 F 2 "" V 6530 3300 50  0001 C CNN
@@
 $EndComp
 $Comp
-L R R34
+L R R48
 U 1 1 5AC8A1A9
 P 6300 3300
-F 0 "R34" H 6425 3350 50  0000 C CNN
+F 0 "R48" H 6425 3350 50  0000 C CNN
 F 1 "100k" H 6450 3250 50  0000 C CNN
 F 2 "" V 6230 3300 50  0001 C CNN
@@
 $EndComp
 $Comp
-L D_Schottky D10
+L D_Schottky D8
 U 1 1 5AC8A554
 P 6000 3300
-F 0 "D10" V 5900 3200 50  0000 C CNN
+F 0 "D8" V 5900 3200 50  0000 C CNN
 F 1 "30V,100mA" V 6100 3050 50  0000 C CNN
 F 2 "" H 6000 3300 50  0001 C CNN
@@
 $EndComp
 $Comp
-L C C45
+L C C32
 U 1 1 5AC8ACD0
 P 5450 3500
-F 0 "C45" V 5500 3600 50  0000 L CNN
+F 0 "C32" V 5500 3600 50  0000 L CNN
 F 1 "2.2uF" V 5500 3250 50  0000 L CNN
 F 2 "" H 5488 3350 50  0001 C CNN
@@
 	5600 3500 6650 3500
 $Comp
-L C C46
+L C C33
 U 1 1 5AC8B0DE
 P 5450 3700
-F 0 "C46" V 5500 3800 50  0000 L CNN
+F 0 "C33" V 5500 3800 50  0000 L CNN
 F 1 "NC" V 5500 3450 50  0000 L CNN
 F 2 "" H 5488 3550 50  0001 C CNN
@@
 $EndComp
 $Comp
-L GND #PWR084
+L GND #PWR076
 U 1 1 5AC8B439
 P 5250 3750
-F 0 "#PWR084" H 5250 3500 50  0001 C CNN
+F 0 "#PWR076" H 5250 3500 50  0001 C CNN
 F 1 "GND" H 5250 3600 50  0000 C CNN
 F 2 "" H 5250 3750 50  0001 C CNN
@@
 	7200 3000 7200 3200
 $Comp
-L R R33
+L R R47
 U 1 1 5AC8B597
 P 5150 3300
-F 0 "R33" H 5275 3350 50  0000 C CNN
+F 0 "R47" H 5275 3350 50  0000 C CNN
 F 1 "21.5k" H 5300 3250 50  0000 C CNN
 F 2 "" V 5080 3300 50  0001 C CNN
@@
 Connection ~ 6000 3500
 $Comp
-L D_Schottky D8
+L D_Schottky D6
 U 1 1 5AC8BA0F
 P 4900 3500
-F 0 "D8" H 4900 3600 50  0000 C CNN
+F 0 "D6" H 4900 3600 50  0000 C CNN
 F 1 "30V,100mA" H 4900 3400 50  0000 C CNN
 F 2 "" H 4900 3500 50  0001 C CNN
@@
 $EndComp
 $Comp
-L D_Schottky D9
+L D_Schottky D7
 U 1 1 5AC8BB44
 P 4900 4100
-F 0 "D9" H 4900 4200 50  0000 C CNN
+F 0 "D7" H 4900 4200 50  0000 C CNN
 F 1 "30V,100mA" H 4900 4000 50  0000 C CNN
 F 2 "" H 4900 4100 50  0001 C CNN
@@
 $EndComp
 $Comp
-L C C44
+L C C31
 U 1 1 5AC8BC45
 P 4600 3700
-F 0 "C44" H 4625 3800 50  0000 L CNN
+F 0 "C31" H 4625 3800 50  0000 L CNN
 F 1 "1nF" H 4625 3600 50  0000 L CNN
 F 2 "" H 4638 3550 50  0001 C CNN
@@
 $EndComp
 $Comp
-L GND #PWR085
+L GND #PWR077
 U 1 1 5AC8BC81
 P 4600 3900
-F 0 "#PWR085" H 4600 3650 50  0001 C CNN
+F 0 "#PWR077" H 4600 3650 50  0001 C CNN
 F 1 "GND" H 4600 3750 50  0000 C CNN
 F 2 "" H 4600 3900 50  0001 C CNN
@@
 Connection ~ 5150 3500
 $Comp
-L R R32
+L R R46
 U 1 1 5AC8C0DB
 P 4600 4300
-F 0 "R32" H 4725 4350 50  0000 C CNN
+F 0 "R46" H 4725 4350 50  0000 C CNN
 F 1 "1M" H 4700 4250 50  0000 C CNN
 F 2 "" V 4530 4300 50  0001 C CNN
@@
 GPIO1_IO02(~WDOG~)
 Wire Wire Line
-	3750 3500 4150 3500
+	3700 3500 4150 3500
 Wire Wire Line
 	4450 3500 4750 3500
@@
 Connection ~ 4600 4100
 $Comp
-L GND #PWR086
+L GND #PWR078
 U 1 1 5AC8CD8F
 P 4600 4500
-F 0 "#PWR086" H 4600 4250 50  0001 C CNN
+F 0 "#PWR078" H 4600 4250 50  0001 C CNN
 F 1 "GND" H 4600 4350 50  0000 C CNN
 F 2 "" H 4600 4500 50  0001 C CNN
@@
 	4600 4500 4600 4450
 $Comp
-L GND #PWR087
+L GND #PWR079
 U 1 1 5AC8D3A2
 P 7200 4250
-F 0 "#PWR087" H 7200 4000 50  0001 C CNN
+F 0 "#PWR079" H 7200 4000 50  0001 C CNN
 F 1 "GND" H 7200 4100 50  0000 C CNN
 F 2 "" H 7200 4250 50  0001 C CNN
@@
 	7200 4250 7200 4200
 $Comp
-L R R36
+L R R50
 U 1 1 5AC8D701
 P 8000 3400
-F 0 "R36" V 8080 3400 50  0000 C CNN
+F 0 "R50" V 8080 3400 50  0000 C CNN
 F 1 "120" V 7900 3400 50  0000 C CNN
 F 2 "" V 7930 3400 50  0001 C CNN
@@
 $EndComp
 $Comp
-L R R37
+L R R51
 U 1 1 5AC8D7F2
 P 8000 3700
-F 0 "R37" V 8080 3700 50  0000 C CNN
+F 0 "R51" V 8080 3700 50  0000 C CNN
 F 1 "0" V 7900 3700 50  0000 C CNN
 F 2 "" V 7930 3700 50  0001 C CNN
@@
 	8150 3700 8200 3700
 $Comp
-L SW_Push SW1
+L SW_Push SW2
 U 1 1 5AC99959
-P 3550 3500
-F 0 "SW1" H 3600 3600 50  0000 L CNN
-F 1 "SW_Push" H 3550 3440 50  0000 C CNN
-F 2 "" H 3550 3700 50  0001 C CNN
-F 3 "" H 3550 3700 50  0001 C CNN
-	1    3550 3500
-	1    0    0    -1
-$EndComp
-$Comp
-L TVS_DIODE D7
+P 3500 3500
+F 0 "SW2" H 3550 3600 50  0000 L CNN
+F 1 "SW_Push" H 3500 3440 50  0000 C CNN
+F 2 "" H 3500 3700 50  0001 C CNN
+F 3 "" H 3500 3700 50  0001 C CNN
+	1    3500 3500
+	1    0    0    -1
+$EndComp
+$Comp
+L TVS_DIODE D5
 U 1 1 5AC99E1E
-P 3550 3750
-F 0 "D7" H 3550 3850 50  0000 C CNN
-F 1 "TPD1E10B09DPYR" H 3550 3650 50  0000 C CNN
-F 2 "" H 3650 3750 50  0001 C CNN
-F 3 "" H 3650 3750 50  0001 C CNN
-	1    3550 3750
-	1    0    0    -1
-$EndComp
-$Comp
-L GND #PWR088
+P 3500 3750
+F 0 "D5" H 3500 3850 50  0000 C CNN
+F 1 "TPD1E10B09DPYR" H 3500 3650 50  0000 C CNN
+F 2 "" H 3600 3750 50  0001 C CNN
+F 3 "" H 3600 3750 50  0001 C CNN
+	1    3500 3750
+	1    0    0    -1
+$EndComp
+$Comp
+L GND #PWR080
 U 1 1 5AC9A292
-P 3150 3800
-F 0 "#PWR088" H 3150 3550 50  0001 C CNN
-F 1 "GND" H 3150 3650 50  0000 C CNN
-F 2 "" H 3150 3800 50  0001 C CNN
-F 3 "" H 3150 3800 50  0001 C CNN
-	1    3150 3800
-	1    0    0    -1
-$EndComp
-Wire Wire Line
-	3150 3500 3150 3800
-Wire Wire Line
-	3150 3500 3350 3500
-Wire Wire Line
-	3400 3750 3150 3750
-Connection ~ 3150 3750
-Wire Wire Line
-	3700 3750 3800 3750
-Wire Wire Line
-	3800 3750 3800 3500
-Connection ~ 3800 3500
+P 3100 3800
+F 0 "#PWR080" H 3100 3550 50  0001 C CNN
+F 1 "GND" H 3100 3650 50  0000 C CNN
+F 2 "" H 3100 3800 50  0001 C CNN
+F 3 "" H 3100 3800 50  0001 C CNN
+	1    3100 3800
+	1    0    0    -1
+$EndComp
+Wire Wire Line
+	3100 3500 3100 3800
+Wire Wire Line
+	3100 3500 3300 3500
+Wire Wire Line
+	3350 3750 3100 3750
+Connection ~ 3100 3750
+Wire Wire Line
+	3650 3750 3750 3750
+Wire Wire Line
+	3750 3750 3750 3500
+Connection ~ 3750 3500
 Text Label 3800 3500 0    60   ~ 0
-~SW_RST
-$Comp
-L R R31
+SW_~RST
+$Comp
+L R R45
 U 1 1 5AC9A911
 P 4300 3500
-F 0 "R31" V 4380 3500 50  0000 C CNN
+F 0 "R45" V 4380 3500 50  0000 C CNN
 F 1 "120" V 4200 3500 50  0000 C CNN
 F 2 "" V 4230 3500 50  0001 C CNN
@@
 $EndComp
 $Comp
-L C C43
+L C C30
 U 1 1 5AC9A94A
 P 4300 4100
-F 0 "C43" V 4350 4200 50  0000 L CNN
+F 0 "C30" V 4350 4200 50  0000 L CNN
 F 1 "1uF" V 4350 3900 50  0000 L CNN
 F 2 "" H 4338 3950 50  0001 C CNN

Commit message: Add MIPI DSI, cap touch interface, and AMOLED display regulator circuits
TPS65632's components were selected based on the best match and price based on suggestions. The RT4720 does not seem to be sold by any distributors.
Parts:
- renumbered C30 to C39, C31 to C40, C32 to C41, C33 to C42, U8 to U9
Changed lines of the file:
@@
 $Descr A4 11693 8268
 encoding utf-8
-Sheet 5 12
+Sheet 5 13
 Title "Reset & Watchdog"
 Date "2018-04-09"
@@
 $EndDescr
 $Comp
-L SOM_SNVS_3V3 #PWR075
+L SOM_SNVS_3V3 #PWR087
 U 1 1 5AC8A151
 P 7200 3000
-F 0 "#PWR075" H 7200 2850 50  0001 C CNN
+F 0 "#PWR087" H 7200 2850 50  0001 C CNN
 F 1 "SOM_SNVS_3V3" H 7200 3140 50  0000 C CNN
 F 2 "" H 7200 3000 50  0001 C CNN
@@
 $EndComp
 $Comp
-L C C32
+L C C41
 U 1 1 5AC8ACD0
 P 5450 3500
-F 0 "C32" V 5500 3600 50  0000 L CNN
+F 0 "C41" V 5500 3600 50  0000 L CNN
 F 1 "2.2uF" V 5500 3250 50  0000 L CNN
 F 2 "" H 5488 3350 50  0001 C CNN
@@
 	5600 3500 6650 3500
 $Comp
-L C C33
+L C C42
 U 1 1 5AC8B0DE
 P 5450 3700
-F 0 "C33" V 5500 3800 50  0000 L CNN
+F 0 "C42" V 5500 3800 50  0000 L CNN
 F 1 "NC" V 5500 3450 50  0000 L CNN
 F 2 "" H 5488 3550 50  0001 C CNN
@@
 $EndComp
 $Comp
-L GND #PWR076
+L GND #PWR088
 U 1 1 5AC8B439
 P 5250 3750
-F 0 "#PWR076" H 5250 3500 50  0001 C CNN
+F 0 "#PWR088" H 5250 3500 50  0001 C CNN
 F 1 "GND" H 5250 3600 50  0000 C CNN
 F 2 "" H 5250 3750 50  0001 C CNN
@@
 $EndComp
 $Comp
-L C C31
+L C C40
 U 1 1 5AC8BC45
 P 4600 3700
-F 0 "C31" H 4625 3800 50  0000 L CNN
+F 0 "C40" H 4625 3800 50  0000 L CNN
 F 1 "1nF" H 4625 3600 50  0000 L CNN
 F 2 "" H 4638 3550 50  0001 C CNN
@@
 $EndComp
 $Comp
-L GND #PWR077
+L GND #PWR089
 U 1 1 5AC8BC81
 P 4600 3900
-F 0 "#PWR077" H 4600 3650 50  0001 C CNN
+F 0 "#PWR089" H 4600 3650 50  0001 C CNN
 F 1 "GND" H 4600 3750 50  0000 C CNN
 F 2 "" H 4600 3900 50  0001 C CNN
@@
 Connection ~ 4600 4100
 $Comp
-L GND #PWR078
+L GND #PWR090
 U 1 1 5AC8CD8F
 P 4600 4500
-F 0 "#PWR078" H 4600 4250 50  0001 C CNN
+F 0 "#PWR090" H 4600 4250 50  0001 C CNN
 F 1 "GND" H 4600 4350 50  0000 C CNN
 F 2 "" H 4600 4500 50  0001 C CNN
@@
 	4600 4500 4600 4450
 $Comp
-L GND #PWR079
+L GND #PWR091
 U 1 1 5AC8D3A2
 P 7200 4250
-F 0 "#PWR079" H 7200 4000 50  0001 C CNN
+F 0 "#PWR091" H 7200 4000 50  0001 C CNN
 F 1 "GND" H 7200 4100 50  0000 C CNN
 F 2 "" H 7200 4250 50  0001 C CNN
@@
 $EndComp
 $Comp
-L GND #PWR080
+L GND #PWR092
 U 1 1 5AC9A292
 P 3100 3800
-F 0 "#PWR080" H 3100 3550 50  0001 C CNN
+F 0 "#PWR092" H 3100 3550 50  0001 C CNN
 F 1 "GND" H 3100 3650 50  0000 C CNN
 F 2 "" H 3100 3800 50  0001 C CNN
@@
 $EndComp
 $Comp
-L C C30
+L C C39
 U 1 1 5AC9A94A
 P 4300 4100
-F 0 "C30" V 4350 4200 50  0000 L CNN
+F 0 "C39" V 4350 4200 50  0000 L CNN
 F 1 "1uF" V 4350 3900 50  0000 L CNN
 F 2 "" H 4338 3950 50  0001 C CNN
@@
 	4150 4100 4100 4100
 $Comp
-L TPS3808G30DBVT U8
+L TPS3808G30DBVT U9
 U 1 1 5AC8A118
 P 7200 3700
-F 0 "U8" H 6900 4050 60  0000 C CNN
+F 0 "U9" H 6900 4050 60  0000 C CNN
 F 1 "TPS3808G30DBVT" H 7600 3350 60  0000 C CNN
 F 2 "" H 7200 3700 60  0001 C CNN

Commit message: Add 3.0V LDO for display's VCI and TP_VCC, include a 3~12ms rise time delay for the 1.8V rail to turn on before the 3.0V rail, begin the WWAN M.2 schematic (found a a low-profile key B connector)
Parts:
- renumbered C39 to C42, C40 to C43, C41 to C44, C42 to C45, R45 to R46, R46 to R47, R47 to R48, R48 to R49, R49 to R50, R50 to R51, R51 to R52, U9 to U10
Changed lines of the file:
@@
 $Descr A4 11693 8268
 encoding utf-8
-Sheet 5 13
+Sheet 5 14
 Title "Reset & Watchdog"
-Date "2018-04-09"
+Date "2018-04-10"
 Rev "v0.1.0"
 Comp "Purism SPC"
@@
 $EndDescr
 $Comp
-L SOM_SNVS_3V3 #PWR087
+L SOM_SNVS_3V3 #PWR092
 U 1 1 5AC8A151
 P 7200 3000
-F 0 "#PWR087" H 7200 2850 50  0001 C CNN
+F 0 "#PWR092" H 7200 2850 50  0001 C CNN
 F 1 "SOM_SNVS_3V3" H 7200 3140 50  0000 C CNN
 F 2 "" H 7200 3000 50  0001 C CNN
@@
 $EndComp
 $Comp
-L R R49
+L R R50
 U 1 1 5AC8A17C
 P 6600 3300
-F 0 "R49" H 6725 3350 50  0000 C CNN
+F 0 "R50" H 6725 3350 50  0000 C CNN
 F 1 "NC" H 6700 3250 50  0000 C CNN
 F 2 "" V 6530 3300 50  0001 C CNN
@@
 $EndComp
 $Comp
-L R R48
+L R R49
 U 1 1 5AC8A1A9
 P 6300 3300
-F 0 "R48" H 6425 3350 50  0000 C CNN
+F 0 "R49" H 6425 3350 50  0000 C CNN
 F 1 "100k" H 6450 3250 50  0000 C CNN
 F 2 "" V 6230 3300 50  0001 C CNN
@@
 $EndComp
 $Comp
-L C C41
+L C C44
 U 1 1 5AC8ACD0
 P 5450 3500
-F 0 "C41" V 5500 3600 50  0000 L CNN
+F 0 "C44" V 5500 3600 50  0000 L CNN
 F 1 "2.2uF" V 5500 3250 50  0000 L CNN
 F 2 "" H 5488 3350 50  0001 C CNN
@@
 	5600 3500 6650 3500
 $Comp
-L C C42
+L C C45
 U 1 1 5AC8B0DE
 P 5450 3700
-F 0 "C42" V 5500 3800 50  0000 L CNN
+F 0 "C45" V 5500 3800 50  0000 L CNN
 F 1 "NC" V 5500 3450 50  0000 L CNN
 F 2 "" H 5488 3550 50  0001 C CNN
@@
 $EndComp
 $Comp
-L GND #PWR088
+L GND #PWR093
 U 1 1 5AC8B439
 P 5250 3750
-F 0 "#PWR088" H 5250 3500 50  0001 C CNN
+F 0 "#PWR093" H 5250 3500 50  0001 C CNN
 F 1 "GND" H 5250 3600 50  0000 C CNN
 F 2 "" H 5250 3750 50  0001 C CNN
@@
 	7200 3000 7200 3200
 $Comp
-L R R47
+L R R48
 U 1 1 5AC8B597
 P 5150 3300
-F 0 "R47" H 5275 3350 50  0000 C CNN
+F 0 "R48" H 5275 3350 50  0000 C CNN
 F 1 "21.5k" H 5300 3250 50  0000 C CNN
 F 2 "" V 5080 3300 50  0001 C CNN
@@
 $EndComp
 $Comp
-L C C40
+L C C43
 U 1 1 5AC8BC45
 P 4600 3700
-F 0 "C40" H 4625 3800 50  0000 L CNN
+F 0 "C43" H 4625 3800 50  0000 L CNN
 F 1 "1nF" H 4625 3600 50  0000 L CNN
 F 2 "" H 4638 3550 50  0001 C CNN
@@
 $EndComp
 $Comp
-L GND #PWR089
+L GND #PWR094
 U 1 1 5AC8BC81
 P 4600 3900
-F 0 "#PWR089" H 4600 3650 50  0001 C CNN
+F 0 "#PWR094" H 4600 3650 50  0001 C CNN
 F 1 "GND" H 4600 3750 50  0000 C CNN
 F 2 "" H 4600 3900 50  0001 C CNN
@@
 Connection ~ 5150 3500
 $Comp
-L R R46
+L R R47
 U 1 1 5AC8C0DB
 P 4600 4300
-F 0 "R46" H 4725 4350 50  0000 C CNN
+F 0 "R47" H 4725 4350 50  0000 C CNN
 F 1 "1M" H 4700 4250 50  0000 C CNN
 F 2 "" V 4530 4300 50  0001 C CNN
@@
 Connection ~ 4600 4100
 $Comp
-L GND #PWR090
+L GND #PWR095
 U 1 1 5AC8CD8F
 P 4600 4500
-F 0 "#PWR090" H 4600 4250 50  0001 C CNN
+F 0 "#PWR095" H 4600 4250 50  0001 C CNN
 F 1 "GND" H 4600 4350 50  0000 C CNN
 F 2 "" H 4600 4500 50  0001 C CNN
@@
 	4600 4500 4600 4450
 $Comp
-L GND #PWR091
+L GND #PWR096
 U 1 1 5AC8D3A2
 P 7200 4250
-F 0 "#PWR091" H 7200 4000 50  0001 C CNN
+F 0 "#PWR096" H 7200 4000 50  0001 C CNN
 F 1 "GND" H 7200 4100 50  0000 C CNN
 F 2 "" H 7200 4250 50  0001 C CNN
@@
 	7200 4250 7200 4200
 $Comp
-L R R50
+L R R51
 U 1 1 5AC8D701
 P 8000 3400
-F 0 "R50" V 8080 3400 50  0000 C CNN
+F 0 "R51" V 8080 3400 50  0000 C CNN
 F 1 "120" V 7900 3400 50  0000 C CNN
 F 2 "" V 7930 3400 50  0001 C CNN
@@
 $EndComp
 $Comp
-L R R51
+L R R52
 U 1 1 5AC8D7F2
 P 8000 3700
-F 0 "R51" V 8080 3700 50  0000 C CNN
+F 0 "R52" V 8080 3700 50  0000 C CNN
 F 1 "0" V 7900 3700 50  0000 C CNN
 F 2 "" V 7930 3700 50  0001 C CNN
@@
 $EndComp
 $Comp
-L GND #PWR092
+L GND #PWR097
 U 1 1 5AC9A292
 P 3100 3800
-F 0 "#PWR092" H 3100 3550 50  0001 C CNN
+F 0 "#PWR097" H 3100 3550 50  0001 C CNN
 F 1 "GND" H 3100 3650 50  0000 C CNN
 F 2 "" H 3100 3800 50  0001 C CNN
@@
 SW_~RST
 $Comp
-L R R45
+L R R46
 U 1 1 5AC9A911
 P 4300 3500
-F 0 "R45" V 4380 3500 50  0000 C CNN
+F 0 "R46" V 4380 3500 50  0000 C CNN
 F 1 "120" V 4200 3500 50  0000 C CNN
 F 2 "" V 4230 3500 50  0001 C CNN
@@
 $EndComp
 $Comp
-L C C39
+L C C42
 U 1 1 5AC9A94A
 P 4300 4100
-F 0 "C39" V 4350 4200 50  0000 L CNN
+F 0 "C42" V 4350 4200 50  0000 L CNN
 F 1 "1uF" V 4350 3900 50  0000 L CNN
 F 2 "" H 4338 3950 50  0001 C CNN
@@
 	4150 4100 4100 4100
 $Comp
-L TPS3808G30DBVT U9
+L TPS3808G30DBVT U10
 U 1 1 5AC8A118
 P 7200 3700
-F 0 "U9" H 6900 4050 60  0000 C CNN
+F 0 "U10" H 6900 4050 60  0000 C CNN
 F 1 "TPS3808G30DBVT" H 7600 3350 60  0000 C CNN
 F 2 "" H 7200 3700 60  0001 C CNN
