File: watchdog.sch (KiCad schematic (older format))
At the start: 17 parts, among them SW2 SW_Push, U10 TPS3808G30DBVT

Commit message: Assign all associated signals to their respective pins on the EmCraft i.MX8M SoM
The ERC is now at the same state as the DART SoM schematic. Need to compare various aspects of the current schematic against the EmCraft reference design. The main buck-boost will likely need to be switched to a 5V regulator, or be configured to output 5V.

A regulator will likely need to be added which will output some VBAT voltage level (3.5~4.2V) for the M.2 cards. The SIM7100 for example requires at least 3.4V!
Parts:
- renumbered C42 to C45, C43 to C46, C44 to C47, C45 to C48
Changed lines of the file:
@@
 $EndDescr
 $Comp
-L SOM_SNVS_3V3 #PWR092
+L SOM_SNVS_3V3 #PWR093
 U 1 1 5AC8A151
 P 7200 3000
-F 0 "#PWR092" H 7200 2850 50  0001 C CNN
+F 0 "#PWR093" H 7200 2850 50  0001 C CNN
 F 1 "SOM_SNVS_3V3" H 7200 3140 50  0000 C CNN
 F 2 "" H 7200 3000 50  0001 C CNN
@@
 $EndComp
 $Comp
-L C C44
+L C C47
 U 1 1 5AC8ACD0
 P 5450 3500
-F 0 "C44" V 5500 3600 50  0000 L CNN
+F 0 "C47" V 5500 3600 50  0000 L CNN
 F 1 "2.2uF" V 5500 3250 50  0000 L CNN
 F 2 "" H 5488 3350 50  0001 C CNN
@@
 	5600 3500 6650 3500
 $Comp
-L C C45
+L C C48
 U 1 1 5AC8B0DE
 P 5450 3700
-F 0 "C45" V 5500 3800 50  0000 L CNN
+F 0 "C48" V 5500 3800 50  0000 L CNN
 F 1 "NC" V 5500 3450 50  0000 L CNN
 F 2 "" H 5488 3550 50  0001 C CNN
@@
 $EndComp
 $Comp
-L GND #PWR093
+L GND #PWR094
 U 1 1 5AC8B439
 P 5250 3750
-F 0 "#PWR093" H 5250 3500 50  0001 C CNN
+F 0 "#PWR094" H 5250 3500 50  0001 C CNN
 F 1 "GND" H 5250 3600 50  0000 C CNN
 F 2 "" H 5250 3750 50  0001 C CNN
@@
 $EndComp
 $Comp
-L C C43
+L C C46
 U 1 1 5AC8BC45
 P 4600 3700
-F 0 "C43" H 4625 3800 50  0000 L CNN
+F 0 "C46" H 4625 3800 50  0000 L CNN
 F 1 "1nF" H 4625 3600 50  0000 L CNN
 F 2 "" H 4638 3550 50  0001 C CNN
@@
 $EndComp
 $Comp
-L GND #PWR094
+L GND #PWR095
 U 1 1 5AC8BC81
 P 4600 3900
-F 0 "#PWR094" H 4600 3650 50  0001 C CNN
+F 0 "#PWR095" H 4600 3650 50  0001 C CNN
 F 1 "GND" H 4600 3750 50  0000 C CNN
 F 2 "" H 4600 3900 50  0001 C CNN
@@
 Connection ~ 4600 4100
 $Comp
-L GND #PWR095
+L GND #PWR096
 U 1 1 5AC8CD8F
 P 4600 4500
-F 0 "#PWR095" H 4600 4250 50  0001 C CNN
+F 0 "#PWR096" H 4600 4250 50  0001 C CNN
 F 1 "GND" H 4600 4350 50  0000 C CNN
 F 2 "" H 4600 4500 50  0001 C CNN
@@
 	4600 4500 4600 4450
 $Comp
-L GND #PWR096
+L GND #PWR097
 U 1 1 5AC8D3A2
 P 7200 4250
-F 0 "#PWR096" H 7200 4000 50  0001 C CNN
+F 0 "#PWR097" H 7200 4000 50  0001 C CNN
 F 1 "GND" H 7200 4100 50  0000 C CNN
 F 2 "" H 7200 4250 50  0001 C CNN
@@
 $EndComp
 $Comp
-L GND #PWR097
+L GND #PWR098
 U 1 1 5AC9A292
 P 3100 3800
-F 0 "#PWR097" H 3100 3550 50  0001 C CNN
+F 0 "#PWR098" H 3100 3550 50  0001 C CNN
 F 1 "GND" H 3100 3650 50  0000 C CNN
 F 2 "" H 3100 3800 50  0001 C CNN
@@
 $EndComp
 $Comp
-L C C42
+L C C45
 U 1 1 5AC9A94A
 P 4300 4100
-F 0 "C42" V 4350 4200 50  0000 L CNN
+F 0 "C45" V 4350 4200 50  0000 L CNN
 F 1 "1uF" V 4350 3900 50  0000 L CNN
 F 2 "" H 4338 3950 50  0001 C CNN

Commit message: Use "Start to sheet number*100 and use first free number" designation, any new component added to the schematic will occupy the next available number in that sheet
For example: if sheet 2 has R201-R215 and we add a new resistor it will become R216.
Parts:
- renumbered C45 to C501, C46 to C502, C47 to C503, C48 to C504, D5 to D501, D6 to D502, D7 to D503, D8 to D504, R46 to R501, R47 to R502, R48 to R503, R49 to R504, R50 to R505, R51 to R506, R52 to R507, SW2 to SW501, U10 to U501
Changed lines of the file:
@@
 $EndDescr
 $Comp
-L SOM_SNVS_3V3 #PWR093
+L SOM_SNVS_3V3 #PWR505
 U 1 1 5AC8A151
 P 7200 3000
-F 0 "#PWR093" H 7200 2850 50  0001 C CNN
+F 0 "#PWR505" H 7200 2850 50  0001 C CNN
 F 1 "SOM_SNVS_3V3" H 7200 3140 50  0000 C CNN
 F 2 "" H 7200 3000 50  0001 C CNN
@@
 $EndComp
 $Comp
-L R R50
+L R R505
 U 1 1 5AC8A17C
 P 6600 3300
-F 0 "R50" H 6725 3350 50  0000 C CNN
+F 0 "R505" H 6725 3350 50  0000 C CNN
 F 1 "NC" H 6700 3250 50  0000 C CNN
 F 2 "" V 6530 3300 50  0001 C CNN
@@
 $EndComp
 $Comp
-L R R49
+L R R504
 U 1 1 5AC8A1A9
 P 6300 3300
-F 0 "R49" H 6425 3350 50  0000 C CNN
+F 0 "R504" H 6425 3350 50  0000 C CNN
 F 1 "100k" H 6450 3250 50  0000 C CNN
 F 2 "" V 6230 3300 50  0001 C CNN
@@
 $EndComp
 $Comp
-L D_Schottky D8
+L D_Schottky D504
 U 1 1 5AC8A554
 P 6000 3300
-F 0 "D8" V 5900 3200 50  0000 C CNN
+F 0 "D504" V 5900 3200 50  0000 C CNN
 F 1 "30V,100mA" V 6100 3050 50  0000 C CNN
 F 2 "" H 6000 3300 50  0001 C CNN
@@
 $EndComp
 $Comp
-L C C47
+L C C503
 U 1 1 5AC8ACD0
 P 5450 3500
-F 0 "C47" V 5500 3600 50  0000 L CNN
+F 0 "C503" V 5500 3600 50  0000 L CNN
 F 1 "2.2uF" V 5500 3250 50  0000 L CNN
 F 2 "" H 5488 3350 50  0001 C CNN
@@
 	5600 3500 6650 3500
 $Comp
-L C C48
+L C C504
 U 1 1 5AC8B0DE
 P 5450 3700
-F 0 "C48" V 5500 3800 50  0000 L CNN
+F 0 "C504" V 5500 3800 50  0000 L CNN
 F 1 "NC" V 5500 3450 50  0000 L CNN
 F 2 "" H 5488 3550 50  0001 C CNN
@@
 $EndComp
 $Comp
-L GND #PWR094
+L GND #PWR504
 U 1 1 5AC8B439
 P 5250 3750
-F 0 "#PWR094" H 5250 3500 50  0001 C CNN
+F 0 "#PWR504" H 5250 3500 50  0001 C CNN
 F 1 "GND" H 5250 3600 50  0000 C CNN
 F 2 "" H 5250 3750 50  0001 C CNN
@@
 	7200 3000 7200 3200
 $Comp
-L R R48
+L R R503
 U 1 1 5AC8B597
 P 5150 3300
-F 0 "R48" H 5275 3350 50  0000 C CNN
+F 0 "R503" H 5275 3350 50  0000 C CNN
 F 1 "21.5k" H 5300 3250 50  0000 C CNN
 F 2 "" V 5080 3300 50  0001 C CNN
@@
 Connection ~ 6000 3500
 $Comp
-L D_Schottky D6
+L D_Schottky D502
 U 1 1 5AC8BA0F
 P 4900 3500
-F 0 "D6" H 4900 3600 50  0000 C CNN
+F 0 "D502" H 4900 3600 50  0000 C CNN
 F 1 "30V,100mA" H 4900 3400 50  0000 C CNN
 F 2 "" H 4900 3500 50  0001 C CNN
@@
 $EndComp
 $Comp
-L D_Schottky D7
+L D_Schottky D503
 U 1 1 5AC8BB44
 P 4900 4100
-F 0 "D7" H 4900 4200 50  0000 C CNN
+F 0 "D503" H 4900 4200 50  0000 C CNN
 F 1 "30V,100mA" H 4900 4000 50  0000 C CNN
 F 2 "" H 4900 4100 50  0001 C CNN
@@
 $EndComp
 $Comp
-L C C46
+L C C502
 U 1 1 5AC8BC45
 P 4600 3700
-F 0 "C46" H 4625 3800 50  0000 L CNN
+F 0 "C502" H 4625 3800 50  0000 L CNN
 F 1 "1nF" H 4625 3600 50  0000 L CNN
 F 2 "" H 4638 3550 50  0001 C CNN
@@
 $EndComp
 $Comp
-L GND #PWR095
+L GND #PWR502
 U 1 1 5AC8BC81
 P 4600 3900
-F 0 "#PWR095" H 4600 3650 50  0001 C CNN
+F 0 "#PWR502" H 4600 3650 50  0001 C CNN
 F 1 "GND" H 4600 3750 50  0000 C CNN
 F 2 "" H 4600 3900 50  0001 C CNN
@@
 Connection ~ 5150 3500
 $Comp
-L R R47
+L R R502
 U 1 1 5AC8C0DB
 P 4600 4300
-F 0 "R47" H 4725 4350 50  0000 C CNN
+F 0 "R502" H 4725 4350 50  0000 C CNN
 F 1 "1M" H 4700 4250 50  0000 C CNN
 F 2 "" V 4530 4300 50  0001 C CNN
@@
 Connection ~ 4600 4100
 $Comp
-L GND #PWR096
+L GND #PWR503
 U 1 1 5AC8CD8F
 P 4600 4500
-F 0 "#PWR096" H 4600 4250 50  0001 C CNN
+F 0 "#PWR503" H 4600 4250 50  0001 C CNN
 F 1 "GND" H 4600 4350 50  0000 C CNN
 F 2 "" H 4600 4500 50  0001 C CNN
@@
 	4600 4500 4600 4450
 $Comp
-L GND #PWR097
+L GND #PWR506
 U 1 1 5AC8D3A2
 P 7200 4250
-F 0 "#PWR097" H 7200 4000 50  0001 C CNN
+F 0 "#PWR506" H 7200 4000 50  0001 C CNN
 F 1 "GND" H 7200 4100 50  0000 C CNN
 F 2 "" H 7200 4250 50  0001 C CNN
@@
 	7200 4250 7200 4200
 $Comp
-L R R51
+L R R506
 U 1 1 5AC8D701
 P 8000 3400
-F 0 "R51" V 8080 3400 50  0000 C CNN
+F 0 "R506" V 8080 3400 50  0000 C CNN
 F 1 "120" V 7900 3400 50  0000 C CNN
 F 2 "" V 7930 3400 50  0001 C CNN
@@
 $EndComp
 $Comp
-L R R52
+L R R507
 U 1 1 5AC8D7F2
 P 8000 3700
-F 0 "R52" V 8080 3700 50  0000 C CNN
+F 0 "R507" V 8080 3700 50  0000 C CNN
 F 1 "0" V 7900 3700 50  0000 C CNN
 F 2 "" V 7930 3700 50  0001 C CNN
@@
 	8150 3700 8200 3700
 $Comp
-L SW_Push SW2
+L SW_Push SW501
 U 1 1 5AC99959
 P 3500 3500
-F 0 "SW2" H 3550 3600 50  0000 L CNN
+F 0 "SW501" H 3550 3600 50  0000 L CNN
 F 1 "SW_Push" H 3500 3440 50  0000 C CNN
 F 2 "" H 3500 3700 50  0001 C CNN
@@
 $EndComp
 $Comp
-L TVS_DIODE D5
+L TVS_DIODE D501
 U 1 1 5AC99E1E
 P 3500 3750
-F 0 "D5" H 3500 3850 50  0000 C CNN
+F 0 "D501" H 3500 3850 50  0000 C CNN
 F 1 "TPD1E10B09DPYR" H 3500 3650 50  0000 C CNN
 F 2 "" H 3600 3750 50  0001 C CNN
@@
 $EndComp
 $Comp
-L GND #PWR098
+L GND #PWR501
 U 1 1 5AC9A292
 P 3100 3800
-F 0 "#PWR098" H 3100 3550 50  0001 C CNN
+F 0 "#PWR501" H 3100 3550 50  0001 C CNN
 F 1 "GND" H 3100 3650 50  0000 C CNN
 F 2 "" H 3100 3800 50  0001 C CNN
@@
 SW_~RST
 $Comp
-L R R46
+L R R501
 U 1 1 5AC9A911
 P 4300 3500
-F 0 "R46" V 4380 3500 50  0000 C CNN
+F 0 "R501" V 4380 3500 50  0000 C CNN
 F 1 "120" V 4200 3500 50  0000 C CNN
 F 2 "" V 4230 3500 50  0001 C CNN
@@
 $EndComp
 $Comp
-L C C45
+L C C501
 U 1 1 5AC9A94A
 P 4300 4100
-F 0 "C45" V 4350 4200 50  0000 L CNN
+F 0 "C501" V 4350 4200 50  0000 L CNN
 F 1 "1uF" V 4350 3900 50  0000 L CNN
 F 2 "" H 4338 3950 50  0001 C CNN
@@
 	4150 4100 4100 4100
 $Comp
-L TPS3808G30DBVT U10
+L TPS3808G30DBVT U501
 U 1 1 5AC8A118
 P 7200 3700
-F 0 "U10" H 6900 4050 60  0000 C CNN
+F 0 "U501" H 6900 4050 60  0000 C CNN
 F 1 "TPS3808G30DBVT" H 7600 3350 60  0000 C CNN
 F 2 "" H 7200 3700 60  0001 C CNN

Commit message: Move reference designators in the schematic so that they are legible
Connections:
- wire segments 38 -> 53
Other:
- moved on the sheet: C501, C502, D501, D502, D503, R501, R502, R503, SW501

Commit message: Include reverse polarity protection circuit along with a simulation showing its effectiveness
Protecting VBAT from when board is sinking current via USB C. Protects against reverse polarity at the DC jack.

In EmCraft's instance VBUS should only be 5V when sinking current but they must protect against the condition when VBUS>12V and DC_IN=12V. This may need testing.
Connections:
- net labels added: 3V3_OUT
- net labels removed: SOM_SNVS_3V3
- wire segments 53 -> 38
Changed lines of the file:
@@
 Sheet 5 14
 Title "Reset & Watchdog"
-Date "2018-04-16"
+Date "2018-04-18"
 Rev "v0.1.0"
 Comp "Purism SPC"
@@
 Comment4 ""
 $EndDescr
-$Comp
-L SOM_SNVS_3V3 #PWR093
-U 1 1 5AC8A151
-P 7200 3000
-F 0 "#PWR093" H 7200 2850 50  0001 C CNN
-F 1 "SOM_SNVS_3V3" H 7200 3140 50  0000 C CNN
-F 2 "" H 7200 3000 50  0001 C CNN
-F 3 "" H 7200 3000 50  0001 C CNN
-	1    7200 3000
-	1    0    0    -1
-$EndComp
 $Comp
 L R R505
@@
 $EndComp
 Wire Wire Line
-	5600 3500 6000 3500
-Wire Wire Line
-	6000 3500 6300 3500
-Wire Wire Line
-	6300 3500 6650 3500
+	5600 3500 6650 3500
 $Comp
 L C C504
@@
 $EndComp
 $Comp
-L GND #PWR094
+L GND #PWR095
 U 1 1 5AC8B439
 P 5200 3750
-F 0 "#PWR094" H 5200 3500 50  0001 C CNN
+F 0 "#PWR095" H 5200 3500 50  0001 C CNN
 F 1 "GND" H 5200 3600 50  0000 C CNN
 F 2 "" H 5200 3750 50  0001 C CNN
@@
 	5300 3500 5200 3500
 Wire Wire Line
-	5200 3500 5200 3700
-Wire Wire Line
-	5200 3700 5200 3750
+	5200 3500 5200 3750
 Wire Wire Line
 	5300 3700 5200 3700
 Connection ~ 5200 3700
 Wire Wire Line
-	5600 3700 6600 3700
-Wire Wire Line
-	6600 3700 6650 3700
+	5600 3700 6650 3700
 Wire Wire Line
 	6600 3450 6600 3700
 Connection ~ 6600 3700
 Wire Wire Line
-	7200 3000 7200 3100
-Wire Wire Line
-	7200 3100 7200 3200
+	7200 3000 7200 3200
 $Comp
 L R R503
@@
 $EndComp
 Wire Wire Line
-	5100 3100 6000 3100
-Wire Wire Line
-	6000 3100 6300 3100
-Wire Wire Line
-	6300 3100 6600 3100
-Wire Wire Line
-	6600 3100 7200 3100
+	5100 3100 7200 3100
 Wire Wire Line
 	5100 3100 5100 3150
@@
 $EndComp
 $Comp
-L GND #PWR095
+L GND #PWR096
 U 1 1 5AC8BC81
 P 4550 3900
-F 0 "#PWR095" H 4550 3650 50  0001 C CNN
+F 0 "#PWR096" H 4550 3650 50  0001 C CNN
 F 1 "GND" H 4550 3750 50  0000 C CNN
 F 2 "" H 4550 3900 50  0001 C CNN
@@
 	6600 3900 6600 4100
 Wire Wire Line
-	6600 4100 5100 4100
-Wire Wire Line
-	5100 4100 5000 4100
-Wire Wire Line
-	5100 3450 5100 3500
-Wire Wire Line
-	5100 3500 5100 4100
+	6600 4100 5000 4100
+Wire Wire Line
+	5100 3450 5100 4100
 Connection ~ 5100 4100
 Wire Wire Line
@@
 GPIO1_IO02(~WDOG~)
 Wire Wire Line
-	3600 3500 3650 3500
-Wire Wire Line
-	3650 3500 4050 3500
-Wire Wire Line
-	4350 3500 4550 3500
-Wire Wire Line
-	4550 3500 4700 3500
+	3600 3500 4050 3500
+Wire Wire Line
+	4350 3500 4700 3500
 Wire Wire Line
 	4550 3550 4550 3500
@@
 	4550 3900 4550 3850
 Wire Wire Line
-	4400 4100 4550 4100
-Wire Wire Line
-	4550 4100 4700 4100
+	4400 4100 4700 4100
 Wire Wire Line
 	4550 4100 4550 4150
 Connection ~ 4550 4100
 $Comp
-L GND #PWR096
+L GND #PWR097
 U 1 1 5AC8CD8F
 P 4550 4500
-F 0 "#PWR096" H 4550 4250 50  0001 C CNN
+F 0 "#PWR097" H 4550 4250 50  0001 C CNN
 F 1 "GND" H 4550 4350 50  0000 C CNN
 F 2 "" H 4550 4500 50  0001 C CNN
@@
 	4550 4500 4550 4450
 $Comp
-L GND #PWR097
+L GND #PWR098
 U 1 1 5AC8D3A2
 P 7200 4250
-F 0 "#PWR097" H 7200 4000 50  0001 C CNN
+F 0 "#PWR098" H 7200 4000 50  0001 C CNN
 F 1 "GND" H 7200 4100 50  0000 C CNN
 F 2 "" H 7200 4250 50  0001 C CNN
@@
 $EndComp
 Wire Wire Line
-	7750 3700 7800 3700
-Wire Wire Line
-	7800 3700 7850 3700
+	7750 3700 7850 3700
 Wire Wire Line
 	7800 3700 7800 3400
@@
 $EndComp
 $Comp
-L GND #PWR098
+L GND #PWR099
 U 1 1 5AC9A292
 P 3000 3800
-F 0 "#PWR098" H 3000 3550 50  0001 C CNN
+F 0 "#PWR099" H 3000 3550 50  0001 C CNN
 F 1 "GND" H 3000 3650 50  0000 C CNN
 F 2 "" H 3000 3800 50  0001 C CNN
@@
 $EndComp
 Wire Wire Line
-	3000 3500 3000 3750
-Wire Wire Line
-	3000 3750 3000 3800
+	3000 3500 3000 3800
 Wire Wire Line
 	3000 3500 3200 3500
@@
 	1    0    0    -1
 $EndComp
+$Comp
+L 3V3_OUT #PWR0100
+U 1 1 5AE83458
+P 7200 3000
+F 0 "#PWR0100" H 7200 2850 50  0001 C CNN
+F 1 "3V3_OUT" H 7200 3140 50  0000 C CNN
+F 2 "" H 7200 3000 50  0001 C CNN
+F 3 "" H 7200 3000 50  0001 C CNN
+	1    7200 3000
+	1    0    0    -1
+$EndComp
