File: audio.sch (KiCad schematic (older format))
At the start: 25 parts, among them J10 CTIA / AHJ, U21 SGTL5000

Commit message: Begin creating the IMX8M-SOM schematic symbol, remove the old DART-MX8M symbol
Parts:
- renumbered C84 to C61, C85 to C62, C86 to C63, C87 to C64, C88 to C65, C89 to C66, C90 to C67, C91 to C68, C92 to C69, C93 to C70, C94 to C71, C95 to C72, C96 to C73, C97 to C74, D20 to D17, D21 to D18, J10 to J7, R87 to R76, R88 to R77, R89 to R78, R90 to R79, R91 to R80, U21 to U17
Changed lines of the file:
@@
 $EndDescr
 $Comp
-L SGTL5000 U21
+L SGTL5000 U17
 U 1 1 5ABE7D8D
 P 3050 3350
-F 0 "U21" H 2600 4250 60  0000 C CNN
+F 0 "U17" H 2600 4250 60  0000 C CNN
 F 1 "SGTL5000" H 3500 4250 60  0000 C CNN
 F 2 "" H 3050 3400 60  0000 C CNN
@@
 	1700 3900 2350 3900
 $Comp
-L C C87
+L C C64
 U 1 1 5ABEEF4C
 P 4700 3300
-F 0 "C87" V 4750 3350 50  0000 L CNN
+F 0 "C64" V 4750 3350 50  0000 L CNN
 F 1 "220u" V 4750 3050 50  0000 L CNN
 F 2 "" H 4738 3150 50  0001 C CNN
@@
 $EndComp
 $Comp
-L C C88
+L C C65
 U 1 1 5ABEEF73
 P 4700 3500
-F 0 "C88" V 4750 3300 50  0000 L CNN
+F 0 "C65" V 4750 3300 50  0000 L CNN
 F 1 "200u" V 4750 3550 50  0000 L CNN
 F 2 "" H 4738 3350 50  0001 C CNN
@@
 	3900 3500 4550 3500
 $Comp
-L C C85
+L C C62
 U 1 1 5ABEF358
 P 4150 3700
-F 0 "C85" H 4175 3800 50  0000 L CNN
+F 0 "C62" H 4175 3800 50  0000 L CNN
 F 1 "NC" H 4175 3600 50  0000 L CNN
 F 2 "" H 4188 3550 50  0001 C CNN
@@
 $EndComp
 $Comp
-L C C86
+L C C63
 U 1 1 5ABEF388
 P 4400 3700
-F 0 "C86" H 4425 3800 50  0000 L CNN
+F 0 "C63" H 4425 3800 50  0000 L CNN
 F 1 "NC" H 4425 3600 50  0000 L CNN
 F 2 "" H 4438 3550 50  0001 C CNN
@@
 	4150 3850 4150 3900
 $Comp
-L R R87
+L R R76
 U 1 1 5ABEFC7B
 P 5000 4050
-F 0 "R87" H 5125 4100 50  0000 C CNN
+F 0 "R76" H 5125 4100 50  0000 C CNN
 F 1 "33" H 5125 4000 50  0000 C CNN
 F 2 "" V 4930 4050 50  0001 C CNN
@@
 $EndComp
 $Comp
-L C C95
+L C C72
 U 1 1 5ABF2943
 P 8500 3700
-F 0 "C95" H 8525 3800 50  0000 L CNN
+F 0 "C72" H 8525 3800 50  0000 L CNN
 F 1 "270p" H 8525 3600 50  0000 L CNN
 F 2 "" H 8538 3550 50  0001 C CNN
@@
 $EndComp
 $Comp
-L C C93
+L C C70
 U 1 1 5ABF2987
 P 7000 3700
-F 0 "C93" H 7025 3800 50  0000 L CNN
+F 0 "C70" H 7025 3800 50  0000 L CNN
 F 1 "270p" H 7025 3600 50  0000 L CNN
 F 2 "" H 7038 3550 50  0001 C CNN
@@
 Connection ~ 4150 3300
 $Comp
-L C C89
+L C C66
 U 1 1 5ABF4002
 P 5000 3700
-F 0 "C89" H 5025 3800 50  0000 L CNN
+F 0 "C66" H 5025 3800 50  0000 L CNN
 F 1 "100n" H 5025 3600 50  0000 L CNN
 F 2 "" H 5038 3550 50  0001 C CNN
@@
 $EndComp
 $Comp
-L C C90
+L C C67
 U 1 1 5ABF490A
 P 5300 3900
-F 0 "C90" H 5325 4000 50  0000 L CNN
+F 0 "C67" H 5325 4000 50  0000 L CNN
 F 1 "100p" H 5325 3800 50  0000 L CNN
 F 2 "" H 5338 3750 50  0001 C CNN
@@
 $EndComp
 $Comp
-L R R88
+L R R77
 U 1 1 5ABF49BF
 P 5600 3900
-F 0 "R88" H 5725 3950 50  0000 C CNN
+F 0 "R77" H 5725 3950 50  0000 C CNN
 F 1 "15k" H 5725 3850 50  0000 C CNN
 F 2 "" V 5530 3900 50  0001 C CNN
@@
 Connection ~ 5600 3300
 $Comp
-L R R89
+L R R78
 U 1 1 5ABF53AE
 P 5900 4050
-F 0 "R89" H 6025 4100 50  0000 C CNN
+F 0 "R78" H 6025 4100 50  0000 C CNN
 F 1 "33" H 6025 4000 50  0000 C CNN
 F 2 "" V 5830 4050 50  0001 C CNN
@@
 	5900 4200 5900 4250
 $Comp
-L C C91
+L C C68
 U 1 1 5ABF53BC
 P 5900 3700
-F 0 "C91" H 5925 3800 50  0000 L CNN
+F 0 "C68" H 5925 3800 50  0000 L CNN
 F 1 "100n" H 5925 3600 50  0000 L CNN
 F 2 "" H 5938 3550 50  0001 C CNN
@@
 $EndComp
 $Comp
-L C C92
+L C C69
 U 1 1 5ABF53C2
 P 6200 3900
-F 0 "C92" H 6225 4000 50  0000 L CNN
+F 0 "C69" H 6225 4000 50  0000 L CNN
 F 1 "100p" H 6225 3800 50  0000 L CNN
 F 2 "" H 6238 3750 50  0001 C CNN
@@
 $EndComp
 $Comp
-L R R90
+L R R79
 U 1 1 5ABF53C8
 P 6500 3900
-F 0 "R90" H 6625 3950 50  0000 C CNN
+F 0 "R79" H 6625 3950 50  0000 C CNN
 F 1 "15k" H 6625 3850 50  0000 C CNN
 F 2 "" V 6430 3900 50  0001 C CNN
@@
 Connection ~ 6500 3500
 $Comp
-L D_TVS_ALT D20
+L D_TVS_ALT D17
 U 1 1 5ABF82C5
 P 7400 3700
-F 0 "D20" V 7350 3800 50  0000 C CNN
+F 0 "D17" V 7350 3800 50  0000 C CNN
 F 1 "ESD5B5.0S" V 7450 3950 50  0000 C CNN
 F 2 "" H 7400 3700 50  0001 C CNN
@@
 	7400 3900 7400 3850
 $Comp
-L D_TVS_ALT D21
+L D_TVS_ALT D18
 U 1 1 5ABF8533
 P 7950 3700
-F 0 "D21" V 7900 3800 50  0000 C CNN
+F 0 "D18" V 7900 3800 50  0000 C CNN
 F 1 "ESD5B5.0S" V 8000 3950 50  0000 C CNN
 F 2 "" H 7950 3700 50  0001 C CNN
@@
 Connection ~ 7950 3500
 $Comp
-L Audio-Jack-5 J10
+L Audio-Jack-5 J7
 U 1 1 5ABF9919
 P 9550 3400
-F 0 "J10" H 9500 3610 50  0000 C CNN
+F 0 "J7" H 9500 3610 50  0000 C CNN
 F 1 "CTIA / AHJ" H 9575 3025 50  0000 C CNN
 F 2 "" H 9800 3500 50  0001 C CNN
@@
 MIC_IN
 $Comp
-L C C84
+L C C61
 U 1 1 5ABFC3EE
 P 3800 3900
-F 0 "C84" H 3825 4000 50  0000 L CNN
+F 0 "C61" H 3825 4000 50  0000 L CNN
 F 1 "100n" H 3825 3800 50  0000 L CNN
 F 2 "" H 3838 3750 50  0001 C CNN
@@
 NoConn ~ 3750 3550
 $Comp
-L C C97
+L C C74
 U 1 1 5AC79EEC
 P 9100 3800
-F 0 "C97" H 9125 3900 50  0000 L CNN
+F 0 "C74" H 9125 3900 50  0000 L CNN
 F 1 "270pF" H 9125 3700 50  0000 L CNN
 F 2 "" H 9138 3650 50  0001 C CNN
@@
 	9000 3600 9350 3600
 $Comp
-L R R91
+L R R80
 U 1 1 5AC7B464
 P 8500 4550
-F 0 "R91" V 8400 4550 50  0000 C CNN
+F 0 "R80" V 8400 4550 50  0000 C CNN
 F 1 "2.2k" V 8600 4550 50  0000 C CNN
 F 2 "" V 8430 4550 50  0001 C CNN
@@
 	8750 3600 8800 3600
 $Comp
-L C C96
+L C C73
 U 1 1 5AC7B848
 P 8500 4300
-F 0 "C96" V 8550 4150 50  0000 L CNN
+F 0 "C73" V 8550 4150 50  0000 L CNN
 F 1 "100nF" V 8625 4175 50  0000 L CNN
 F 2 "" H 8538 4150 50  0001 C CNN
@@
 Connection ~ 8750 4300
 $Comp
-L C C94
+L C C71
 U 1 1 5AC7BC8A
 P 8300 4750
-F 0 "C94" H 8325 4850 50  0000 L CNN
+F 0 "C71" H 8325 4850 50  0000 L CNN
 F 1 "1uF" H 8325 4650 50  0000 L CNN
 F 2 "" H 8338 4600 50  0001 C CNN

Commit message: Assign all associated signals to their respective pins on the EmCraft i.MX8M SoM
The ERC is now at the same state as the DART SoM schematic. Need to compare various aspects of the current schematic against the EmCraft reference design. The main buck-boost will likely need to be switched to a 5V regulator, or be configured to output 5V.

A regulator will likely need to be added which will output some VBAT voltage level (3.5~4.2V) for the M.2 cards. The SIM7100 for example requires at least 3.4V!
Parts:
- renumbered C61 to C64, C62 to C65, C63 to C66, C64 to C67, C65 to C68, C66 to C69, C67 to C70, C68 to C71, C69 to C72, C70 to C73, C71 to C74, C72 to C75, C73 to C76, C74 to C77
Changed lines of the file:
@@
 $EndComp
 $Comp
-L GND #PWR0157
+L GND #PWR0159
 U 1 1 5ABE80CA
 P 3050 4450
-F 0 "#PWR0157" H 3050 4200 50  0001 C CNN
+F 0 "#PWR0159" H 3050 4200 50  0001 C CNN
 F 1 "GND" H 3050 4300 50  0000 C CNN
 F 2 "" H 3050 4450 50  0001 C CNN
@@
 	1700 3900 2350 3900
 $Comp
-L C C64
+L C C67
 U 1 1 5ABEEF4C
 P 4700 3300
-F 0 "C64" V 4750 3350 50  0000 L CNN
+F 0 "C67" V 4750 3350 50  0000 L CNN
 F 1 "220u" V 4750 3050 50  0000 L CNN
 F 2 "" H 4738 3150 50  0001 C CNN
@@
 $EndComp
 $Comp
-L C C65
+L C C68
 U 1 1 5ABEEF73
 P 4700 3500
-F 0 "C65" V 4750 3300 50  0000 L CNN
+F 0 "C68" V 4750 3300 50  0000 L CNN
 F 1 "200u" V 4750 3550 50  0000 L CNN
 F 2 "" H 4738 3350 50  0001 C CNN
@@
 	3900 3500 4550 3500
 $Comp
-L C C62
+L C C65
 U 1 1 5ABEF358
 P 4150 3700
-F 0 "C62" H 4175 3800 50  0000 L CNN
+F 0 "C65" H 4175 3800 50  0000 L CNN
 F 1 "NC" H 4175 3600 50  0000 L CNN
 F 2 "" H 4188 3550 50  0001 C CNN
@@
 $EndComp
 $Comp
-L C C63
+L C C66
 U 1 1 5ABEF388
 P 4400 3700
-F 0 "C63" H 4425 3800 50  0000 L CNN
+F 0 "C66" H 4425 3800 50  0000 L CNN
 F 1 "NC" H 4425 3600 50  0000 L CNN
 F 2 "" H 4438 3550 50  0001 C CNN
@@
 $EndComp
 $Comp
-L GND #PWR0158
+L GND #PWR0160
 U 1 1 5ABEF777
 P 4400 3900
-F 0 "#PWR0158" H 4400 3650 50  0001 C CNN
+F 0 "#PWR0160" H 4400 3650 50  0001 C CNN
 F 1 "GND" H 4400 3750 50  0000 C CNN
 F 2 "" H 4400 3900 50  0001 C CNN
@@
 $EndComp
 $Comp
-L GND #PWR0159
+L GND #PWR0161
 U 1 1 5ABEF798
 P 4150 3900
-F 0 "#PWR0159" H 4150 3650 50  0001 C CNN
+F 0 "#PWR0161" H 4150 3650 50  0001 C CNN
 F 1 "GND" H 4150 3750 50  0000 C CNN
 F 2 "" H 4150 3900 50  0001 C CNN
@@
 	5000 3850 5000 3900
 $Comp
-L GND #PWR0160
+L GND #PWR0162
 U 1 1 5ABF0047
 P 5300 4300
-F 0 "#PWR0160" H 5300 4050 50  0001 C CNN
+F 0 "#PWR0162" H 5300 4050 50  0001 C CNN
 F 1 "GND" H 5300 4150 50  0000 C CNN
 F 2 "" H 5300 4300 50  0001 C CNN
@@
 $EndComp
 $Comp
-L C C72
+L C C75
 U 1 1 5ABF2943
 P 8500 3700
-F 0 "C72" H 8525 3800 50  0000 L CNN
+F 0 "C75" H 8525 3800 50  0000 L CNN
 F 1 "270p" H 8525 3600 50  0000 L CNN
 F 2 "" H 8538 3550 50  0001 C CNN
@@
 $EndComp
 $Comp
-L C C70
+L C C73
 U 1 1 5ABF2987
 P 7000 3700
-F 0 "C70" H 7025 3800 50  0000 L CNN
+F 0 "C73" H 7025 3800 50  0000 L CNN
 F 1 "270p" H 7025 3600 50  0000 L CNN
 F 2 "" H 7038 3550 50  0001 C CNN
@@
 	8500 3500 8500 3550
 $Comp
-L GND #PWR0161
+L GND #PWR0163
 U 1 1 5ABF2BDF
 P 8500 3900
-F 0 "#PWR0161" H 8500 3650 50  0001 C CNN
+F 0 "#PWR0163" H 8500 3650 50  0001 C CNN
 F 1 "GND" H 8500 3750 50  0000 C CNN
 F 2 "" H 8500 3900 50  0001 C CNN
@@
 	8500 3900 8500 3850
 $Comp
-L GND #PWR0162
+L GND #PWR0164
 U 1 1 5ABF2C32
 P 7000 3900
-F 0 "#PWR0162" H 7000 3650 50  0001 C CNN
+F 0 "#PWR0164" H 7000 3650 50  0001 C CNN
 F 1 "GND" H 7000 3750 50  0000 C CNN
 F 2 "" H 7000 3900 50  0001 C CNN
@@
 Connection ~ 4150 3300
 $Comp
-L C C66
+L C C69
 U 1 1 5ABF4002
 P 5000 3700
-F 0 "C66" H 5025 3800 50  0000 L CNN
+F 0 "C69" H 5025 3800 50  0000 L CNN
 F 1 "100n" H 5025 3600 50  0000 L CNN
 F 2 "" H 5038 3550 50  0001 C CNN
@@
 $EndComp
 $Comp
-L C C67
+L C C70
 U 1 1 5ABF490A
 P 5300 3900
-F 0 "C67" H 5325 4000 50  0000 L CNN
+F 0 "C70" H 5325 4000 50  0000 L CNN
 F 1 "100p" H 5325 3800 50  0000 L CNN
 F 2 "" H 5338 3750 50  0001 C CNN
@@
 	5900 3850 5900 3900
 $Comp
-L GND #PWR0163
+L GND #PWR0165
 U 1 1 5ABF53B5
 P 6200 4300
-F 0 "#PWR0163" H 6200 4050 50  0001 C CNN
+F 0 "#PWR0165" H 6200 4050 50  0001 C CNN
 F 1 "GND" H 6200 4150 50  0000 C CNN
 F 2 "" H 6200 4300 50  0001 C CNN
@@
 	5900 4200 5900 4250
 $Comp
-L C C68
+L C C71
 U 1 1 5ABF53BC
 P 5900 3700
-F 0 "C68" H 5925 3800 50  0000 L CNN
+F 0 "C71" H 5925 3800 50  0000 L CNN
 F 1 "100n" H 5925 3600 50  0000 L CNN
 F 2 "" H 5938 3550 50  0001 C CNN
@@
 $EndComp
 $Comp
-L C C69
+L C C72
 U 1 1 5ABF53C2
 P 6200 3900
-F 0 "C69" H 6225 4000 50  0000 L CNN
+F 0 "C72" H 6225 4000 50  0000 L CNN
 F 1 "100p" H 6225 3800 50  0000 L CNN
 F 2 "" H 6238 3750 50  0001 C CNN
@@
 $EndComp
 $Comp
-L GND #PWR0164
+L GND #PWR0166
 U 1 1 5ABF847B
 P 7400 3900
-F 0 "#PWR0164" H 7400 3650 50  0001 C CNN
+F 0 "#PWR0166" H 7400 3650 50  0001 C CNN
 F 1 "GND" H 7400 3750 50  0000 C CNN
 F 2 "" H 7400 3900 50  0001 C CNN
@@
 	7950 3500 7950 3550
 $Comp
-L GND #PWR0165
+L GND #PWR0167
 U 1 1 5ABF8745
 P 7950 3900
-F 0 "#PWR0165" H 7950 3650 50  0001 C CNN
+F 0 "#PWR0167" H 7950 3650 50  0001 C CNN
 F 1 "GND" H 7950 3750 50  0000 C CNN
 F 2 "" H 7950 3900 50  0001 C CNN
@@
 Connection ~ 9300 3300
 $Comp
-L GND #PWR0166
+L GND #PWR0168
 U 1 1 5ABFAC4D
 P 9850 3850
-F 0 "#PWR0166" H 9850 3600 50  0001 C CNN
+F 0 "#PWR0168" H 9850 3600 50  0001 C CNN
 F 1 "GND" H 9850 3700 50  0000 C CNN
 F 2 "" H 9850 3850 50  0001 C CNN
@@
 MIC_IN
 $Comp
-L C C61
+L C C64
 U 1 1 5ABFC3EE
 P 3800 3900
-F 0 "C61" H 3825 4000 50  0000 L CNN
+F 0 "C64" H 3825 4000 50  0000 L CNN
 F 1 "100n" H 3825 3800 50  0000 L CNN
 F 2 "" H 3838 3750 50  0001 C CNN
@@
 $EndComp
 $Comp
-L GND #PWR0167
+L GND #PWR0169
 U 1 1 5ABFCB56
 P 3800 4100
-F 0 "#PWR0167" H 3800 3850 50  0001 C CNN
+F 0 "#PWR0169" H 3800 3850 50  0001 C CNN
 F 1 "GND" H 3800 3950 50  0000 C CNN
 F 2 "" H 3800 4100 50  0001 C CNN
@@
 NoConn ~ 3750 3550
 $Comp
-L C C74
+L C C77
 U 1 1 5AC79EEC
 P 9100 3800
-F 0 "C74" H 9125 3900 50  0000 L CNN
+F 0 "C77" H 9125 3900 50  0000 L CNN
 F 1 "270pF" H 9125 3700 50  0000 L CNN
 F 2 "" H 9138 3650 50  0001 C CNN
@@
 $EndComp
 $Comp
-L GND #PWR0168
+L GND #PWR0170
 U 1 1 5AC7A8FB
 P 9100 4000
-F 0 "#PWR0168" H 9100 3750 50  0001 C CNN
+F 0 "#PWR0170" H 9100 3750 50  0001 C CNN
 F 1 "GND" H 9100 3850 50  0000 C CNN
 F 2 "" H 9100 4000 50  0001 C CNN
@@
 	8750 3600 8800 3600
 $Comp
-L C C73
+L C C76
 U 1 1 5AC7B848
 P 8500 4300
-F 0 "C73" V 8550 4150 50  0000 L CNN
+F 0 "C76" V 8550 4150 50  0000 L CNN
 F 1 "100nF" V 8625 4175 50  0000 L CNN
 F 2 "" H 8538 4150 50  0001 C CNN
@@
 Connection ~ 8750 4300
 $Comp
-L C C71
+L C C74
 U 1 1 5AC7BC8A
 P 8300 4750
-F 0 "C71" H 8325 4850 50  0000 L CNN
+F 0 "C74" H 8325 4850 50  0000 L CNN
 F 1 "1uF" H 8325 4650 50  0000 L CNN
 F 2 "" H 8338 4600 50  0001 C CNN
@@
 Connection ~ 8300 4550
 $Comp
-L GND #PWR0169
+L GND #PWR0171
 U 1 1 5AC7C780
 P 8300 4950
-F 0 "#PWR0169" H 8300 4700 50  0001 C CNN
+F 0 "#PWR0171" H 8300 4700 50  0001 C CNN
 F 1 "GND" H 8300 4800 50  0000 C CNN
 F 2 "" H 8300 4950 50  0001 C CNN

Commit message: Use "Start to sheet number*100 and use first free number" designation, any new component added to the schematic will occupy the next available number in that sheet
For example: if sheet 2 has R201-R215 and we add a new resistor it will become R216.
Parts:
- renumbered C64 to C1301, C65 to C1302, C66 to C1303, C67 to C1304, C68 to C1305, C69 to C1306, C70 to C1307, C71 to C1308, C72 to C1309, C73 to C1310, C74 to C1311, C75 to C1312, C76 to C1313, C77 to C1314, D17 to D1301, D18 to D1302, FB2 to FB1301, FL2 to FL1301, J7 to J1301, R76 to R1301, R77 to R1302, R78 to R1303, R79 to R1304, R80 to R1305, U17 to U1301
Changed lines of the file:
@@
 $EndDescr
 $Comp
-L SGTL5000 U17
+L SGTL5000 U1301
 U 1 1 5ABE7D8D
 P 3050 3350
-F 0 "U17" H 2600 4250 60  0000 C CNN
+F 0 "U1301" H 2600 4250 60  0000 C CNN
 F 1 "SGTL5000" H 3500 4250 60  0000 C CNN
 F 2 "" H 3050 3400 60  0000 C CNN
@@
 $EndComp
 $Comp
-L GND #PWR0159
+L GND #PWR1301
 U 1 1 5ABE80CA
 P 3050 4450
-F 0 "#PWR0159" H 3050 4200 50  0001 C CNN
+F 0 "#PWR1301" H 3050 4200 50  0001 C CNN
 F 1 "GND" H 3050 4300 50  0000 C CNN
 F 2 "" H 3050 4450 50  0001 C CNN
@@
 	1700 3900 2350 3900
 $Comp
-L C C67
+L C C1304
 U 1 1 5ABEEF4C
 P 4700 3300
-F 0 "C67" V 4750 3350 50  0000 L CNN
+F 0 "C1304" V 4750 3350 50  0000 L CNN
 F 1 "220u" V 4750 3050 50  0000 L CNN
 F 2 "" H 4738 3150 50  0001 C CNN
@@
 $EndComp
 $Comp
-L C C68
+L C C1305
 U 1 1 5ABEEF73
 P 4700 3500
-F 0 "C68" V 4750 3300 50  0000 L CNN
+F 0 "C1305" V 4750 3300 50  0000 L CNN
 F 1 "200u" V 4750 3550 50  0000 L CNN
 F 2 "" H 4738 3350 50  0001 C CNN
@@
 	3900 3500 4550 3500
 $Comp
-L C C65
+L C C1302
 U 1 1 5ABEF358
 P 4150 3700
-F 0 "C65" H 4175 3800 50  0000 L CNN
+F 0 "C1302" H 4175 3800 50  0000 L CNN
 F 1 "NC" H 4175 3600 50  0000 L CNN
 F 2 "" H 4188 3550 50  0001 C CNN
@@
 $EndComp
 $Comp
-L C C66
+L C C1303
 U 1 1 5ABEF388
 P 4400 3700
-F 0 "C66" H 4425 3800 50  0000 L CNN
+F 0 "C1303" H 4425 3800 50  0000 L CNN
 F 1 "NC" H 4425 3600 50  0000 L CNN
 F 2 "" H 4438 3550 50  0001 C CNN
@@
 $EndComp
 $Comp
-L GND #PWR0160
+L GND #PWR1304
 U 1 1 5ABEF777
 P 4400 3900
-F 0 "#PWR0160" H 4400 3650 50  0001 C CNN
+F 0 "#PWR1304" H 4400 3650 50  0001 C CNN
 F 1 "GND" H 4400 3750 50  0000 C CNN
 F 2 "" H 4400 3900 50  0001 C CNN
@@
 $EndComp
 $Comp
-L GND #PWR0161
+L GND #PWR1303
 U 1 1 5ABEF798
 P 4150 3900
-F 0 "#PWR0161" H 4150 3650 50  0001 C CNN
+F 0 "#PWR1303" H 4150 3650 50  0001 C CNN
 F 1 "GND" H 4150 3750 50  0000 C CNN
 F 2 "" H 4150 3900 50  0001 C CNN
@@
 	4150 3850 4150 3900
 $Comp
-L R R76
+L R R1301
 U 1 1 5ABEFC7B
 P 5000 4050
-F 0 "R76" H 5125 4100 50  0000 C CNN
+F 0 "R1301" H 5125 4100 50  0000 C CNN
 F 1 "33" H 5125 4000 50  0000 C CNN
 F 2 "" V 4930 4050 50  0001 C CNN
@@
 	5000 3850 5000 3900
 $Comp
-L GND #PWR0162
+L GND #PWR1305
 U 1 1 5ABF0047
 P 5300 4300
-F 0 "#PWR0162" H 5300 4050 50  0001 C CNN
+F 0 "#PWR1305" H 5300 4050 50  0001 C CNN
 F 1 "GND" H 5300 4150 50  0000 C CNN
 F 2 "" H 5300 4300 50  0001 C CNN
@@
 	5000 4200 5000 4250
 $Comp
-L EMI_Filter_CommonMode FL2
+L EMI_Filter_CommonMode FL1301
 U 1 1 5ABF2412
 P 6750 3400
-F 0 "FL2" H 6750 3550 50  0000 C CNN
+F 0 "FL1301" H 6750 3550 50  0000 C CNN
 F 1 "DLW21SN900SQ2L" H 6750 3200 50  0000 C CNN
 F 2 "" V 6750 3440 50  0000 C CNN
@@
 $EndComp
 $Comp
-L C C75
+L C C1312
 U 1 1 5ABF2943
 P 8500 3700
-F 0 "C75" H 8525 3800 50  0000 L CNN
+F 0 "C1312" H 8525 3800 50  0000 L CNN
 F 1 "270p" H 8525 3600 50  0000 L CNN
 F 2 "" H 8538 3550 50  0001 C CNN
@@
 $EndComp
 $Comp
-L C C73
+L C C1310
 U 1 1 5ABF2987
 P 7000 3700
-F 0 "C73" H 7025 3800 50  0000 L CNN
+F 0 "C1310" H 7025 3800 50  0000 L CNN
 F 1 "270p" H 7025 3600 50  0000 L CNN
 F 2 "" H 7038 3550 50  0001 C CNN
@@
 	8500 3500 8500 3550
 $Comp
-L GND #PWR0163
+L GND #PWR1311
 U 1 1 5ABF2BDF
 P 8500 3900
-F 0 "#PWR0163" H 8500 3650 50  0001 C CNN
+F 0 "#PWR1311" H 8500 3650 50  0001 C CNN
 F 1 "GND" H 8500 3750 50  0000 C CNN
 F 2 "" H 8500 3900 50  0001 C CNN
@@
 	8500 3900 8500 3850
 $Comp
-L GND #PWR0164
+L GND #PWR1307
 U 1 1 5ABF2C32
 P 7000 3900
-F 0 "#PWR0164" H 7000 3650 50  0001 C CNN
+F 0 "#PWR1307" H 7000 3650 50  0001 C CNN
 F 1 "GND" H 7000 3750 50  0000 C CNN
 F 2 "" H 7000 3900 50  0001 C CNN
@@
 Connection ~ 4150 3300
 $Comp
-L C C69
+L C C1306
 U 1 1 5ABF4002
 P 5000 3700
-F 0 "C69" H 5025 3800 50  0000 L CNN
+F 0 "C1306" H 5025 3800 50  0000 L CNN
 F 1 "100n" H 5025 3600 50  0000 L CNN
 F 2 "" H 5038 3550 50  0001 C CNN
@@
 $EndComp
 $Comp
-L C C70
+L C C1307
 U 1 1 5ABF490A
 P 5300 3900
-F 0 "C70" H 5325 4000 50  0000 L CNN
+F 0 "C1307" H 5325 4000 50  0000 L CNN
 F 1 "100p" H 5325 3800 50  0000 L CNN
 F 2 "" H 5338 3750 50  0001 C CNN
@@
 $EndComp
 $Comp
-L R R77
+L R R1302
 U 1 1 5ABF49BF
 P 5600 3900
-F 0 "R77" H 5725 3950 50  0000 C CNN
+F 0 "R1302" H 5725 3950 50  0000 C CNN
 F 1 "15k" H 5725 3850 50  0000 C CNN
 F 2 "" V 5530 3900 50  0001 C CNN
@@
 Connection ~ 5600 3300
 $Comp
-L R R78
+L R R1303
 U 1 1 5ABF53AE
 P 5900 4050
-F 0 "R78" H 6025 4100 50  0000 C CNN
+F 0 "R1303" H 6025 4100 50  0000 C CNN
 F 1 "33" H 6025 4000 50  0000 C CNN
 F 2 "" V 5830 4050 50  0001 C CNN
@@
 	5900 3850 5900 3900
 $Comp
-L GND #PWR0165
+L GND #PWR1306
 U 1 1 5ABF53B5
 P 6200 4300
-F 0 "#PWR0165" H 6200 4050 50  0001 C CNN
+F 0 "#PWR1306" H 6200 4050 50  0001 C CNN
 F 1 "GND" H 6200 4150 50  0000 C CNN
 F 2 "" H 6200 4300 50  0001 C CNN
@@
 	5900 4200 5900 4250
 $Comp
-L C C71
+L C C1308
 U 1 1 5ABF53BC
 P 5900 3700
-F 0 "C71" H 5925 3800 50  0000 L CNN
+F 0 "C1308" H 5925 3800 50  0000 L CNN
 F 1 "100n" H 5925 3600 50  0000 L CNN
 F 2 "" H 5938 3550 50  0001 C CNN
@@
 $EndComp
 $Comp
-L C C72
+L C C1309
 U 1 1 5ABF53C2
 P 6200 3900
-F 0 "C72" H 6225 4000 50  0000 L CNN
+F 0 "C1309" H 6225 4000 50  0000 L CNN
 F 1 "100p" H 6225 3800 50  0000 L CNN
 F 2 "" H 6238 3750 50  0001 C CNN
@@
 $EndComp
 $Comp
-L R R79
+L R R1304
 U 1 1 5ABF53C8
 P 6500 3900
-F 0 "R79" H 6625 3950 50  0000 C CNN
+F 0 "R1304" H 6625 3950 50  0000 C CNN
 F 1 "15k" H 6625 3850 50  0000 C CNN
 F 2 "" V 6430 3900 50  0001 C CNN
@@
 Connection ~ 6500 3500
 $Comp
-L D_TVS_ALT D17
+L D_TVS_ALT D1301
 U 1 1 5ABF82C5
 P 7400 3700
-F 0 "D17" V 7350 3800 50  0000 C CNN
+F 0 "D1301" V 7350 3800 50  0000 C CNN
 F 1 "ESD5B5.0S" V 7450 3950 50  0000 C CNN
 F 2 "" H 7400 3700 50  0001 C CNN
@@
 $EndComp
 $Comp
-L GND #PWR0166
+L GND #PWR1308
 U 1 1 5ABF847B
 P 7400 3900
-F 0 "#PWR0166" H 7400 3650 50  0001 C CNN
+F 0 "#PWR1308" H 7400 3650 50  0001 C CNN
 F 1 "GND" H 7400 3750 50  0000 C CNN
 F 2 "" H 7400 3900 50  0001 C CNN
@@
 	7400 3900 7400 3850
 $Comp
-L D_TVS_ALT D18
+L D_TVS_ALT D1302
 U 1 1 5ABF8533
 P 7950 3700
-F 0 "D18" V 7900 3800 50  0000 C CNN
+F 0 "D1302" V 7900 3800 50  0000 C CNN
 F 1 "ESD5B5.0S" V 8000 3950 50  0000 C CNN
 F 2 "" H 7950 3700 50  0001 C CNN
@@
 	7950 3500 7950 3550
 $Comp
-L GND #PWR0167
+L GND #PWR1309
 U 1 1 5ABF8745
 P 7950 3900
-F 0 "#PWR0167" H 7950 3650 50  0001 C CNN
+F 0 "#PWR1309" H 7950 3650 50  0001 C CNN
 F 1 "GND" H 7950 3750 50  0000 C CNN
 F 2 "" H 7950 3900 50  0001 C CNN
@@
 Connection ~ 7950 3500
 $Comp
-L Audio-Jack-5 J7
+L Audio-Jack-5 J1301
 U 1 1 5ABF9919
 P 9550 3400
-F 0 "J7" H 9500 3610 50  0000 C CNN
+F 0 "J1301" H 9500 3610 50  0000 C CNN
 F 1 "CTIA / AHJ" H 9575 3025 50  0000 C CNN
 F 2 "" H 9800 3500 50  0001 C CNN
@@
 Connection ~ 9300 3300
 $Comp
-L GND #PWR0168
+L GND #PWR1313
 U 1 1 5ABFAC4D
 P 9850 3850
-F 0 "#PWR0168" H 9850 3600 50  0001 C CNN
+F 0 "#PWR1313" H 9850 3600 50  0001 C CNN
 F 1 "GND" H 9850 3700 50  0000 C CNN
 F 2 "" H 9850 3850 50  0001 C CNN
@@
 MIC_IN
 $Comp
-L C C64
+L C C1301
 U 1 1 5ABFC3EE
 P 3800 3900
-F 0 "C64" H 3825 4000 50  0000 L CNN
+F 0 "C1301" H 3825 4000 50  0000 L CNN
 F 1 "100n" H 3825 3800 50  0000 L CNN
 F 2 "" H 3838 3750 50  0001 C CNN
@@
 $EndComp
 $Comp
-L GND #PWR0169
+L GND #PWR1302
 U 1 1 5ABFCB56
 P 3800 4100
-F 0 "#PWR0169" H 3800 3850 50  0001 C CNN
+F 0 "#PWR1302" H 3800 3850 50  0001 C CNN
 F 1 "GND" H 3800 3950 50  0000 C CNN
 F 2 "" H 3800 4100 50  0001 C CNN
@@
 NoConn ~ 3750 3550
 $Comp
-L C C77
+L C C1314
 U 1 1 5AC79EEC
 P 9100 3800
-F 0 "C77" H 9125 3900 50  0000 L CNN
+F 0 "C1314" H 9125 3900 50  0000 L CNN
 F 1 "270pF" H 9125 3700 50  0000 L CNN
 F 2 "" H 9138 3650 50  0001 C CNN
@@
 $EndComp
 $Comp
-L Ferrite_Bead_Small FB2
+L Ferrite_Bead_Small FB1301
 U 1 1 5AC7A038
 P 8900 3600
-F 0 "FB2" V 9050 3550 50  0000 L CNN
+F 0 "FB1301" V 9050 3550 50  0000 L CNN
 F 1 "BLM15AX601SN1D" V 8750 3300 50  0000 L CNN
 F 2 "" V 8830 3600 50  0001 C CNN
@@
 $EndComp
 $Comp
-L GND #PWR0170
+L GND #PWR1312
 U 1 1 5AC7A8FB
 P 9100 4000
-F 0 "#PWR0170" H 9100 3750 50  0001 C CNN
+F 0 "#PWR1312" H 9100 3750 50  0001 C CNN
 F 1 "GND" H 9100 3850 50  0000 C CNN
 F 2 "" H 9100 4000 50  0001 C CNN
@@
 	9000 3600 9350 3600
 $Comp
-L R R80
+L R R1305
 U 1 1 5AC7B464
 P 8500 4550
-F 0 "R80" V 8400 4550 50  0000 C CNN
+F 0 "R1305" V 8400 4550 50  0000 C CNN
 F 1 "2.2k" V 8600 4550 50  0000 C CNN
 F 2 "" V 8430 4550 50  0001 C CNN
@@
 	8750 3600 8800 3600
 $Comp
-L C C76
+L C C1313
 U 1 1 5AC7B848
 P 8500 4300
-F 0 "C76" V 8550 4150 50  0000 L CNN
+F 0 "C1313" V 8550 4150 50  0000 L CNN
 F 1 "100nF" V 8625 4175 50  0000 L CNN
 F 2 "" H 8538 4150 50  0001 C CNN
@@
 Connection ~ 8750 4300
 $Comp
-L C C74
+L C C1311
 U 1 1 5AC7BC8A
 P 8300 4750
-F 0 "C74" H 8325 4850 50  0000 L CNN
+F 0 "C1311" H 8325 4850 50  0000 L CNN
 F 1 "1uF" H 8325 4650 50  0000 L CNN
 F 2 "" H 8338 4600 50  0001 C CNN
@@
 Connection ~ 8300 4550
 $Comp
-L GND #PWR0171
+L GND #PWR1310
 U 1 1 5AC7C780
 P 8300 4950
-F 0 "#PWR0171" H 8300 4700 50  0001 C CNN
+F 0 "#PWR1310" H 8300 4700 50  0001 C CNN
 F 1 "GND" H 8300 4800 50  0000 C CNN
 F 2 "" H 8300 4950 50  0001 C CNN
