File: boot.sch (KiCad schematic (older format))
At the start: 30 parts, among them SW1 TDA01H0SB1R, U7 SN74LVC1G34, U8 SN74LVC1G34, U9 SN74LVC1G04

Commit message: Assign all associated signals to their respective pins on the EmCraft i.MX8M SoM
The ERC is now at the same state as the DART SoM schematic. Need to compare various aspects of the current schematic against the EmCraft reference design. The main buck-boost will likely need to be switched to a 5V regulator, or be configured to output 5V.

A regulator will likely need to be added which will output some VBAT voltage level (3.5~4.2V) for the M.2 cards. The SIM7100 for example requires at least 3.4V!
Parts:
- renumbered C39 to C42, C40 to C43, C41 to C44
Changed lines of the file:
@@
 $EndComp
 $Comp
-L GND #PWR077
+L GND #PWR078
 U 1 1 5ACC0FBD
 P 2050 3850
-F 0 "#PWR077" H 2050 3600 50  0001 C CNN
+F 0 "#PWR078" H 2050 3600 50  0001 C CNN
 F 1 "GND" H 2050 3700 50  0000 C CNN
 F 2 "" H 2050 3850 50  0001 C CNN
@@
 $EndComp
 $Comp
-L GND #PWR078
+L GND #PWR079
 U 1 1 5ACC1D74
 P 4800 3650
-F 0 "#PWR078" H 4800 3400 50  0001 C CNN
+F 0 "#PWR079" H 4800 3400 50  0001 C CNN
 F 1 "GND" H 4800 3500 50  0000 C CNN
 F 2 "" H 4800 3650 50  0001 C CNN
@@
 $EndComp
 $Comp
-L SOM_NVCC_3V3 #PWR079
+L SOM_NVCC_3V3 #PWR080
 U 1 1 5ACC3732
 P 4800 2650
-F 0 "#PWR079" H 4800 2500 50  0001 C CNN
+F 0 "#PWR080" H 4800 2500 50  0001 C CNN
 F 1 "SOM_NVCC_3V3" H 4800 2790 50  0000 C CNN
 F 2 "" H 4800 2650 50  0001 C CNN
@@
 $EndComp
 $Comp
-L C C41
+L C C44
 U 1 1 5ACC6E61
 P 6500 4950
-F 0 "C41" H 6525 5050 50  0000 L CNN
+F 0 "C44" H 6525 5050 50  0000 L CNN
 F 1 "100nF" H 6525 4850 50  0000 L CNN
 F 2 "" H 6538 4800 50  0001 C CNN
@@
 $EndComp
 $Comp
-L GND #PWR080
+L GND #PWR081
 U 1 1 5ACC6EBC
 P 6500 5150
-F 0 "#PWR080" H 6500 4900 50  0001 C CNN
+F 0 "#PWR081" H 6500 4900 50  0001 C CNN
 F 1 "GND" H 6500 5000 50  0000 C CNN
 F 2 "" H 6500 5150 50  0001 C CNN
@@
 $EndComp
 $Comp
-L C C40
+L C C43
 U 1 1 5ACC73C7
 P 6500 3800
-F 0 "C40" H 6525 3900 50  0000 L CNN
+F 0 "C43" H 6525 3900 50  0000 L CNN
 F 1 "100nF" H 6525 3700 50  0000 L CNN
 F 2 "" H 6538 3650 50  0001 C CNN
@@
 $EndComp
 $Comp
-L GND #PWR081
+L GND #PWR082
 U 1 1 5ACC7769
 P 6500 4000
-F 0 "#PWR081" H 6500 3750 50  0001 C CNN
+F 0 "#PWR082" H 6500 3750 50  0001 C CNN
 F 1 "GND" H 6500 3850 50  0000 C CNN
 F 2 "" H 6500 4000 50  0001 C CNN
@@
 $EndComp
 $Comp
-L C C39
+L C C42
 U 1 1 5ACC7D43
 P 6500 2650
-F 0 "C39" H 6525 2750 50  0000 L CNN
+F 0 "C42" H 6525 2750 50  0000 L CNN
 F 1 "100nF" H 6525 2550 50  0000 L CNN
 F 2 "" H 6538 2500 50  0001 C CNN
@@
 $EndComp
 $Comp
-L GND #PWR082
+L GND #PWR083
 U 1 1 5ACC7DC1
 P 6500 2850
-F 0 "#PWR082" H 6500 2600 50  0001 C CNN
+F 0 "#PWR083" H 6500 2600 50  0001 C CNN
 F 1 "GND" H 6500 2700 50  0000 C CNN
 F 2 "" H 6500 2850 50  0001 C CNN
@@
 $EndComp
 $Comp
-L GND #PWR083
+L GND #PWR084
 U 1 1 5ACC80EC
 P 6100 3350
-F 0 "#PWR083" H 6100 3100 50  0001 C CNN
+F 0 "#PWR084" H 6100 3100 50  0001 C CNN
 F 1 "GND" H 6100 3200 50  0000 C CNN
 F 2 "" H 6100 3350 50  0001 C CNN
@@
 $EndComp
 $Comp
-L SOM_NVCC_3V3 #PWR084
+L SOM_NVCC_3V3 #PWR085
 U 1 1 5ACC8DC6
 P 6100 2400
-F 0 "#PWR084" H 6100 2250 50  0001 C CNN
+F 0 "#PWR085" H 6100 2250 50  0001 C CNN
 F 1 "SOM_NVCC_3V3" H 6100 2540 50  0000 C CNN
 F 2 "" H 6100 2400 50  0001 C CNN
@@
 $EndComp
 $Comp
-L GND #PWR085
+L GND #PWR086
 U 1 1 5ACC980A
 P 6100 4500
-F 0 "#PWR085" H 6100 4250 50  0001 C CNN
+F 0 "#PWR086" H 6100 4250 50  0001 C CNN
 F 1 "GND" H 6100 4350 50  0000 C CNN
 F 2 "" H 6100 4500 50  0001 C CNN
@@
 $EndComp
 $Comp
-L GND #PWR086
+L GND #PWR087
 U 1 1 5ACD1FAC
 P 6500 2200
-F 0 "#PWR086" H 6500 1950 50  0001 C CNN
+F 0 "#PWR087" H 6500 1950 50  0001 C CNN
 F 1 "GND" H 6500 2050 50  0000 C CNN
 F 2 "" H 6500 2200 50  0001 C CNN
@@
 $EndComp
 $Comp
-L GND #PWR087
+L GND #PWR088
 U 1 1 5ACD42FB
 P 6500 3400
-F 0 "#PWR087" H 6500 3150 50  0001 C CNN
+F 0 "#PWR088" H 6500 3150 50  0001 C CNN
 F 1 "GND" H 6500 3250 50  0000 C CNN
 F 2 "" H 6500 3400 50  0001 C CNN
@@
 SW_VOLDN
 $Comp
-L GND #PWR088
+L GND #PWR089
 U 1 1 5ACD6BAB
 P 6100 5650
-F 0 "#PWR088" H 6100 5400 50  0001 C CNN
+F 0 "#PWR089" H 6100 5400 50  0001 C CNN
 F 1 "GND" H 6100 5500 50  0000 C CNN
 F 2 "" H 6100 5650 50  0001 C CNN
@@
 $EndComp
 $Comp
-L GND #PWR089
+L GND #PWR090
 U 1 1 5ACDBA57
 P 6500 6000
-F 0 "#PWR089" H 6500 5750 50  0001 C CNN
+F 0 "#PWR090" H 6500 5750 50  0001 C CNN
 F 1 "GND" H 6500 5850 50  0000 C CNN
 F 2 "" H 6500 6000 50  0001 C CNN
@@
 $EndComp
 $Comp
-L SOM_NVCC_3V3 #PWR090
+L SOM_NVCC_3V3 #PWR091
 U 1 1 5AD4F627
 P 3450 4300
-F 0 "#PWR090" H 3450 4150 50  0001 C CNN
+F 0 "#PWR091" H 3450 4150 50  0001 C CNN
 F 1 "SOM_NVCC_3V3" H 3450 4440 50  0000 C CNN
 F 2 "" H 3450 4300 50  0001 C CNN
@@
 Connection ~ 3450 4350
 $Comp
-L GND #PWR091
+L GND #PWR092
 U 1 1 5AD4F7AA
 P 3450 5300
-F 0 "#PWR091" H 3450 5050 50  0001 C CNN
+F 0 "#PWR092" H 3450 5050 50  0001 C CNN
 F 1 "GND" H 3450 5150 50  0000 C CNN
 F 2 "" H 3450 5300 50  0001 C CNN

Commit message: Use "Start to sheet number*100 and use first free number" designation, any new component added to the schematic will occupy the next available number in that sheet
For example: if sheet 2 has R201-R215 and we add a new resistor it will become R216.
Parts:
- renumbered C42 to C401, C43 to C402, C44 to C403, D4 to D401, R24 to R401, R25 to R402, R26 to R403, R27 to R404, R28 to R405, R29 to R406, R30 to R407, R31 to R408, R32 to R409, R33 to R410, R34 to R411, R35 to R412, R36 to R413, R37 to R414, R38 to R415, R39 to R416, R40 to R417, R41 to R418, R42 to R419, R43 to R420, R44 to R421, R45 to R422, SW1 to SW401, U7 to U401, U8 to U402, U9 to U403

Commit message: Move reference designators in the schematic so that they are legible
Connections:
- wire segments 80 -> 105
Other:
- moved on the sheet: R401, R402, R403, R404, R405, R406, R407, R408

Commit message: Include reverse polarity protection circuit along with a simulation showing its effectiveness
Protecting VBAT from when board is sinking current via USB C. Protects against reverse polarity at the DC jack.

In EmCraft's instance VBUS should only be 5V when sinking current but they must protect against the condition when VBUS>12V and DC_IN=12V. This may need testing.
Connections:
- net labels added: 3V3_OUT
- net labels removed: SOM_NVCC_3V3
- wire segments 105 -> 80
Changed lines of the file:
@@
 Sheet 4 14
 Title "Boot Configuration"
-Date "2018-04-16"
+Date "2018-04-18"
 Rev "v0.1.0"
 Comp "Purism SPC"
@@
 $EndComp
 $Comp
-L GND #PWR078
+L GND #PWR080
 U 1 1 5ACC0FBD
 P 2000 3850
-F 0 "#PWR078" H 2000 3600 50  0001 C CNN
+F 0 "#PWR080" H 2000 3600 50  0001 C CNN
 F 1 "GND" H 2000 3700 50  0000 C CNN
 F 2 "" H 2000 3850 50  0001 C CNN
@@
 $EndComp
 $Comp
-L GND #PWR079
+L GND #PWR081
 U 1 1 5ACC1D74
 P 4800 3650
-F 0 "#PWR079" H 4800 3400 50  0001 C CNN
+F 0 "#PWR081" H 4800 3400 50  0001 C CNN
 F 1 "GND" H 4800 3500 50  0000 C CNN
 F 2 "" H 4800 3650 50  0001 C CNN
@@
 F 3 "" H 4800 2900 50  0001 C CNN
 	1    4800 2900
-	1    0    0    -1
-$EndComp
-$Comp
-L SOM_NVCC_3V3 #PWR080
-U 1 1 5ACC3732
-P 4800 2650
-F 0 "#PWR080" H 4800 2500 50  0001 C CNN
-F 1 "SOM_NVCC_3V3" H 4800 2790 50  0000 C CNN
-F 2 "" H 4800 2650 50  0001 C CNN
-F 3 "" H 4800 2650 50  0001 C CNN
-	1    4800 2650
 	1    0    0    -1
 $EndComp
@@
 $EndComp
 $Comp
-L GND #PWR081
+L GND #PWR082
 U 1 1 5ACC6EBC
 P 6500 5150
-F 0 "#PWR081" H 6500 4900 50  0001 C CNN
+F 0 "#PWR082" H 6500 4900 50  0001 C CNN
 F 1 "GND" H 6500 5000 50  0000 C CNN
 F 2 "" H 6500 5150 50  0001 C CNN
@@
 $EndComp
 $Comp
-L GND #PWR082
+L GND #PWR083
 U 1 1 5ACC7769
 P 6500 4000
-F 0 "#PWR082" H 6500 3750 50  0001 C CNN
+F 0 "#PWR083" H 6500 3750 50  0001 C CNN
 F 1 "GND" H 6500 3850 50  0000 C CNN
 F 2 "" H 6500 4000 50  0001 C CNN
@@
 $EndComp
 $Comp
-L GND #PWR083
+L GND #PWR084
 U 1 1 5ACC7DC1
 P 6500 2850
-F 0 "#PWR083" H 6500 2600 50  0001 C CNN
+F 0 "#PWR084" H 6500 2600 50  0001 C CNN
 F 1 "GND" H 6500 2700 50  0000 C CNN
 F 2 "" H 6500 2850 50  0001 C CNN
@@
 $EndComp
 $Comp
-L GND #PWR084
+L GND #PWR085
 U 1 1 5ACC80EC
 P 6100 3350
-F 0 "#PWR084" H 6100 3100 50  0001 C CNN
+F 0 "#PWR085" H 6100 3100 50  0001 C CNN
 F 1 "GND" H 6100 3200 50  0000 C CNN
 F 2 "" H 6100 3350 50  0001 C CNN
 F 3 "" H 6100 3350 50  0001 C CNN
 	1    6100 3350
-	1    0    0    -1
-$EndComp
-$Comp
-L SOM_NVCC_3V3 #PWR085
-U 1 1 5ACC8DC6
-P 6100 2400
-F 0 "#PWR085" H 6100 2250 50  0001 C CNN
-F 1 "SOM_NVCC_3V3" H 6100 2540 50  0000 C CNN
-F 2 "" H 6100 2400 50  0001 C CNN
-F 3 "" H 6100 2400 50  0001 C CNN
-	1    6100 2400
 	1    0    0    -1
 $EndComp
@@
 	6500 5700 6650 5700
 Wire Wire Line
-	6500 5700 6500 5950
-Wire Wire Line
-	6500 5950 6500 6000
+	6500 5700 6500 6000
 Wire Wire Line
 	6950 5950 8350 5950
@@
 	6500 1900 6650 1900
 Wire Wire Line
-	6500 1900 6500 2150
-Wire Wire Line
-	6500 2150 6500 2200
+	6500 1900 6500 2200
 Wire Wire Line
 	6950 5400 8350 5400
@@
 Connection ~ 5550 3100
 Wire Wire Line
-	5550 3100 5550 4250
-Wire Wire Line
-	5550 4250 5550 5400
+	5550 3100 5550 5400
 Wire Wire Line
 	5550 5400 5750 5400
@@
 Connection ~ 6100 3600
 Wire Wire Line
-	5650 2450 5650 3600
-Wire Wire Line
-	5650 3600 5650 4750
+	5650 2450 5650 4750
 Wire Wire Line
 	6100 4500 6100 4450
@@
 	6500 2450 6500 2500
 Wire Wire Line
-	5650 2450 6100 2450
-Wire Wire Line
-	6100 2450 6500 2450
-Wire Wire Line
-	6100 2400 6100 2450
-Wire Wire Line
-	6100 2450 6100 2900
+	5650 2450 6500 2450
+Wire Wire Line
+	6100 2400 6100 2900
 Wire Wire Line
 	6500 4000 6500 3950
@@
 	6500 3600 6500 3650
 Wire Wire Line
-	5650 3600 6100 3600
-Wire Wire Line
-	6100 3600 6500 3600
+	5650 3600 6500 3600
 Wire Wire Line
 	6100 4050 6100 3600
@@
 	6500 4750 6500 4800
 Wire Wire Line
-	5650 4750 6100 4750
-Wire Wire Line
-	6100 4750 6500 4750
+	5650 4750 6500 4750
 Wire Wire Line
 	6100 5200 6100 4750
@@
 Connection ~ 4800 2700
 Wire Wire Line
-	2500 2700 2800 2700
-Wire Wire Line
-	2800 2700 4800 2700
+	2500 2700 4800 2700
 Wire Wire Line
 	2500 2750 2500 2700
@@
 	2350 3600 3600 3600
 Wire Wire Line
-	2350 3500 2500 3500
-Wire Wire Line
-	2500 3500 3600 3500
+	2350 3500 3600 3500
 Wire Wire Line
 	2350 3400 3600 3400
@@
 	2350 3100 3600 3100
 Wire Wire Line
-	4800 2650 4800 2700
-Wire Wire Line
-	4800 2700 4800 2750
+	4800 2650 4800 2750
 Connection ~ 4800 3100
 Wire Wire Line
@@
 	4900 3100 4900 3150
 Wire Wire Line
-	4700 3100 4800 3100
-Wire Wire Line
-	4800 3100 4900 3100
-Wire Wire Line
-	4900 3100 5550 3100
-Wire Wire Line
-	5550 3100 5750 3100
+	4700 3100 5750 3100
 Wire Wire Line
 	4700 3200 4700 3100
@@
 	4900 3600 4900 3550
 Wire Wire Line
-	4700 3600 4800 3600
-Wire Wire Line
-	4800 3600 4900 3600
+	4700 3600 4900 3600
 Wire Wire Line
 	4700 3500 4700 3600
@@
 	2000 3100 2050 3100
 Wire Wire Line
-	2000 3100 2000 3300
-Wire Wire Line
-	2000 3300 2000 3400
-Wire Wire Line
-	2000 3400 2000 3500
-Wire Wire Line
-	2000 3500 2000 3600
-Wire Wire Line
-	2000 3600 2000 3700
-Wire Wire Line
-	2000 3700 2000 3800
-Wire Wire Line
-	2000 3800 2000 3850
+	2000 3100 2000 3850
 Text HLabel 3850 4750 2    60   Output ~ 0
 BOOT_MODE0
@@
 	1    0    0    -1
 $EndComp
-$Comp
-L SOM_NVCC_3V3 #PWR091
-U 1 1 5AD4F627
-P 3450 4300
-F 0 "#PWR091" H 3450 4150 50  0001 C CNN
-F 1 "SOM_NVCC_3V3" H 3450 4440 50  0000 C CNN
-F 2 "" H 3450 4300 50  0001 C CNN
-F 3 "" H 3450 4300 50  0001 C CNN
-	1    3450 4300
-	1    0    0    -1
-$EndComp
 Wire Wire Line
 	3300 4400 3300 4350
 Wire Wire Line
-	3300 4350 3450 4350
-Wire Wire Line
-	3450 4350 3600 4350
+	3300 4350 3600 4350
 Wire Wire Line
 	3600 4350 3600 4400
@@
 Connection ~ 3450 4350
 $Comp
-L GND #PWR092
+L GND #PWR091
 U 1 1 5AD4F7AA
 P 3450 5300
-F 0 "#PWR092" H 3450 5050 50  0001 C CNN
+F 0 "#PWR091" H 3450 5050 50  0001 C CNN
 F 1 "GND" H 3450 5150 50  0000 C CNN
 F 2 "" H 3450 5300 50  0001 C CNN
@@
 	3600 5250 3600 5200
 Wire Wire Line
-	3300 5250 3450 5250
-Wire Wire Line
-	3450 5250 3600 5250
+	3300 5250 3600 5250
 Wire Wire Line
 	3450 5300 3450 5250
 Connection ~ 3450 5250
 Wire Wire Line
-	3300 4700 3300 4850
-Wire Wire Line
-	3300 4850 3300 4900
-Wire Wire Line
-	3600 4700 3600 4750
-Wire Wire Line
-	3600 4750 3600 4900
+	3300 4700 3300 4900
+Wire Wire Line
+	3600 4700 3600 4900
 Wire Wire Line
 	3300 4850 3850 4850
@@
 EndData
 $EndBitmap
+$Comp
+L 3V3_OUT #PWR092
+U 1 1 5AEA3D45
+P 4800 2650
+F 0 "#PWR092" H 4800 2500 50  0001 C CNN
+F 1 "3V3_OUT" H 4800 2790 50  0000 C CNN
+F 2 "" H 4800 2650 50  0001 C CNN
+F 3 "" H 4800 2650 50  0001 C CNN
+	1    4800 2650
+	1    0    0    -1
+$EndComp
+$Comp
+L 3V3_OUT #PWR093
+U 1 1 5AEA3DF0
+P 6100 2400
+F 0 "#PWR093" H 6100 2250 50  0001 C CNN
+F 1 "3V3_OUT" H 6100 2540 50  0000 C CNN
+F 2 "" H 6100 2400 50  0001 C CNN
+F 3 "" H 6100 2400 50  0001 C CNN
+	1    6100 2400
+	1    0    0    -1
+$EndComp
+$Comp
+L 3V3_OUT #PWR094
+U 1 1 5AEA3E9B
+P 3450 4300
+F 0 "#PWR094" H 3450 4150 50  0001 C CNN
+F 1 "3V3_OUT" H 3450 4440 50  0000 C CNN
+F 2 "" H 3450 4300 50  0001 C CNN
+F 3 "" H 3450 4300 50  0001 C CNN
+	1    3450 4300
+	1    0    0    -1
+$EndComp
 $EndSCHEMATC

Commit message: Modify the boot config pins such that the eMMC is an 8-bit bus, depressing a momentary push button switch during boot causes SD boot, and relevant options
Parts:
- removed SW401: TDA01H0SB1R, symbol SW_SPST
- removed U401: SN74LVC1G34, symbol SN74LVC1G34
- added SW401: SW_Push, symbol SW_Push
- added U401: SN74LVC1G04, symbol SN74LVC1G04
- R401, R402, R403, R404, R405, R406, R407, R415, R416, R421, R422: value NC -> 10k
- R409: value 4.7k -> 10k
- R410, R413: value 1k -> 10k
- R417, R419, R420: value 47k -> 10k
- renumbered U403 to U402, U402 to U403
Connections:
- net 3V3_OUT: now also R405.1, U401.5
- net BOOT_CFG: now also SW401.1, U401.2
- net BOOT_CFG00: no longer R416.2, R419.2
- net GND: now also SW401.2, U401.3; no longer R405.1
- net at U402.4: now also R419.1; no longer R420.1
- net at R417.1: now also U401.4
- net at U403.4: now also R420.1; no longer R419.1
- new net BOOT_CFG09: R416.2
- new net BOOT_CFG12: R419.2
Other:
- note added: "BOOT CFG PRIORITY:\nH Int. eMMC\nL Ext. SD Card"
- note added: "BOOT_CFG04:\n0 - 1-bit SD bus\n0 - 4-bit SD bus\n(pull-up DATA1-3?)"
- note added: "BOOT_CFG05:\n1 - 8-bit eMMC bus"
- note added: "No SD power cycle"
- note added: "only eMMC/SD!"
- note added: "was LED1"
- note removed: ""Low – Represents pull down or floating.""
- note removed: "4.7k"
- note removed: "SoM's datasheet Table 57\nhas CFG10 mistakenly inverted,\ninconsistent with schematic and\nthe i.MX8M reference manual"
- moved on the sheet: R401, R402, R403, R404, R406, R407, R408, U402, U403
