File: boot.sch (KiCad schematic (older format))
At the start: 26 parts, among them SW501 DPDT

Commit message: Give the DPDT switches descriptive values
Parts:
- SW501: value DPDT -> BOOT_SW
Changed lines of the file:
@@
 P 3100 5500
 F 0 "SW501" V 3150 5225 50  0000 C CNN
-F 1 "DPDT" V 3050 5225 50  0000 C CNN
+F 1 "BOOT_SW" V 3050 5225 50  0000 C CNN
 F 2 "dvk-mx8m-bsb:Switch_CK_DPDT_JS202011JAQN" H 3100 5500 50  0001 C CNN
 F 3 "https://www.ckswitches.com/media/1422/js.pdf" H 3100 5500 50  0001 C CNN
@@
 P 3800 4950
 F 0 "SW501" V 3850 4675 50  0000 C CNN
-F 1 "DPDT" V 3750 4675 50  0000 C CNN
+F 1 "BOOT_SW" V 3750 4675 50  0000 C CNN
 F 2 "dvk-mx8m-bsb:Switch_CK_DPDT_JS202011JAQN" H 3800 4950 50  0001 C CNN
 F 3 "https://www.ckswitches.com/media/1422/js.pdf" H 3800 4950 50  0001 C CNN

Commit message: Move CAPTOUCH_~RST from BOOT_CFG_03 to GPIO1_IO05/P3.33 (was CSI_P2_PWDN), add a 10k pull-down to LCD_~RESET, make the corresponding changes to the BoM and netlist/layout
Having CAPTOUCH_~RST on BOOT_CFG_03 caused a voltage divider on the pin.
Connections:
- net labels removed: CAPTOUCH_~RST, CSI_P2_PWRDN, GP_LED3, SW_BACK
Changed lines of the file:
@@
 Text Label 3200 2950 0    60   ~ 0
 <CB_Function>
-Text Label 3200 3150 0    60   ~ 0
-GP_LED3
-Text Label 3200 3250 0    60   ~ 0
-CAPTOUCH_~RST
-Text Label 3200 3350 0    60   ~ 0
-SW_BACK
 Text Label 3200 3550 0    60   ~ 0
 SAI6_TXFS/RXFS
-Text Label 3200 3650 0    60   ~ 0
-CSI_P2_PWRDN
 Text Label 7000 3250 0    60   ~ 0
 BOOT_CFG10

Commit message: Update project files to KiCad 5.0.0
Parts:
- C501, C502: symbol C -> dvk-mx8m-bsb-rescue:C
- D501, D502: symbol D_TVS_ALT -> dvk-mx8m-bsb-rescue:D_TVS_ALT
- R501, R502, R503, R504, R505, R506, R507, R508, R509, R510, R511, R512, R513, R514, R515, R516, R517, R518, R519, R520, R521: symbol R -> dvk-mx8m-bsb-rescue:R
- SW501: symbol SW_DPDT_x2 -> dvk-mx8m-bsb-rescue:SW_DPDT_x2
Changed lines of the file:
@@
-EESchema Schematic File Version 2
-LIBS:power
-LIBS:device
-LIBS:switches
-LIBS:relays
-LIBS:motors
-LIBS:transistors
-LIBS:conn
-LIBS:linear
-LIBS:regul
-LIBS:74xx
-LIBS:cmos4000
-LIBS:adc-dac
-LIBS:memory
-LIBS:xilinx
-LIBS:microcontrollers
-LIBS:dsp
-LIBS:microchip
-LIBS:analog_switches
-LIBS:motorola
-LIBS:texas
-LIBS:intel
-LIBS:audio
-LIBS:interface
-LIBS:digital-audio
-LIBS:philips
-LIBS:display
-LIBS:cypress
-LIBS:siliconi
-LIBS:opto
-LIBS:atmel
-LIBS:contrib
-LIBS:valves
-LIBS:dvk-mx8m-bsb
+EESchema Schematic File Version 4
 LIBS:dvk-mx8m-bsb-cache
-EELAYER 25 0
+EELAYER 26 0
 EELAYER END
 $Descr A4 11693 8268
@@
 $EndDescr
 $Comp
-L GND #PWR0128
+L power:GND #PWR0128
 U 1 1 5ACC0FBD
 P 2050 3700
@@
 $EndComp
 $Comp
-L R R507
+L dvk-mx8m-bsb-rescue:R R507
 U 1 1 5ACC15C6
 P 2550 2750
@@
 BOOT_CFG09
 $Comp
-L GND #PWR0129
+L power:GND #PWR0129
 U 1 1 5ACD1FAC
 P 6600 2350
@@
 BOOT_CFG15
 $Comp
-L GND #PWR0130
+L power:GND #PWR0130
 U 1 1 5ACDBA57
 P 6600 6150
@@
 BOOT_MODE1
 $Comp
-L GND #PWR0131
+L power:GND #PWR0131
 U 1 1 5AD4F7AA
 P 3450 5800
@@
 	4150 5200 4250 5200
 $Comp
-L R R501
+L dvk-mx8m-bsb-rescue:R R501
 U 1 1 5B305194
 P 2250 2950
@@
 $EndComp
 $Comp
-L R R502
+L dvk-mx8m-bsb-rescue:R R502
 U 1 1 5B305386
 P 2250 3150
@@
 $EndComp
 $Comp
-L R R503
+L dvk-mx8m-bsb-rescue:R R503
 U 1 1 5B305401
 P 2250 3250
@@
 $EndComp
 $Comp
-L R R504
+L dvk-mx8m-bsb-rescue:R R504
 U 1 1 5B30547B
 P 2250 3350
@@
 $EndComp
 $Comp
-L R R505
+L dvk-mx8m-bsb-rescue:R R505
 U 1 1 5B3054F4
 P 2250 3550
@@
 $EndComp
 $Comp
-L R R506
+L dvk-mx8m-bsb-rescue:R R506
 U 1 1 5B305574
 P 2250 3650
@@
 $EndComp
 $Comp
-L R R508
+L dvk-mx8m-bsb-rescue:R R508
 U 1 1 5B307580
 P 2850 2750
@@
 $EndComp
 $Comp
-L R R510
+L dvk-mx8m-bsb-rescue:R R510
 U 1 1 5B3075F3
 P 3150 2750
@@
 $EndComp
 $Comp
-L R R514
+L dvk-mx8m-bsb-rescue:R R514
 U 1 1 5B307AAD
 P 6800 2050
@@
 $EndComp
 $Comp
-L R R515
+L dvk-mx8m-bsb-rescue:R R515
 U 1 1 5B3095E1
 P 6800 2300
@@
 $EndComp
 $Comp
-L R R516
+L dvk-mx8m-bsb-rescue:R R516
 U 1 1 5B309654
 P 6800 3250
@@
 $EndComp
 $Comp
-L R R517
+L dvk-mx8m-bsb-rescue:R R517
 U 1 1 5B3096EC
 P 6800 3500
@@
 $EndComp
 $Comp
-L R R518
+L dvk-mx8m-bsb-rescue:R R518
 U 1 1 5B309B05
 P 6800 4400
@@
 $EndComp
 $Comp
-L R R519
+L dvk-mx8m-bsb-rescue:R R519
 U 1 1 5B309B9F
 P 6800 5550
@@
 $EndComp
 $Comp
-L R R520
+L dvk-mx8m-bsb-rescue:R R520
 U 1 1 5B309C4A
 P 6800 5850
@@
 $EndComp
 $Comp
-L R R521
+L dvk-mx8m-bsb-rescue:R R521
 U 1 1 5B309CCE
 P 6800 6100
@@
 $EndComp
 $Comp
-L R R513
+L dvk-mx8m-bsb-rescue:R R513
 U 1 1 5B30A633
 P 4000 5200
@@
 $EndComp
 $Comp
-L R R509
+L dvk-mx8m-bsb-rescue:R R509
 U 1 1 5B30A6F1
 P 3000 5200
@@
 $EndComp
 $Comp
-L R R512
+L dvk-mx8m-bsb-rescue:R R512
 U 1 1 5B30B2F4
 P 3800 5550
@@
 $EndComp
 $Comp
-L R R511
+L dvk-mx8m-bsb-rescue:R R511
 U 1 1 5B30BB41
 P 3200 4900
@@
 $EndComp
 $Comp
-L SW_DPDT_x2 SW501
+L dvk-mx8m-bsb-rescue:SW_DPDT_x2 SW501
 U 1 1 5B0CA9C7
 P 3100 5500
@@
 NoConn ~ 3700 4750
 $Comp
-L SW_DPDT_x2 SW501
+L dvk-mx8m-bsb-rescue:SW_DPDT_x2 SW501
 U 2 1 5B0D695F
 P 3800 4950
@@
 $EndComp
 $Comp
-L GND #PWR0132
+L power:GND #PWR0132
 U 1 1 5B0E7810
 P 6600 3550
@@
 Connection ~ 6600 3500
 $Comp
-L GND #PWR0133
+L power:GND #PWR0133
 U 1 1 5B0E79B9
 P 6600 4450
@@
 	6600 4400 6650 4400
 $Comp
-L 3V3 #PWR0134
+L dvk-mx8m-bsb:3V3 #PWR0134
 U 1 1 5B0E8A3A
 P 6600 5500
@@
 	5300 6100 1600 6100
 $Comp
-L 3V3_SNVS #PWR0135
+L dvk-mx8m-bsb:3V3_SNVS #PWR0135
 U 1 1 5B12988B
 P 3550 4050
@@
 $EndComp
 $Comp
-L 3V3 #PWR0136
+L dvk-mx8m-bsb:3V3 #PWR0136
 U 1 1 5B129EC7
 P 2850 1900
@@
 $EndComp
 $Comp
-L C C502
+L dvk-mx8m-bsb-rescue:C C502
 U 1 1 5B12AE9C
 P 3700 4300
@@
 $EndComp
 $Comp
-L C C501
+L dvk-mx8m-bsb-rescue:C C501
 U 1 1 5B12B02A
 P 3000 2150
@@
 $EndComp
 $Comp
-L GND #PWR0137
+L power:GND #PWR0137
 U 1 1 5B12B357
 P 3000 2350
@@
 	3000 2300 3000 2350
 $Comp
-L GND #PWR0138
+L power:GND #PWR0138
 U 1 1 5B12BC91
 P 3700 4500
@@
 	3700 4450 3700 4500
 $Comp
-L D_TVS_ALT D501
+L dvk-mx8m-bsb-rescue:D_TVS_ALT D501
 U 1 1 5B21861F
 P 2800 5500
@@
 $EndComp
 $Comp
-L D_TVS_ALT D502
+L dvk-mx8m-bsb-rescue:D_TVS_ALT D502
 U 1 1 5B218688
 P 4200 5500

Commit message: Update the schematic symbols and footprints after upgrading to KiCad 5.0.0, fix all ERC and DRC violations after the new update/upgrade
Parts:
- C501, C502: footprint Capacitors_SMD:C_0603 -> Capacitor_SMD:C_0603_1608Metric; symbol dvk-mx8m-bsb-rescue:C -> Device:C
- D501, D502: symbol dvk-mx8m-bsb-rescue:D_TVS_ALT -> Device:D_TVS_ALT
- R501, R502, R503, R504, R505, R506, R507, R508, R509, R510, R511, R512, R513, R514, R515, R516, R517, R518, R519, R520, R521: footprint Resistors_SMD:R_0603 -> Resistor_SMD:R_0603_1608Metric; symbol dvk-mx8m-bsb-rescue:R -> Device:R
- SW501: symbol dvk-mx8m-bsb-rescue:SW_DPDT_x2 -> Switch:SW_DPDT_x2

Commit message: Reduce all 0603 resistor sizes to 0402
Parts:
- R501, R502, R503, R504, R505, R506, R507, R508, R509, R510, R511, R512, R513, R514, R515, R516, R517, R518, R519, R520, R521: footprint Resistor_SMD:R_0603_1608Metric -> Resistor_SMD:R_0402_1005Metric
Changed lines of the file:
@@
 F 0 "R507" H 2700 2800 50  0000 C CNN
 F 1 "NC" H 2650 2700 50  0000 C CNN
-F 2 "Resistor_SMD:R_0603_1608Metric" V 2480 2750 50  0001 C CNN
+F 2 "Resistor_SMD:R_0402_1005Metric" V 2480 2750 50  0001 C CNN
 F 3 "" H 2550 2750 50  0001 C CNN
 	1    2550 2750
@@
 F 0 "R501" V 2300 3150 50  0000 C CNN
 F 1 "10k" V 2250 2950 50  0000 C CNN
-F 2 "Resistor_SMD:R_0603_1608Metric" V 2180 2950 50  0001 C CNN
+F 2 "Resistor_SMD:R_0402_1005Metric" V 2180 2950 50  0001 C CNN
 F 3 "https://www.seielect.com/Catalog/SEI-RMCF_RMCP.pdf" H 2250 2950 50  0001 C CNN
 F 4 "Stackpole" H 2250 2950 60  0001 C CNN "MFG Name"
@@
 F 0 "R502" V 2300 3350 50  0000 C CNN
 F 1 "10k" V 2250 3150 50  0000 C CNN
-F 2 "Resistor_SMD:R_0603_1608Metric" V 2180 3150 50  0001 C CNN
+F 2 "Resistor_SMD:R_0402_1005Metric" V 2180 3150 50  0001 C CNN
 F 3 "https://www.seielect.com/Catalog/SEI-RMCF_RMCP.pdf" H 2250 3150 50  0001 C CNN
 F 4 "Stackpole" H 2250 3150 60  0001 C CNN "MFG Name"
@@
 F 0 "R503" V 2300 3450 50  0000 C CNN
 F 1 "10k" V 2250 3250 50  0000 C CNN
-F 2 "Resistor_SMD:R_0603_1608Metric" V 2180 3250 50  0001 C CNN
+F 2 "Resistor_SMD:R_0402_1005Metric" V 2180 3250 50  0001 C CNN
 F 3 "https://www.seielect.com/Catalog/SEI-RMCF_RMCP.pdf" H 2250 3250 50  0001 C CNN
 F 4 "Stackpole" H 2250 3250 60  0001 C CNN "MFG Name"
@@
 F 0 "R504" V 2300 3550 50  0000 C CNN
 F 1 "10k" V 2250 3350 50  0000 C CNN
-F 2 "Resistor_SMD:R_0603_1608Metric" V 2180 3350 50  0001 C CNN
+F 2 "Resistor_SMD:R_0402_1005Metric" V 2180 3350 50  0001 C CNN
 F 3 "https://www.seielect.com/Catalog/SEI-RMCF_RMCP.pdf" H 2250 3350 50  0001 C CNN
 F 4 "Stackpole" H 2250 3350 60  0001 C CNN "MFG Name"
@@
 F 0 "R505" V 2300 3750 50  0000 C CNN
 F 1 "10k" V 2250 3550 50  0000 C CNN
-F 2 "Resistor_SMD:R_0603_1608Metric" V 2180 3550 50  0001 C CNN
+F 2 "Resistor_SMD:R_0402_1005Metric" V 2180 3550 50  0001 C CNN
 F 3 "https://www.seielect.com/Catalog/SEI-RMCF_RMCP.pdf" H 2250 3550 50  0001 C CNN
 F 4 "Stackpole" H 2250 3550 60  0001 C CNN "MFG Name"
@@
 F 0 "R506" V 2300 3850 50  0000 C CNN
 F 1 "10k" V 2250 3650 50  0000 C CNN
-F 2 "Resistor_SMD:R_0603_1608Metric" V 2180 3650 50  0001 C CNN
+F 2 "Resistor_SMD:R_0402_1005Metric" V 2180 3650 50  0001 C CNN
 F 3 "https://www.seielect.com/Catalog/SEI-RMCF_RMCP.pdf" H 2250 3650 50  0001 C CNN
 F 4 "Stackpole" H 2250 3650 60  0001 C CNN "MFG Name"
@@
 F 0 "R508" H 3000 2800 50  0000 C CNN
 F 1 "10k" H 2975 2700 50  0000 C CNN
-F 2 "Resistor_SMD:R_0603_1608Metric" V 2780 2750 50  0001 C CNN
+F 2 "Resistor_SMD:R_0402_1005Metric" V 2780 2750 50  0001 C CNN
 F 3 "https://www.seielect.com/Catalog/SEI-RMCF_RMCP.pdf" H 2850 2750 50  0001 C CNN
 F 4 "Stackpole" H 2850 2750 60  0001 C CNN "MFG Name"
@@
 F 0 "R510" H 3300 2800 50  0000 C CNN
 F 1 "10k" H 3275 2700 50  0000 C CNN
-F 2 "Resistor_SMD:R_0603_1608Metric" V 3080 2750 50  0001 C CNN
+F 2 "Resistor_SMD:R_0402_1005Metric" V 3080 2750 50  0001 C CNN
 F 3 "https://www.seielect.com/Catalog/SEI-RMCF_RMCP.pdf" H 3150 2750 50  0001 C CNN
 F 4 "Stackpole" H 3150 2750 60  0001 C CNN "MFG Name"
@@
 F 0 "R514" V 6725 2050 50  0000 C CNN
 F 1 "10k" V 6875 2050 50  0000 C CNN
-F 2 "Resistor_SMD:R_0603_1608Metric" V 6730 2050 50  0001 C CNN
+F 2 "Resistor_SMD:R_0402_1005Metric" V 6730 2050 50  0001 C CNN
 F 3 "https://www.seielect.com/Catalog/SEI-RMCF_RMCP.pdf" H 6800 2050 50  0001 C CNN
 F 4 "Stackpole" H 6800 2050 60  0001 C CNN "MFG Name"
@@
 F 0 "R515" V 6725 2300 50  0000 C CNN
 F 1 "10k" V 6875 2300 50  0000 C CNN
-F 2 "Resistor_SMD:R_0603_1608Metric" V 6730 2300 50  0001 C CNN
+F 2 "Resistor_SMD:R_0402_1005Metric" V 6730 2300 50  0001 C CNN
 F 3 "https://www.seielect.com/Catalog/SEI-RMCF_RMCP.pdf" H 6800 2300 50  0001 C CNN
 F 4 "Stackpole" H 6800 2300 60  0001 C CNN "MFG Name"
@@
 F 0 "R516" V 6725 3250 50  0000 C CNN
 F 1 "10k" V 6875 3250 50  0000 C CNN
-F 2 "Resistor_SMD:R_0603_1608Metric" V 6730 3250 50  0001 C CNN
+F 2 "Resistor_SMD:R_0402_1005Metric" V 6730 3250 50  0001 C CNN
 F 3 "https://www.seielect.com/Catalog/SEI-RMCF_RMCP.pdf" H 6800 3250 50  0001 C CNN
 F 4 "Stackpole" H 6800 3250 60  0001 C CNN "MFG Name"
@@
 F 0 "R517" V 6725 3500 50  0000 C CNN
 F 1 "10k" V 6875 3500 50  0000 C CNN
-F 2 "Resistor_SMD:R_0603_1608Metric" V 6730 3500 50  0001 C CNN
+F 2 "Resistor_SMD:R_0402_1005Metric" V 6730 3500 50  0001 C CNN
 F 3 "https://www.seielect.com/Catalog/SEI-RMCF_RMCP.pdf" H 6800 3500 50  0001 C CNN
 F 4 "Stackpole" H 6800 3500 60  0001 C CNN "MFG Name"
@@
 F 0 "R518" V 6725 4400 50  0000 C CNN
 F 1 "10k" V 6875 4400 50  0000 C CNN
-F 2 "Resistor_SMD:R_0603_1608Metric" V 6730 4400 50  0001 C CNN
+F 2 "Resistor_SMD:R_0402_1005Metric" V 6730 4400 50  0001 C CNN
 F 3 "https://www.seielect.com/Catalog/SEI-RMCF_RMCP.pdf" H 6800 4400 50  0001 C CNN
 F 4 "Stackpole" H 6800 4400 60  0001 C CNN "MFG Name"
@@
 F 0 "R519" V 6725 5550 50  0000 C CNN
 F 1 "10k" V 6875 5550 50  0000 C CNN
-F 2 "Resistor_SMD:R_0603_1608Metric" V 6730 5550 50  0001 C CNN
+F 2 "Resistor_SMD:R_0402_1005Metric" V 6730 5550 50  0001 C CNN
 F 3 "https://www.seielect.com/Catalog/SEI-RMCF_RMCP.pdf" H 6800 5550 50  0001 C CNN
 F 4 "Stackpole" H 6800 5550 60  0001 C CNN "MFG Name"
@@
 F 0 "R520" V 6725 5850 50  0000 C CNN
 F 1 "10k" V 6875 5850 50  0000 C CNN
-F 2 "Resistor_SMD:R_0603_1608Metric" V 6730 5850 50  0001 C CNN
+F 2 "Resistor_SMD:R_0402_1005Metric" V 6730 5850 50  0001 C CNN
 F 3 "https://www.seielect.com/Catalog/SEI-RMCF_RMCP.pdf" H 6800 5850 50  0001 C CNN
 F 4 "Stackpole" H 6800 5850 60  0001 C CNN "MFG Name"
@@
 F 0 "R521" V 6725 6100 50  0000 C CNN
 F 1 "10k" V 6875 6100 50  0000 C CNN
-F 2 "Resistor_SMD:R_0603_1608Metric" V 6730 6100 50  0001 C CNN
+F 2 "Resistor_SMD:R_0402_1005Metric" V 6730 6100 50  0001 C CNN
 F 3 "https://www.seielect.com/Catalog/SEI-RMCF_RMCP.pdf" H 6800 6100 50  0001 C CNN
 F 4 "Stackpole" H 6800 6100 60  0001 C CNN "MFG Name"
@@
 F 0 "R513" V 3925 5200 50  0000 C CNN
 F 1 "10k" V 4075 5200 50  0000 C CNN
-F 2 "Resistor_SMD:R_0603_1608Metric" V 3930 5200 50  0001 C CNN
+F 2 "Resistor_SMD:R_0402_1005Metric" V 3930 5200 50  0001 C CNN
 F 3 "https://www.seielect.com/Catalog/SEI-RMCF_RMCP.pdf" H 4000 5200 50  0001 C CNN
 F 4 "Stackpole" H 4000 5200 60  0001 C CNN "MFG Name"
@@
 F 0 "R509" V 2850 5200 50  0000 C CNN
 F 1 "10k" V 2925 5200 50  0000 C CNN
-F 2 "Resistor_SMD:R_0603_1608Metric" V 2930 5200 50  0001 C CNN
+F 2 "Resistor_SMD:R_0402_1005Metric" V 2930 5200 50  0001 C CNN
 F 3 "https://www.seielect.com/Catalog/SEI-RMCF_RMCP.pdf" H 3000 5200 50  0001 C CNN
 F 4 "Stackpole" H 3000 5200 60  0001 C CNN "MFG Name"
@@
 F 0 "R512" H 3650 5600 50  0000 C CNN
 F 1 "10k" H 3675 5500 50  0000 C CNN
-F 2 "Resistor_SMD:R_0603_1608Metric" V 3730 5550 50  0001 C CNN
+F 2 "Resistor_SMD:R_0402_1005Metric" V 3730 5550 50  0001 C CNN
 F 3 "https://www.seielect.com/Catalog/SEI-RMCF_RMCP.pdf" H 3800 5550 50  0001 C CNN
 F 4 "Stackpole" H 3800 5550 60  0001 C CNN "MFG Name"
@@
 F 0 "R511" H 3050 4950 50  0000 C CNN
 F 1 "10k" H 3075 4850 50  0000 C CNN
-F 2 "Resistor_SMD:R_0603_1608Metric" V 3130 4900 50  0001 C CNN
+F 2 "Resistor_SMD:R_0402_1005Metric" V 3130 4900 50  0001 C CNN
 F 3 "https://www.seielect.com/Catalog/SEI-RMCF_RMCP.pdf" H 3200 4900 50  0001 C CNN
 F 4 "Stackpole" H 3200 4900 60  0001 C CNN "MFG Name"
