File: buttons_led.sch (KiCad schematic (older format))
At the start: 13 parts, among them Q10 2N7002P, SW3 SW_Push, SW4 SW_Push, SW5 SW_Push, SW6 SW_Push, SW7 SW_Push

Commit message: Use "Start to sheet number*100 and use first free number" designation, any new component added to the schematic will occupy the next available number in that sheet
For example: if sheet 2 has R201-R215 and we add a new resistor it will become R216.
Parts:
- renumbered D11 to D1201, D12 to D1202, D13 to D1203, D14 to D1204, D15 to D1205, D16 to D1206, Q10 to Q1201, R75 to R1201, SW3 to SW1201, SW4 to SW1202, SW5 to SW1203, SW6 to SW1204, SW7 to SW1205
Changed lines of the file:
@@
 $EndDescr
 $Comp
-L SW_Push SW3
+L SW_Push SW1201
 U 1 1 5ACC398C
 P 3200 1700
-F 0 "SW3" H 3250 1800 50  0000 L CNN
+F 0 "SW1201" H 3250 1800 50  0000 L CNN
 F 1 "SW_Push" H 3200 1640 50  0000 C CNN
 F 2 "" H 3200 1900 50  0001 C CNN
@@
 $EndComp
 $Comp
-L SW_Push SW4
+L SW_Push SW1202
 U 1 1 5ACC39A6
 P 3200 2400
-F 0 "SW4" H 3250 2500 50  0000 L CNN
+F 0 "SW1202" H 3250 2500 50  0000 L CNN
 F 1 "SW_Push" H 3200 2340 50  0000 C CNN
 F 2 "" H 3200 2600 50  0001 C CNN
@@
 $EndComp
 $Comp
-L SW_Push SW5
+L SW_Push SW1203
 U 1 1 5ACC3A06
 P 3200 3100
-F 0 "SW5" H 3250 3200 50  0000 L CNN
+F 0 "SW1203" H 3250 3200 50  0000 L CNN
 F 1 "SW_Push" H 3200 3040 50  0000 C CNN
 F 2 "" H 3200 3300 50  0001 C CNN
@@
 $EndComp
 $Comp
-L SW_Push SW6
+L SW_Push SW1204
 U 1 1 5ACC3A3E
 P 3200 3800
-F 0 "SW6" H 3250 3900 50  0000 L CNN
+F 0 "SW1204" H 3250 3900 50  0000 L CNN
 F 1 "SW_Push" H 3200 3740 50  0000 C CNN
 F 2 "" H 3200 4000 50  0001 C CNN
@@
 $EndComp
 $Comp
-L SW_Push SW7
+L SW_Push SW1205
 U 1 1 5ACC3AC2
 P 3200 4500
-F 0 "SW7" H 3250 4600 50  0000 L CNN
+F 0 "SW1205" H 3250 4600 50  0000 L CNN
 F 1 "SW_Push" H 3200 4440 50  0000 C CNN
 F 2 "" H 3200 4700 50  0001 C CNN
@@
 $EndComp
 $Comp
-L TVS_DIODE D11
+L TVS_DIODE D1201
 U 1 1 5ACC3B61
 P 3200 1950
-F 0 "D11" H 3200 2050 50  0000 C CNN
+F 0 "D1201" H 3200 2050 50  0000 C CNN
 F 1 "TPD1E10B09DPYR" H 3200 1850 50  0000 C CNN
 F 2 "" H 3300 1950 50  0001 C CNN
@@
 $EndComp
 $Comp
-L TVS_DIODE D12
+L TVS_DIODE D1202
 U 1 1 5ACC3BD8
 P 3200 2650
-F 0 "D12" H 3200 2750 50  0000 C CNN
+F 0 "D1202" H 3200 2750 50  0000 C CNN
 F 1 "TPD1E10B09DPYR" H 3200 2550 50  0000 C CNN
 F 2 "" H 3300 2650 50  0001 C CNN
@@
 $EndComp
 $Comp
-L TVS_DIODE D13
+L TVS_DIODE D1203
 U 1 1 5ACC3D42
 P 3200 3350
-F 0 "D13" H 3200 3450 50  0000 C CNN
+F 0 "D1203" H 3200 3450 50  0000 C CNN
 F 1 "TPD1E10B09DPYR" H 3200 3250 50  0000 C CNN
 F 2 "" H 3300 3350 50  0001 C CNN
@@
 $EndComp
 $Comp
-L TVS_DIODE D14
+L TVS_DIODE D1204
 U 1 1 5ACC3EAF
 P 3200 4050
-F 0 "D14" H 3200 4150 50  0000 C CNN
+F 0 "D1204" H 3200 4150 50  0000 C CNN
 F 1 "TPD1E10B09DPYR" H 3200 3950 50  0000 C CNN
 F 2 "" H 3300 4050 50  0001 C CNN
@@
 $EndComp
 $Comp
-L TVS_DIODE D15
+L TVS_DIODE D1205
 U 1 1 5ACC3FE9
 P 3200 4750
-F 0 "D15" H 3200 4850 50  0000 C CNN
+F 0 "D1205" H 3200 4850 50  0000 C CNN
 F 1 "TPD1E10B09DPYR" H 3200 4650 50  0000 C CNN
 F 2 "" H 3300 4750 50  0001 C CNN
@@
 	2800 1700 3000 1700
 $Comp
-L GND #PWR0152
+L GND #PWR1201
 U 1 1 5ACC4A3B
 P 2800 2000
-F 0 "#PWR0152" H 2800 1750 50  0001 C CNN
+F 0 "#PWR1201" H 2800 1750 50  0001 C CNN
 F 1 "GND" H 2800 1850 50  0000 C CNN
 F 2 "" H 2800 2000 50  0001 C CNN
@@
 	2800 2400 3000 2400
 $Comp
-L GND #PWR0153
+L GND #PWR1202
 U 1 1 5ACC4CAE
 P 2800 2700
-F 0 "#PWR0153" H 2800 2450 50  0001 C CNN
+F 0 "#PWR1202" H 2800 2450 50  0001 C CNN
 F 1 "GND" H 2800 2550 50  0000 C CNN
 F 2 "" H 2800 2700 50  0001 C CNN
@@
 	2800 3100 3000 3100
 $Comp
-L GND #PWR0154
+L GND #PWR1203
 U 1 1 5ACC4CDD
 P 2800 3400
-F 0 "#PWR0154" H 2800 3150 50  0001 C CNN
+F 0 "#PWR1203" H 2800 3150 50  0001 C CNN
 F 1 "GND" H 2800 3250 50  0000 C CNN
 F 2 "" H 2800 3400 50  0001 C CNN
@@
 	2800 3800 3000 3800
 $Comp
-L GND #PWR0155
+L GND #PWR1204
 U 1 1 5ACC4E99
 P 2800 4100
-F 0 "#PWR0155" H 2800 3850 50  0001 C CNN
+F 0 "#PWR1204" H 2800 3850 50  0001 C CNN
 F 1 "GND" H 2800 3950 50  0000 C CNN
 F 2 "" H 2800 4100 50  0001 C CNN
@@
 	2800 4500 3000 4500
 $Comp
-L GND #PWR0156
+L GND #PWR1205
 U 1 1 5ACC4EB3
 P 2800 4800
-F 0 "#PWR0156" H 2800 4550 50  0001 C CNN
+F 0 "#PWR1205" H 2800 4550 50  0001 C CNN
 F 1 "GND" H 2800 4650 50  0000 C CNN
 F 2 "" H 2800 4800 50  0001 C CNN
@@
 Connection ~ 3450 4500
 $Comp
-L LED D16
+L LED D1206
 U 1 1 5ACC7C6F
 P 8750 3300
-F 0 "D16" V 8800 3450 50  0000 C CNN
+F 0 "D1206" V 8800 3450 50  0000 C CNN
 F 1 "LED" V 8700 3450 50  0000 C CNN
 F 2 "" H 8750 3300 50  0001 C CNN
@@
 $EndComp
 $Comp
-L Q_NMOS_GSD Q10
+L Q_NMOS_GSD Q1201
 U 1 1 5ACC7CF3
 P 8650 3700
-F 0 "Q10" H 8850 3750 50  0000 L CNN
+F 0 "Q1201" H 8850 3750 50  0000 L CNN
 F 1 "2N7002P" H 8850 3650 50  0000 L CNN
 F 2 "" H 8850 3800 50  0001 C CNN
@@
 $EndComp
 $Comp
-L GND #PWR0157
+L GND #PWR1207
 U 1 1 5ACC7D2C
 P 8750 3950
-F 0 "#PWR0157" H 8750 3700 50  0001 C CNN
+F 0 "#PWR1207" H 8750 3700 50  0001 C CNN
 F 1 "GND" H 8750 3800 50  0000 C CNN
 F 2 "" H 8750 3950 50  0001 C CNN
@@
 $EndComp
 $Comp
-L R R75
+L R R1201
 U 1 1 5ACC7E2E
 P 8750 2950
-F 0 "R75" H 8850 3000 50  0000 C CNN
+F 0 "R1201" H 8850 3000 50  0000 C CNN
 F 1 "330" H 8875 2900 50  0000 C CNN
 F 2 "" V 8680 2950 50  0001 C CNN
@@
 $EndComp
 $Comp
-L BASE_PER_3V3 #PWR0158
+L BASE_PER_3V3 #PWR1206
 U 1 1 5ACC7FBC
 P 8750 2750
-F 0 "#PWR0158" H 8750 2600 50  0001 C CNN
+F 0 "#PWR1206" H 8750 2600 50  0001 C CNN
 F 1 "BASE_PER_3V3" H 8750 2890 50  0000 C CNN
 F 2 "" H 8750 2750 50  0001 C CNN

Commit message: Move reference designators in the schematic so that they are legible
Connections:
- wire segments 35 -> 45
Changed lines of the file:
@@
 	3050 1950 2800 1950
 Wire Wire Line
-	2800 1700 2800 2000
+	2800 1700 2800 1950
+Wire Wire Line
+	2800 1950 2800 2000
 Wire Wire Line
 	2800 1700 3000 1700
 $Comp
-L GND #PWR1201
+L GND #PWR0152
 U 1 1 5ACC4A3B
 P 2800 2000
-F 0 "#PWR1201" H 2800 1750 50  0001 C CNN
+F 0 "#PWR0152" H 2800 1750 50  0001 C CNN
 F 1 "GND" H 2800 1850 50  0000 C CNN
 F 2 "" H 2800 2000 50  0001 C CNN
@@
 	3050 2650 2800 2650
 Wire Wire Line
-	2800 2400 2800 2700
+	2800 2400 2800 2650
+Wire Wire Line
+	2800 2650 2800 2700
 Wire Wire Line
 	2800 2400 3000 2400
 $Comp
-L GND #PWR1202
+L GND #PWR0153
 U 1 1 5ACC4CAE
 P 2800 2700
-F 0 "#PWR1202" H 2800 2450 50  0001 C CNN
+F 0 "#PWR0153" H 2800 2450 50  0001 C CNN
 F 1 "GND" H 2800 2550 50  0000 C CNN
 F 2 "" H 2800 2700 50  0001 C CNN
@@
 	3050 3350 2800 3350
 Wire Wire Line
-	2800 3100 2800 3400
+	2800 3100 2800 3350
+Wire Wire Line
+	2800 3350 2800 3400
 Wire Wire Line
 	2800 3100 3000 3100
 $Comp
-L GND #PWR1203
+L GND #PWR0154
 U 1 1 5ACC4CDD
 P 2800 3400
-F 0 "#PWR1203" H 2800 3150 50  0001 C CNN
+F 0 "#PWR0154" H 2800 3150 50  0001 C CNN
 F 1 "GND" H 2800 3250 50  0000 C CNN
 F 2 "" H 2800 3400 50  0001 C CNN
@@
 	3050 4050 2800 4050
 Wire Wire Line
-	2800 3800 2800 4100
+	2800 3800 2800 4050
+Wire Wire Line
+	2800 4050 2800 4100
 Wire Wire Line
 	2800 3800 3000 3800
 $Comp
-L GND #PWR1204
+L GND #PWR0155
 U 1 1 5ACC4E99
 P 2800 4100
-F 0 "#PWR1204" H 2800 3850 50  0001 C CNN
+F 0 "#PWR0155" H 2800 3850 50  0001 C CNN
 F 1 "GND" H 2800 3950 50  0000 C CNN
 F 2 "" H 2800 4100 50  0001 C CNN
@@
 	3050 4750 2800 4750
 Wire Wire Line
-	2800 4500 2800 4800
+	2800 4500 2800 4750
+Wire Wire Line
+	2800 4750 2800 4800
 Wire Wire Line
 	2800 4500 3000 4500
 $Comp
-L GND #PWR1205
+L GND #PWR0156
 U 1 1 5ACC4EB3
 P 2800 4800
-F 0 "#PWR1205" H 2800 4550 50  0001 C CNN
+F 0 "#PWR0156" H 2800 4550 50  0001 C CNN
 F 1 "GND" H 2800 4650 50  0000 C CNN
 F 2 "" H 2800 4800 50  0001 C CNN
@@
 	3450 1950 3450 1700
 Wire Wire Line
-	3400 1700 4100 1700
+	3400 1700 3450 1700
+Wire Wire Line
+	3450 1700 4150 1700
 Connection ~ 3450 1700
 Wire Wire Line
@@
 	3450 2650 3450 2400
 Wire Wire Line
-	3400 2400 4100 2400
+	3400 2400 3450 2400
+Wire Wire Line
+	3450 2400 4150 2400
 Connection ~ 3450 2400
 Wire Wire Line
@@
 	3450 3350 3450 3100
 Wire Wire Line
-	3400 3100 4100 3100
+	3400 3100 3450 3100
+Wire Wire Line
+	3450 3100 4150 3100
 Connection ~ 3450 3100
 Wire Wire Line
@@
 	3450 4050 3450 3800
 Wire Wire Line
-	3400 3800 4100 3800
+	3400 3800 3450 3800
+Wire Wire Line
+	3450 3800 4150 3800
 Connection ~ 3450 3800
 Wire Wire Line
@@
 	3450 4750 3450 4500
 Wire Wire Line
-	3400 4500 4100 4500
+	3400 4500 3450 4500
+Wire Wire Line
+	3450 4500 4150 4500
 Connection ~ 3450 4500
 $Comp
@@
 U 1 1 5ACC7C6F
 P 8750 3300
-F 0 "D1206" V 8800 3450 50  0000 C CNN
+F 0 "D1206" V 8800 3475 50  0000 C CNN
 F 1 "LED" V 8700 3450 50  0000 C CNN
 F 2 "" H 8750 3300 50  0001 C CNN
@@
 $EndComp
 $Comp
-L GND #PWR1207
+L GND #PWR0157
 U 1 1 5ACC7D2C
 P 8750 3950
-F 0 "#PWR1207" H 8750 3700 50  0001 C CNN
+F 0 "#PWR0157" H 8750 3700 50  0001 C CNN
 F 1 "GND" H 8750 3800 50  0000 C CNN
 F 2 "" H 8750 3950 50  0001 C CNN
@@
 U 1 1 5ACC7E2E
 P 8750 2950
-F 0 "R1201" H 8850 3000 50  0000 C CNN
+F 0 "R1201" H 8925 3000 50  0000 C CNN
 F 1 "330" H 8875 2900 50  0000 C CNN
 F 2 "" V 8680 2950 50  0001 C CNN
@@
 $EndComp
 $Comp
-L BASE_PER_3V3 #PWR1206
+L BASE_PER_3V3 #PWR0158
 U 1 1 5ACC7FBC
 P 8750 2750
-F 0 "#PWR1206" H 8750 2600 50  0001 C CNN
+F 0 "#PWR0158" H 8750 2600 50  0001 C CNN
 F 1 "BASE_PER_3V3" H 8750 2890 50  0000 C CNN
 F 2 "" H 8750 2750 50  0001 C CNN
@@
 Wire Wire Line
 	8450 3700 7750 3700
-Text Label 3500 1700 0    60   ~ 0
+Text Label 3550 1700 0    60   ~ 0
 BOOT_CFG04
-Text Label 3500 2400 0    60   ~ 0
+Text Label 3550 2400 0    60   ~ 0
 BOOT_CFG11
-Text Label 3500 3100 0    60   ~ 0
+Text Label 3550 3100 0    60   ~ 0
 BOOT_CFG14
-Text Label 3500 3800 0    60   ~ 0
+Text Label 3550 3800 0    60   ~ 0
 BOOT_CFG09
-Text HLabel 4100 1700 2    60   Output ~ 0
+Text HLabel 4150 1700 2    60   Output ~ 0
 SW_BACK
-Text HLabel 4100 2400 2    60   Output ~ 0
+Text HLabel 4150 2400 2    60   Output ~ 0
 SW_VOLDN
-Text HLabel 4100 3100 2    60   Output ~ 0
+Text HLabel 4150 3100 2    60   Output ~ 0
 SW_VOLUP
-Text HLabel 4100 3800 2    60   Output ~ 0
+Text HLabel 4150 3800 2    60   Output ~ 0
 SW_HOME
-Text HLabel 4100 4500 2    60   Output ~ 0
+Text HLabel 4150 4500 2    60   Output ~ 0
 ONOFF
 Text Label 7850 3700 0    60   ~ 0

Commit message: Include reverse polarity protection circuit along with a simulation showing its effectiveness
Protecting VBAT from when board is sinking current via USB C. Protects against reverse polarity at the DC jack.

In EmCraft's instance VBUS should only be 5V when sinking current but they must protect against the condition when VBUS>12V and DC_IN=12V. This may need testing.
Connections:
- net labels added: 3V3_P
- net labels removed: BASE_PER_3V3
- wire segments 45 -> 35
Changed lines of the file:
@@
 Sheet 12 14
 Title "Buttons & LED"
-Date "2018-04-16"
+Date "2018-04-18"
 Rev "v0.1.0"
 Comp "Purism SPC"
@@
 	3050 1950 2800 1950
 Wire Wire Line
-	2800 1700 2800 1950
-Wire Wire Line
-	2800 1950 2800 2000
+	2800 1700 2800 2000
 Wire Wire Line
 	2800 1700 3000 1700
 $Comp
-L GND #PWR0152
+L GND #PWR0153
 U 1 1 5ACC4A3B
 P 2800 2000
-F 0 "#PWR0152" H 2800 1750 50  0001 C CNN
+F 0 "#PWR0153" H 2800 1750 50  0001 C CNN
 F 1 "GND" H 2800 1850 50  0000 C CNN
 F 2 "" H 2800 2000 50  0001 C CNN
@@
 	3050 2650 2800 2650
 Wire Wire Line
-	2800 2400 2800 2650
-Wire Wire Line
-	2800 2650 2800 2700
+	2800 2400 2800 2700
 Wire Wire Line
 	2800 2400 3000 2400
 $Comp
-L GND #PWR0153
+L GND #PWR0154
 U 1 1 5ACC4CAE
 P 2800 2700
-F 0 "#PWR0153" H 2800 2450 50  0001 C CNN
+F 0 "#PWR0154" H 2800 2450 50  0001 C CNN
 F 1 "GND" H 2800 2550 50  0000 C CNN
 F 2 "" H 2800 2700 50  0001 C CNN
@@
 	3050 3350 2800 3350
 Wire Wire Line
-	2800 3100 2800 3350
-Wire Wire Line
-	2800 3350 2800 3400
+	2800 3100 2800 3400
 Wire Wire Line
 	2800 3100 3000 3100
 $Comp
-L GND #PWR0154
+L GND #PWR0155
 U 1 1 5ACC4CDD
 P 2800 3400
-F 0 "#PWR0154" H 2800 3150 50  0001 C CNN
+F 0 "#PWR0155" H 2800 3150 50  0001 C CNN
 F 1 "GND" H 2800 3250 50  0000 C CNN
 F 2 "" H 2800 3400 50  0001 C CNN
@@
 	3050 4050 2800 4050
 Wire Wire Line
-	2800 3800 2800 4050
-Wire Wire Line
-	2800 4050 2800 4100
+	2800 3800 2800 4100
 Wire Wire Line
 	2800 3800 3000 3800
 $Comp
-L GND #PWR0155
+L GND #PWR0156
 U 1 1 5ACC4E99
 P 2800 4100
-F 0 "#PWR0155" H 2800 3850 50  0001 C CNN
+F 0 "#PWR0156" H 2800 3850 50  0001 C CNN
 F 1 "GND" H 2800 3950 50  0000 C CNN
 F 2 "" H 2800 4100 50  0001 C CNN
@@
 	3050 4750 2800 4750
 Wire Wire Line
-	2800 4500 2800 4750
-Wire Wire Line
-	2800 4750 2800 4800
+	2800 4500 2800 4800
 Wire Wire Line
 	2800 4500 3000 4500
 $Comp
-L GND #PWR0156
+L GND #PWR0157
 U 1 1 5ACC4EB3
 P 2800 4800
-F 0 "#PWR0156" H 2800 4550 50  0001 C CNN
+F 0 "#PWR0157" H 2800 4550 50  0001 C CNN
 F 1 "GND" H 2800 4650 50  0000 C CNN
 F 2 "" H 2800 4800 50  0001 C CNN
@@
 	3450 1950 3450 1700
 Wire Wire Line
-	3400 1700 3450 1700
-Wire Wire Line
-	3450 1700 4150 1700
+	3400 1700 4150 1700
 Connection ~ 3450 1700
 Wire Wire Line
@@
 	3450 2650 3450 2400
 Wire Wire Line
-	3400 2400 3450 2400
-Wire Wire Line
-	3450 2400 4150 2400
+	3400 2400 4150 2400
 Connection ~ 3450 2400
 Wire Wire Line
@@
 	3450 3350 3450 3100
 Wire Wire Line
-	3400 3100 3450 3100
-Wire Wire Line
-	3450 3100 4150 3100
+	3400 3100 4150 3100
 Connection ~ 3450 3100
 Wire Wire Line
@@
 	3450 4050 3450 3800
 Wire Wire Line
-	3400 3800 3450 3800
-Wire Wire Line
-	3450 3800 4150 3800
+	3400 3800 4150 3800
 Connection ~ 3450 3800
 Wire Wire Line
@@
 	3450 4750 3450 4500
 Wire Wire Line
-	3400 4500 3450 4500
-Wire Wire Line
-	3450 4500 4150 4500
+	3400 4500 4150 4500
 Connection ~ 3450 4500
 $Comp
@@
 $EndComp
 $Comp
-L GND #PWR0157
+L GND #PWR0158
 U 1 1 5ACC7D2C
 P 8750 3950
-F 0 "#PWR0157" H 8750 3700 50  0001 C CNN
+F 0 "#PWR0158" H 8750 3700 50  0001 C CNN
 F 1 "GND" H 8750 3800 50  0000 C CNN
 F 2 "" H 8750 3950 50  0001 C CNN
@@
 	1    8750 2950
 	-1   0    0    -1
-$EndComp
-$Comp
-L BASE_PER_3V3 #PWR0158
-U 1 1 5ACC7FBC
-P 8750 2750
-F 0 "#PWR0158" H 8750 2600 50  0001 C CNN
-F 1 "BASE_PER_3V3" H 8750 2890 50  0000 C CNN
-F 2 "" H 8750 2750 50  0001 C CNN
-F 3 "" H 8750 2750 50  0001 C CNN
-	1    8750 2750
-	1    0    0    -1
 $EndComp
 Wire Wire Line
@@
 Text Notes 9100 3350 0    60   ~ 0
 LTST-C19HE1WT\n  RBG Option
+$Comp
+L 3V3_P #PWR0159
+U 1 1 5AEA32FD
+P 8750 2750
+F 0 "#PWR0159" H 8750 2600 50  0001 C CNN
+F 1 "3V3_P" H 8750 2890 50  0000 C CNN
+F 2 "" H 8750 2750 50  0001 C CNN
+F 3 "" H 8750 2750 50  0001 C CNN
+	1    8750 2750
+	1    0    0    -1
+$EndComp
 $EndSCHEMATC
