File: mipi_dsi.sch (KiCad schematic (older format))
At the start: 19 parts, among them J6 WP7B-P040VA1-R500, Q6 2SK3018, Q7 2SK3018, Q8 2SK3018, Q9 2SK3018

Commit message: Assign all associated signals to their respective pins on the EmCraft i.MX8M SoM
The ERC is now at the same state as the DART SoM schematic. Need to compare various aspects of the current schematic against the EmCraft reference design. The main buck-boost will likely need to be switched to a 5V regulator, or be configured to output 5V.

A regulator will likely need to be added which will output some VBAT voltage level (3.5~4.2V) for the M.2 cards. The SIM7100 for example requires at least 3.4V!
Parts:
- renumbered C53 to C56, C54 to C57, C55 to C58, C56 to C59, C57 to C60, C58 to C61, C59 to C62, C60 to C63
Changed lines of the file:
@@
 NoConn ~ 4800 4750
 $Comp
-L GND #PWR0135
+L GND #PWR0137
 U 1 1 5AD63824
 P 4050 4950
-F 0 "#PWR0135" H 4050 4700 50  0001 C CNN
+F 0 "#PWR0137" H 4050 4700 50  0001 C CNN
 F 1 "GND" H 4050 4800 50  0000 C CNN
 F 2 "" H 4050 4950 50  0001 C CNN
@@
 Connection ~ 4050 4850
 $Comp
-L GND #PWR0136
+L GND #PWR0138
 U 1 1 5AD638B9
 P 5050 4950
-F 0 "#PWR0136" H 5050 4700 50  0001 C CNN
+F 0 "#PWR0138" H 5050 4700 50  0001 C CNN
 F 1 "GND" H 5050 4800 50  0000 C CNN
 F 2 "" H 5050 4950 50  0001 C CNN
@@
 D3_N
 $Comp
-L BASE_PER_1V8 #PWR0137
+L BASE_PER_1V8 #PWR0139
 U 1 1 5AD9C3F5
 P 4550 2000
-F 0 "#PWR0137" H 4550 1850 50  0001 C CNN
+F 0 "#PWR0139" H 4550 1850 50  0001 C CNN
 F 1 "BASE_PER_1V8" H 4550 2140 50  0000 C CNN
 F 2 "" H 4550 2000 50  0001 C CNN
@@
 Connection ~ 5300 3550
 $Comp
-L C C53
+L C C56
 U 1 1 5AD9EFD9
 P 4100 2250
-F 0 "C53" H 4125 2350 50  0000 L CNN
+F 0 "C56" H 4125 2350 50  0000 L CNN
 F 1 "100pF" H 4125 2150 50  0000 L CNN
 F 2 "" H 4138 2100 50  0001 C CNN
@@
 $EndComp
 $Comp
-L C C54
+L C C57
 U 1 1 5AD9F01C
 P 4400 2250
-F 0 "C54" H 4425 2350 50  0000 L CNN
+F 0 "C57" H 4425 2350 50  0000 L CNN
 F 1 "1nF" H 4425 2150 50  0000 L CNN
 F 2 "" H 4438 2100 50  0001 C CNN
@@
 $EndComp
 $Comp
-L C C55
+L C C58
 U 1 1 5AD9F039
 P 4700 2250
-F 0 "C55" H 4725 2350 50  0000 L CNN
+F 0 "C58" H 4725 2350 50  0000 L CNN
 F 1 "10nF" H 4725 2150 50  0000 L CNN
 F 2 "" H 4738 2100 50  0001 C CNN
@@
 $EndComp
 $Comp
-L C C56
+L C C59
 U 1 1 5AD9F0C9
 P 5000 2250
-F 0 "C56" H 5025 2350 50  0000 L CNN
+F 0 "C59" H 5025 2350 50  0000 L CNN
 F 1 "100nF" H 5025 2150 50  0000 L CNN
 F 2 "" H 5038 2100 50  0001 C CNN
@@
 	4100 2050 5300 2050
 $Comp
-L GND #PWR0138
+L GND #PWR0140
 U 1 1 5AD9F1A8
 P 4550 2500
-F 0 "#PWR0138" H 4550 2250 50  0001 C CNN
+F 0 "#PWR0140" H 4550 2250 50  0001 C CNN
 F 1 "GND" H 4550 2350 50  0000 C CNN
 F 2 "" H 4550 2500 50  0001 C CNN
@@
 	5400 2050 5400 4250
 $Comp
-L C C57
+L C C60
 U 1 1 5ADA269A
 P 5550 2250
-F 0 "C57" H 5575 2350 50  0000 L CNN
+F 0 "C60" H 5575 2350 50  0000 L CNN
 F 1 "100pF" H 5575 2150 50  0000 L CNN
 F 2 "" H 5588 2100 50  0001 C CNN
@@
 $EndComp
 $Comp
-L C C58
+L C C61
 U 1 1 5ADA26A0
 P 5850 2250
-F 0 "C58" H 5875 2350 50  0000 L CNN
+F 0 "C61" H 5875 2350 50  0000 L CNN
 F 1 "1nF" H 5875 2150 50  0000 L CNN
 F 2 "" H 5888 2100 50  0001 C CNN
@@
 $EndComp
 $Comp
-L C C59
+L C C62
 U 1 1 5ADA26A6
 P 6150 2250
-F 0 "C59" H 6175 2350 50  0000 L CNN
+F 0 "C62" H 6175 2350 50  0000 L CNN
 F 1 "10nF" H 6175 2150 50  0000 L CNN
 F 2 "" H 6188 2100 50  0001 C CNN
@@
 $EndComp
 $Comp
-L C C60
+L C C63
 U 1 1 5ADA26AC
 P 6450 2250
-F 0 "C60" H 6475 2350 50  0000 L CNN
+F 0 "C63" H 6475 2350 50  0000 L CNN
 F 1 "100nF" H 6475 2150 50  0000 L CNN
 F 2 "" H 6488 2100 50  0001 C CNN
@@
 $EndComp
 $Comp
-L GND #PWR0139
+L GND #PWR0141
 U 1 1 5ADA26B2
 P 6000 2500
-F 0 "#PWR0139" H 6000 2250 50  0001 C CNN
+F 0 "#PWR0141" H 6000 2250 50  0001 C CNN
 F 1 "GND" H 6000 2350 50  0000 C CNN
 F 2 "" H 6000 2500 50  0001 C CNN
@@
 Connection ~ 5900 4150
 $Comp
-L BASE_PER_1V8 #PWR0140
+L BASE_PER_1V8 #PWR0142
 U 1 1 5ADCA156
 P 6150 3700
-F 0 "#PWR0140" H 6150 3550 50  0001 C CNN
+F 0 "#PWR0142" H 6150 3550 50  0001 C CNN
 F 1 "BASE_PER_1V8" H 6150 3840 50  0000 C CNN
 F 2 "" H 6150 3700 50  0001 C CNN
@@
 $EndComp
 $Comp
-L BASE_PER_1V8 #PWR0141
+L BASE_PER_1V8 #PWR0143
 U 1 1 5ADCB88E
 P 7800 3800
-F 0 "#PWR0141" H 7800 3650 50  0001 C CNN
+F 0 "#PWR0143" H 7800 3650 50  0001 C CNN
 F 1 "BASE_PER_1V8" H 7800 3940 50  0000 C CNN
 F 2 "" H 7800 3800 50  0001 C CNN
@@
 	8650 4250 8650 4200
 $Comp
-L BASE_PER_3V3 #PWR0142
+L BASE_PER_3V3 #PWR0144
 U 1 1 5ADCBF34
 P 8650 3800
-F 0 "#PWR0142" H 8650 3650 50  0001 C CNN
+F 0 "#PWR0144" H 8650 3650 50  0001 C CNN
 F 1 "BASE_PER_3V3" H 8650 3940 50  0000 C CNN
 F 2 "" H 8650 3800 50  0001 C CNN
@@
 Connection ~ 5850 3400
 $Comp
-L BASE_PER_1V8 #PWR0143
+L BASE_PER_1V8 #PWR0145
 U 1 1 5ADCE85A
 P 6150 2950
-F 0 "#PWR0143" H 6150 2800 50  0001 C CNN
+F 0 "#PWR0145" H 6150 2800 50  0001 C CNN
 F 1 "BASE_PER_1V8" H 6150 3090 50  0000 C CNN
 F 2 "" H 6150 2950 50  0001 C CNN
@@
 $EndComp
 $Comp
-L BASE_PER_1V8 #PWR0144
+L BASE_PER_1V8 #PWR0146
 U 1 1 5ADD4F70
 P 7450 2950
-F 0 "#PWR0144" H 7450 2800 50  0001 C CNN
+F 0 "#PWR0146" H 7450 2800 50  0001 C CNN
 F 1 "BASE_PER_1V8" H 7450 3090 50  0000 C CNN
 F 2 "" H 7450 2950 50  0001 C CNN
@@
 $EndComp
 $Comp
-L BASE_PER_3V3 #PWR0145
+L BASE_PER_3V3 #PWR0147
 U 1 1 5ADCACA8
 P 6750 3700
-F 0 "#PWR0145" H 6750 3550 50  0001 C CNN
+F 0 "#PWR0147" H 6750 3550 50  0001 C CNN
 F 1 "BASE_PER_3V3" H 6750 3840 50  0000 C CNN
 F 2 "" H 6750 3700 50  0001 C CNN
@@
 $EndBitmap
 $Comp
-L OVSS #PWR0146
+L OVSS #PWR0148
 U 1 1 5AE7CB26
 P 4250 2900
-F 0 "#PWR0146" H 4250 2750 50  0001 C CNN
+F 0 "#PWR0148" H 4250 2750 50  0001 C CNN
 F 1 "OVSS" H 4250 3040 50  0000 C CNN
 F 2 "" H 4250 2900 50  0001 C CNN
@@
 Connection ~ 4250 2950
 $Comp
-L OVDD #PWR0147
+L OVDD #PWR0149
 U 1 1 5AE7D1B4
 P 4850 2900
-F 0 "#PWR0147" H 4850 2750 50  0001 C CNN
+F 0 "#PWR0149" H 4850 2750 50  0001 C CNN
 F 1 "OVDD" H 4850 3040 50  0000 C CNN
 F 2 "" H 4850 2900 50  0001 C CNN
@@
 Connection ~ 4850 2950
 $Comp
-L VCI_TP_VCC #PWR0148
+L VCI_TP_VCC #PWR0150
 U 1 1 5AD63D0F
 P 6000 2000
-F 0 "#PWR0148" H 6000 1850 50  0001 C CNN
+F 0 "#PWR0150" H 6000 1850 50  0001 C CNN
 F 1 "VCI_TP_VCC" H 6000 2140 50  0000 C CNN
 F 2 "" H 6000 2000 50  0001 C CNN
@@
 1.8V rises ~~12ms after 3.0V
 $Comp
-L AVDD #PWR0149
+L AVDD #PWR0151
 U 1 1 5ACF9758
 P 5200 3250
-F 0 "#PWR0149" H 5200 3100 50  0001 C CNN
+F 0 "#PWR0151" H 5200 3100 50  0001 C CNN
 F 1 "AVDD" H 5200 3390 50  0000 C CNN
 F 2 "" H 5200 3250 50  0001 C CNN

Commit message: Use "Start to sheet number*100 and use first free number" designation, any new component added to the schematic will occupy the next available number in that sheet
For example: if sheet 2 has R201-R215 and we add a new resistor it will become R216.
Parts:
- renumbered C56 to C1101, C57 to C1102, C58 to C1103, C59 to C1104, C60 to C1105, C61 to C1106, C62 to C1107, C63 to C1108, J6 to J1101, Q6 to Q1101, Q7 to Q1102, Q8 to Q1103, Q9 to Q1104, R69 to R1101, R70 to R1102, R71 to R1103, R72 to R1104, R73 to R1105, R74 to R1106
Changed lines of the file:
@@
 $EndDescr
 $Comp
-L Conn_02x20_Odd_Even J6
+L Conn_02x20_Odd_Even J1101
 U 1 1 5AD62C84
 P 4500 3850
-F 0 "J6" H 4550 4850 50  0000 C CNN
+F 0 "J1101" H 4550 4850 50  0000 C CNN
 F 1 "WP7B-P040VA1-R500" H 4550 2750 50  0000 C CNN
 F 2 "" H 4500 3850 50  0001 C CNN
@@
 NoConn ~ 4800 4750
 $Comp
-L GND #PWR0137
+L GND #PWR1101
 U 1 1 5AD63824
 P 4050 4950
-F 0 "#PWR0137" H 4050 4700 50  0001 C CNN
+F 0 "#PWR1101" H 4050 4700 50  0001 C CNN
 F 1 "GND" H 4050 4800 50  0000 C CNN
 F 2 "" H 4050 4950 50  0001 C CNN
@@
 Connection ~ 4050 4850
 $Comp
-L GND #PWR0138
+L GND #PWR1106
 U 1 1 5AD638B9
 P 5050 4950
-F 0 "#PWR0138" H 5050 4700 50  0001 C CNN
+F 0 "#PWR1106" H 5050 4700 50  0001 C CNN
 F 1 "GND" H 5050 4800 50  0000 C CNN
 F 2 "" H 5050 4950 50  0001 C CNN
@@
 D3_N
 $Comp
-L BASE_PER_1V8 #PWR0139
+L BASE_PER_1V8 #PWR1103
 U 1 1 5AD9C3F5
 P 4550 2000
-F 0 "#PWR0139" H 4550 1850 50  0001 C CNN
+F 0 "#PWR1103" H 4550 1850 50  0001 C CNN
 F 1 "BASE_PER_1V8" H 4550 2140 50  0000 C CNN
 F 2 "" H 4550 2000 50  0001 C CNN
@@
 Connection ~ 5300 3550
 $Comp
-L C C56
+L C C1101
 U 1 1 5AD9EFD9
 P 4100 2250
-F 0 "C56" H 4125 2350 50  0000 L CNN
+F 0 "C1101" H 4125 2350 50  0000 L CNN
 F 1 "100pF" H 4125 2150 50  0000 L CNN
 F 2 "" H 4138 2100 50  0001 C CNN
@@
 $EndComp
 $Comp
-L C C57
+L C C1102
 U 1 1 5AD9F01C
 P 4400 2250
-F 0 "C57" H 4425 2350 50  0000 L CNN
+F 0 "C1102" H 4425 2350 50  0000 L CNN
 F 1 "1nF" H 4425 2150 50  0000 L CNN
 F 2 "" H 4438 2100 50  0001 C CNN
@@
 $EndComp
 $Comp
-L C C58
+L C C1103
 U 1 1 5AD9F039
 P 4700 2250
-F 0 "C58" H 4725 2350 50  0000 L CNN
+F 0 "C1103" H 4725 2350 50  0000 L CNN
 F 1 "10nF" H 4725 2150 50  0000 L CNN
 F 2 "" H 4738 2100 50  0001 C CNN
@@
 $EndComp
 $Comp
-L C C59
+L C C1104
 U 1 1 5AD9F0C9
 P 5000 2250
-F 0 "C59" H 5025 2350 50  0000 L CNN
+F 0 "C1104" H 5025 2350 50  0000 L CNN
 F 1 "100nF" H 5025 2150 50  0000 L CNN
 F 2 "" H 5038 2100 50  0001 C CNN
@@
 	4100 2050 5300 2050
 $Comp
-L GND #PWR0140
+L GND #PWR1104
 U 1 1 5AD9F1A8
 P 4550 2500
-F 0 "#PWR0140" H 4550 2250 50  0001 C CNN
+F 0 "#PWR1104" H 4550 2250 50  0001 C CNN
 F 1 "GND" H 4550 2350 50  0000 C CNN
 F 2 "" H 4550 2500 50  0001 C CNN
@@
 	5400 2050 5400 4250
 $Comp
-L C C60
+L C C1105
 U 1 1 5ADA269A
 P 5550 2250
-F 0 "C60" H 5575 2350 50  0000 L CNN
+F 0 "C1105" H 5575 2350 50  0000 L CNN
 F 1 "100pF" H 5575 2150 50  0000 L CNN
 F 2 "" H 5588 2100 50  0001 C CNN
@@
 $EndComp
 $Comp
-L C C61
+L C C1106
 U 1 1 5ADA26A0
 P 5850 2250
-F 0 "C61" H 5875 2350 50  0000 L CNN
+F 0 "C1106" H 5875 2350 50  0000 L CNN
 F 1 "1nF" H 5875 2150 50  0000 L CNN
 F 2 "" H 5888 2100 50  0001 C CNN
@@
 $EndComp
 $Comp
-L C C62
+L C C1107
 U 1 1 5ADA26A6
 P 6150 2250
-F 0 "C62" H 6175 2350 50  0000 L CNN
+F 0 "C1107" H 6175 2350 50  0000 L CNN
 F 1 "10nF" H 6175 2150 50  0000 L CNN
 F 2 "" H 6188 2100 50  0001 C CNN
@@
 $EndComp
 $Comp
-L C C63
+L C C1108
 U 1 1 5ADA26AC
 P 6450 2250
-F 0 "C63" H 6475 2350 50  0000 L CNN
+F 0 "C1108" H 6475 2350 50  0000 L CNN
 F 1 "100nF" H 6475 2150 50  0000 L CNN
 F 2 "" H 6488 2100 50  0001 C CNN
@@
 $EndComp
 $Comp
-L GND #PWR0141
+L GND #PWR1109
 U 1 1 5ADA26B2
 P 6000 2500
-F 0 "#PWR0141" H 6000 2250 50  0001 C CNN
+F 0 "#PWR1109" H 6000 2250 50  0001 C CNN
 F 1 "GND" H 6000 2350 50  0000 C CNN
 F 2 "" H 6000 2500 50  0001 C CNN
@@
 SWIRE
 $Comp
-L Q_NMOS_SGD Q8
+L Q_NMOS_SGD Q1103
 U 1 1 5ADC2CF3
 P 7450 3300
-F 0 "Q8" V 7350 3400 50  0000 L CNN
+F 0 "Q1103" V 7350 3400 50  0000 L CNN
 F 1 "2SK3018" V 7450 3450 50  0000 L CNN
 F 2 "" H 7650 3400 50  0001 C CNN
@@
 $EndComp
 $Comp
-L Q_NMOS_SGD Q6
+L Q_NMOS_SGD Q1101
 U 1 1 5ADC87D2
 P 6150 3300
-F 0 "Q6" V 6050 3400 50  0000 L CNN
+F 0 "Q1101" V 6050 3400 50  0000 L CNN
 F 1 "2SK3018" V 6150 3450 50  0000 L CNN
 F 2 "" H 6350 3400 50  0001 C CNN
@@
 $EndComp
 $Comp
-L Q_NMOS_SGD Q7
+L Q_NMOS_SGD Q1102
 U 1 1 5ADC894E
 P 6150 4050
-F 0 "Q7" V 6050 4150 50  0000 L CNN
+F 0 "Q1102" V 6050 4150 50  0000 L CNN
 F 1 "2SK3018" V 6150 4200 50  0000 L CNN
 F 2 "" H 6350 4150 50  0001 C CNN
@@
 $EndComp
 $Comp
-L Q_NMOS_SGD Q9
+L Q_NMOS_SGD Q1104
 U 1 1 5ADC89B8
 P 8050 4150
-F 0 "Q9" V 7950 4250 50  0000 L CNN
+F 0 "Q1104" V 7950 4250 50  0000 L CNN
 F 1 "2SK3018" V 8050 4300 50  0000 L CNN
 F 2 "" H 8250 4250 50  0001 C CNN
@@
 Connection ~ 5900 4150
 $Comp
-L BASE_PER_1V8 #PWR0142
+L BASE_PER_1V8 #PWR1111
 U 1 1 5ADCA156
 P 6150 3700
-F 0 "#PWR0142" H 6150 3550 50  0001 C CNN
+F 0 "#PWR1111" H 6150 3550 50  0001 C CNN
 F 1 "BASE_PER_1V8" H 6150 3840 50  0000 C CNN
 F 2 "" H 6150 3700 50  0001 C CNN
@@
 Connection ~ 6150 3750
 $Comp
-L R R71
+L R R1103
 U 1 1 5ADCAB95
 P 6750 3950
-F 0 "R71" H 6875 4000 50  0000 C CNN
+F 0 "R1103" H 6875 4000 50  0000 C CNN
 F 1 "10k" H 6875 3900 50  0000 C CNN
 F 2 "" V 6680 3950 50  0001 C CNN
@@
 	6750 3800 6750 3700
 $Comp
-L R R73
+L R R1105
 U 1 1 5ADCB77A
 P 7800 4050
-F 0 "R73" H 7925 4000 50  0000 C CNN
+F 0 "R1105" H 7925 4000 50  0000 C CNN
 F 1 "10k" H 7925 4100 50  0000 C CNN
 F 2 "" V 7730 4050 50  0001 C CNN
@@
 $EndComp
 $Comp
-L BASE_PER_1V8 #PWR0143
+L BASE_PER_1V8 #PWR1114
 U 1 1 5ADCB88E
 P 7800 3800
-F 0 "#PWR0143" H 7800 3650 50  0001 C CNN
+F 0 "#PWR1114" H 7800 3650 50  0001 C CNN
 F 1 "BASE_PER_1V8" H 7800 3940 50  0000 C CNN
 F 2 "" H 7800 3800 50  0001 C CNN
@@
 	8650 4250 8650 4200
 $Comp
-L BASE_PER_3V3 #PWR0144
+L BASE_PER_3V3 #PWR1115
 U 1 1 5ADCBF34
 P 8650 3800
-F 0 "#PWR0144" H 8650 3650 50  0001 C CNN
+F 0 "#PWR1115" H 8650 3650 50  0001 C CNN
 F 1 "BASE_PER_3V3" H 8650 3940 50  0000 C CNN
 F 2 "" H 8650 3800 50  0001 C CNN
@@
 Connection ~ 5850 3400
 $Comp
-L BASE_PER_1V8 #PWR0145
+L BASE_PER_1V8 #PWR1110
 U 1 1 5ADCE85A
 P 6150 2950
-F 0 "#PWR0145" H 6150 2800 50  0001 C CNN
+F 0 "#PWR1110" H 6150 2800 50  0001 C CNN
 F 1 "BASE_PER_1V8" H 6150 3090 50  0000 C CNN
 F 2 "" H 6150 2950 50  0001 C CNN
@@
 Connection ~ 6750 4150
 $Comp
-L R R70
+L R R1102
 U 1 1 5ADD2F2F
 P 5900 3950
-F 0 "R70" H 6025 3900 50  0000 C CNN
+F 0 "R1102" H 6025 3900 50  0000 C CNN
 F 1 "10k" H 6025 4000 50  0000 C CNN
 F 2 "" V 5830 3950 50  0001 C CNN
@@
 $EndComp
 $Comp
-L R R69
+L R R1101
 U 1 1 5ADD2F9F
 P 5850 3200
-F 0 "R69" H 5975 3150 50  0000 C CNN
+F 0 "R1101" H 5975 3150 50  0000 C CNN
 F 1 "10k" H 5975 3250 50  0000 C CNN
 F 2 "" V 5780 3200 50  0001 C CNN
@@
 $EndComp
 $Comp
-L R R74
+L R R1106
 U 1 1 5ADD38F2
 P 8650 4050
-F 0 "R74" H 8775 4100 50  0000 C CNN
+F 0 "R1106" H 8775 4100 50  0000 C CNN
 F 1 "10k" H 8775 4000 50  0000 C CNN
 F 2 "" V 8580 4050 50  0001 C CNN
@@
 	6950 3400 7250 3400
 $Comp
-L R R72
+L R R1104
 U 1 1 5ADD4E48
 P 7200 3200
-F 0 "R72" H 7325 3150 50  0000 C CNN
+F 0 "R1104" H 7325 3150 50  0000 C CNN
 F 1 "10k" H 7325 3250 50  0000 C CNN
 F 2 "" V 7130 3200 50  0001 C CNN
@@
 $EndComp
 $Comp
-L BASE_PER_1V8 #PWR0146
+L BASE_PER_1V8 #PWR1113
 U 1 1 5ADD4F70
 P 7450 2950
-F 0 "#PWR0146" H 7450 2800 50  0001 C CNN
+F 0 "#PWR1113" H 7450 2800 50  0001 C CNN
 F 1 "BASE_PER_1V8" H 7450 3090 50  0000 C CNN
 F 2 "" H 7450 2950 50  0001 C CNN
@@
 $EndComp
 $Comp
-L BASE_PER_3V3 #PWR0147
+L BASE_PER_3V3 #PWR1112
 U 1 1 5ADCACA8
 P 6750 3700
-F 0 "#PWR0147" H 6750 3550 50  0001 C CNN
+F 0 "#PWR1112" H 6750 3550 50  0001 C CNN
 F 1 "BASE_PER_3V3" H 6750 3840 50  0000 C CNN
 F 2 "" H 6750 3700 50  0001 C CNN
@@
 $EndBitmap
 $Comp
-L OVSS #PWR0148
+L OVSS #PWR1102
 U 1 1 5AE7CB26
 P 4250 2900
-F 0 "#PWR0148" H 4250 2750 50  0001 C CNN
+F 0 "#PWR1102" H 4250 2750 50  0001 C CNN
 F 1 "OVSS" H 4250 3040 50  0000 C CNN
 F 2 "" H 4250 2900 50  0001 C CNN
@@
 Connection ~ 4250 2950
 $Comp
-L OVDD #PWR0149
+L OVDD #PWR1105
 U 1 1 5AE7D1B4
 P 4850 2900
-F 0 "#PWR0149" H 4850 2750 50  0001 C CNN
+F 0 "#PWR1105" H 4850 2750 50  0001 C CNN
 F 1 "OVDD" H 4850 3040 50  0000 C CNN
 F 2 "" H 4850 2900 50  0001 C CNN
@@
 Connection ~ 4850 2950
 $Comp
-L VCI_TP_VCC #PWR0150
+L VCI_TP_VCC #PWR1108
 U 1 1 5AD63D0F
 P 6000 2000
-F 0 "#PWR0150" H 6000 1850 50  0001 C CNN
+F 0 "#PWR1108" H 6000 1850 50  0001 C CNN
 F 1 "VCI_TP_VCC" H 6000 2140 50  0000 C CNN
 F 2 "" H 6000 2000 50  0001 C CNN
@@
 1.8V rises ~~12ms after 3.0V
 $Comp
-L AVDD #PWR0151
+L AVDD #PWR1107
 U 1 1 5ACF9758
 P 5200 3250
-F 0 "#PWR0151" H 5200 3100 50  0001 C CNN
+F 0 "#PWR1107" H 5200 3100 50  0001 C CNN
 F 1 "AVDD" H 5200 3390 50  0000 C CNN
 F 2 "" H 5200 3250 50  0001 C CNN

Commit message: Move reference designators in the schematic so that they are legible
Connections:
- wire segments 99 -> 134
Other:
- moved on the sheet: Q1101, Q1102, Q1103, Q1104, R1101, R1102, R1103, R1104, R1105, R1106
