File: mipi_dsi.sch (KiCad schematic (older format))
At the start: 19 parts, among them J1101 WP7B-P040VA1-R500, Q1101 2SK3018, Q1102 2SK3018, Q1103 2SK3018, Q1104 2SK3018

Commit message: Include reverse polarity protection circuit along with a simulation showing its effectiveness
Protecting VBAT from when board is sinking current via USB C. Protects against reverse polarity at the DC jack.

In EmCraft's instance VBUS should only be 5V when sinking current but they must protect against the condition when VBUS>12V and DC_IN=12V. This may need testing.
Connections:
- net labels added: 3V3_P
- net labels removed: BASE_PER_3V3
- wire segments 134 -> 99
Changed lines of the file:
@@
 Sheet 11 14
 Title "MIPI DSI"
-Date "2018-04-16"
+Date "2018-04-18"
 Rev "v0.1.0"
 Comp "Purism SPC"
@@
 NoConn ~ 4800 4750
 $Comp
-L GND #PWR0137
+L GND #PWR0138
 U 1 1 5AD63824
 P 4050 4950
-F 0 "#PWR0137" H 4050 4700 50  0001 C CNN
+F 0 "#PWR0138" H 4050 4700 50  0001 C CNN
 F 1 "GND" H 4050 4800 50  0000 C CNN
 F 2 "" H 4050 4950 50  0001 C CNN
@@
 	4300 3350 4050 3350
 Wire Wire Line
-	4050 3350 4050 3650
-Wire Wire Line
-	4050 3650 4050 3950
-Wire Wire Line
-	4050 3950 4050 4250
-Wire Wire Line
-	4050 4250 4050 4550
-Wire Wire Line
-	4050 4550 4050 4850
-Wire Wire Line
-	4050 4850 4050 4950
+	4050 3350 4050 4950
 Wire Wire Line
 	4300 3650 4050 3650
@@
 Connection ~ 4050 4850
 $Comp
-L GND #PWR0138
+L GND #PWR0139
 U 1 1 5AD638B9
 P 5050 4950
-F 0 "#PWR0138" H 5050 4700 50  0001 C CNN
+F 0 "#PWR0139" H 5050 4700 50  0001 C CNN
 F 1 "GND" H 5050 4800 50  0000 C CNN
 F 2 "" H 5050 4950 50  0001 C CNN
@@
 D3_N
 $Comp
-L BASE_PER_1V8 #PWR0139
+L BASE_PER_1V8 #PWR0140
 U 1 1 5AD9C3F5
 P 4550 2000
-F 0 "#PWR0139" H 4550 1850 50  0001 C CNN
+F 0 "#PWR0140" H 4550 1850 50  0001 C CNN
 F 1 "BASE_PER_1V8" H 4550 2140 50  0000 C CNN
 F 2 "" H 4550 2000 50  0001 C CNN
@@
 $EndComp
 Wire Wire Line
-	5300 2050 5300 3550
-Wire Wire Line
-	5300 3550 5300 4350
+	5300 2050 5300 4350
 Wire Wire Line
 	4800 3550 5300 3550
@@
 	4100 2100 4100 2050
 Wire Wire Line
-	4100 2050 4400 2050
-Wire Wire Line
-	4400 2050 4550 2050
-Wire Wire Line
-	4550 2050 4700 2050
-Wire Wire Line
-	4700 2050 5000 2050
-Wire Wire Line
-	5000 2050 5300 2050
-$Comp
-L GND #PWR0140
+	4100 2050 5300 2050
+$Comp
+L GND #PWR0141
 U 1 1 5AD9F1A8
 P 4550 2500
-F 0 "#PWR0140" H 4550 2250 50  0001 C CNN
+F 0 "#PWR0141" H 4550 2250 50  0001 C CNN
 F 1 "GND" H 4550 2350 50  0000 C CNN
 F 2 "" H 4550 2500 50  0001 C CNN
@@
 	4100 2400 4100 2450
 Wire Wire Line
-	4100 2450 4400 2450
-Wire Wire Line
-	4400 2450 4550 2450
-Wire Wire Line
-	4550 2450 4700 2450
-Wire Wire Line
-	4700 2450 5000 2450
+	4100 2450 5000 2450
 Wire Wire Line
 	5000 2450 5000 2400
@@
 Connection ~ 4550 2050
 Wire Wire Line
-	5400 2050 5400 3450
-Wire Wire Line
-	5400 3450 5400 4250
+	5400 2050 5400 4250
 $Comp
 L C C1105
@@
 $EndComp
 $Comp
-L GND #PWR0141
+L GND #PWR0142
 U 1 1 5ADA26B2
 P 6000 2500
-F 0 "#PWR0141" H 6000 2250 50  0001 C CNN
+F 0 "#PWR0142" H 6000 2250 50  0001 C CNN
 F 1 "GND" H 6000 2350 50  0000 C CNN
 F 2 "" H 6000 2500 50  0001 C CNN
@@
 	5550 2400 5550 2450
 Wire Wire Line
-	5550 2450 5850 2450
-Wire Wire Line
-	5850 2450 6000 2450
-Wire Wire Line
-	6000 2450 6150 2450
-Wire Wire Line
-	6150 2450 6450 2450
+	5550 2450 6450 2450
 Wire Wire Line
 	6450 2450 6450 2400
@@
 Connection ~ 6000 2450
 Wire Wire Line
-	5400 2050 5550 2050
-Wire Wire Line
-	5550 2050 5850 2050
-Wire Wire Line
-	5850 2050 6000 2050
-Wire Wire Line
-	6000 2050 6150 2050
-Wire Wire Line
-	6150 2050 6450 2050
+	5400 2050 6450 2050
 Wire Wire Line
 	6450 2050 6450 2100
@@
 	5500 3950 5500 4250
 Wire Wire Line
-	5500 4250 7850 4250
-Wire Wire Line
-	7850 4250 7900 4250
+	5500 4250 7900 4250
 Wire Wire Line
 	4800 3850 5600 3850
@@
 	5600 3850 5600 4150
 Wire Wire Line
-	5600 4150 5950 4150
-Wire Wire Line
-	5950 4150 6000 4150
+	5600 4150 6000 4150
 Wire Wire Line
 	5950 4150 5950 4100
 Connection ~ 5950 4150
 $Comp
-L BASE_PER_1V8 #PWR0142
+L BASE_PER_1V8 #PWR0143
 U 1 1 5ADCA156
 P 6200 3700
-F 0 "#PWR0142" H 6200 3550 50  0001 C CNN
+F 0 "#PWR0143" H 6200 3550 50  0001 C CNN
 F 1 "BASE_PER_1V8" H 6200 3840 50  0000 C CNN
 F 2 "" H 6200 3700 50  0001 C CNN
@@
 $EndComp
 Wire Wire Line
-	6200 3700 6200 3750
-Wire Wire Line
-	6200 3750 6200 3850
+	6200 3700 6200 3850
 Wire Wire Line
 	5950 3800 5950 3750
@@
 $EndComp
 Wire Wire Line
-	6400 4150 6800 4150
-Wire Wire Line
-	6800 4150 6850 4150
+	6400 4150 6850 4150
 Wire Wire Line
 	6800 4150 6800 4100
@@
 $EndComp
 $Comp
-L BASE_PER_1V8 #PWR0143
+L BASE_PER_1V8 #PWR0144
 U 1 1 5ADCB88E
-P 7900 3800
-F 0 "#PWR0143" H 7900 3650 50  0001 C CNN
-F 1 "BASE_PER_1V8" H 7900 3940 50  0000 C CNN
-F 2 "" H 7900 3800 50  0001 C CNN
-F 3 "" H 7900 3800 50  0001 C CNN
-	1    7900 3800
+P 7850 3800
+F 0 "#PWR0144" H 7850 3650 50  0001 C CNN
+F 1 "BASE_PER_1V8" H 7850 3940 50  0000 C CNN
+F 2 "" H 7850 3800 50  0001 C CNN
+F 3 "" H 7850 3800 50  0001 C CNN
+	1    7850 3800
 	1    0    0    -1
 $EndComp
@@
 Connection ~ 7850 4250
 Wire Wire Line
-	7900 3800 7850 3850
-Wire Wire Line
-	7850 3850 7850 3900
+	7850 3800 7850 3900
 Wire Wire Line
 	7850 3850 8100 3850
@@
 Connection ~ 7850 3850
 Wire Wire Line
-	8300 4250 8700 4250
-Wire Wire Line
-	8700 4250 8750 4250
+	8300 4250 8750 4250
 Wire Wire Line
 	8700 4250 8700 4200
-$Comp
-L BASE_PER_3V3 #PWR0144
-U 1 1 5ADCBF34
-P 8700 3800
-F 0 "#PWR0144" H 8700 3650 50  0001 C CNN
-F 1 "BASE_PER_3V3" H 8700 3940 50  0000 C CNN
-F 2 "" H 8700 3800 50  0001 C CNN
-F 3 "" H 8700 3800 50  0001 C CNN
-	1    8700 3800
-	1    0    0    -1
-$EndComp
 Wire Wire Line
 	8700 3900 8700 3800
@@
 	5900 3750 4800 3750
 Wire Wire Line
-	5900 3350 5900 3400
-Wire Wire Line
-	5900 3400 5900 3750
+	5900 3350 5900 3750
 Wire Wire Line
 	5900 3400 6000 3400
@@
 $EndComp
 Wire Wire Line
-	6200 2950 6200 3000
-Wire Wire Line
-	6200 3000 6200 3100
+	6200 2950 6200 3100
 Wire Wire Line
 	5900 3050 5900 3000
@@
 	7000 2750 7000 3400
 Wire Wire Line
-	7000 3400 7300 3400
-Wire Wire Line
-	7300 3400 7350 3400
+	7000 3400 7350 3400
 $Comp
 L R R1104
@@
 	1    0    0    -1
 $EndComp
-$Comp
-L BASE_PER_3V3 #PWR0147
-U 1 1 5ADCACA8
-P 6800 3700
-F 0 "#PWR0147" H 6800 3550 50  0001 C CNN
-F 1 "BASE_PER_3V3" H 6800 3840 50  0000 C CNN
-F 2 "" H 6800 3700 50  0001 C CNN
-F 3 "" H 6800 3700 50  0001 C CNN
-	1    6800 3700
-	1    0    0    -1
-$EndComp
 Wire Wire Line
 	6450 3400 6400 3400
@@
 Connection ~ 7300 3400
 Wire Wire Line
-	7550 2950 7550 3000
-Wire Wire Line
-	7550 3000 7550 3100
+	7550 2950 7550 3100
 Wire Wire Line
 	7300 3050 7300 3000
@@
 $EndBitmap
 $Comp
-L OVSS #PWR0148
+L OVSS #PWR0147
 U 1 1 5AE7CB26
 P 4250 2900
-F 0 "#PWR0148" H 4250 2750 50  0001 C CNN
+F 0 "#PWR0147" H 4250 2750 50  0001 C CNN
 F 1 "OVSS" H 4250 3040 50  0000 C CNN
 F 2 "" H 4250 2900 50  0001 C CNN
@@
 	4250 3150 4300 3150
 Wire Wire Line
-	4250 2900 4250 2950
-Wire Wire Line
-	4250 2950 4250 3050
-Wire Wire Line
-	4250 3050 4250 3150
+	4250 2900 4250 3150
 Wire Wire Line
 	4300 3050 4250 3050
@@
 Connection ~ 4250 2950
 $Comp
-L OVDD #PWR0149
+L OVDD #PWR0148
 U 1 1 5AE7D1B4
 P 4850 2900
-F 0 "#PWR0149" H 4850 2750 50  0001 C CNN
+F 0 "#PWR0148" H 4850 2750 50  0001 C CNN
 F 1 "OVDD" H 4850 3040 50  0000 C CNN
 F 2 "" H 4850 2900 50  0001 C CNN
@@
 	4850 3150 4800 3150
 Wire Wire Line
-	4850 2900 4850 2950
-Wire Wire Line
-	4850 2950 4850 3050
-Wire Wire Line
-	4850 3050 4850 3150
+	4850 2900 4850 3150
 Wire Wire Line
 	4800 3050 4850 3050
@@
 Connection ~ 4850 2950
 $Comp
-L VCI_TP_VCC #PWR0150
+L VCI_TP_VCC #PWR0149
 U 1 1 5AD63D0F
 P 6000 2000
-F 0 "#PWR0150" H 6000 1850 50  0001 C CNN
+F 0 "#PWR0149" H 6000 1850 50  0001 C CNN
 F 1 "VCI_TP_VCC" H 6000 2140 50  0000 C CNN
 F 2 "" H 6000 2000 50  0001 C CNN
@@
 1.8V rises ~~12ms after 3.0V
 $Comp
-L AVDD #PWR0151
+L AVDD #PWR0150
 U 1 1 5ACF9758
 P 5200 3250
-F 0 "#PWR0151" H 5200 3100 50  0001 C CNN
+F 0 "#PWR0150" H 5200 3100 50  0001 C CNN
 F 1 "AVDD" H 5200 3390 50  0000 C CNN
 F 2 "" H 5200 3250 50  0001 C CNN
@@
 Wire Wire Line
 	5200 3350 5200 3250
+$Comp
+L 3V3_P #PWR0151
+U 1 1 5AEA3227
+P 8700 3800
+F 0 "#PWR0151" H 8700 3650 50  0001 C CNN
+F 1 "3V3_P" H 8700 3940 50  0000 C CNN
+F 2 "" H 8700 3800 50  0001 C CNN
+F 3 "" H 8700 3800 50  0001 C CNN
+	1    8700 3800
+	1    0    0    -1
+$EndComp
+$Comp
+L 3V3_P #PWR0152
+U 1 1 5AEA329B
+P 6800 3700
+F 0 "#PWR0152" H 6800 3550 50  0001 C CNN
+F 1 "3V3_P" H 6800 3840 50  0000 C CNN
+F 2 "" H 6800 3700 50  0001 C CNN
+F 3 "" H 6800 3700 50  0001 C CNN
+	1    6800 3700
+	1    0    0    -1
+$EndComp
 $EndSCHEMATC

Commit message: Add USB type C circuit with DRP PD capability, should sink near 2A @ 5-6.5V and source 550mA @ 5V
Removed the reverse current protection circuit from the last commit due to the requirement changing to only 18650 battery and USB-C being possible power sources

Next thing to add is the charging circuit when the USB-C is in sink mode/role
Parts:
- renumbered C1101 to C1201, C1102 to C1202, C1103 to C1203, C1104 to C1204, C1105 to C1205, C1106 to C1206, C1107 to C1207, C1108 to C1208, J1101 to J1201, Q1101 to Q1201, Q1102 to Q1202, Q1103 to Q1203, Q1104 to Q1204, R1101 to R1201, R1102 to R1202, R1103 to R1203, R1104 to R1204, R1105 to R1205, R1106 to R1206
Connections:
- net labels added: 1V8_P
- net labels removed: BASE_PER_1V8
