File: uart.sch (KiCad schematic (older format))
At the start: 4 parts, among them J3 Conn_01x06, U13 74LVC2G241

Commit message: Assign all associated signals to their respective pins on the EmCraft i.MX8M SoM
The ERC is now at the same state as the DART SoM schematic. Need to compare various aspects of the current schematic against the EmCraft reference design. The main buck-boost will likely need to be switched to a 5V regulator, or be configured to output 5V.

A regulator will likely need to be added which will output some VBAT voltage level (3.5~4.2V) for the M.2 cards. The SIM7100 for example requires at least 3.4V!
Parts:
- renumbered C48 to C51
Changed lines of the file:
@@
 $EndComp
 $Comp
-L GND #PWR0108
+L GND #PWR0110
 U 1 1 5ACD6027
 P 6500 3800
-F 0 "#PWR0108" H 6500 3550 50  0001 C CNN
+F 0 "#PWR0110" H 6500 3550 50  0001 C CNN
 F 1 "GND" H 6500 3650 50  0000 C CNN
 F 2 "" H 6500 3800 50  0001 C CNN
@@
 NoConn ~ 6650 3950
 $Comp
-L GND #PWR0109
+L GND #PWR0111
 U 1 1 5ACD61E3
 P 5550 4200
-F 0 "#PWR0109" H 5550 3950 50  0001 C CNN
+F 0 "#PWR0111" H 5550 3950 50  0001 C CNN
 F 1 "GND" H 5550 4050 50  0000 C CNN
 F 2 "" H 5550 4200 50  0001 C CNN
@@
 $EndComp
 $Comp
-L SOM_NVCC_3V3 #PWR0110
+L SOM_NVCC_3V3 #PWR0112
 U 1 1 5ACD624F
 P 5550 3550
-F 0 "#PWR0110" H 5550 3400 50  0001 C CNN
+F 0 "#PWR0112" H 5550 3400 50  0001 C CNN
 F 1 "SOM_NVCC_3V3" H 5550 3690 50  0000 C CNN
 F 2 "" H 5550 3550 50  0001 C CNN
@@
 $EndComp
 $Comp
-L GND #PWR0111
+L GND #PWR0113
 U 1 1 5ACD62CD
 P 4750 3750
-F 0 "#PWR0111" H 4750 3500 50  0001 C CNN
+F 0 "#PWR0113" H 4750 3500 50  0001 C CNN
 F 1 "GND" H 4750 3600 50  0000 C CNN
 F 2 "" H 4750 3750 50  0001 C CNN
@@
 $EndComp
 $Comp
-L SOM_NVCC_3V3 #PWR0112
+L SOM_NVCC_3V3 #PWR0114
 U 1 1 5ACD631A
 P 4550 3750
-F 0 "#PWR0112" H 4550 3600 50  0001 C CNN
+F 0 "#PWR0114" H 4550 3600 50  0001 C CNN
 F 1 "SOM_NVCC_3V3" H 4550 3890 50  0000 C CNN
 F 2 "" H 4550 3750 50  0001 C CNN
@@
 	4850 3350 6000 3350
 $Comp
-L GND #PWR0113
+L GND #PWR0115
 U 1 1 5ACD6CF4
 P 5900 3750
-F 0 "#PWR0113" H 5900 3500 50  0001 C CNN
+F 0 "#PWR0115" H 5900 3500 50  0001 C CNN
 F 1 "GND" H 5900 3600 50  0000 C CNN
 F 2 "" H 5900 3750 50  0001 C CNN
@@
 RX<-TX
 $Comp
-L C C48
+L C C51
 U 1 1 5ACD7D29
 P 6250 3350
-F 0 "C48" H 6275 3450 50  0000 L CNN
+F 0 "C51" H 6275 3450 50  0000 L CNN
 F 1 "100nF" H 6275 3250 50  0000 L CNN
 F 2 "" H 6288 3200 50  0001 C CNN
@@
 $EndComp
 $Comp
-L GND #PWR0114
+L GND #PWR0116
 U 1 1 5ACD7D5E
 P 6250 3550
-F 0 "#PWR0114" H 6250 3300 50  0001 C CNN
+F 0 "#PWR0116" H 6250 3300 50  0001 C CNN
 F 1 "GND" H 6250 3400 50  0000 C CNN
 F 2 "" H 6250 3550 50  0001 C CNN
@@
 $EndComp
 $Comp
-L SOM_NVCC_3V3 #PWR0115
+L SOM_NVCC_3V3 #PWR0117
 U 1 1 5ACD7D75
 P 6250 3150
-F 0 "#PWR0115" H 6250 3000 50  0001 C CNN
+F 0 "#PWR0117" H 6250 3000 50  0001 C CNN
 F 1 "SOM_NVCC_3V3" H 6250 3290 50  0000 C CNN
 F 2 "" H 6250 3150 50  0001 C CNN

Commit message: Use "Start to sheet number*100 and use first free number" designation, any new component added to the schematic will occupy the next available number in that sheet
For example: if sheet 2 has R201-R215 and we add a new resistor it will become R216.
Parts:
- renumbered C51 to C701, J3 to J701, R56 to R701, U13 to U701
Changed lines of the file:
@@
 $EndDescr
 $Comp
-L 74LVC2G241 U13
+L 74LVC2G241 U701
 U 1 1 5ACD5FC3
 P 5200 3900
-F 0 "U13" H 5200 4300 60  0000 C CNN
+F 0 "U701" H 5200 4300 60  0000 C CNN
 F 1 "74LVC2G241" H 5200 4225 60  0000 C CNN
 F 2 "" H 5250 3650 60  0001 C CNN
@@
 $EndComp
 $Comp
-L Conn_01x06 J3
+L Conn_01x06 J701
 U 1 1 5ACD600C
 P 6850 3950
-F 0 "J3" H 6850 4250 50  0000 C CNN
+F 0 "J701" H 6850 4250 50  0000 C CNN
 F 1 "Conn_01x06" H 6850 3550 50  0000 C CNN
 F 2 "" H 6850 3950 50  0001 C CNN
@@
 $EndComp
 $Comp
-L GND #PWR0110
+L GND #PWR708
 U 1 1 5ACD6027
 P 6500 3800
-F 0 "#PWR0110" H 6500 3550 50  0001 C CNN
+F 0 "#PWR708" H 6500 3550 50  0001 C CNN
 F 1 "GND" H 6500 3650 50  0000 C CNN
 F 2 "" H 6500 3800 50  0001 C CNN
@@
 NoConn ~ 6650 3950
 $Comp
-L GND #PWR0111
+L GND #PWR704
 U 1 1 5ACD61E3
 P 5550 4200
-F 0 "#PWR0111" H 5550 3950 50  0001 C CNN
+F 0 "#PWR704" H 5550 3950 50  0001 C CNN
 F 1 "GND" H 5550 4050 50  0000 C CNN
 F 2 "" H 5550 4200 50  0001 C CNN
@@
 $EndComp
 $Comp
-L SOM_NVCC_3V3 #PWR0112
+L SOM_NVCC_3V3 #PWR703
 U 1 1 5ACD624F
 P 5550 3550
-F 0 "#PWR0112" H 5550 3400 50  0001 C CNN
+F 0 "#PWR703" H 5550 3400 50  0001 C CNN
 F 1 "SOM_NVCC_3V3" H 5550 3690 50  0000 C CNN
 F 2 "" H 5550 3550 50  0001 C CNN
@@
 $EndComp
 $Comp
-L GND #PWR0113
+L GND #PWR702
 U 1 1 5ACD62CD
 P 4750 3750
-F 0 "#PWR0113" H 4750 3500 50  0001 C CNN
+F 0 "#PWR702" H 4750 3500 50  0001 C CNN
 F 1 "GND" H 4750 3600 50  0000 C CNN
 F 2 "" H 4750 3750 50  0001 C CNN
@@
 $EndComp
 $Comp
-L SOM_NVCC_3V3 #PWR0114
+L SOM_NVCC_3V3 #PWR701
 U 1 1 5ACD631A
 P 4550 3750
-F 0 "#PWR0114" H 4550 3600 50  0001 C CNN
+F 0 "#PWR701" H 4550 3600 50  0001 C CNN
 F 1 "SOM_NVCC_3V3" H 4550 3890 50  0000 C CNN
 F 2 "" H 4550 3750 50  0001 C CNN
@@
 UART1_RXD
 $Comp
-L R R56
+L R R701
 U 1 1 5ACD6464
 P 5900 3550
-F 0 "R56" H 6000 3600 50  0000 C CNN
+F 0 "R701" H 6000 3600 50  0000 C CNN
 F 1 "100k" H 6050 3500 50  0000 C CNN
 F 2 "" V 5830 3550 50  0001 C CNN
@@
 	4850 3350 6000 3350
 $Comp
-L GND #PWR0115
+L GND #PWR705
 U 1 1 5ACD6CF4
 P 5900 3750
-F 0 "#PWR0115" H 5900 3500 50  0001 C CNN
+F 0 "#PWR705" H 5900 3500 50  0001 C CNN
 F 1 "GND" H 5900 3600 50  0000 C CNN
 F 2 "" H 5900 3750 50  0001 C CNN
@@
 RX<-TX
 $Comp
-L C C51
+L C C701
 U 1 1 5ACD7D29
 P 6250 3350
-F 0 "C51" H 6275 3450 50  0000 L CNN
+F 0 "C701" H 6275 3450 50  0000 L CNN
 F 1 "100nF" H 6275 3250 50  0000 L CNN
 F 2 "" H 6288 3200 50  0001 C CNN
@@
 $EndComp
 $Comp
-L GND #PWR0116
+L GND #PWR707
 U 1 1 5ACD7D5E
 P 6250 3550
-F 0 "#PWR0116" H 6250 3300 50  0001 C CNN
+F 0 "#PWR707" H 6250 3300 50  0001 C CNN
 F 1 "GND" H 6250 3400 50  0000 C CNN
 F 2 "" H 6250 3550 50  0001 C CNN
@@
 $EndComp
 $Comp
-L SOM_NVCC_3V3 #PWR0117
+L SOM_NVCC_3V3 #PWR706
 U 1 1 5ACD7D75
 P 6250 3150
-F 0 "#PWR0117" H 6250 3000 50  0001 C CNN
+F 0 "#PWR706" H 6250 3000 50  0001 C CNN
 F 1 "SOM_NVCC_3V3" H 6250 3290 50  0000 C CNN
 F 2 "" H 6250 3150 50  0001 C CNN

Commit message: Move reference designators in the schematic so that they are legible
Changed lines of the file:
@@
 $EndComp
 $Comp
-L GND #PWR708
+L GND #PWR0110
 U 1 1 5ACD6027
 P 6500 3800
-F 0 "#PWR708" H 6500 3550 50  0001 C CNN
+F 0 "#PWR0110" H 6500 3550 50  0001 C CNN
 F 1 "GND" H 6500 3650 50  0000 C CNN
 F 2 "" H 6500 3800 50  0001 C CNN
@@
 NoConn ~ 6650 3950
 $Comp
-L GND #PWR704
+L GND #PWR0111
 U 1 1 5ACD61E3
 P 5550 4200
-F 0 "#PWR704" H 5550 3950 50  0001 C CNN
+F 0 "#PWR0111" H 5550 3950 50  0001 C CNN
 F 1 "GND" H 5550 4050 50  0000 C CNN
 F 2 "" H 5550 4200 50  0001 C CNN
@@
 $EndComp
 $Comp
-L SOM_NVCC_3V3 #PWR703
+L SOM_NVCC_3V3 #PWR0112
 U 1 1 5ACD624F
 P 5550 3550
-F 0 "#PWR703" H 5550 3400 50  0001 C CNN
+F 0 "#PWR0112" H 5550 3400 50  0001 C CNN
 F 1 "SOM_NVCC_3V3" H 5550 3690 50  0000 C CNN
 F 2 "" H 5550 3550 50  0001 C CNN
@@
 $EndComp
 $Comp
-L GND #PWR702
+L GND #PWR0113
 U 1 1 5ACD62CD
 P 4750 3750
-F 0 "#PWR702" H 4750 3500 50  0001 C CNN
+F 0 "#PWR0113" H 4750 3500 50  0001 C CNN
 F 1 "GND" H 4750 3600 50  0000 C CNN
 F 2 "" H 4750 3750 50  0001 C CNN
@@
 $EndComp
 $Comp
-L SOM_NVCC_3V3 #PWR701
+L SOM_NVCC_3V3 #PWR0114
 U 1 1 5ACD631A
 P 4550 3750
-F 0 "#PWR701" H 4550 3600 50  0001 C CNN
+F 0 "#PWR0114" H 4550 3600 50  0001 C CNN
 F 1 "SOM_NVCC_3V3" H 4550 3890 50  0000 C CNN
 F 2 "" H 4550 3750 50  0001 C CNN
@@
 U 1 1 5ACD6464
 P 5900 3550
-F 0 "R701" H 6000 3600 50  0000 C CNN
+F 0 "R701" H 6050 3600 50  0000 C CNN
 F 1 "100k" H 6050 3500 50  0000 C CNN
 F 2 "" V 5830 3550 50  0001 C CNN
@@
 	4850 3350 6000 3350
 $Comp
-L GND #PWR705
+L GND #PWR0115
 U 1 1 5ACD6CF4
 P 5900 3750
-F 0 "#PWR705" H 5900 3500 50  0001 C CNN
+F 0 "#PWR0115" H 5900 3500 50  0001 C CNN
 F 1 "GND" H 5900 3600 50  0000 C CNN
 F 2 "" H 5900 3750 50  0001 C CNN
@@
 $EndComp
 $Comp
-L GND #PWR707
+L GND #PWR0116
 U 1 1 5ACD7D5E
 P 6250 3550
-F 0 "#PWR707" H 6250 3300 50  0001 C CNN
+F 0 "#PWR0116" H 6250 3300 50  0001 C CNN
 F 1 "GND" H 6250 3400 50  0000 C CNN
 F 2 "" H 6250 3550 50  0001 C CNN
@@
 $EndComp
 $Comp
-L SOM_NVCC_3V3 #PWR706
+L SOM_NVCC_3V3 #PWR0117
 U 1 1 5ACD7D75
 P 6250 3150
-F 0 "#PWR706" H 6250 3000 50  0001 C CNN
+F 0 "#PWR0117" H 6250 3000 50  0001 C CNN
 F 1 "SOM_NVCC_3V3" H 6250 3290 50  0000 C CNN
 F 2 "" H 6250 3150 50  0001 C CNN

Commit message: Include reverse polarity protection circuit along with a simulation showing its effectiveness
Protecting VBAT from when board is sinking current via USB C. Protects against reverse polarity at the DC jack.

In EmCraft's instance VBUS should only be 5V when sinking current but they must protect against the condition when VBUS>12V and DC_IN=12V. This may need testing.
Connections:
- net labels added: 3V3_OUT
- net labels removed: SOM_NVCC_3V3
Changed lines of the file:
@@
 Sheet 7 14
 Title "UART Debug"
-Date "2018-04-16"
+Date "2018-04-18"
 Rev "v0.1.0"
 Comp "Purism SPC"
@@
 $EndComp
 $Comp
-L SOM_NVCC_3V3 #PWR0112
-U 1 1 5ACD624F
-P 5550 3550
-F 0 "#PWR0112" H 5550 3400 50  0001 C CNN
-F 1 "SOM_NVCC_3V3" H 5550 3690 50  0000 C CNN
-F 2 "" H 5550 3550 50  0001 C CNN
-F 3 "" H 5550 3550 50  0001 C CNN
-	1    5550 3550
-	1    0    0    -1
-$EndComp
-$Comp
-L GND #PWR0113
+L GND #PWR0112
 U 1 1 5ACD62CD
 P 4750 3750
-F 0 "#PWR0113" H 4750 3500 50  0001 C CNN
+F 0 "#PWR0112" H 4750 3500 50  0001 C CNN
 F 1 "GND" H 4750 3600 50  0000 C CNN
 F 2 "" H 4750 3750 50  0001 C CNN
 F 3 "" H 4750 3750 50  0001 C CNN
 	1    4750 3750
-	1    0    0    -1
-$EndComp
-$Comp
-L SOM_NVCC_3V3 #PWR0114
-U 1 1 5ACD631A
-P 4550 3750
-F 0 "#PWR0114" H 4550 3600 50  0001 C CNN
-F 1 "SOM_NVCC_3V3" H 4550 3890 50  0000 C CNN
-F 2 "" H 4550 3750 50  0001 C CNN
-F 3 "" H 4550 3750 50  0001 C CNN
-	1    4550 3750
 	1    0    0    -1
 $EndComp
@@
 	4850 3350 6000 3350
 $Comp
-L GND #PWR0115
+L GND #PWR0113
 U 1 1 5ACD6CF4
 P 5900 3750
-F 0 "#PWR0115" H 5900 3500 50  0001 C CNN
+F 0 "#PWR0113" H 5900 3500 50  0001 C CNN
 F 1 "GND" H 5900 3600 50  0000 C CNN
 F 2 "" H 5900 3750 50  0001 C CNN
@@
 $EndComp
 $Comp
-L GND #PWR0116
+L GND #PWR0114
 U 1 1 5ACD7D5E
 P 6250 3550
-F 0 "#PWR0116" H 6250 3300 50  0001 C CNN
+F 0 "#PWR0114" H 6250 3300 50  0001 C CNN
 F 1 "GND" H 6250 3400 50  0000 C CNN
 F 2 "" H 6250 3550 50  0001 C CNN
@@
 	1    0    0    -1
 $EndComp
-$Comp
-L SOM_NVCC_3V3 #PWR0117
-U 1 1 5ACD7D75
+Wire Wire Line
+	6250 3550 6250 3500
+Wire Wire Line
+	6250 3200 6250 3150
+Text Notes 6650 3600 0    60   ~ 0
+Accepts 3.3V \nor 5V Logic
+$Comp
+L 3V3_OUT #PWR0115
+U 1 1 5AEA3EFC
+P 5550 3550
+F 0 "#PWR0115" H 5550 3400 50  0001 C CNN
+F 1 "3V3_OUT" H 5550 3690 50  0000 C CNN
+F 2 "" H 5550 3550 50  0001 C CNN
+F 3 "" H 5550 3550 50  0001 C CNN
+	1    5550 3550
+	1    0    0    -1
+$EndComp
+$Comp
+L 3V3_OUT #PWR0116
+U 1 1 5AEA3F25
+P 4550 3750
+F 0 "#PWR0116" H 4550 3600 50  0001 C CNN
+F 1 "3V3_OUT" H 4550 3890 50  0000 C CNN
+F 2 "" H 4550 3750 50  0001 C CNN
+F 3 "" H 4550 3750 50  0001 C CNN
+	1    4550 3750
+	1    0    0    -1
+$EndComp
+$Comp
+L 3V3_OUT #PWR0117
+U 1 1 5AEA3F4E
 P 6250 3150
 F 0 "#PWR0117" H 6250 3000 50  0001 C CNN
-F 1 "SOM_NVCC_3V3" H 6250 3290 50  0000 C CNN
+F 1 "3V3_OUT" H 6250 3290 50  0000 C CNN
 F 2 "" H 6250 3150 50  0001 C CNN
 F 3 "" H 6250 3150 50  0001 C CNN
@@
 	1    0    0    -1
 $EndComp
-Wire Wire Line
-	6250 3550 6250 3500
-Wire Wire Line
-	6250 3200 6250 3150
-Text Notes 6650 3600 0    60   ~ 0
-Accepts 3.3V \nor 5V Logic
 $EndSCHEMATC
