File: uart.sch (KiCad schematic (older format))
At the start: 4 parts, among them J701 Conn_01x06, U701 74LVC2G241

Commit message: Assign most of the capacitors their respective footprints (most are 0603s), add camera/CSI connector component info, source cheaper distributors for 3.5mm headset jack and RJ45
Parts:
- C701: footprint (none) -> Capacitors_SMD:C_0603
Changed lines of the file:
@@
 $EndComp
 $Comp
-L GND #PWR708
+L GND #PWR0137
 U 1 1 5ACD6027
 P 6500 3800
-F 0 "#PWR708" H 6500 3550 50  0001 C CNN
+F 0 "#PWR0137" H 6500 3550 50  0001 C CNN
 F 1 "GND" H 6500 3650 50  0000 C CNN
 F 2 "" H 6500 3800 50  0001 C CNN
@@
 NoConn ~ 6650 3950
 $Comp
-L GND #PWR704
+L GND #PWR0138
 U 1 1 5ACD61E3
 P 5550 4200
-F 0 "#PWR704" H 5550 3950 50  0001 C CNN
+F 0 "#PWR0138" H 5550 3950 50  0001 C CNN
 F 1 "GND" H 5550 4050 50  0000 C CNN
 F 2 "" H 5550 4200 50  0001 C CNN
@@
 $EndComp
 $Comp
-L GND #PWR702
+L GND #PWR0139
 U 1 1 5ACD62CD
 P 4750 3750
-F 0 "#PWR702" H 4750 3500 50  0001 C CNN
+F 0 "#PWR0139" H 4750 3500 50  0001 C CNN
 F 1 "GND" H 4750 3600 50  0000 C CNN
 F 2 "" H 4750 3750 50  0001 C CNN
@@
 	4850 3350 6000 3350
 $Comp
-L GND #PWR705
+L GND #PWR0140
 U 1 1 5ACD6CF4
 P 5900 3750
-F 0 "#PWR705" H 5900 3500 50  0001 C CNN
+F 0 "#PWR0140" H 5900 3500 50  0001 C CNN
 F 1 "GND" H 5900 3600 50  0000 C CNN
 F 2 "" H 5900 3750 50  0001 C CNN
@@
 F 0 "C701" H 6275 3450 50  0000 L CNN
 F 1 "100nF" H 6275 3250 50  0000 L CNN
-F 2 "" H 6288 3200 50  0001 C CNN
+F 2 "Capacitors_SMD:C_0603" H 6288 3200 50  0001 C CNN
 F 3 "" H 6250 3350 50  0001 C CNN
 	1    6250 3350
@@
 $EndComp
 $Comp
-L GND #PWR707
+L GND #PWR0141
 U 1 1 5ACD7D5E
 P 6250 3550
-F 0 "#PWR707" H 6250 3300 50  0001 C CNN
+F 0 "#PWR0141" H 6250 3300 50  0001 C CNN
 F 1 "GND" H 6250 3400 50  0000 C CNN
 F 2 "" H 6250 3550 50  0001 C CNN
@@
 Accepts 3.3V \nor 5V Logic
 $Comp
-L 3V3_OUT #PWR703
+L 3V3_OUT #PWR0142
 U 1 1 5AEA3EFC
 P 5550 3550
-F 0 "#PWR703" H 5550 3400 50  0001 C CNN
+F 0 "#PWR0142" H 5550 3400 50  0001 C CNN
 F 1 "3V3_OUT" H 5550 3690 50  0000 C CNN
 F 2 "" H 5550 3550 50  0001 C CNN
@@
 $EndComp
 $Comp
-L 3V3_OUT #PWR701
+L 3V3_OUT #PWR0143
 U 1 1 5AEA3F25
 P 4550 3750
-F 0 "#PWR701" H 4550 3600 50  0001 C CNN
+F 0 "#PWR0143" H 4550 3600 50  0001 C CNN
 F 1 "3V3_OUT" H 4550 3890 50  0000 C CNN
 F 2 "" H 4550 3750 50  0001 C CNN
@@
 $EndComp
 $Comp
-L 3V3_OUT #PWR706
+L 3V3_OUT #PWR0144
 U 1 1 5AEA3F4E
 P 6250 3150
-F 0 "#PWR706" H 6250 3000 50  0001 C CNN
+F 0 "#PWR0144" H 6250 3000 50  0001 C CNN
 F 1 "3V3_OUT" H 6250 3290 50  0000 C CNN
 F 2 "" H 6250 3150 50  0001 C CNN

Commit message: Connect VCC of the USB1_VBUS comparitor (TLV3201AIDBVR) to 5V_SOM instead of 5V_P so that VBUS presence can be detected quickly enough for the USB Serial Downloader bootmode, connect the TVS diodes on the HDMI receptacle to the proper pins
Parts:
- J701: value Conn_01x06 -> Debug_UART
Changed lines of the file:
@@
 P 6850 3950
 F 0 "J701" H 6850 4250 50  0000 C CNN
-F 1 "Conn_01x06" H 6850 3550 50  0000 C CNN
+F 1 "Debug_UART" H 6850 3550 50  0000 C CNN
 F 2 "" H 6850 3950 50  0001 C CNN
 F 3 "https://media.digikey.com/PDF/Data%20Sheets/Sullins%20PDFs/z%20RzCzzzSzzN-RC,%20ST,11635-B.pdf" H 6850 3950 50  0001 C CNN
@@
 $EndComp
 $Comp
-L GND #PWR0149
+L GND #PWR0150
 U 1 1 5ACD6027
 P 6500 3800
-F 0 "#PWR0149" H 6500 3550 50  0001 C CNN
+F 0 "#PWR0150" H 6500 3550 50  0001 C CNN
 F 1 "GND" H 6500 3650 50  0000 C CNN
 F 2 "" H 6500 3800 50  0001 C CNN
@@
 NoConn ~ 6650 3950
 $Comp
-L GND #PWR0150
+L GND #PWR0151
 U 1 1 5ACD61E3
 P 5550 4200
-F 0 "#PWR0150" H 5550 3950 50  0001 C CNN
+F 0 "#PWR0151" H 5550 3950 50  0001 C CNN
 F 1 "GND" H 5550 4050 50  0000 C CNN
 F 2 "" H 5550 4200 50  0001 C CNN
@@
 $EndComp
 $Comp
-L GND #PWR0151
+L GND #PWR0152
 U 1 1 5ACD62CD
 P 4750 3750
-F 0 "#PWR0151" H 4750 3500 50  0001 C CNN
+F 0 "#PWR0152" H 4750 3500 50  0001 C CNN
 F 1 "GND" H 4750 3600 50  0000 C CNN
 F 2 "" H 4750 3750 50  0001 C CNN
@@
 	4850 3350 6000 3350
 $Comp
-L GND #PWR0152
+L GND #PWR0153
 U 1 1 5ACD6CF4
 P 5900 3750
-F 0 "#PWR0152" H 5900 3500 50  0001 C CNN
+F 0 "#PWR0153" H 5900 3500 50  0001 C CNN
 F 1 "GND" H 5900 3600 50  0000 C CNN
 F 2 "" H 5900 3750 50  0001 C CNN
@@
 $EndComp
 $Comp
-L GND #PWR0153
+L GND #PWR0154
 U 1 1 5ACD7D5E
 P 6250 3550
-F 0 "#PWR0153" H 6250 3300 50  0001 C CNN
+F 0 "#PWR0154" H 6250 3300 50  0001 C CNN
 F 1 "GND" H 6250 3400 50  0000 C CNN
 F 2 "" H 6250 3550 50  0001 C CNN
@@
 Accepts 3.3V \nor 5V Logic
 $Comp
-L 3V3_OUT #PWR0154
+L 3V3_OUT #PWR0155
 U 1 1 5AEA3EFC
 P 5550 3550
-F 0 "#PWR0154" H 5550 3400 50  0001 C CNN
+F 0 "#PWR0155" H 5550 3400 50  0001 C CNN
 F 1 "3V3_OUT" H 5550 3690 50  0000 C CNN
 F 2 "" H 5550 3550 50  0001 C CNN
@@
 $EndComp
 $Comp
-L 3V3_OUT #PWR0155
+L 3V3_OUT #PWR0156
 U 1 1 5AEA3F25
 P 4550 3750
-F 0 "#PWR0155" H 4550 3600 50  0001 C CNN
+F 0 "#PWR0156" H 4550 3600 50  0001 C CNN
 F 1 "3V3_OUT" H 4550 3890 50  0000 C CNN
 F 2 "" H 4550 3750 50  0001 C CNN
@@
 $EndComp
 $Comp
-L 3V3_OUT #PWR0156
+L 3V3_OUT #PWR0157
 U 1 1 5AEA3F4E
 P 6250 3150
-F 0 "#PWR0156" H 6250 3000 50  0001 C CNN
+F 0 "#PWR0157" H 6250 3000 50  0001 C CNN
 F 1 "3V3_OUT" H 6250 3290 50  0000 C CNN
 F 2 "" H 6250 3150 50  0001 C CNN

Commit message: Add haptic motor and debug UART headers/connectors, include notes in schematic r egarding the DPDT switches' & logic gates' pins being interchangeable
Used right-angled JST 2.5mm connector scaled in half as the motor connector footprint & 3D model, included 1cm distance from haptic motor placement from the edge of the connector (shown on silkscreen).
Parts:
- J701: footprint (none) -> Pin_Headers:Pin_Header_Straight_1x06_Pitch2.54mm
Changed lines of the file:
@@
 F 0 "J701" H 6850 4250 50  0000 C CNN
 F 1 "Debug_UART" H 6850 3550 50  0000 C CNN
-F 2 "" H 6850 3950 50  0001 C CNN
+F 2 "Pin_Headers:Pin_Header_Straight_1x06_Pitch2.54mm" H 6850 3950 50  0001 C CNN
 F 3 "https://media.digikey.com/PDF/Data%20Sheets/Sullins%20PDFs/z%20RzCzzzSzzN-RC,%20ST,11635-B.pdf" H 6850 3950 50  0001 C CNN
 F 4 "Sullins" H 6850 3950 60  0001 C CNN "MFG Name"
