File: sdio_demux.sch (KiCad schematic (older format))
At the start: 4 parts, among them U1601 TS3A27518E

Commit message: Footprints of SD card socket and demultiplexer assigned
Parts:
- U1601: footprint (none) -> dvk-mx8m-bsb:TS3A27518E
Changed lines of the file:
@@
 F 0 "U1601" H 5600 4900 60  0000 C CNN
 F 1 "TS3A27518E" H 5800 1950 60  0000 C CNN
-F 2 "" H 5850 4900 60  0001 C CNN
-F 3 "http://www.ti.com/lit/ds/symlink/ts3a27518e.pdf" H 6750 4550 60  0000 C CNN
+F 2 "dvk-mx8m-bsb:TS3A27518E" H 5850 4900 60  0001 C CNN
+F 3 "http://www.ti.com/lit/ds/symlink/ts3a27518e.pdf" H 6750 4550 60  0001 C CNN
 F 4 "Texas Instruments" H 5800 3450 60  0001 C CNN "MFG Name"
 F 5 "TS3A27518ERTWR" H 5800 3450 60  0001 C CNN "MFG Part Num"
@@
 $Bitmap
 Pos 4050 1400
-Scale 1.000000
+Scale 1,000000
 Data
 89 50 4E 47 0D 0A 1A 0A 00 00 00 0D 49 48 44 52 00 00 02 A0 00 00 00 76 08 02 00 00 00 98 A6 B6
