File: usb_hub.sch (KiCad schematic (older format))
At the start: 25 parts, among them U1001 USB2422, Y1001 24MHz

Commit message: Add NOR flash chip schematic, use mini-HDMI (requested) instead of micro and add its corresponding properties and footprint, use 3.5mm CTIA headset jack with through-hole pins rather than an SMD one for extra "mechanical rigidity"
Will likely want to use a USB-C receptacle with through-hole shield pins.
Other:
- note added: "TODO:\nUse USB4640???"
Changed lines of the file:
@@
 $Descr A4 11693 8268
 encoding utf-8
-Sheet 10 19
+Sheet 10 20
 Title ""
-Date "2018-05-02"
+Date "2018-05-14"
 Rev "v0.1.0"
 Comp "Purism SPC"
@@
 Text Notes 4975 5900 0    60   ~ 0
 Where Cxout and Cxin are capacitance to GND\nand Cxout_xin is capacitance between XOUT/XIN
+Text Notes 5650 1200 0    60   ~ 0
+TODO:\nUse USB4640???
 $EndSCHEMATC

Commit message: Include power load switch ICs to the 3.3V and 5V rails so that the SoC can disable the peripherals' power using the PWR_EN signal
Need to verify that 3V3's capacitance is greater than 3V3_P!

Next step is to have PWR_EN control the various logic translator chips EN pins.
Connections:
- net +5V renamed 5V_P
Changed lines of the file:
@@
 $EndComp
 $Comp
-L GND #PWR0133
+L GND #PWR0152
 U 1 1 5AFCAB4E
 P 7900 4700
-F 0 "#PWR0133" H 7900 4450 50  0001 C CNN
+F 0 "#PWR0152" H 7900 4450 50  0001 C CNN
 F 1 "GND" H 7900 4550 50  0000 C CNN
 F 2 "" H 7900 4700 50  0001 C CNN
@@
 $EndComp
 $Comp
-L GND #PWR0134
+L GND #PWR0153
 U 1 1 5AFCB041
 P 7650 5350
-F 0 "#PWR0134" H 7650 5100 50  0001 C CNN
+F 0 "#PWR0153" H 7650 5100 50  0001 C CNN
 F 1 "GND" H 7650 5200 50  0000 C CNN
 F 2 "" H 7650 5350 50  0001 C CNN
@@
 $EndComp
 $Comp
-L 3V3_P #PWR0135
+L 3V3_P #PWR0154
 U 1 1 5AFCD0CA
 P 8200 4200
-F 0 "#PWR0135" H 8200 4050 50  0001 C CNN
+F 0 "#PWR0154" H 8200 4050 50  0001 C CNN
 F 1 "3V3_P" H 8200 4340 50  0000 C CNN
 F 2 "" H 8200 4200 50  0001 C CNN
@@
 $EndComp
 $Comp
-L GND #PWR0136
+L GND #PWR0155
 U 1 1 5AFD0B06
 P 8400 4050
-F 0 "#PWR0136" H 8400 3800 50  0001 C CNN
+F 0 "#PWR0155" H 8400 3800 50  0001 C CNN
 F 1 "GND" H 8400 3900 50  0000 C CNN
 F 2 "" H 8400 4050 50  0001 C CNN
@@
 $EndComp
 $Comp
-L GND #PWR0137
+L GND #PWR0156
 U 1 1 5AFD409A
 P 5100 4350
-F 0 "#PWR0137" H 5100 4100 50  0001 C CNN
+F 0 "#PWR0156" H 5100 4100 50  0001 C CNN
 F 1 "GND" H 5100 4200 50  0000 C CNN
 F 2 "" H 5100 4350 50  0001 C CNN
@@
 $EndComp
 $Comp
-L GND #PWR0138
+L GND #PWR0157
 U 1 1 5AFD422F
 P 5100 3750
-F 0 "#PWR0138" H 5100 3500 50  0001 C CNN
+F 0 "#PWR0157" H 5100 3500 50  0001 C CNN
 F 1 "GND" H 5100 3600 50  0000 C CNN
 F 2 "" H 5100 3750 50  0001 C CNN
@@
 $EndComp
 $Comp
-L GND #PWR0139
+L GND #PWR0158
 U 1 1 5AFD5419
 P 4400 5100
-F 0 "#PWR0139" H 4400 4850 50  0001 C CNN
+F 0 "#PWR0158" H 4400 4850 50  0001 C CNN
 F 1 "GND" H 4400 4950 50  0000 C CNN
 F 2 "" H 4400 5100 50  0001 C CNN
@@
 $EndComp
 $Comp
-L GND #PWR0140
+L GND #PWR0159
 U 1 1 5AE5E881
 P 4700 3900
-F 0 "#PWR0140" H 4700 3650 50  0001 C CNN
+F 0 "#PWR0159" H 4700 3650 50  0001 C CNN
 F 1 "GND" H 4700 3750 50  0000 C CNN
 F 2 "" H 4700 3900 50  0001 C CNN
@@
 $EndComp
 $Comp
-L 3V3_P #PWR0141
+L 3V3_P #PWR0160
 U 1 1 5AE604F2
 P 4700 3100
-F 0 "#PWR0141" H 4700 2950 50  0001 C CNN
+F 0 "#PWR0160" H 4700 2950 50  0001 C CNN
 F 1 "3V3_P" H 4700 3240 50  0000 C CNN
 F 2 "" H 4700 3100 50  0001 C CNN
@@
 NoConn ~ 7000 3100
 NoConn ~ 7000 3200
-$Comp
-L +5V #PWR0142
-U 1 1 5AE74EE5
-P 3700 1700
-F 0 "#PWR0142" H 3700 1550 50  0001 C CNN
-F 1 "+5V" H 3700 1840 50  0000 C CNN
-F 2 "" H 3700 1700 50  0001 C CNN
-F 3 "" H 3700 1700 50  0001 C CNN
-	1    3700 1700
-	1    0    0    -1
-$EndComp
 $Comp
 L R R1003
@@
 $EndComp
 $Comp
-L GND #PWR0143
+L GND #PWR0161
 U 1 1 5AE75200
 P 3950 2200
-F 0 "#PWR0143" H 3950 1950 50  0001 C CNN
+F 0 "#PWR0161" H 3950 1950 50  0001 C CNN
 F 1 "GND" H 3950 2050 50  0000 C CNN
 F 2 "" H 3950 2200 50  0001 C CNN
@@
 $EndComp
 $Comp
-L GND #PWR0144
+L GND #PWR0162
 U 1 1 5AE8DF47
 P 5150 3000
-F 0 "#PWR0144" H 5150 2750 50  0001 C CNN
+F 0 "#PWR0162" H 5150 2750 50  0001 C CNN
 F 1 "GND" H 5150 2850 50  0000 C CNN
 F 2 "" H 5150 3000 50  0001 C CNN
@@
 $EndComp
 $Comp
-L GND #PWR0145
+L GND #PWR0163
 U 1 1 5AF52101
 P 3050 2200
-F 0 "#PWR0145" H 3050 1950 50  0001 C CNN
+F 0 "#PWR0163" H 3050 1950 50  0001 C CNN
 F 1 "GND" H 3050 2050 50  0000 C CNN
 F 2 "" H 3050 2200 50  0001 C CNN
@@
 Text Notes 5650 1200 0    60   ~ 0
 TODO:\nUse USB4640???
+$Comp
+L 5V_P #PWR0164
+U 1 1 5B3E4C16
+P 3700 1700
+F 0 "#PWR0164" H 3700 1550 50  0001 C CNN
+F 1 "5V_P" H 3700 1840 50  0000 C CNN
+F 2 "" H 3700 1700 50  0001 C CNN
+F 3 "" H 3700 1700 50  0001 C CNN
+	1    3700 1700
+	1    0    0    -1
+$EndComp
 $EndSCHEMATC
