File: csi.sch (KiCad schematic (older format))
At the start: 16 parts, among them J1301 OV5640, SW1301 DPDT, U1301 74LVC1G32

Commit message: Make corrections to schematic based on Emcraft's baseboard revision changes
Connections:
- net CLKO2 renamed CLKO1
Changed lines of the file:
@@
 Sheet 13 24
 Title ""
-Date "2018-05-31"
+Date "2018-06-01"
 Rev "v0.1.0"
 Comp "Purism SPC"
@@
 $EndComp
 $Comp
-L GND #PWR0194
+L GND #PWR0196
 U 1 1 5B1EAF19
 P 6800 4350
-F 0 "#PWR0194" H 6800 4100 50  0001 C CNN
+F 0 "#PWR0196" H 6800 4100 50  0001 C CNN
 F 1 "GND" H 6800 4200 50  0000 C CNN
 F 2 "" H 6800 4350 50  0001 C CNN
@@
 $EndComp
 $Comp
-L 1V8_P #PWR0195
+L 1V8_P #PWR0197
 U 1 1 5B1DBE6F
 P 6300 3450
-F 0 "#PWR0195" H 6300 3300 50  0001 C CNN
+F 0 "#PWR0197" H 6300 3300 50  0001 C CNN
 F 1 "1V8_P" H 6300 3590 50  0000 C CNN
 F 2 "" H 6300 3450 50  0001 C CNN
@@
 $EndComp
 $Comp
-L GND #PWR0196
+L GND #PWR0198
 U 1 1 5B1A278C
 P 7650 3450
-F 0 "#PWR0196" H 7650 3200 50  0001 C CNN
+F 0 "#PWR0198" H 7650 3200 50  0001 C CNN
 F 1 "GND" H 7650 3300 50  0000 C CNN
 F 2 "" H 7650 3450 50  0001 C CNN
@@
 $EndComp
 $Comp
-L GND #PWR0197
+L GND #PWR0199
 U 1 1 5B1964B5
 P 7800 4100
-F 0 "#PWR0197" H 7800 3850 50  0001 C CNN
+F 0 "#PWR0199" H 7800 3850 50  0001 C CNN
 F 1 "GND" H 7800 3950 50  0000 C CNN
 F 2 "" H 7800 4100 50  0001 C CNN
@@
 $EndComp
 Text HLabel 10750 3650 2    60   Input ~ 0
-CLKO2
+CLKO1
 $Comp
-L 1V8_P #PWR0198
+L 1V8_P #PWR0200
 U 1 1 5B105CDE
 P 10350 3250
-F 0 "#PWR0198" H 10350 3100 50  0001 C CNN
+F 0 "#PWR0200" H 10350 3100 50  0001 C CNN
 F 1 "1V8_P" H 10350 3390 50  0000 C CNN
 F 2 "" H 10350 3250 50  0001 C CNN
@@
 $EndComp
 $Comp
-L 1V8_P #PWR0199
+L 1V8_P #PWR0201
 U 1 1 5B0F8E1D
 P 9800 2600
-F 0 "#PWR0199" H 9800 2450 50  0001 C CNN
+F 0 "#PWR0201" H 9800 2450 50  0001 C CNN
 F 1 "1V8_P" H 9800 2740 50  0000 C CNN
 F 2 "" H 9800 2600 50  0001 C CNN
@@
 C0_P
 $Comp
-L 1V8_P #PWR0200
+L 1V8_P #PWR0202
 U 1 1 5B19049B
 P 7800 3000
-F 0 "#PWR0200" H 7800 2850 50  0001 C CNN
+F 0 "#PWR0202" H 7800 2850 50  0001 C CNN
 F 1 "1V8_P" H 7800 3140 50  0000 C CNN
 F 2 "" H 7800 3000 50  0001 C CNN
@@
 $EndComp
 $Comp
-L 2V8_P #PWR0201
+L 2V8_P #PWR0203
 U 1 1 5B2B0429
 P 8900 2600
-F 0 "#PWR0201" H 8900 2450 50  0001 C CNN
+F 0 "#PWR0203" H 8900 2450 50  0001 C CNN
 F 1 "2V8_P" H 8900 2740 50  0000 C CNN
 F 2 "" H 8900 2600 50  0001 C CNN
@@
 NoConn ~ 9200 2650
 $Comp
-L GND #PWR0202
+L GND #PWR0204
 U 1 1 5B11F1A4
 P 9150 4100
-F 0 "#PWR0202" H 9150 3850 50  0001 C CNN
+F 0 "#PWR0204" H 9150 3850 50  0001 C CNN
 F 1 "GND" H 9150 3950 50  0000 C CNN
 F 2 "" H 9150 4100 50  0001 C CNN
@@
 NoConn ~ 9200 3550
 $Comp
-L GND #PWR0203
+L GND #PWR0205
 U 1 1 5B11FD52
 P 9750 4100
-F 0 "#PWR0203" H 9750 3850 50  0001 C CNN
+F 0 "#PWR0205" H 9750 3850 50  0001 C CNN
 F 1 "GND" H 9750 3950 50  0000 C CNN
 F 2 "" H 9750 4100 50  0001 C CNN
@@
 	9800 2600 9800 2850
 $Comp
-L GND #PWR0204
+L GND #PWR0206
 U 1 1 5B164232
 P 6400 4350
-F 0 "#PWR0204" H 6400 4100 50  0001 C CNN
+F 0 "#PWR0206" H 6400 4100 50  0001 C CNN
 F 1 "GND" H 6400 4200 50  0000 C CNN
 F 2 "" H 6400 4350 50  0001 C CNN
