File: csi.sch (KiCad schematic (older format))
At the start: 19 parts, among them J1301 OV5640, SW1301 MIC_CAM_HKS, U1301 74LVC1G32, U1302 TXB0101

Commit message: Use I2C3 bus instead of I2C1 bus based on EmCraft's feedback
Connections:
- net labels added: I2C3_SCL_1V8, I2C3_SDA_1V8
- net labels removed: I2C1_SCL_1V8, I2C1_SDA_1V8
Changed lines of the file:
@@
 $EndComp
 Text HLabel 8750 3250 0    60   Input ~ 0
-I2C1_SCL_1V8
+I2C3_SCL_1V8
 Text HLabel 8750 3350 0    60   BiDi ~ 0
-I2C1_SDA_1V8
+I2C3_SDA_1V8
 Text HLabel 9450 3650 2    60   Input ~ 0
 CLK_N

Commit message: Update project files to KiCad 5.0.0
Parts:
- C1301, C1302, C1303, C1304, C1305, C1306, C1307, C1308, C1309, C1310: symbol C -> dvk-mx8m-bsb-rescue:C
- CAM1301: symbol OV5640_Camera -> dvk-mx8m-bsb:OV5640_Camera
- D1301, D1302: symbol D_Schottky_ALT -> dvk-mx8m-bsb-rescue:D_Schottky_ALT
- J1301: symbol Conn_02x15_Counter_Clockwise -> dvk-mx8m-bsb-rescue:Conn_02x15_Counter_Clockwise
- R1301, R1302: symbol R -> dvk-mx8m-bsb-rescue:R
- SW1301: symbol SW_DPDT_x2 -> dvk-mx8m-bsb-rescue:SW_DPDT_x2
- U1301: symbol 74LVC1G32 -> dvk-mx8m-bsb:74LVC1G32
- U1302: symbol TXB0101 -> dvk-mx8m-bsb:TXB0101
Changed lines of the file:
@@
-EESchema Schematic File Version 2
-LIBS:power
-LIBS:device
-LIBS:switches
-LIBS:relays
-LIBS:motors
-LIBS:transistors
-LIBS:conn
-LIBS:linear
-LIBS:regul
-LIBS:74xx
-LIBS:cmos4000
-LIBS:adc-dac
-LIBS:memory
-LIBS:xilinx
-LIBS:microcontrollers
-LIBS:dsp
-LIBS:microchip
-LIBS:analog_switches
-LIBS:motorola
-LIBS:texas
-LIBS:intel
-LIBS:audio
-LIBS:interface
-LIBS:digital-audio
-LIBS:philips
-LIBS:display
-LIBS:cypress
-LIBS:siliconi
-LIBS:opto
-LIBS:atmel
-LIBS:contrib
-LIBS:valves
-LIBS:dvk-mx8m-bsb
+EESchema Schematic File Version 4
 LIBS:dvk-mx8m-bsb-cache
-EELAYER 25 0
+EELAYER 26 0
 EELAYER END
 $Descr A4 11693 8268
@@
 DPDT with\nmicrophone
 $Comp
-L R R1301
+L dvk-mx8m-bsb-rescue:R R1301
 U 1 1 5B1ED51C
 P 6100 4150
@@
 $EndComp
 $Comp
-L GND #PWR0201
+L power:GND #PWR0201
 U 1 1 5B1EAF19
 P 6500 4350
@@
 $EndComp
 $Comp
-L C C1301
+L dvk-mx8m-bsb-rescue:C C1301
 U 1 1 5B1EAF12
 P 6500 4150
@@
 $EndComp
 $Comp
-L D_Schottky_ALT D1301
+L dvk-mx8m-bsb-rescue:D_Schottky_ALT D1301
 U 1 1 5B1EAB95
 P 6300 3700
@@
 $EndComp
 $Comp
-L R R1302
+L dvk-mx8m-bsb-rescue:R R1302
 U 1 1 5B1E9C00
 P 6300 3950
@@
 $EndComp
 $Comp
-L 1V8_P #PWR0202
+L dvk-mx8m-bsb:1V8_P #PWR0202
 U 1 1 5B1DBE6F
 P 6000 3450
@@
 $EndComp
 $Comp
-L GND #PWR0203
+L power:GND #PWR0203
 U 1 1 5B1A278C
 P 7350 3450
@@
 $EndComp
 $Comp
-L C C1302
+L dvk-mx8m-bsb-rescue:C C1302
 U 1 1 5B197A0E
 P 7350 3250
@@
 $EndComp
 $Comp
-L GND #PWR0204
+L power:GND #PWR0204
 U 1 1 5B1964B5
 P 7500 4100
@@
 $EndComp
 $Comp
-L 74LVC1G32 U1301
+L dvk-mx8m-bsb:74LVC1G32 U1301
 U 1 1 5B196213
 P 7700 3850
@@
 internal pull-up
 $Comp
-L D_Schottky_ALT D1302
+L dvk-mx8m-bsb-rescue:D_Schottky_ALT D1302
 U 1 1 5B15603B
 P 8150 3450
@@
 CLKO1
 $Comp
-L 1V8_P #PWR0205
+L dvk-mx8m-bsb:1V8_P #PWR0205
 U 1 1 5B105CDE
 P 10250 3300
@@
 V_IH(min)=1.26V
 $Comp
-L C C1309
+L dvk-mx8m-bsb-rescue:C C1309
 U 1 1 5B0F9030
 P 10400 2850
@@
 $EndComp
 $Comp
-L C C1307
+L dvk-mx8m-bsb-rescue:C C1307
 U 1 1 5B0F8FA9
 P 10150 2850
@@
 $EndComp
 $Comp
-L C C1306
+L dvk-mx8m-bsb-rescue:C C1306
 U 1 1 5B0F8F0F
 P 9900 2850
@@
 $EndComp
 $Comp
-L C C1305
+L dvk-mx8m-bsb-rescue:C C1305
 U 1 1 5B0F8E57
 P 9650 2850
@@
 $EndComp
 $Comp
-L 1V8_P #PWR0206
+L dvk-mx8m-bsb:1V8_P #PWR0206
 U 1 1 5B0F8E1D
 P 9450 2600
@@
 C0_P
 $Comp
-L 1V8_P #PWR0207
+L dvk-mx8m-bsb:1V8_P #PWR0207
 U 1 1 5B19049B
 P 7500 3000
@@
 $EndComp
 $Comp
-L 2V8_P #PWR0208
+L dvk-mx8m-bsb:2V8_P #PWR0208
 U 1 1 5B2B0429
 P 8550 2600
@@
 $EndComp
 $Comp
-L C C1304
+L dvk-mx8m-bsb-rescue:C C1304
 U 1 1 5B2B061C
 P 8550 2850
@@
 OV5640 CMOS Image Sensor Datasheet:\nhttps://cdn.sparkfun.com/datasheets/\nSensors/LightImaging/OV5640_datasheet.pdf
 $Comp
-L SW_DPDT_x2 SW1301
+L dvk-mx8m-bsb-rescue:SW_DPDT_x2 SW1301
 U 1 1 5B126541
 P 5900 3700
@@
 NoConn ~ 5800 3500
 $Comp
-L Conn_02x15_Counter_Clockwise J1301
+L dvk-mx8m-bsb-rescue:Conn_02x15_Counter_Clockwise J1301
 U 1 1 5B11E3C0
 P 9050 3350
@@
 NoConn ~ 8850 2650
 $Comp
-L GND #PWR0209
+L power:GND #PWR0209
 U 1 1 5B11F1A4
 P 8800 4100
@@
 NoConn ~ 8850 3550
 $Comp
-L GND #PWR0210
+L power:GND #PWR0210
 U 1 1 5B11FD52
 P 9400 4100
@@
 NoConn ~ 9350 2950
 $Comp
-L GND #PWR0211
+L power:GND #PWR0211
 U 1 1 5B164232
 P 6100 4350
@@
 Camera
 $Comp
-L OV5640_Camera CAM1301
+L dvk-mx8m-bsb:OV5640_Camera CAM1301
 U 1 1 5B2ACE32
 P 8450 5850
@@
 $EndComp
 $Comp
-L C C1303
+L dvk-mx8m-bsb-rescue:C C1303
 U 1 1 5B30A24C
 P 8250 2850
@@
 $EndComp
 $Comp
-L 3V3_P #PWR0212
+L dvk-mx8m-bsb:3V3_P #PWR0212
 U 1 1 5B333E35
 P 10550 3300
@@
 $EndComp
 $Comp
-L TXB0101 U1302
+L dvk-mx8m-bsb:TXB0101 U1302
 U 1 1 5B33432B
 P 10400 4300
@@
 $EndComp
 $Comp
-L C C1310
+L dvk-mx8m-bsb-rescue:C C1310
 U 1 1 5B334AE4
 P 10650 3550
@@
 $EndComp
 $Comp
-L GND #PWR0213
+L power:GND #PWR0213
 U 1 1 5B334B49
 P 10650 3750
@@
 $EndComp
 $Comp
-L C C1308
+L dvk-mx8m-bsb-rescue:C C1308
 U 1 1 5B334D05
 P 10150 3550
@@
 $EndComp
 $Comp
-L GND #PWR0214
+L power:GND #PWR0214
 U 1 1 5B334D7C
 P 10150 3750
@@
 $EndComp
 $Comp
-L GND #PWR0215
+L power:GND #PWR0215
 U 1 1 5B334EEB
 P 10400 4750

Commit message: Update the schematic symbols and footprints after upgrading to KiCad 5.0.0, fix all ERC and DRC violations after the new update/upgrade
Parts:
- C1301, C1302, C1303, C1304, C1305, C1306, C1307, C1308, C1309, C1310: footprint Capacitors_SMD:C_0603 -> Capacitor_SMD:C_0603_1608Metric; symbol dvk-mx8m-bsb-rescue:C -> Device:C
- D1301, D1302: symbol dvk-mx8m-bsb-rescue:D_Schottky_ALT -> Device:D_Schottky_ALT
- J1301: symbol dvk-mx8m-bsb-rescue:Conn_02x15_Counter_Clockwise -> Connector_Generic:Conn_02x15_Counter_Clockwise
- R1301, R1302: footprint Resistors_SMD:R_0603 -> Resistor_SMD:R_0603_1608Metric; symbol dvk-mx8m-bsb-rescue:R -> Device:R
- SW1301: symbol dvk-mx8m-bsb-rescue:SW_DPDT_x2 -> Switch:SW_DPDT_x2
Changed lines of the file:
@@
 Sheet 13 24
 Title "MIPI CSI"
-Date "2018-06-18"
+Date "2018-07-17"
 Rev "v0.1.0"
 Comp "Copyright 2018 GNU GPLv3"
@@
 DPDT with\nmicrophone
 $Comp
-L dvk-mx8m-bsb-rescue:R R1301
+L Device:R R1301
 U 1 1 5B1ED51C
 P 6100 4150
 F 0 "R1301" H 6275 4200 50  0000 C CNN
 F 1 "100k" H 6250 4100 50  0000 C CNN
-F 2 "Resistors_SMD:R_0603" V 6030 4150 50  0001 C CNN
+F 2 "Resistor_SMD:R_0603_1608Metric" V 6030 4150 50  0001 C CNN
 F 3 "" H 6100 4150 50  0001 C CNN
 	1    6100 4150
@@
 $EndComp
 $Comp
-L dvk-mx8m-bsb-rescue:C C1301
+L Device:C C1301
 U 1 1 5B1EAF12
 P 6500 4150
 F 0 "C1301" H 6525 4250 50  0000 L CNN
 F 1 "100nF" H 6525 4050 50  0000 L CNN
-F 2 "Capacitors_SMD:C_0603" H 6538 4000 50  0001 C CNN
+F 2 "Capacitor_SMD:C_0603_1608Metric" H 6538 4000 50  0001 C CNN
 F 3 "" H 6500 4150 50  0001 C CNN
 	1    6500 4150
@@
 $EndComp
 $Comp
-L dvk-mx8m-bsb-rescue:D_Schottky_ALT D1301
+L Device:D_Schottky_ALT D1301
 U 1 1 5B1EAB95
 P 6300 3700
@@
 $EndComp
 $Comp
-L dvk-mx8m-bsb-rescue:R R1302
+L Device:R R1302
 U 1 1 5B1E9C00
 P 6300 3950
 F 0 "R1302" V 6380 3950 50  0000 C CNN
 F 1 "100k" V 6200 3950 50  0000 C CNN
-F 2 "Resistors_SMD:R_0603" V 6230 3950 50  0001 C CNN
+F 2 "Resistor_SMD:R_0603_1608Metric" V 6230 3950 50  0001 C CNN
 F 3 "" H 6300 3950 50  0001 C CNN
 	1    6300 3950
@@
 $EndComp
 $Comp
-L dvk-mx8m-bsb-rescue:C C1302
+L Device:C C1302
 U 1 1 5B197A0E
 P 7350 3250
 F 0 "C1302" H 7375 3350 50  0000 L CNN
 F 1 "100nF" H 7375 3150 50  0000 L CNN
-F 2 "Capacitors_SMD:C_0603" H 7388 3100 50  0001 C CNN
+F 2 "Capacitor_SMD:C_0603_1608Metric" H 7388 3100 50  0001 C CNN
 F 3 "" H 7350 3250 50  0001 C CNN
 	1    7350 3250
@@
 internal pull-up
 $Comp
-L dvk-mx8m-bsb-rescue:D_Schottky_ALT D1302
+L Device:D_Schottky_ALT D1302
 U 1 1 5B15603B
 P 8150 3450
@@
 V_IH(min)=1.26V
 $Comp
-L dvk-mx8m-bsb-rescue:C C1309
+L Device:C C1309
 U 1 1 5B0F9030
 P 10400 2850
 F 0 "C1309" H 10425 2950 50  0000 L CNN
 F 1 "4.7uF" H 10425 2750 50  0000 L CNN
-F 2 "Capacitors_SMD:C_0603" H 10438 2700 50  0001 C CNN
+F 2 "Capacitor_SMD:C_0603_1608Metric" H 10438 2700 50  0001 C CNN
 F 3 "" H 10400 2850 50  0001 C CNN
 	1    10400 2850
@@
 $EndComp
 $Comp
-L dvk-mx8m-bsb-rescue:C C1307
+L Device:C C1307
 U 1 1 5B0F8FA9
 P 10150 2850
 F 0 "C1307" H 10150 2950 50  0000 L CNN
 F 1 "10nF" H 10175 2750 50  0000 L CNN
-F 2 "Capacitors_SMD:C_0603" H 10188 2700 50  0001 C CNN
+F 2 "Capacitor_SMD:C_0603_1608Metric" H 10188 2700 50  0001 C CNN
 F 3 "" H 10150 2850 50  0001 C CNN
 	1    10150 2850
@@
 $EndComp
 $Comp
-L dvk-mx8m-bsb-rescue:C C1306
+L Device:C C1306
 U 1 1 5B0F8F0F
 P 9900 2850
 F 0 "C1306" H 9900 2950 50  0000 L CNN
 F 1 "1nF" H 9925 2750 50  0000 L CNN
-F 2 "Capacitors_SMD:C_0603" H 9938 2700 50  0001 C CNN
+F 2 "Capacitor_SMD:C_0603_1608Metric" H 9938 2700 50  0001 C CNN
 F 3 "" H 9900 2850 50  0001 C CNN
 	1    9900 2850
@@
 $EndComp
 $Comp
-L dvk-mx8m-bsb-rescue:C C1305
+L Device:C C1305
 U 1 1 5B0F8E57
 P 9650 2850
 F 0 "C1305" H 9650 2950 50  0000 L CNN
 F 1 "100pF" H 9650 2750 50  0000 L CNN
-F 2 "Capacitors_SMD:C_0603" H 9688 2700 50  0001 C CNN
+F 2 "Capacitor_SMD:C_0603_1608Metric" H 9688 2700 50  0001 C CNN
 F 3 "" H 9650 2850 50  0001 C CNN
 	1    9650 2850
@@
 $EndComp
 $Comp
-L dvk-mx8m-bsb-rescue:C C1304
+L Device:C C1304
 U 1 1 5B2B061C
 P 8550 2850
 F 0 "C1304" H 8575 2950 50  0000 L CNN
 F 1 "100nF" H 8575 2750 50  0000 L CNN
-F 2 "Capacitors_SMD:C_0603" H 8588 2700 50  0001 C CNN
+F 2 "Capacitor_SMD:C_0603_1608Metric" H 8588 2700 50  0001 C CNN
 F 3 "" H 8550 2850 50  0001 C CNN
 	1    8550 2850
@@
 OV5640 CMOS Image Sensor Datasheet:\nhttps://cdn.sparkfun.com/datasheets/\nSensors/LightImaging/OV5640_datasheet.pdf
 $Comp
-L dvk-mx8m-bsb-rescue:SW_DPDT_x2 SW1301
+L Switch:SW_DPDT_x2 SW1301
 U 1 1 5B126541
 P 5900 3700
@@
 NoConn ~ 5800 3500
 $Comp
-L dvk-mx8m-bsb-rescue:Conn_02x15_Counter_Clockwise J1301
+L Connector_Generic:Conn_02x15_Counter_Clockwise J1301
 U 1 1 5B11E3C0
 P 9050 3350
@@
 $EndComp
 $Comp
-L dvk-mx8m-bsb-rescue:C C1303
+L Device:C C1303
 U 1 1 5B30A24C
 P 8250 2850
 F 0 "C1303" H 8275 2950 50  0000 L CNN
 F 1 "4.7uF" H 8275 2750 50  0000 L CNN
-F 2 "Capacitors_SMD:C_0603" H 8288 2700 50  0001 C CNN
+F 2 "Capacitor_SMD:C_0603_1608Metric" H 8288 2700 50  0001 C CNN
 F 3 "" H 8250 2850 50  0001 C CNN
 	1    8250 2850
@@
 $EndComp
 $Comp
-L dvk-mx8m-bsb-rescue:C C1310
+L Device:C C1310
 U 1 1 5B334AE4
 P 10650 3550
 F 0 "C1310" H 10650 3650 50  0000 L CNN
 F 1 "100nF" H 10650 3450 50  0000 L CNN
-F 2 "Capacitors_SMD:C_0603" H 10688 3400 50  0001 C CNN
+F 2 "Capacitor_SMD:C_0603_1608Metric" H 10688 3400 50  0001 C CNN
 F 3 "" H 10650 3550 50  0001 C CNN
 	1    10650 3550
@@
 $EndComp
 $Comp
-L dvk-mx8m-bsb-rescue:C C1308
+L Device:C C1308
 U 1 1 5B334D05
 P 10150 3550
 F 0 "C1308" H 10150 3650 50  0000 L CNN
 F 1 "100nF" H 10150 3450 50  0000 L CNN
-F 2 "Capacitors_SMD:C_0603" H 10188 3400 50  0001 C CNN
+F 2 "Capacitor_SMD:C_0603_1608Metric" H 10188 3400 50  0001 C CNN
 F 3 "" H 10150 3550 50  0001 C CNN
 	1    10150 3550

Commit message: Update all of the 3D model paths to the new directory name structure, use the correct camera mating connector part number AXT530124 instead of AXT630124 which is the one found on the camera, add the camera connector's 3D model
Parts:
- J1301: footprint dvk-mx8m-bsb:Conn_Pan_AXT630124 -> dvk-mx8m-bsb:Conn_Pan_AXT530124; Distrib Link https://www.mouser.com/ProductDetail/Panasonic-Industrial-Devices/AXT630124?qs=%2fha2pyFaduhWgBlnq%2f5GKY1ayWUWO5uKyvuPHSGZuvc%3d -> https://www.mouser.com/ProductDetail/Panasonic-Industrial-Devices/AXT530124?qs=2rFUEsTwVNyiwPOEKkiHLw%3D%3D; Distrib PN 769-AXT630124 -> 769-AXT530124; MFG Part Num AXT630124 -> AXT530124; Others https://octopart.com/search?q=AXT630124&start=0 -> https://octopart.com/search?q=AXT530124&start=0
Connections:
- wire segments 79 -> 110
Changed lines of the file:
@@
 F 0 "J1301" H 9100 4225 50  0000 C CNN
 F 1 "OV5640" H 9100 4150 50  0000 C CNN
-F 2 "dvk-mx8m-bsb:Conn_Pan_AXT630124" H 9050 3350 50  0001 C CNN
+F 2 "dvk-mx8m-bsb:Conn_Pan_AXT530124" H 9050 3350 50  0001 C CNN
 F 3 "https://www3.panasonic.biz/ac/cdn/e/control/connector/base-fpc/catalog/con_eng_f4s.pdf" H 9050 3350 50  0001 C CNN
 F 4 "Panasonic" H 9050 3350 60  0001 C CNN "MFG Name"
-F 5 "AXT630124" H 9050 3350 60  0001 C CNN "MFG Part Num"
-F 6 "769-AXT630124" H 9050 3350 60  0001 C CNN "Distrib PN"
-F 7 "https://www.mouser.com/ProductDetail/Panasonic-Industrial-Devices/AXT630124?qs=%2fha2pyFaduhWgBlnq%2f5GKY1ayWUWO5uKyvuPHSGZuvc%3d" H 9050 3350 60  0001 C CNN "Distrib Link"
+F 5 "AXT530124" H 9050 3350 60  0001 C CNN "MFG Part Num"
+F 6 "769-AXT530124" H 9050 3350 60  0001 C CNN "Distrib PN"
+F 7 "https://www.mouser.com/ProductDetail/Panasonic-Industrial-Devices/AXT530124?qs=2rFUEsTwVNyiwPOEKkiHLw%3D%3D" H 9050 3350 60  0001 C CNN "Distrib Link"
 F 8 "-" H 9050 3350 60  0001 C CNN "Tolerance"
-F 9 "https://octopart.com/search?q=AXT630124&start=0" H 9050 3350 60  0001 C CNN "Others"
+F 9 "https://octopart.com/search?q=AXT530124&start=0" H 9050 3350 60  0001 C CNN "Others"
 	1    9050 3350
 	1    0    0    -1
@@
 Connection ~ 10250 3350
 Wire Wire Line
-	9900 3350 10250 3350
+	9900 3350 10150 3350
 Wire Wire Line
 	10150 3400 10150 3350
@@
 	10650 3400 10650 3350
 Wire Wire Line
-	10250 3300 10250 3900
-Wire Wire Line
-	10550 3300 10550 3900
-Wire Wire Line
-	8250 2650 8750 2650
-Wire Wire Line
-	8250 3150 8850 3150
+	10250 3300 10250 3350
+Wire Wire Line
+	10550 3300 10550 3350
+Wire Wire Line
+	8250 2650 8550 2650
+Wire Wire Line
+	8250 3150 8550 3150
 Connection ~ 8550 3150
 Wire Wire Line
@@
 	10400 3050 10400 3000
 Wire Wire Line
-	9350 3050 10400 3050
-Wire Wire Line
-	9450 2600 9450 2850
+	9350 3050 9400 3050
+Wire Wire Line
+	9450 2600 9450 2650
 Wire Wire Line
 	9450 2850 9350 2850
 Connection ~ 8550 2650
 Wire Wire Line
-	8750 2650 8750 3050
-Wire Wire Line
-	8800 2750 8800 4100
+	8750 2650 8750 2850
+Wire Wire Line
+	8800 2750 8800 2950
 Wire Wire Line
 	8750 2850 8850 2850
@@
 	9400 2750 9350 2750
 Wire Wire Line
-	9400 2750 9400 4100
+	9400 2750 9400 3050
 Connection ~ 8800 4050
 Wire Wire Line
@@
 	3600 5050 3600 7750
 Wire Wire Line
-	5900 3950 6150 3950
-Wire Wire Line
-	6500 3700 6500 4000
-Wire Wire Line
-	6100 3700 6100 4000
+	5900 3950 6100 3950
+Wire Wire Line
+	6500 3700 6500 3950
+Wire Wire Line
+	6100 3700 6100 3950
 Wire Wire Line
 	6450 3700 6500 3700
@@
 Connection ~ 6500 3950
 Wire Wire Line
-	6450 3950 7100 3950
+	6450 3950 6500 3950
 Wire Wire Line
 	6500 4350 6500 4300
@@
 	7500 4050 7500 4100
 Wire Wire Line
-	7500 3000 7500 3650
+	7500 3000 7500 3050
 Wire Wire Line
 	9850 4300 9850 3150
@@
 Connection ~ 9450 2650
 Wire Wire Line
-	9450 2650 10400 2650
+	9450 2650 9650 2650
 Wire Wire Line
 	10400 2650 10400 2700
@@
 	8550 3150 8550 3000
 Wire Wire Line
-	8550 2600 8550 2700
+	8550 2600 8550 2650
 Wire Wire Line
 	8750 3250 8850 3250
+Wire Wire Line
+	10150 3350 10250 3350
+Wire Wire Line
+	10250 3350 10250 3900
+Wire Wire Line
+	10550 3350 10550 3900
+Wire Wire Line
+	8550 3150 8800 3150
+Wire Wire Line
+	9650 3050 9900 3050
+Wire Wire Line
+	8550 2650 8750 2650
+Wire Wire Line
+	8550 2650 8550 2700
+Wire Wire Line
+	8750 2850 8750 3050
+Wire Wire Line
+	9400 3050 9650 3050
+Wire Wire Line
+	9400 3050 9400 3250
+Wire Wire Line
+	9400 3250 9400 3550
+Wire Wire Line
+	9400 3550 9400 3850
+Wire Wire Line
+	9400 3850 9400 4100
+Wire Wire Line
+	8800 4050 8800 4100
+Wire Wire Line
+	8800 3950 8800 4050
+Wire Wire Line
+	8800 3750 8800 3950
+Wire Wire Line
+	8800 3650 8800 3750
+Wire Wire Line
+	8800 3150 8800 3650
+Wire Wire Line
+	8800 3150 8850 3150
+Wire Wire Line
+	8800 2950 8800 3150
+Wire Wire Line
+	6100 3950 6150 3950
+Wire Wire Line
+	6100 3950 6100 4000
+Wire Wire Line
+	6500 3950 6500 4000
+Wire Wire Line
+	6500 3950 7100 3950
+Wire Wire Line
+	7500 3050 7500 3650
+Wire Wire Line
+	9650 2650 9900 2650
+Wire Wire Line
+	9900 2650 10150 2650
+Wire Wire Line
+	10150 2650 10400 2650
+Wire Wire Line
+	9900 3050 10150 3050
+Wire Wire Line
+	10150 3050 10400 3050
+Wire Wire Line
+	9450 2650 9450 2850
 $EndSCHEMATC

Commit message: Reduce all 0603 resistor sizes to 0402
Parts:
- R1301, R1302: footprint Resistor_SMD:R_0603_1608Metric -> Resistor_SMD:R_0402_1005Metric
Changed lines of the file:
@@
 F 0 "R1301" H 6275 4200 50  0000 C CNN
 F 1 "100k" H 6250 4100 50  0000 C CNN
-F 2 "Resistor_SMD:R_0603_1608Metric" V 6030 4150 50  0001 C CNN
+F 2 "Resistor_SMD:R_0402_1005Metric" V 6030 4150 50  0001 C CNN
 F 3 "" H 6100 4150 50  0001 C CNN
 	1    6100 4150
@@
 F 0 "R1302" V 6380 3950 50  0000 C CNN
 F 1 "100k" V 6200 3950 50  0000 C CNN
-F 2 "Resistor_SMD:R_0603_1608Metric" V 6230 3950 50  0001 C CNN
+F 2 "Resistor_SMD:R_0402_1005Metric" V 6230 3950 50  0001 C CNN
 F 3 "" H 6300 3950 50  0001 C CNN
 	1    6300 3950

Commit message: Change all 0603 capacitors _EXCEPT_ the 2.2uF, 4.7uF, 8.2uF, 10uF, and 22uF caps to 0402
Parts:
- C1301, C1302, C1304, C1305, C1306, C1307, C1308, C1310: footprint Capacitor_SMD:C_0603_1608Metric -> Capacitor_SMD:C_0402_1005Metric
Changed lines of the file:
@@
 F 0 "C1301" H 6525 4250 50  0000 L CNN
 F 1 "100nF" H 6525 4050 50  0000 L CNN
-F 2 "Capacitor_SMD:C_0603_1608Metric" H 6538 4000 50  0001 C CNN
+F 2 "Capacitor_SMD:C_0402_1005Metric" H 6538 4000 50  0001 C CNN
 F 3 "" H 6500 4150 50  0001 C CNN
 	1    6500 4150
@@
 F 0 "C1302" H 7375 3350 50  0000 L CNN
 F 1 "100nF" H 7375 3150 50  0000 L CNN
-F 2 "Capacitor_SMD:C_0603_1608Metric" H 7388 3100 50  0001 C CNN
+F 2 "Capacitor_SMD:C_0402_1005Metric" H 7388 3100 50  0001 C CNN
 F 3 "" H 7350 3250 50  0001 C CNN
 	1    7350 3250
@@
 F 0 "C1307" H 10150 2950 50  0000 L CNN
 F 1 "10nF" H 10175 2750 50  0000 L CNN
-F 2 "Capacitor_SMD:C_0603_1608Metric" H 10188 2700 50  0001 C CNN
+F 2 "Capacitor_SMD:C_0402_1005Metric" H 10188 2700 50  0001 C CNN
 F 3 "" H 10150 2850 50  0001 C CNN
 	1    10150 2850
@@
 F 0 "C1306" H 9900 2950 50  0000 L CNN
 F 1 "1nF" H 9925 2750 50  0000 L CNN
-F 2 "Capacitor_SMD:C_0603_1608Metric" H 9938 2700 50  0001 C CNN
+F 2 "Capacitor_SMD:C_0402_1005Metric" H 9938 2700 50  0001 C CNN
 F 3 "" H 9900 2850 50  0001 C CNN
 	1    9900 2850
@@
 F 0 "C1305" H 9650 2950 50  0000 L CNN
 F 1 "100pF" H 9650 2750 50  0000 L CNN
-F 2 "Capacitor_SMD:C_0603_1608Metric" H 9688 2700 50  0001 C CNN
+F 2 "Capacitor_SMD:C_0402_1005Metric" H 9688 2700 50  0001 C CNN
 F 3 "" H 9650 2850 50  0001 C CNN
 	1    9650 2850
@@
 F 0 "C1304" H 8575 2950 50  0000 L CNN
 F 1 "100nF" H 8575 2750 50  0000 L CNN
-F 2 "Capacitor_SMD:C_0603_1608Metric" H 8588 2700 50  0001 C CNN
+F 2 "Capacitor_SMD:C_0402_1005Metric" H 8588 2700 50  0001 C CNN
 F 3 "" H 8550 2850 50  0001 C CNN
 	1    8550 2850
@@
 F 0 "C1310" H 10650 3650 50  0000 L CNN
 F 1 "100nF" H 10650 3450 50  0000 L CNN
-F 2 "Capacitor_SMD:C_0603_1608Metric" H 10688 3400 50  0001 C CNN
+F 2 "Capacitor_SMD:C_0402_1005Metric" H 10688 3400 50  0001 C CNN
 F 3 "" H 10650 3550 50  0001 C CNN
 	1    10650 3550
@@
 F 0 "C1308" H 10150 3650 50  0000 L CNN
 F 1 "100nF" H 10150 3450 50  0000 L CNN
-F 2 "Capacitor_SMD:C_0603_1608Metric" H 10188 3400 50  0001 C CNN
+F 2 "Capacitor_SMD:C_0402_1005Metric" H 10188 3400 50  0001 C CNN
 F 3 "" H 10150 3550 50  0001 C CNN
 	1    10150 3550
