File: usb-c.sch (KiCad schematic (older format))
At the start: 55 parts, among them J201 USB_C_Receptacle, U201 PTN5110HQZ, U202 PTN36043BXZ, U203 PCMF3HDMI2SZ, U204 PCMF2HDMI2SZ, U205 TLV3201AIDBVR

Commit message: Add preliminary Bill-of-Materials, fill in more missing component information such as inductor selection for the 3V3(_P) rail
Most critical components should now be getting ordered.
Parts:
- R201: value 4.7 -> 4.7k
- R226: value 100 -> 0
Changed lines of the file:
@@
 P 1100 6500
 F 0 "R201" V 1150 6725 50  0000 C CNN
-F 1 "4.7" V 1100 6500 50  0000 C CNN
+F 1 "4.7k" V 1100 6500 50  0000 C CNN
 F 2 "Resistors_SMD:R_0603" V 1030 6500 50  0001 C CNN
 F 3 "" H 1100 6500 50  0001 C CNN
@@
 P 10600 6150
 F 0 "R226" V 10680 6150 50  0000 C CNN
-F 1 "100" V 10500 6150 50  0000 C CNN
+F 1 "0" V 10500 6150 50  0000 C CNN
 F 2 "Resistors_SMD:R_0603" V 10530 6150 50  0001 C CNN
 F 3 "" H 10600 6150 50  0001 C CNN
