File: sensors.sch (KiCad schematic (older format))
At the start: 13 parts, among them U2001 VCNL4040, U2002 LSM9DS1, U2003 74LVC1G332

Commit message: Use the MX25L1606EZNI manufacturer's recommended land pattern
A combination of Macronix's "Recommended PCB Pad Layouts for 8-USON & 8-WSON Packages" (page 4) and "Macronix 209mil 8-SOP and 6x5mm 8-WSON Dual Layout" app notes were used in conjunction with KiCad's official DFN-S-8-1EP_6x5mm_Pitch1.27mm footprint to give a well-rounded pattern.
Changed lines of the file:
@@
 $Bitmap
 Pos 7450 5900
-Scale 1,000000
+Scale 1.000000
 Data
 89 50 4E 47 0D 0A 1A 0A 00 00 00 0D 49 48 44 52 00 00 03 77 00 00 01 45 08 02 00 00 00 C0 7C 83
@@
 $Bitmap
 Pos 10050 5900
-Scale 1,000000
+Scale 1.000000
 Data
 89 50 4E 47 0D 0A 1A 0A 00 00 00 0D 49 48 44 52 00 00 02 A2 00 00 01 63 08 02 00 00 00 69 3F FE
@@
 	9350 2960 10050 2960
 Wire Wire Line
-	9250 2900 9250 2950
-Wire Wire Line
-	9250 2950 9250 3050
+	9250 2900 9250 3050
 Wire Wire Line
 	9000 2950 9250 2950
@@
 	9350 2250 9050 2250
 Wire Wire Line
-	9050 4400 8400 4400
-Wire Wire Line
-	8400 4400 8200 4400
-Wire Wire Line
-	8200 4400 7550 4400
-Wire Wire Line
-	7550 4400 7250 4400
+	9050 4400 7250 4400
 Connection ~ 7550 4400
 Wire Wire Line
@@
 	4550 3050 4350 3050
 Wire Wire Line
-	4550 2200 4550 2250
-Wire Wire Line
-	4550 2250 4550 3050
-Wire Wire Line
-	4550 3050 4550 3100
+	4550 2200 4550 3100
 Wire Wire Line
-	3800 2200 3800 2250
-Wire Wire Line
-	3800 2250 3800 2750
+	3800 2200 3800 2750
 Wire Wire Line
 	4550 3450 4550 3400
@@
 	2600 3500 2600 3550
 Wire Wire Line
-	2550 3550 2600 3550
-Wire Wire Line
-	2600 3550 3250 3550
+	2550 3550 3250 3550
 Wire Wire Line
 	2600 3150 2600 3200
@@
 	4350 3500 4400 3500
 Wire Wire Line
-	3600 2250 3800 2250
-Wire Wire Line
-	3800 2250 4000 2250
+	3600 2250 4000 2250
 Wire Wire Line
 	4300 2250 4550 2250
 Connection ~ 4550 2250
 Wire Wire Line
-	9050 3450 9050 3550
-Wire Wire Line
-	9050 3550 9050 3650
-Wire Wire Line
-	9050 3650 9050 3750
-Wire Wire Line
-	9050 3750 9050 3850
-Wire Wire Line
-	9050 3850 9050 4400
+	9050 3450 9050 4400
 Wire Wire Line
 	9050 3450 9000 3450
@@
 Connection ~ 8400 4400
 Wire Wire Line
-	8200 4150 8200 4400
-Wire Wire Line
-	8200 4400 8200 4450
+	8200 4150 8200 4450
 Connection ~ 8200 4400
 Wire Wire Line
 	8300 2550 8300 2500
 Wire Wire Line
-	8300 2500 8400 2500
-Wire Wire Line
-	8400 2500 8500 2500
-Wire Wire Line
-	8500 2500 8600 2500
-Wire Wire Line
-	8600 2500 8700 2500
+	8300 2500 8700 2500
 Wire Wire Line
 	8700 2500 8700 2550
 Wire Wire Line
-	8500 1800 8500 1850
-Wire Wire Line
-	8500 1850 8500 2500
+	8500 1800 8500 2500
 Connection ~ 8500 2500
 Wire Wire Line
@@
 	8650 1850 8650 1900
 Wire Wire Line
-	8000 1850 8300 1850
-Wire Wire Line
-	8300 1850 8500 1850
-Wire Wire Line
-	8500 1850 8650 1850
+	8000 1850 8650 1850
 Wire Wire Line
 	8000 1850 8000 1900
@@
 $EndComp
 Wire Wire Line
-	9750 1500 9750 1550
-Wire Wire Line
-	9750 1550 9750 2150
+	9750 1500 9750 2150
 $Comp
 L C C2008

Commit message: Add BLM18PG121SN1D chip ferrite beads to the GNSS, proximity+ambient light sensor, and IMU +3.3V power pins
Parts:
- added FB2001, FB2002: BLM18PG121SN1D, dvk-mx8m-bsb:FER-0603, symbol Ferrite_Bead
Connections:
- net 3V3_P: now also FB2001.2, FB2002.2; no longer C2002.1, C2005.1, C2006.1, C2007.1, R2002.2, U2001.4 (LEDA), U2002.1 (VDDIO), U2002.22 (VDD), U2002.23 (VDD), U2002.3 (VDDIO)
- new net: C2002.1, FB2001.1, R2002.2, U2001.4 (LEDA)
- new net: C2005.1, C2006.1, C2007.1, FB2002.1, U2002.1 (VDDIO), U2002.22 (VDD), U2002.23 (VDD), U2002.3 (VDDIO)
Other:
- moved on the sheet: C2001, C2002, C2003, C2004, C2005, C2006, C2007, C2008, R2001, R2002, U2001, U2002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

Commit message: Use LSM9DS1 manufacturer's recommended land and solder mask design pattern, include silkscreen notes on the axis directions, import LGA24 3D model and assign it
Parts:
- U2002: footprint Housings_LGA:LGA-24L_3x3.5mm_Pitch0.43mm -> dvk-mx8m-bsb:LSM9DS1
Changed lines of the file:
@@
 F 0 "U2002" H 7550 4550 50  0000 L CNN
 F 1 "LSM9DS1" H 7550 4450 50  0000 L CNN
-F 2 "Housings_LGA:LGA-24L_3x3.5mm_Pitch0.43mm" H 9650 4450 50  0001 C CNN
+F 2 "dvk-mx8m-bsb:LSM9DS1" H 9650 4450 50  0001 C CNN
 F 3 "http://www.st.com/content/ccc/resource/technical/document/datasheet/1e/3f/2a/d6/25/eb/48/46/DM00103319.pdf/files/DM00103319.pdf/jcr:content/translations/en.DM00103319.pdf" H 8150 3800 50  0001 C CNN
 F 4 "STMicroelectronics" H 8150 3700 60  0001 C CNN "MFG Name"

Commit message: Create SN74LVC1G332DCKR footprint based on the manufacturer's given example and assign it to the respective schematic symbol, assign it the official KiCad SC-70-6 3D model
Parts:
- U2003: footprint (none) -> dvk-mx8m-bsb:SN74LVC1G332DCKR
Changed lines of the file:
@@
 F 0 "U2003" H 9900 2750 50  0000 C CNN
 F 1 "74LVC1G332" H 9930 2690 50  0000 C CNN
-F 2 "" H 9900 2700 50  0001 C CNN
+F 2 "dvk-mx8m-bsb:SN74LVC1G332DCKR" H 9900 2700 50  0001 C CNN
 F 3 "http://www.ti.com/lit/ds/symlink/sn74lvc1g332.pdf" H 9900 2700 50  0001 C CNN
 F 4 "Texas Instruments" H 9900 2700 60  0001 C CNN "MFG Name"
