File: wifi_bt_m2.sch (KiCad schematic (older format))
At the start: 40 parts, among them J1801 MHF4, J1802 MHF4, J1803 Key_E, Q1801 FDV301N, Q1802 FDV301N, SW1801 WLAN_HKS, U1801 NTB0104GU12, U1802 NTB0104GU12, U1803 74AUP2G08

Commit message: Assign u.FL to the coax connectors in the WLAN+BT circuit
Parts:
- J1801, J1802: value MHF4 -> u.FL; footprint dvk-mx8m-bsb:MHF4_20449-001E -> dvk-mx8m-bsb:U.FL_Hirose_U.FL-R-SMT-1_Vertical; Distrib Link https://www.mouser.com/ProductDetail/Taoglas/RECE-20449-001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 -> https://www.mouser.com/ProductDetail/Linx-Technologies/CONU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; Distrib PN 960-RECE20449-001E01 -> 712-CONUFL001-SMD-T; MFG Name Taoglas -> Linx; MFG Part Num RECE-20449-001E-01 -> CONUFL001-SMD-T; Others https://octopart.com/search?q=20449-001E&start=0 -> https://octopart.com/search?q=CONUFL001-SMD-T&oq=CONUFL001-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
Changed lines of the file:
@@
 P 1900 2050
 F 0 "J1801" H 1910 2170 50  0000 C CNN
-F 1 "MHF4" H 2100 2050 50  0000 C CNN
-F 2 "dvk-mx8m-bsb:MHF4_20449-001E" H 1900 2050 50  0001 C CNN
-F 3 "https://www.taoglas.com/wp-content/uploads/2016/04/RECE.20449.001E.01.pdf" H 1900 2050 50  0001 C CNN
-F 4 "Taoglas" H 1900 2050 60  0001 C CNN "MFG Name"
-F 5 "RECE-20449-001E-01" H 1900 2050 60  0001 C CNN "MFG Part Num"
-F 6 "960-RECE20449-001E01" H 1900 2050 60  0001 C CNN "Distrib PN"
-F 7 "https://www.mouser.com/ProductDetail/Taoglas/RECE-20449-001E-01?qs=60YbxKv0rtCt8UzaWSJTyg%3D%3D" H 1900 2050 60  0001 C CNN "Distrib Link"
+F 1 "u.FL" H 2100 2050 50  0000 C CNN
+F 2 "dvk-mx8m-bsb:U.FL_Hirose_U.FL-R-SMT-1_Vertical" H 1900 2050 50  0001 C CNN
+F 3 "https://linxtechnologies.com/wp/wp-content/uploads/conufl001-smd.pdf" H 1900 2050 50  0001 C CNN
+F 4 "Linx" H 1900 2050 60  0001 C CNN "MFG Name"
+F 5 "CONUFL001-SMD-T" H 1900 2050 60  0001 C CNN "MFG Part Num"
+F 6 "712-CONUFL001-SMD-T" H 1900 2050 60  0001 C CNN "Distrib PN"
+F 7 "https://www.mouser.com/ProductDetail/Linx-Technologies/CONUFL001-SMD-T?qs=%2fha2pyFaduivK93xHKUivxg4VjfDQlObuMZMwyaL26SpKX%252bySjigOg%3d%3d" H 1900 2050 60  0001 C CNN "Distrib Link"
 F 8 "-" H 1900 2050 60  0001 C CNN "Tolerance"
-F 9 "https://octopart.com/search?q=20449-001E&start=0" H 1900 2050 60  0001 C CNN "Others"
+F 9 "https://octopart.com/search?q=CONUFL001-SMD-T&oq=CONUFL001-SMD-T&start=0" H 1900 2050 60  0001 C CNN "Others"
 	1    1900 2050
-	1    0    0    -1
-$EndComp
-$Comp
-L Conn_Coaxial J1802
-U 1 1 5B6AA2C1
-P 1900 2900
-F 0 "J1802" H 1910 3020 50  0000 C CNN
-F 1 "MHF4" H 2100 2900 50  0000 C CNN
-F 2 "dvk-mx8m-bsb:MHF4_20449-001E" H 1900 2900 50  0001 C CNN
-F 3 "https://www.taoglas.com/wp-content/uploads/2016/04/RECE.20449.001E.01.pdf" H 1900 2900 50  0001 C CNN
-F 4 "Taoglas" H 1900 2900 60  0001 C CNN "MFG Name"
-F 5 "RECE-20449-001E-01" H 1900 2900 60  0001 C CNN "MFG Part Num"
-F 6 "960-RECE20449-001E01" H 1900 2900 60  0001 C CNN "Distrib PN"
-F 7 "https://www.mouser.com/ProductDetail/Taoglas/RECE-20449-001E-01?qs=60YbxKv0rtCt8UzaWSJTyg%3D%3D" H 1900 2900 60  0001 C CNN "Distrib Link"
-F 8 "-" H 1900 2900 60  0001 C CNN "Tolerance"
-F 9 "https://octopart.com/search?q=20449-001E&start=0" H 1900 2900 60  0001 C CNN "Others"
-	1    1900 2900
 	1    0    0    -1
 $EndComp
@@
 	0    1    1    0
 $EndComp
+$Comp
+L Conn_Coaxial J1802
+U 1 1 5B29F847
+P 1900 2900
+F 0 "J1802" H 1910 3020 50  0000 C CNN
+F 1 "u.FL" H 2100 2900 50  0000 C CNN
+F 2 "dvk-mx8m-bsb:U.FL_Hirose_U.FL-R-SMT-1_Vertical" H 1900 2900 50  0001 C CNN
+F 3 "https://linxtechnologies.com/wp/wp-content/uploads/conufl001-smd.pdf" H 1900 2900 50  0001 C CNN
+F 4 "Linx" H 1900 2900 60  0001 C CNN "MFG Name"
+F 5 "CONUFL001-SMD-T" H 1900 2900 60  0001 C CNN "MFG Part Num"
+F 6 "712-CONUFL001-SMD-T" H 1900 2900 60  0001 C CNN "Distrib PN"
+F 7 "https://www.mouser.com/ProductDetail/Linx-Technologies/CONUFL001-SMD-T?qs=%2fha2pyFaduivK93xHKUivxg4VjfDQlObuMZMwyaL26SpKX%252bySjigOg%3d%3d" H 1900 2900 60  0001 C CNN "Distrib Link"
+F 8 "-" H 1900 2900 60  0001 C CNN "Tolerance"
+F 9 "https://octopart.com/search?q=CONUFL001-SMD-T&oq=CONUFL001-SMD-T&start=0" H 1900 2900 60  0001 C CNN "Others"
+	1    1900 2900
+	1    0    0    -1
+$EndComp
 $EndSCHEMATC

Commit message: Add FDV301N footprint based on the manufacturer's given recommended land pattern, use lower ESR 220uF tantalum capacitors in place of previously selected ones, re-export the BoM
Double checked FET footprints to make sure those assigned to the official SOT-23 footprint are correct.
Parts:
- C1816, C1817: Distrib Link https://www.arrow.com/en/products/293d227x9010d2te3/vishay -> https://www.tme.eu/en/details/tpsd227k010r010/smd-tantalum-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; Distrib PN 293D227X9010D2TE3 -> TPSD227K010R0100; MFG Name Vishay -> AVX; MFG Part Num 293D227X9010D2TE3 -> TPSD227K010R0100; Others https://www.digikey.com/products/en/capacitors/tantalum-cap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 -> https://www.arrow.com/en/products/293d227x9010d2te3/vishay
- Q1801, Q1802: footprint TO_SOT_Packages_SMD:SOT-23 -> dvk-mx8m-bsb:FDV301N

Commit message: For better BoM generation, added placeholders for SOM, disṕlay, camera, WWAN card and wifi/BT card. Datasheet links and supplier information can be stored in these new library symbols.
Parts:
- added MOD1801: WifiBTCard, dvk-mx8m-bsb:M2Card_E_2230, symbol WifiBTCard
Changed lines of the file:
@@
 WLAN_DN
 $Comp
-L GND #PWR1811
+L GND #PWR0302
 U 1 1 5B01D9F9
 P 5300 5050
-F 0 "#PWR1811" H 5300 4800 50  0001 C CNN
+F 0 "#PWR0302" H 5300 4800 50  0001 C CNN
 F 1 "GND" H 5300 4900 50  0000 C CNN
 F 2 "" H 5300 5050 50  0001 C CNN
@@
 $EndComp
 $Comp
-L GND #PWR1813
+L GND #PWR0303
 U 1 1 5B01E5BE
 P 5900 5050
-F 0 "#PWR1813" H 5900 4800 50  0001 C CNN
+F 0 "#PWR0303" H 5900 4800 50  0001 C CNN
 F 1 "GND" H 5900 4900 50  0000 C CNN
 F 2 "" H 5900 5050 50  0001 C CNN
@@
 $EndComp
 $Comp
-L 3V3_P #PWR1814
+L 3V3_P #PWR0304
 U 1 1 5B01E6B8
 P 5950 900
-F 0 "#PWR1814" H 5950 750 50  0001 C CNN
+F 0 "#PWR0304" H 5950 750 50  0001 C CNN
 F 1 "3V3_P" H 5950 1040 50  0000 C CNN
 F 2 "" H 5950 900 50  0001 C CNN
@@
 $Bitmap
 Pos 9300 2400
-Scale 1.000000
+Scale 1,000000
 Data
 89 50 4E 47 0D 0A 1A 0A 00 00 00 0D 49 48 44 52 00 00 01 9A 00 00 00 E2 08 02 00 00 00 F8 62 96
@@
 BT_HOST_WAKE
 $Comp
-L 3V3_P #PWR1826
+L 3V3_P #PWR0305
 U 1 1 5B0C3C8A
 P 9600 3600
-F 0 "#PWR1826" H 9600 3450 50  0001 C CNN
+F 0 "#PWR0305" H 9600 3450 50  0001 C CNN
 F 1 "3V3_P" H 9600 3740 50  0000 C CNN
 F 2 "" H 9600 3600 50  0001 C CNN
@@
 NoConn ~ 6500 3750
 $Comp
-L 3V3_P #PWR1818
+L 3V3_P #PWR0306
 U 1 1 5B0D90EE
 P 7750 2700
-F 0 "#PWR1818" H 7750 2550 50  0001 C CNN
+F 0 "#PWR0306" H 7750 2550 50  0001 C CNN
 F 1 "3V3_P" H 7750 2840 50  0000 C CNN
 F 2 "" H 7750 2700 50  0001 C CNN
@@
 $EndComp
 $Comp
-L GND #PWR1821
+L GND #PWR0307
 U 1 1 5B0D91C5
 P 7750 4700
-F 0 "#PWR1821" H 7750 4450 50  0001 C CNN
+F 0 "#PWR0307" H 7750 4450 50  0001 C CNN
 F 1 "GND" H 7750 4550 50  0000 C CNN
 F 2 "" H 7750 4700 50  0001 C CNN
@@
 WIFI_WAKE
 $Comp
-L 1V8_P #PWR1808
+L 1V8_P #PWR0308
 U 1 1 5AEFAF82
 P 4550 2000
-F 0 "#PWR1808" H 4550 1850 50  0001 C CNN
+F 0 "#PWR0308" H 4550 1850 50  0001 C CNN
 F 1 "1V8_P" H 4550 2140 50  0000 C CNN
 F 2 "" H 4550 2000 50  0001 C CNN
@@
 NoConn ~ 5850 2050
 $Comp
-L 1V8_P #PWR1817
+L 1V8_P #PWR0309
 U 1 1 5AEB9155
 P 7000 5050
-F 0 "#PWR1817" H 7000 4900 50  0001 C CNN
+F 0 "#PWR0309" H 7000 4900 50  0001 C CNN
 F 1 "1V8_P" H 7000 5190 50  0000 C CNN
 F 2 "" H 7000 5050 50  0001 C CNN
@@
 M2_I2C_SCL
 $Comp
-L 3V3_P #PWR1820
+L 3V3_P #PWR0310
 U 1 1 5AF2CD0D
 P 7750 4200
-F 0 "#PWR1820" H 7750 4050 50  0001 C CNN
+F 0 "#PWR0310" H 7750 4050 50  0001 C CNN
 F 1 "3V3_P" H 7750 4340 50  0000 C CNN
 F 2 "" H 7750 4200 50  0001 C CNN
@@
 $EndComp
 $Comp
-L GND #PWR1819
+L GND #PWR0311
 U 1 1 5AF2CDB4
 P 7750 3800
-F 0 "#PWR1819" H 7750 3550 50  0001 C CNN
+F 0 "#PWR0311" H 7750 3550 50  0001 C CNN
 F 1 "GND" H 7750 3650 50  0000 C CNN
 F 2 "" H 7750 3800 50  0001 C CNN
@@
 $EndComp
 $Comp
-L GND #PWR1824
+L GND #PWR0312
 U 1 1 5AF3C984
 P 9000 4500
-F 0 "#PWR1824" H 9000 4250 50  0001 C CNN
+F 0 "#PWR0312" H 9000 4250 50  0001 C CNN
 F 1 "GND" H 9000 4350 50  0000 C CNN
 F 2 "" H 9000 4500 50  0001 C CNN
@@
 $EndComp
 $Comp
-L GND #PWR1827
+L GND #PWR0313
 U 1 1 5AF3C98A
 P 9600 4500
-F 0 "#PWR1827" H 9600 4250 50  0001 C CNN
+F 0 "#PWR0313" H 9600 4250 50  0001 C CNN
 F 1 "GND" H 9600 4350 50  0000 C CNN
 F 2 "" H 9600 4500 50  0001 C CNN
@@
 $EndComp
 $Comp
-L 1V8_P #PWR1825
+L 1V8_P #PWR0314
 U 1 1 5AEBC081
 P 9400 5050
-F 0 "#PWR1825" H 9400 4900 50  0001 C CNN
+F 0 "#PWR0314" H 9400 4900 50  0001 C CNN
 F 1 "1V8_P" H 9400 5190 50  0000 C CNN
 F 2 "" H 9400 5050 50  0001 C CNN
@@
 $EndComp
 $Comp
-L GND #PWR1816
+L GND #PWR0315
 U 1 1 5B2489BD
 P 6350 6200
-F 0 "#PWR1816" H 6350 5950 50  0001 C CNN
+F 0 "#PWR0315" H 6350 5950 50  0001 C CNN
 F 1 "GND" H 6350 6050 50  0000 C CNN
 F 2 "" H 6350 6200 50  0001 C CNN
@@
 $EndComp
 $Comp
-L GND #PWR1809
+L GND #PWR0316
 U 1 1 5B2489DB
 P 4600 6200
-F 0 "#PWR1809" H 4600 5950 50  0001 C CNN
+F 0 "#PWR0316" H 4600 5950 50  0001 C CNN
 F 1 "GND" H 4600 6050 50  0000 C CNN
 F 2 "" H 4600 6200 50  0001 C CNN
@@
 $EndComp
 $Comp
-L GND #PWR1812
+L GND #PWR0317
 U 1 1 5B2489F2
 P 5400 7550
-F 0 "#PWR1812" H 5400 7300 50  0001 C CNN
+F 0 "#PWR0317" H 5400 7300 50  0001 C CNN
 F 1 "GND" H 5400 7400 50  0000 C CNN
 F 2 "" H 5400 7550 50  0001 C CNN
@@
 BCLK
 $Comp
-L 3V3_P #PWR1815
+L 3V3_P #PWR0318
 U 1 1 5B248A11
 P 6200 5700
-F 0 "#PWR1815" H 6200 5550 50  0001 C CNN
+F 0 "#PWR0318" H 6200 5550 50  0001 C CNN
 F 1 "3V3_P" H 6200 5840 50  0000 C CNN
 F 2 "" H 6200 5700 50  0001 C CNN
@@
 $EndComp
 $Comp
-L 1V8_P #PWR1810
+L 1V8_P #PWR0319
 U 1 1 5B248A1D
 P 4950 5700
-F 0 "#PWR1810" H 4950 5550 50  0001 C CNN
+F 0 "#PWR0319" H 4950 5550 50  0001 C CNN
 F 1 "1V8_P" H 4950 5840 50  0000 C CNN
 F 2 "" H 4950 5700 50  0001 C CNN
@@
 $EndComp
 $Comp
-L GND #PWR1807
+L GND #PWR0320
 U 1 1 5B337EDE
 P 3200 6200
-F 0 "#PWR1807" H 3200 5950 50  0001 C CNN
+F 0 "#PWR0320" H 3200 5950 50  0001 C CNN
 F 1 "GND" H 3200 6050 50  0000 C CNN
 F 2 "" H 3200 6200 50  0001 C CNN
@@
 $EndComp
 $Comp
-L GND #PWR1801
+L GND #PWR0321
 U 1 1 5B337EFC
 P 1450 6200
-F 0 "#PWR1801" H 1450 5950 50  0001 C CNN
+F 0 "#PWR0321" H 1450 5950 50  0001 C CNN
 F 1 "GND" H 1450 6050 50  0000 C CNN
 F 2 "" H 1450 6200 50  0001 C CNN
@@
 $EndComp
 $Comp
-L GND #PWR1805
+L GND #PWR0322
 U 1 1 5B337F13
 P 2250 7550
-F 0 "#PWR1805" H 2250 7300 50  0001 C CNN
+F 0 "#PWR0322" H 2250 7300 50  0001 C CNN
 F 1 "GND" H 2250 7400 50  0000 C CNN
 F 2 "" H 2250 7550 50  0001 C CNN
@@
 $EndComp
 $Comp
-L 3V3_P #PWR1806
+L 3V3_P #PWR0323
 U 1 1 5B337F23
 P 3050 5700
-F 0 "#PWR1806" H 3050 5550 50  0001 C CNN
+F 0 "#PWR0323" H 3050 5550 50  0001 C CNN
 F 1 "3V3_P" H 3050 5840 50  0000 C CNN
 F 2 "" H 3050 5700 50  0001 C CNN
@@
 $EndComp
 $Comp
-L 1V8_P #PWR1802
+L 1V8_P #PWR0324
 U 1 1 5B337F29
 P 1800 5700
-F 0 "#PWR1802" H 1800 5550 50  0001 C CNN
+F 0 "#PWR0324" H 1800 5550 50  0001 C CNN
 F 1 "1V8_P" H 1800 5840 50  0000 C CNN
 F 2 "" H 1800 5700 50  0001 C CNN
@@
 $EndComp
 $Comp
-L GND #PWR1822
+L GND #PWR0325
 U 1 1 5B0D6FE3
 P 7900 3150
-F 0 "#PWR1822" H 7900 2900 50  0001 C CNN
+F 0 "#PWR0325" H 7900 2900 50  0001 C CNN
 F 1 "GND" H 7900 3000 50  0000 C CNN
 F 2 "" H 7900 3150 50  0001 C CNN
@@
 NoConn ~ 19750 8050
 $Comp
-L GND #PWR1803
+L GND #PWR0326
 U 1 1 5B1205DC
 P 1900 2300
-F 0 "#PWR1803" H 1900 2050 50  0001 C CNN
+F 0 "#PWR0326" H 1900 2050 50  0001 C CNN
 F 1 "GND" H 1900 2150 50  0000 C CNN
 F 2 "" H 1900 2300 50  0001 C CNN
@@
 	1700 2050 1700 2000
 $Comp
-L GND #PWR1804
+L GND #PWR0327
 U 1 1 5B1206B3
 P 1900 3150
-F 0 "#PWR1804" H 1900 2900 50  0001 C CNN
+F 0 "#PWR0327" H 1900 2900 50  0001 C CNN
 F 1 "GND" H 1900 3000 50  0000 C CNN
 F 2 "" H 1900 3150 50  0001 C CNN
@@
 $EndComp
 $Comp
-L GND #PWR1823
+L GND #PWR0328
 U 1 1 5B1DE1E8
 P 8300 1450
-F 0 "#PWR1823" H 8300 1200 50  0001 C CNN
+F 0 "#PWR0328" H 8300 1200 50  0001 C CNN
 F 1 "GND" H 8300 1300 50  0000 C CNN
 F 2 "" H 8300 1450 50  0001 C CNN
@@
 	1    0    0    -1
 $EndComp
+$Comp
+L WifiBTCard MOD1801
+U 1 1 5B2AC34E
+P 3350 4100
+F 0 "MOD1801" H 3350 4450 60  0000 C CNN
+F 1 "WifiBTCard" H 3350 4350 60  0000 C CNN
+F 2 "dvk-mx8m-bsb:M2Card_E_2230" H 3350 4050 60  0001 C CNN
+F 3 "http://www.redpinesignals.com/pdfs/RS9116_Connectivity_Product_Brief.pdf" H 3350 4050 60  0001 C CNN
+	1    3350 4100
+	1    0    0    -1
+$EndComp

Commit message: Update WWAN mPCIe sheet by organizing a few things and fixing the component properties order
Parts:
- C1817: footprint Capacitors_Tantalum_SMD:CP_Tantalum_Case-D_EIA-7343-31_Reflow -> Capacitors_SMD:CP_Elec_6.3x7.7; Distrib Link https://www.tme.eu/en/details/tpsd227k010r010/smd-tantalum-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 -> https://www.tme.eu/en/details/eeefpa221xap/smd-low-imp-elec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; Distrib PN TPSD227K010R0100 -> EEEFPA221XAP; MFG Name AVX -> Panasonic; MFG Part Num TPSD227K010R0100 -> EEEFPA221XAP; Others https://www.arrow.com/en/products/293d227x9010d2te3/vishay -> http://uk.farnell.com/panasonic-electronic-components/eeefp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; Tolerance 10% -> 20%
Changed lines of the file:
@@
 WLAN_DN
 $Comp
-L GND #PWR0302
+L GND #PWR0307
 U 1 1 5B01D9F9
 P 5300 5050
-F 0 "#PWR0302" H 5300 4800 50  0001 C CNN
+F 0 "#PWR0307" H 5300 4800 50  0001 C CNN
 F 1 "GND" H 5300 4900 50  0000 C CNN
 F 2 "" H 5300 5050 50  0001 C CNN
@@
 $EndComp
 $Comp
-L GND #PWR0303
+L GND #PWR0308
 U 1 1 5B01E5BE
 P 5900 5050
-F 0 "#PWR0303" H 5900 4800 50  0001 C CNN
+F 0 "#PWR0308" H 5900 4800 50  0001 C CNN
 F 1 "GND" H 5900 4900 50  0000 C CNN
 F 2 "" H 5900 5050 50  0001 C CNN
@@
 $EndComp
 $Comp
-L 3V3_P #PWR0304
+L 3V3_P #PWR0309
 U 1 1 5B01E6B8
 P 5950 900
-F 0 "#PWR0304" H 5950 750 50  0001 C CNN
+F 0 "#PWR0309" H 5950 750 50  0001 C CNN
 F 1 "3V3_P" H 5950 1040 50  0000 C CNN
 F 2 "" H 5950 900 50  0001 C CNN
@@
 BT_HOST_WAKE
 $Comp
-L 3V3_P #PWR0305
+L 3V3_P #PWR0310
 U 1 1 5B0C3C8A
 P 9600 3600
-F 0 "#PWR0305" H 9600 3450 50  0001 C CNN
+F 0 "#PWR0310" H 9600 3450 50  0001 C CNN
 F 1 "3V3_P" H 9600 3740 50  0000 C CNN
 F 2 "" H 9600 3600 50  0001 C CNN
@@
 NoConn ~ 6500 3750
 $Comp
-L 3V3_P #PWR0306
+L 3V3_P #PWR0311
 U 1 1 5B0D90EE
 P 7750 2700
-F 0 "#PWR0306" H 7750 2550 50  0001 C CNN
+F 0 "#PWR0311" H 7750 2550 50  0001 C CNN
 F 1 "3V3_P" H 7750 2840 50  0000 C CNN
 F 2 "" H 7750 2700 50  0001 C CNN
@@
 $EndComp
 $Comp
-L GND #PWR0307
+L GND #PWR0312
 U 1 1 5B0D91C5
 P 7750 4700
-F 0 "#PWR0307" H 7750 4450 50  0001 C CNN
+F 0 "#PWR0312" H 7750 4450 50  0001 C CNN
 F 1 "GND" H 7750 4550 50  0000 C CNN
 F 2 "" H 7750 4700 50  0001 C CNN
@@
 WIFI_WAKE
 $Comp
-L 1V8_P #PWR0308
+L 1V8_P #PWR0313
 U 1 1 5AEFAF82
 P 4550 2000
-F 0 "#PWR0308" H 4550 1850 50  0001 C CNN
+F 0 "#PWR0313" H 4550 1850 50  0001 C CNN
 F 1 "1V8_P" H 4550 2140 50  0000 C CNN
 F 2 "" H 4550 2000 50  0001 C CNN
@@
 NoConn ~ 5850 2050
 $Comp
-L 1V8_P #PWR0309
+L 1V8_P #PWR0314
 U 1 1 5AEB9155
 P 7000 5050
-F 0 "#PWR0309" H 7000 4900 50  0001 C CNN
+F 0 "#PWR0314" H 7000 4900 50  0001 C CNN
 F 1 "1V8_P" H 7000 5190 50  0000 C CNN
 F 2 "" H 7000 5050 50  0001 C CNN
@@
 M2_I2C_SCL
 $Comp
-L 3V3_P #PWR0310
+L 3V3_P #PWR0315
 U 1 1 5AF2CD0D
 P 7750 4200
-F 0 "#PWR0310" H 7750 4050 50  0001 C CNN
+F 0 "#PWR0315" H 7750 4050 50  0001 C CNN
 F 1 "3V3_P" H 7750 4340 50  0000 C CNN
 F 2 "" H 7750 4200 50  0001 C CNN
@@
 $EndComp
 $Comp
-L GND #PWR0311
+L GND #PWR0316
 U 1 1 5AF2CDB4
 P 7750 3800
-F 0 "#PWR0311" H 7750 3550 50  0001 C CNN
+F 0 "#PWR0316" H 7750 3550 50  0001 C CNN
 F 1 "GND" H 7750 3650 50  0000 C CNN
 F 2 "" H 7750 3800 50  0001 C CNN
@@
 $EndComp
 $Comp
-L GND #PWR0312
+L GND #PWR0317
 U 1 1 5AF3C984
 P 9000 4500
-F 0 "#PWR0312" H 9000 4250 50  0001 C CNN
+F 0 "#PWR0317" H 9000 4250 50  0001 C CNN
 F 1 "GND" H 9000 4350 50  0000 C CNN
 F 2 "" H 9000 4500 50  0001 C CNN
@@
 $EndComp
 $Comp
-L GND #PWR0313
+L GND #PWR0318
 U 1 1 5AF3C98A
 P 9600 4500
-F 0 "#PWR0313" H 9600 4250 50  0001 C CNN
+F 0 "#PWR0318" H 9600 4250 50  0001 C CNN
 F 1 "GND" H 9600 4350 50  0000 C CNN
 F 2 "" H 9600 4500 50  0001 C CNN
@@
 $EndComp
 $Comp
-L 1V8_P #PWR0314
+L 1V8_P #PWR0319
 U 1 1 5AEBC081
 P 9400 5050
-F 0 "#PWR0314" H 9400 4900 50  0001 C CNN
+F 0 "#PWR0319" H 9400 4900 50  0001 C CNN
 F 1 "1V8_P" H 9400 5190 50  0000 C CNN
 F 2 "" H 9400 5050 50  0001 C CNN
@@
 $EndComp
 $Comp
-L GND #PWR0315
+L GND #PWR0320
 U 1 1 5B2489BD
 P 6350 6200
-F 0 "#PWR0315" H 6350 5950 50  0001 C CNN
+F 0 "#PWR0320" H 6350 5950 50  0001 C CNN
 F 1 "GND" H 6350 6050 50  0000 C CNN
 F 2 "" H 6350 6200 50  0001 C CNN
@@
 $EndComp
 $Comp
-L GND #PWR0316
+L GND #PWR0321
 U 1 1 5B2489DB
 P 4600 6200
-F 0 "#PWR0316" H 4600 5950 50  0001 C CNN
+F 0 "#PWR0321" H 4600 5950 50  0001 C CNN
 F 1 "GND" H 4600 6050 50  0000 C CNN
 F 2 "" H 4600 6200 50  0001 C CNN
@@
 $EndComp
 $Comp
-L GND #PWR0317
+L GND #PWR0322
 U 1 1 5B2489F2
 P 5400 7550
-F 0 "#PWR0317" H 5400 7300 50  0001 C CNN
+F 0 "#PWR0322" H 5400 7300 50  0001 C CNN
 F 1 "GND" H 5400 7400 50  0000 C CNN
 F 2 "" H 5400 7550 50  0001 C CNN
@@
 BCLK
 $Comp
-L 3V3_P #PWR0318
+L 3V3_P #PWR0323
 U 1 1 5B248A11
 P 6200 5700
-F 0 "#PWR0318" H 6200 5550 50  0001 C CNN
+F 0 "#PWR0323" H 6200 5550 50  0001 C CNN
 F 1 "3V3_P" H 6200 5840 50  0000 C CNN
 F 2 "" H 6200 5700 50  0001 C CNN
@@
 $EndComp
 $Comp
-L 1V8_P #PWR0319
+L 1V8_P #PWR0324
 U 1 1 5B248A1D
 P 4950 5700
-F 0 "#PWR0319" H 4950 5550 50  0001 C CNN
+F 0 "#PWR0324" H 4950 5550 50  0001 C CNN
 F 1 "1V8_P" H 4950 5840 50  0000 C CNN
 F 2 "" H 4950 5700 50  0001 C CNN
@@
 $EndComp
 $Comp
-L GND #PWR0320
+L GND #PWR0325
 U 1 1 5B337EDE
 P 3200 6200
-F 0 "#PWR0320" H 3200 5950 50  0001 C CNN
+F 0 "#PWR0325" H 3200 5950 50  0001 C CNN
 F 1 "GND" H 3200 6050 50  0000 C CNN
 F 2 "" H 3200 6200 50  0001 C CNN
@@
 $EndComp
 $Comp
-L GND #PWR0321
+L GND #PWR0326
 U 1 1 5B337EFC
 P 1450 6200
-F 0 "#PWR0321" H 1450 5950 50  0001 C CNN
+F 0 "#PWR0326" H 1450 5950 50  0001 C CNN
 F 1 "GND" H 1450 6050 50  0000 C CNN
 F 2 "" H 1450 6200 50  0001 C CNN
@@
 $EndComp
 $Comp
-L GND #PWR0322
+L GND #PWR0327
 U 1 1 5B337F13
 P 2250 7550
-F 0 "#PWR0322" H 2250 7300 50  0001 C CNN
+F 0 "#PWR0327" H 2250 7300 50  0001 C CNN
 F 1 "GND" H 2250 7400 50  0000 C CNN
 F 2 "" H 2250 7550 50  0001 C CNN
@@
 $EndComp
 $Comp
-L 3V3_P #PWR0323
+L 3V3_P #PWR0328
 U 1 1 5B337F23
 P 3050 5700
-F 0 "#PWR0323" H 3050 5550 50  0001 C CNN
+F 0 "#PWR0328" H 3050 5550 50  0001 C CNN
 F 1 "3V3_P" H 3050 5840 50  0000 C CNN
 F 2 "" H 3050 5700 50  0001 C CNN
@@
 $EndComp
 $Comp
-L 1V8_P #PWR0324
+L 1V8_P #PWR0329
 U 1 1 5B337F29
 P 1800 5700
-F 0 "#PWR0324" H 1800 5550 50  0001 C CNN
+F 0 "#PWR0329" H 1800 5550 50  0001 C CNN
 F 1 "1V8_P" H 1800 5840 50  0000 C CNN
 F 2 "" H 1800 5700 50  0001 C CNN
@@
 $EndComp
 $Comp
-L GND #PWR0325
+L GND #PWR0330
 U 1 1 5B0D6FE3
 P 7900 3150
-F 0 "#PWR0325" H 7900 2900 50  0001 C CNN
+F 0 "#PWR0330" H 7900 2900 50  0001 C CNN
 F 1 "GND" H 7900 3000 50  0000 C CNN
 F 2 "" H 7900 3150 50  0001 C CNN
@@
 NoConn ~ 19750 8050
 $Comp
-L GND #PWR0326
+L GND #PWR0331
 U 1 1 5B1205DC
 P 1900 2300
-F 0 "#PWR0326" H 1900 2050 50  0001 C CNN
+F 0 "#PWR0331" H 1900 2050 50  0001 C CNN
 F 1 "GND" H 1900 2150 50  0000 C CNN
 F 2 "" H 1900 2300 50  0001 C CNN
@@
 	1700 2050 1700 2000
 $Comp
-L GND #PWR0327
+L GND #PWR0332
 U 1 1 5B1206B3
 P 1900 3150
-F 0 "#PWR0327" H 1900 2900 50  0001 C CNN
+F 0 "#PWR0332" H 1900 2900 50  0001 C CNN
 F 1 "GND" H 1900 3000 50  0000 C CNN
 F 2 "" H 1900 3150 50  0001 C CNN
@@
 $EndComp
 $Comp
-L GND #PWR0328
+L GND #PWR0333
 U 1 1 5B1DE1E8
 P 8300 1450
-F 0 "#PWR0328" H 8300 1200 50  0001 C CNN
+F 0 "#PWR0333" H 8300 1200 50  0001 C CNN
 F 1 "GND" H 8300 1300 50  0000 C CNN
 F 2 "" H 8300 1450 50  0001 C CNN
@@
 	8300 1300 8300 1450
 Wire Wire Line
-	8050 1300 8050 1400
+	8050 1400 8050 1300
 Connection ~ 8050 1400
 Wire Wire Line
-	7800 1300 7800 1400
+	7800 1400 7800 1300
 Connection ~ 7800 1400
 Wire Wire Line
-	7550 1300 7550 1400
+	7550 1400 7550 1300
 Connection ~ 7550 1400
 Wire Wire Line
-	7300 1300 7300 1400
+	7300 1400 7300 1300
 Connection ~ 7300 1400
 Wire Wire Line
-	7050 1300 7050 1400
+	7050 1400 7050 1300
 Connection ~ 7050 1400
 Wire Wire Line
@@
 	6550 1400 8300 1400
 Wire Wire Line
-	8300 950  5950 950
+	5950 950  8300 950
 Connection ~ 6100 950
 Text Notes 5350 900  0    60   ~ 0
@@
 $EndComp
 $Comp
-L CP1 C1817
-U 1 1 5B300AB8
-P 8300 1150
-F 0 "C1817" H 8325 1250 50  0000 L CNN
-F 1 "220uF" H 8325 1050 50  0000 L CNN
-F 2 "Capacitors_Tantalum_SMD:CP_Tantalum_Case-D_EIA-7343-31_Reflow" H 8300 1150 50  0001 C CNN
-F 3 "http://datasheets.avx.com/TPS.pdf" H 8300 1150 50  0001 C CNN
-F 4 "AVX" H 8300 1150 60  0001 C CNN "MFG Name"
-F 5 "TPSD227K010R0100" H 8300 1150 60  0001 C CNN "MFG Part Num"
-F 6 "TPSD227K010R0100" H 8300 1150 60  0001 C CNN "Distrib PN"
-F 7 "https://www.tme.eu/en/details/tpsd227k010r010/smd-tantalum-capacitors/avx/tpsd227k010r0100/" H 8300 1150 60  0001 C CNN "Distrib Link"
-F 8 "10%" H 8300 1150 60  0001 C CNN "Tolerance"
-F 9 "https://www.arrow.com/en/products/293d227x9010d2te3/vishay" H 8300 1150 60  0001 C CNN "Others"
-	1    8300 1150
-	1    0    0    -1
-$EndComp
-$Comp
 L WifiBTCard MOD1801
 U 1 1 5B2AC34E
@@
 	1    0    0    -1
 $EndComp
+$Comp
+L CP1 C1817
+U 1 1 5B32B987
+P 8300 1150
+F 0 "C1817" H 8300 1250 50  0000 L CNN
+F 1 "220uF" H 8300 1050 50  0000 L CNN
+F 2 "Capacitors_SMD:CP_Elec_6.3x7.7" H 8300 1150 50  0001 C CNN
+F 3 "https://industrial.panasonic.com/cdbs/www-data/pdf/RDE0000/ABA0000C1184.pdf" H 8300 1150 50  0001 C CNN
+F 4 "Panasonic" H 8300 1150 60  0001 C CNN "MFG Name"
+F 5 "EEEFPA221XAP" H 8300 1150 60  0001 C CNN "MFG Part Num"
+F 6 "EEEFPA221XAP" H 8300 1150 60  0001 C CNN "Distrib PN"
+F 7 "https://www.tme.eu/en/details/eeefpa221xap/smd-low-imp-electrolytic-capacitors/panasonic/" H 8300 1150 60  0001 C CNN "Distrib Link"
+F 8 "20%" H 8300 1150 60  0001 C CNN "Tolerance"
+F 9 "http://uk.farnell.com/panasonic-electronic-components/eeefpa221xap/cap-alu-elec-220uf-10v-smd/dp/1539464" H 8300 1150 60  0001 C CNN "Others"
+	1    8300 1150
+	1    0    0    -1
+$EndComp
