File: jtag.sch (KiCad schematic (older format))
At the start: 9 parts, among them J801 NC

Commit message: Update project files to KiCad 5.0.0
Parts:
- D801: symbol D_Schottky_ALT -> dvk-mx8m-bsb-rescue:D_Schottky_ALT
- J801: symbol Conn_02x05_Odd_Even -> dvk-mx8m-bsb-rescue:Conn_02x05_Odd_Even
- R801, R802, R803, R804, R805, R806, R807: symbol R -> dvk-mx8m-bsb-rescue:R
Changed lines of the file:
@@
-EESchema Schematic File Version 2
-LIBS:power
-LIBS:device
-LIBS:switches
-LIBS:relays
-LIBS:motors
-LIBS:transistors
-LIBS:conn
-LIBS:linear
-LIBS:regul
-LIBS:74xx
-LIBS:cmos4000
-LIBS:adc-dac
-LIBS:memory
-LIBS:xilinx
-LIBS:microcontrollers
-LIBS:dsp
-LIBS:microchip
-LIBS:analog_switches
-LIBS:motorola
-LIBS:texas
-LIBS:intel
-LIBS:audio
-LIBS:interface
-LIBS:digital-audio
-LIBS:philips
-LIBS:display
-LIBS:cypress
-LIBS:siliconi
-LIBS:opto
-LIBS:atmel
-LIBS:contrib
-LIBS:valves
-LIBS:dvk-mx8m-bsb
+EESchema Schematic File Version 4
 LIBS:dvk-mx8m-bsb-cache
-EELAYER 25 0
+EELAYER 26 0
 EELAYER END
 $Descr A4 11693 8268
@@
 $EndDescr
 $Comp
-L Conn_02x05_Odd_Even J801
+L dvk-mx8m-bsb-rescue:Conn_02x05_Odd_Even J801
 U 1 1 5AD052A0
 P 6200 3550
@@
 $EndComp
 $Comp
-L R R806
+L dvk-mx8m-bsb-rescue:R R806
 U 1 1 5AD052F0
 P 6750 3650
@@
 $EndComp
 $Comp
-L R R807
+L dvk-mx8m-bsb-rescue:R R807
 U 1 1 5AD0530D
 P 6750 3750
@@
 $EndComp
 $Comp
-L R R804
+L dvk-mx8m-bsb-rescue:R R804
 U 1 1 5AD058A3
 P 6150 3950
@@
 $EndComp
 $Comp
-L R R805
+L dvk-mx8m-bsb-rescue:R R805
 U 1 1 5AD0593B
 P 6450 3150
@@
 Connection ~ 6550 3750
 $Comp
-L GND #PWR0152
+L power:GND #PWR0152
 U 1 1 5AD06B94
 P 6950 3800
@@
 	5750 3450 5750 4000
 $Comp
-L GND #PWR0153
+L power:GND #PWR0153
 U 1 1 5AD075E7
 P 5750 4350
@@
 ARM DStream
 $Comp
-L 3V3_OUT #PWR0154
+L dvk-mx8m-bsb:3V3_OUT #PWR0154
 U 1 1 5AEA3F80
 P 6450 2950
@@
 $EndComp
 $Comp
-L 3V3_OUT #PWR0155
+L dvk-mx8m-bsb:3V3_OUT #PWR0155
 U 1 1 5AE5744F
 P 5300 2900
@@
 Connection ~ 5350 3650
 $Comp
-L D_Schottky_ALT D801
+L dvk-mx8m-bsb-rescue:D_Schottky_ALT D801
 U 1 1 5B170CAA
 P 5550 3750
@@
 $EndComp
 $Comp
-L R R803
+L dvk-mx8m-bsb-rescue:R R803
 U 1 1 5B31E00F
 P 5750 4150
@@
 $EndComp
 $Comp
-L R R801
+L dvk-mx8m-bsb-rescue:R R801
 U 1 1 5B31E065
 P 5250 3150
@@
 $EndComp
 $Comp
-L R R802
+L dvk-mx8m-bsb-rescue:R R802
 U 1 1 5B31E0A4
 P 5350 3150

Commit message: Update the schematic symbols and footprints after upgrading to KiCad 5.0.0, fix all ERC and DRC violations after the new update/upgrade
Parts:
- D801: symbol dvk-mx8m-bsb-rescue:D_Schottky_ALT -> Device:D_Schottky_ALT
- J801: footprint Pin_Headers:Pin_Header_Straight_2x05_Pitch1.27mm_SMD -> Connector_PinHeader_1.27mm:PinHeader_2x05_P1.27mm_Vertical_SMD; symbol dvk-mx8m-bsb-rescue:Conn_02x05_Odd_Even -> Connector_Generic:Conn_02x05_Odd_Even
- R801, R802, R803, R804, R805, R806, R807: footprint Resistors_SMD:R_0603 -> Resistor_SMD:R_0603_1608Metric; symbol dvk-mx8m-bsb-rescue:R -> Device:R
Changed lines of the file:
@@
 Sheet 8 24
 Title "JTAG"
-Date "2018-06-18"
+Date "2018-07-17"
 Rev "v0.1.0"
 Comp "Copyright 2018 GNU GPLv3"
@@
 $EndDescr
 $Comp
-L dvk-mx8m-bsb-rescue:Conn_02x05_Odd_Even J801
+L Connector_Generic:Conn_02x05_Odd_Even J801
 U 1 1 5AD052A0
 P 6200 3550
 F 0 "J801" H 6250 3850 50  0000 C CNN
 F 1 "NC" H 6250 3250 50  0000 C CNN
-F 2 "Pin_Headers:Pin_Header_Straight_2x05_Pitch1.27mm_SMD" H 6200 3550 50  0001 C CNN
+F 2 "Connector_PinHeader_1.27mm:PinHeader_2x05_P1.27mm_Vertical_SMD" H 6200 3550 50  0001 C CNN
 F 3 "https://media.digikey.com/pdf/Data%20Sheets/Sullins%20PDFs/GRPB_%20_2VWQS-RC%2010958-C.pdf" H 6200 3550 50  0001 C CNN
 F 4 "Sullins" H 6200 3550 60  0001 C CNN "MFG Name"
@@
 $EndComp
 $Comp
-L dvk-mx8m-bsb-rescue:R R806
+L Device:R R806
 U 1 1 5AD052F0
 P 6750 3650
 F 0 "R806" V 6800 3850 50  0000 C CNN
 F 1 "NC" V 6750 3650 50  0000 C CNN
-F 2 "Resistors_SMD:R_0603" V 6680 3650 50  0001 C CNN
+F 2 "Resistor_SMD:R_0603_1608Metric" V 6680 3650 50  0001 C CNN
 F 3 "" H 6750 3650 50  0001 C CNN
 	1    6750 3650
@@
 $EndComp
 $Comp
-L dvk-mx8m-bsb-rescue:R R807
+L Device:R R807
 U 1 1 5AD0530D
 P 6750 3750
 F 0 "R807" V 6830 3750 50  0000 C CNN
 F 1 "0" V 6750 3750 50  0000 C CNN
-F 2 "Resistors_SMD:R_0603" V 6680 3750 50  0001 C CNN
+F 2 "Resistor_SMD:R_0603_1608Metric" V 6680 3750 50  0001 C CNN
 F 3 "" H 6750 3750 50  0001 C CNN
 	1    6750 3750
@@
 $EndComp
 $Comp
-L dvk-mx8m-bsb-rescue:R R804
+L Device:R R804
 U 1 1 5AD058A3
 P 6150 3950
 F 0 "R804" V 6230 3950 50  0000 C CNN
 F 1 "NC" V 6150 3950 50  0000 C CNN
-F 2 "Resistors_SMD:R_0603" V 6080 3950 50  0001 C CNN
+F 2 "Resistor_SMD:R_0603_1608Metric" V 6080 3950 50  0001 C CNN
 F 3 "" H 6150 3950 50  0001 C CNN
 	1    6150 3950
@@
 $EndComp
 $Comp
-L dvk-mx8m-bsb-rescue:R R805
+L Device:R R805
 U 1 1 5AD0593B
 P 6450 3150
 F 0 "R805" H 6300 3100 50  0000 C CNN
 F 1 "120" H 6325 3200 50  0000 C CNN
-F 2 "Resistors_SMD:R_0603" V 6380 3150 50  0001 C CNN
+F 2 "Resistor_SMD:R_0603_1608Metric" V 6380 3150 50  0001 C CNN
 F 3 "" H 6450 3150 50  0001 C CNN
 	1    6450 3150
@@
 Connection ~ 5350 3650
 $Comp
-L dvk-mx8m-bsb-rescue:D_Schottky_ALT D801
+L Device:D_Schottky_ALT D801
 U 1 1 5B170CAA
 P 5550 3750
@@
 $EndComp
 $Comp
-L dvk-mx8m-bsb-rescue:R R803
+L Device:R R803
 U 1 1 5B31E00F
 P 5750 4150
 F 0 "R803" H 5900 4200 50  0000 C CNN
 F 1 "10k" H 5875 4100 50  0000 C CNN
-F 2 "Resistors_SMD:R_0603" V 5680 4150 50  0001 C CNN
+F 2 "Resistor_SMD:R_0603_1608Metric" V 5680 4150 50  0001 C CNN
 F 3 "https://www.seielect.com/Catalog/SEI-RMCF_RMCP.pdf" H 5750 4150 50  0001 C CNN
 F 4 "Stackpole" H 5750 4150 60  0001 C CNN "MFG Name"
@@
 $EndComp
 $Comp
-L dvk-mx8m-bsb-rescue:R R801
+L Device:R R801
 U 1 1 5B31E065
 P 5250 3150
 F 0 "R801" H 5400 3200 50  0000 C CNN
 F 1 "10k" H 5375 3100 50  0000 C CNN
-F 2 "Resistors_SMD:R_0603" V 5180 3150 50  0001 C CNN
+F 2 "Resistor_SMD:R_0603_1608Metric" V 5180 3150 50  0001 C CNN
 F 3 "https://www.seielect.com/Catalog/SEI-RMCF_RMCP.pdf" H 5250 3150 50  0001 C CNN
 F 4 "Stackpole" H 5250 3150 60  0001 C CNN "MFG Name"
@@
 $EndComp
 $Comp
-L dvk-mx8m-bsb-rescue:R R802
+L Device:R R802
 U 1 1 5B31E0A4
 P 5350 3150
 F 0 "R802" H 5500 3200 50  0000 C CNN
 F 1 "10k" H 5475 3100 50  0000 C CNN
-F 2 "Resistors_SMD:R_0603" V 5280 3150 50  0001 C CNN
+F 2 "Resistor_SMD:R_0603_1608Metric" V 5280 3150 50  0001 C CNN
 F 3 "https://www.seielect.com/Catalog/SEI-RMCF_RMCP.pdf" H 5350 3150 50  0001 C CNN
 F 4 "Stackpole" H 5350 3150 60  0001 C CNN "MFG Name"
