File: ethernet.sch (KiCad schematic (older format))
At the start: 57 parts, among them J1701 RJ45, U1701 AR8031, Y1701 25MHz

Commit message: Add a 100k pull-down resistor to the the class-D audio amplifier's SD# / MUTE pin
Parts:
- R1718: Distrib Link https://www.digikey.com/product-detail/en/stackpole-electro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 -> (none); Distrib PN RMCF0603JG10K0CT-ND -> (none); MFG Name Stackpole -> (none); MFG Part Num RMCF0603JG10K0 -> (none); Others https://www.digikey.com/products/en/resistors/chip-resistor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 -> (none); Tolerance 5% -> (none)
Changed lines of the file:
@@
 $EndComp
 $Comp
-L GND #PWR0298
+L GND #PWR0299
 U 1 1 5AF1A655
 P 5100 6650
-F 0 "#PWR0298" H 5100 6400 50  0001 C CNN
+F 0 "#PWR0299" H 5100 6400 50  0001 C CNN
 F 1 "GND" H 5100 6500 50  0000 C CNN
 F 2 "" H 5100 6650 50  0001 C CNN
@@
 $EndComp
 $Comp
-L GND #PWR0299
+L GND #PWR0300
 U 1 1 5AF1A6B7
 P 4000 6700
-F 0 "#PWR0299" H 4000 6450 50  0001 C CNN
+F 0 "#PWR0300" H 4000 6450 50  0001 C CNN
 F 1 "GND" H 4000 6550 50  0000 C CNN
 F 2 "" H 4000 6700 50  0001 C CNN
@@
 $EndComp
 $Comp
-L GND #PWR0300
+L GND #PWR0301
 U 1 1 5AF1C035
 P 3050 6900
-F 0 "#PWR0300" H 3050 6650 50  0001 C CNN
+F 0 "#PWR0301" H 3050 6650 50  0001 C CNN
 F 1 "GND" H 3050 6750 50  0000 C CNN
 F 2 "" H 3050 6900 50  0001 C CNN
@@
 $EndComp
 $Comp
-L GND #PWR0301
+L GND #PWR0302
 U 1 1 5AF1D077
 P 2150 6550
-F 0 "#PWR0301" H 2150 6300 50  0001 C CNN
+F 0 "#PWR0302" H 2150 6300 50  0001 C CNN
 F 1 "GND" H 2150 6400 50  0000 C CNN
 F 2 "" H 2150 6550 50  0001 C CNN
@@
 $EndComp
 $Comp
-L GND #PWR0302
+L GND #PWR0303
 U 1 1 5AF23D63
 P 6500 6550
-F 0 "#PWR0302" H 6500 6300 50  0001 C CNN
+F 0 "#PWR0303" H 6500 6300 50  0001 C CNN
 F 1 "GND" H 6500 6400 50  0000 C CNN
 F 2 "" H 6500 6550 50  0001 C CNN
@@
 $EndComp
 $Comp
-L GND #PWR0303
+L GND #PWR0304
 U 1 1 5AF27185
 P 6950 3550
-F 0 "#PWR0303" H 6950 3300 50  0001 C CNN
+F 0 "#PWR0304" H 6950 3300 50  0001 C CNN
 F 1 "GND" H 6950 3400 50  0000 C CNN
 F 2 "" H 6950 3550 50  0001 C CNN
@@
 $EndComp
 $Comp
-L GND #PWR0304
+L GND #PWR0305
 U 1 1 5AF2ADD1
 P 6850 2600
-F 0 "#PWR0304" H 6850 2350 50  0001 C CNN
+F 0 "#PWR0305" H 6850 2350 50  0001 C CNN
 F 1 "GND" H 6850 2450 50  0000 C CNN
 F 2 "" H 6850 2600 50  0001 C CNN
@@
 $EndComp
 $Comp
-L GND #PWR0305
+L GND #PWR0306
 U 1 1 5AF2DC02
 P 4200 1450
-F 0 "#PWR0305" H 4200 1200 50  0001 C CNN
+F 0 "#PWR0306" H 4200 1200 50  0001 C CNN
 F 1 "GND" H 4200 1300 50  0000 C CNN
 F 2 "" H 4200 1450 50  0001 C CNN
@@
 $EndComp
 $Comp
-L GND #PWR0306
+L GND #PWR0307
 U 1 1 5AF2E0B5
 P 4200 2100
-F 0 "#PWR0306" H 4200 1850 50  0001 C CNN
+F 0 "#PWR0307" H 4200 1850 50  0001 C CNN
 F 1 "GND" H 4200 1950 50  0000 C CNN
 F 2 "" H 4200 2100 50  0001 C CNN
@@
 $EndComp
 $Comp
-L 3V3_P #PWR0307
+L 3V3_P #PWR0308
 U 1 1 5AF325F5
 P 3000 950
-F 0 "#PWR0307" H 3000 800 50  0001 C CNN
+F 0 "#PWR0308" H 3000 800 50  0001 C CNN
 F 1 "3V3_P" H 3000 1090 50  0000 C CNN
 F 2 "" H 3000 950 50  0001 C CNN
@@
 $EndComp
 $Comp
-L GND #PWR0308
+L GND #PWR0309
 U 1 1 5AF33215
 P 6000 1800
-F 0 "#PWR0308" H 6000 1550 50  0001 C CNN
+F 0 "#PWR0309" H 6000 1550 50  0001 C CNN
 F 1 "GND" H 6000 1650 50  0000 C CNN
 F 2 "" H 6000 1800 50  0001 C CNN
@@
 ENET_2V5
 $Comp
-L 3V3_P #PWR0309
+L 3V3_P #PWR0310
 U 1 1 5AF58308
 P 2150 4500
-F 0 "#PWR0309" H 2150 4350 50  0001 C CNN
+F 0 "#PWR0310" H 2150 4350 50  0001 C CNN
 F 1 "3V3_P" H 2150 4640 50  0000 C CNN
 F 2 "" H 2150 4500 50  0001 C CNN
@@
 $EndComp
 $Comp
-L GND #PWR0310
+L GND #PWR0311
 U 1 1 5AFCAFF1
 P 1900 3550
-F 0 "#PWR0310" H 1900 3300 50  0001 C CNN
+F 0 "#PWR0311" H 1900 3300 50  0001 C CNN
 F 1 "GND" H 1900 3400 50  0000 C CNN
 F 2 "" H 1900 3550 50  0001 C CNN
@@
 $EndComp
 $Comp
-L GND #PWR0311
+L GND #PWR0312
 U 1 1 5B00F44D
 P 8800 5150
-F 0 "#PWR0311" H 8800 4900 50  0001 C CNN
+F 0 "#PWR0312" H 8800 4900 50  0001 C CNN
 F 1 "GND" H 8800 5000 50  0000 C CNN
 F 2 "" H 8800 5150 50  0001 C CNN
@@
 Connection ~ 7400 3100
 $Comp
-L GND #PWR0312
+L GND #PWR0313
 U 1 1 5B0467F8
 P 8300 3900
-F 0 "#PWR0312" H 8300 3650 50  0001 C CNN
+F 0 "#PWR0313" H 8300 3650 50  0001 C CNN
 F 1 "GND" H 8300 3750 50  0000 C CNN
 F 2 "" H 8300 3900 50  0001 C CNN
@@
 RGMII 10/100/1000 Ethernet
 $Comp
-L PWR_FLAG #FLG0313
+L PWR_FLAG #FLG0314
 U 1 1 5B0C2224
 P 4750 950
-F 0 "#FLG0313" H 4750 1025 50  0001 C CNN
+F 0 "#FLG0314" H 4750 1025 50  0001 C CNN
 F 1 "PWR_FLAG" H 4750 1100 50  0000 C CNN
 F 2 "" H 4750 950 50  0001 C CNN
@@
 Connection ~ 4750 1000
 $Comp
-L PWR_FLAG #FLG0314
+L PWR_FLAG #FLG0315
 U 1 1 5B0C422C
 P 8200 2100
-F 0 "#FLG0314" H 8200 2175 50  0001 C CNN
+F 0 "#FLG0315" H 8200 2175 50  0001 C CNN
 F 1 "PWR_FLAG" H 8200 2250 50  0000 C CNN
 F 2 "" H 8200 2100 50  0001 C CNN
@@
 Connection ~ 8200 2150
 $Comp
-L PWR_FLAG #FLG0315
+L PWR_FLAG #FLG0316
 U 1 1 5B0C4B7D
 P 6200 3050
-F 0 "#FLG0315" H 6200 3125 50  0001 C CNN
+F 0 "#FLG0316" H 6200 3125 50  0001 C CNN
 F 1 "PWR_FLAG" H 6200 3200 50  0000 C CNN
 F 2 "" H 6200 3050 50  0001 C CNN
@@
 F 1 "1.62k" H 3400 4700 50  0000 C CNN
 F 2 "Resistors_SMD:R_0603" V 3180 4750 50  0001 C CNN
-F 3 "https://www.seielect.com/Catalog/SEI-RMCF_RMCP.pdf" H 3250 4750 50  0001 C CNN
-F 4 "Stackpole" H 3250 4750 60  0001 C CNN "MFG Name"
-F 5 "RMCF0603JG10K0" H 3250 4750 60  0001 C CNN "MFG Part Num"
-F 6 "RMCF0603JG10K0CT-ND" H 3250 4750 60  0001 C CNN "Distrib PN"
-F 7 "https://www.digikey.com/product-detail/en/stackpole-electronics-inc/RMCF0603JG10K0/RMCF0603JG10K0CT-ND/4425128" H 3250 4750 60  0001 C CNN "Distrib Link"
-F 8 "5%" H 3250 4750 60  0001 C CNN "Tolerance"
-F 9 "https://www.digikey.com/products/en/resistors/chip-resistor-surface-mount/52?FV=ffe00034%2C400005%2C1f140000%2Cmu10+kOhms%7C2085&quantity=&ColumnSort=1000011&page=1&pageSize=500" H 3250 4750 60  0001 C CNN "Others"
+F 3 "" H 3250 4750 50  0001 C CNN
 	1    3250 4750
 	1    0    0    -1

Commit message: Update project files to KiCad 5.0.0
Parts:
- C1701, C1702, C1703, C1704, C1705, C1706, C1707, C1708, C1709, C1710, C1711, C1712, C1713, C1714, C1715, C1716, C1717, C1718, C1719, C1720, C1721: symbol C -> dvk-mx8m-bsb-rescue:C
- D1701: symbol D_Schottky_ALT -> dvk-mx8m-bsb-rescue:D_Schottky_ALT
- D1702: symbol LED_ALT -> dvk-mx8m-bsb-rescue:LED_ALT
- FB1701, FB1702, FB1703: symbol Ferrite_Bead -> dvk-mx8m-bsb-rescue:Ferrite_Bead
- J1701: symbol RJHSE-5381 -> dvk-mx8m-bsb:RJHSE-5381
- L1701: symbol L -> dvk-mx8m-bsb-rescue:L
- R1701, R1702, R1703, R1704, R1705, R1706, R1707, R1708, R1709, R1710, R1711, R1712, R1713, R1714, R1715, R1716, R1717, R1718, R1719, R1720, R1721, R1722, R1723, R1724, R1725: symbol R -> dvk-mx8m-bsb-rescue:R
- TP1701, TP1702: symbol TEST_1P -> dvk-mx8m-bsb-rescue:TEST_1P
- U1701: symbol AR8031 -> dvk-mx8m-bsb:AR8031
- Y1701: symbol Crystal_GND24 -> dvk-mx8m-bsb-rescue:Crystal_GND24

Commit message: Update the schematic symbols and footprints after upgrading to KiCad 5.0.0, fix all ERC and DRC violations after the new update/upgrade
Parts:
- C1701, C1702, C1703, C1704, C1705, C1706, C1707, C1708, C1709, C1710, C1711, C1712, C1713, C1714, C1715, C1716, C1717, C1718, C1719, C1720, C1721: footprint Capacitors_SMD:C_0603 -> Capacitor_SMD:C_0603_1608Metric; symbol dvk-mx8m-bsb-rescue:C -> Device:C
- D1701: symbol dvk-mx8m-bsb-rescue:D_Schottky_ALT -> Device:D_Schottky_ALT
- D1702: symbol dvk-mx8m-bsb-rescue:LED_ALT -> Device:LED_ALT
- FB1701, FB1702, FB1703: symbol dvk-mx8m-bsb-rescue:Ferrite_Bead -> Device:Ferrite_Bead
- L1701: symbol dvk-mx8m-bsb-rescue:L -> Device:L
- R1701, R1702, R1703, R1704, R1705, R1706, R1707, R1708, R1709, R1710, R1711, R1712, R1713, R1714, R1715, R1716, R1717, R1718, R1719, R1720, R1721, R1722, R1723, R1724, R1725: footprint Resistors_SMD:R_0603 -> Resistor_SMD:R_0603_1608Metric; symbol dvk-mx8m-bsb-rescue:R -> Device:R
- TP1701, TP1702: symbol dvk-mx8m-bsb-rescue:TEST_1P -> Connector:TestPoint
- Y1701: symbol dvk-mx8m-bsb-rescue:Crystal_GND24 -> Device:Crystal_GND24

Commit message: Use the new 1.5mm diameter test point footprint from KiCad 5's library
Parts:
- TP1701, TP1702: footprint Measurement_Points:Measurement_Point_Round-SMD-Pad_Small -> TestPoint:TestPoint_Pad_D1.5mm
Changed lines of the file:
@@
 F 0 "TP1701" H 750 6120 50  0000 C CNN
 F 1 "TEST_1P" H 750 6050 50  0000 C CNN
-F 2 "Measurement_Points:Measurement_Point_Round-SMD-Pad_Small" H 950 5850 50  0001 C CNN
+F 2 "TestPoint:TestPoint_Pad_D1.5mm" H 950 5850 50  0001 C CNN
 F 3 "" H 950 5850 50  0001 C CNN
 	1    750  5850
@@
 F 0 "TP1702" H 1050 6020 50  0000 C CNN
 F 1 "TEST_1P" H 1050 5950 50  0000 C CNN
-F 2 "Measurement_Points:Measurement_Point_Round-SMD-Pad_Small" H 1250 5750 50  0001 C CNN
+F 2 "TestPoint:TestPoint_Pad_D1.5mm" H 1250 5750 50  0001 C CNN
 F 3 "" H 1250 5750 50  0001 C CNN
 	1    1050 5750

Commit message: Routed and connected some passive components around the ethernet interfaces.
Detected and corrected numbering error with MagJack J1701.
Eventually error with missing VCC of Pin 1 of J1707 (to be checked).
Connections:
- wire segments 198 -> 270
Changed lines of the file:
@@
 	2850 6450 2900 6450
 Wire Wire Line
-	2100 6150 4050 6150
+	2100 6150 2150 6150
 Wire Wire Line
 	2150 6550 2150 6500
 Wire Wire Line
-	2850 6050 2850 6500
+	2850 6050 2850 6450
 Connection ~ 2850 6450
 Wire Wire Line
@@
 	3550 6200 3550 6850
 Wire Wire Line
-	3550 6850 2850 6850
+	3550 6850 3250 6850
 Wire Wire Line
 	2850 6850 2850 6800
 Wire Wire Line
-	3050 6650 3050 6900
+	3050 6650 3050 6850
 Connection ~ 3050 6850
 Wire Wire Line
@@
 	3200 6450 3250 6450
 Wire Wire Line
-	3250 6150 3250 6500
+	3250 6150 3250 6450
 Wire Wire Line
 	2150 6200 2150 6150
@@
 	6200 6450 6200 6500
 Wire Wire Line
-	6200 6500 6800 6500
+	6200 6500 6500 6500
 Wire Wire Line
 	6800 6500 6800 6450
 Wire Wire Line
-	6500 6450 6500 6550
+	6500 6450 6500 6500
 Connection ~ 6500 6500
 Wire Wire Line
-	6150 5800 7550 5800
-Wire Wire Line
-	6150 5950 7550 5950
-Wire Wire Line
-	6150 6100 7550 6100
+	6150 5800 6800 5800
+Wire Wire Line
+	6150 5950 6500 5950
+Wire Wire Line
+	6150 6100 6200 6100
 Wire Wire Line
 	6200 6150 6200 6100
@@
 	6150 4500 6700 4500
 Wire Wire Line
-	6150 3100 7650 3100
+	6150 3100 6200 3100
 Wire Wire Line
 	6200 3400 6150 3400
 Wire Wire Line
-	6200 3050 6200 3400
+	6200 3050 6200 3100
 Connection ~ 6200 3100
 Wire Wire Line
@@
 	8200 3100 7950 3100
 Wire Wire Line
-	8200 2100 8200 3100
-Wire Wire Line
-	6150 2150 8200 2150
+	8200 2100 8200 2150
+Wire Wire Line
+	6150 2150 6200 2150
 Wire Wire Line
 	6150 2700 6200 2700
@@
 	6700 2500 6700 2550
 Wire Wire Line
-	6700 2550 7000 2550
+	6700 2550 6850 2550
 Wire Wire Line
 	7000 2550 7000 2500
@@
 	4600 1650 4600 2200
 Wire Wire Line
-	3000 1650 4600 1650
-Wire Wire Line
-	3000 950  3000 1650
+	3000 1650 4050 1650
+Wire Wire Line
+	3000 950  3000 1000
 Wire Wire Line
 	4050 2000 4050 2050
 Wire Wire Line
-	4050 2050 4350 2050
+	4050 2050 4200 2050
 Wire Wire Line
 	4350 2050 4350 2000
@@
 	4050 1350 4050 1400
 Wire Wire Line
-	4050 1400 4350 1400
+	4050 1400 4200 1400
 Wire Wire Line
 	4350 1400 4350 1350
@@
 Connection ~ 3000 1000
 Wire Wire Line
-	3550 1000 4750 1000
-Wire Wire Line
-	4750 950  4750 2200
+	3550 1000 4050 1000
+Wire Wire Line
+	4750 950  4750 1000
 Wire Wire Line
 	4050 1050 4050 1000
@@
 	5700 1700 5700 1750
 Wire Wire Line
-	5700 1750 6300 1750
+	5700 1750 6000 1750
 Wire Wire Line
 	6300 1750 6300 1700
 Wire Wire Line
-	6000 1700 6000 1800
+	6000 1700 6000 1750
 Connection ~ 6000 1750
 Wire Wire Line
 	5100 2200 5100 1350
 Wire Wire Line
-	5100 1350 6350 1350
+	5100 1350 5350 1350
 Wire Wire Line
 	6300 1350 6300 1400
@@
 	4050 4950 4000 4950
 Wire Wire Line
-	3950 5100 4050 5100
-Wire Wire Line
-	3950 5200 4050 5200
-Wire Wire Line
-	1750 5300 2550 5300
-Wire Wire Line
-	2850 5300 4050 5300
-Wire Wire Line
-	1750 5200 3650 5200
+	3950 5100 4000 5100
+Wire Wire Line
+	3950 5200 4000 5200
+Wire Wire Line
+	1750 5300 2500 5300
+Wire Wire Line
+	2850 5300 2900 5300
+Wire Wire Line
+	1750 5200 3250 5200
 Wire Wire Line
 	2500 4900 2500 5300
@@
 Connection ~ 2900 5300
 Wire Wire Line
-	1750 5100 3650 5100
-Wire Wire Line
-	1750 5500 4050 5500
-Wire Wire Line
-	1750 5600 4050 5600
+	1750 5100 3600 5100
+Wire Wire Line
+	1750 5500 2150 5500
+Wire Wire Line
+	1750 5600 1800 5600
 Wire Wire Line
 	2150 4900 2150 5500
@@
 	1800 4600 1800 4550
 Wire Wire Line
-	1800 4550 2500 4550
+	1800 4550 2150 4550
 Wire Wire Line
 	2500 4550 2500 4600
@@
 	3700 4950 3300 4950
 Wire Wire Line
-	2150 4500 2150 4600
+	2150 4500 2150 4550
 Wire Wire Line
 	1850 1700 1900 1700
 Wire Wire Line
-	1900 1700 1900 3550
+	1900 1700 1900 1900
 Wire Wire Line
 	1850 1900 1900 1900
@@
 	1850 2100 2350 2100
 Wire Wire Line
-	850  1700 1550 1700
+	850  1700 1500 1700
 Wire Wire Line
 	1550 1900 850  1900
 Wire Wire Line
-	850  2300 1550 2300
+	850  2300 1500 2300
 Wire Wire Line
 	1550 2500 850  2500
@@
 Connection ~ 8800 4250
 Wire Wire Line
-	9350 3900 9550 3900
+	9350 3900 9500 3900
 Wire Wire Line
 	9550 4000 9500 4000
@@
 	6500 3450 6500 3500
 Wire Wire Line
-	6500 3500 7400 3500
+	6500 3500 6800 3500
 Wire Wire Line
 	7400 3500 7400 3450
@@
 	9550 3750 8800 3750
 Wire Wire Line
-	8800 3750 8800 5150
+	8800 3750 8800 3900
 Wire Wire Line
 	9550 3600 8800 3600
@@
 	8000 3800 8000 3850
 Wire Wire Line
-	8000 3850 8600 3850
+	8000 3850 8300 3850
 Wire Wire Line
 	8600 3850 8600 3800
@@
 $EndComp
 Wire Wire Line
-	8800 3450 8000 3450
-Wire Wire Line
-	8300 3800 8300 3900
+	8800 3450 8600 3450
+Wire Wire Line
+	8300 3800 8300 3850
 $Comp
 L Device:R R1712
@@
 Text Notes 3516 4832 0    39   ~ 0
 1%
+Wire Wire Line
+	2850 6450 2850 6500
+Wire Wire Line
+	3050 6850 2850 6850
+Wire Wire Line
+	3050 6850 3050 6900
+Wire Wire Line
+	3250 6850 3050 6850
+Wire Wire Line
+	2150 6150 3250 6150
+Wire Wire Line
+	3250 6450 3250 6500
+Wire Wire Line
+	3250 6150 4050 6150
+Wire Wire Line
+	6500 6500 6800 6500
+Wire Wire Line
+	6500 6500 6500 6550
+Wire Wire Line
+	6200 6100 7550 6100
+Wire Wire Line
+	6500 5950 7550 5950
+Wire Wire Line
+	6800 5800 7550 5800
+Wire Wire Line
+	6200 3100 6500 3100
+Wire Wire Line
+	6200 3100 6200 3200
+Wire Wire Line
+	6500 3100 6800 3100
+Wire Wire Line
+	6800 3100 7100 3100
+Wire Wire Line
+	7100 3100 7400 3100
+Wire Wire Line
+	6200 3200 6200 3300
+Wire Wire Line
+	6200 3300 6200 3400
+Wire Wire Line
+	6200 2150 6700 2150
+Wire Wire Line
+	6850 2550 7000 2550
+Wire Wire Line
+	6700 2150 7000 2150
+Wire Wire Line
+	7000 2150 8200 2150
+Wire Wire Line
+	4200 2050 4350 2050
+Wire Wire Line
+	4050 1650 4350 1650
+Wire Wire Line
+	4350 1650 4600 1650
+Wire Wire Line
+	4200 1400 4350 1400
+Wire Wire Line
+	3000 1000 3000 1650
+Wire Wire Line
+	4050 1000 4350 1000
+Wire Wire Line
+	4350 1000 4750 1000
+Wire Wire Line
+	6000 1750 6300 1750
+Wire Wire Line
+	6000 1750 6000 1800
+Wire Wire Line
+	5350 1350 5700 1350
+Wire Wire Line
+	5700 1350 6000 1350
+Wire Wire Line
+	6000 1350 6300 1350
+Wire Wire Line
+	6300 1350 6350 1350
+Wire Wire Line
+	2500 5300 2550 5300
+Wire Wire Line
+	2900 5300 4050 5300
+Wire Wire Line
+	2150 5500 4050 5500
+Wire Wire Line
+	1800 5600 4050 5600
+Wire Wire Line
+	2150 4550 2500 4550
+Wire Wire Line
+	2150 4550 2150 4600
+Wire Wire Line
+	1900 1900 1900 2300
+Wire Wire Line
+	1900 2300 1900 2500
+Wire Wire Line
+	1900 2500 1900 2700
+Wire Wire Line
+	1900 2700 1900 2900
+Wire Wire Line
+	1900 2900 1900 3100
+Wire Wire Line
+	1900 3100 1900 3300
+Wire Wire Line
+	1900 3300 1900 3500
+Wire Wire Line
+	1900 3500 1900 3550
+Wire Wire Line
+	1500 1700 1550 1700
+Wire Wire Line
+	1500 2300 1550 2300
+Wire Wire Line
+	8800 4500 8800 5100
+Wire Wire Line
+	8800 5100 8800 5150
+Wire Wire Line
+	8800 4250 8800 4500
+Wire Wire Line
+	9500 3900 9550 3900
+Wire Wire Line
+	8800 3900 8800 4250
+Wire Wire Line
+	6800 3500 6950 3500
+Wire Wire Line
+	7100 3500 7400 3500
+Wire Wire Line
+	6950 3500 7100 3500
+Wire Wire Line
+	7400 3100 7650 3100
+Wire Wire Line
+	8300 3850 8600 3850
+Wire Wire Line
+	8300 3850 8300 3900
+Wire Wire Line
+	8300 3450 8000 3450
+Wire Wire Line
+	8600 3450 8300 3450
+Wire Wire Line
+	4750 1000 4750 2200
+Wire Wire Line
+	8200 2150 8200 3100
+Wire Wire Line
+	4000 5200 4050 5200
+Wire Wire Line
+	3600 5200 3650 5200
+Wire Wire Line
+	4000 5100 4050 5100
+Wire Wire Line
+	3600 5100 3650 5100
+Wire Wire Line
+	3250 5200 3600 5200
 $EndSCHEMATC
