File: battery.sch (KiCad schematic (older format))
At the start: 36 parts, among them Q301 FDV301N, U301 BQ25896

Commit message: Place and begin routing the charge controller circuit
Connections:
- wire segments 112 -> 157
Other:
- note added: "1.658≤ILIM≤2.063\nILIM(nom)≅1.859A\n 3.9≤VIN≤6"
- note removed: "1.658≤ILIM≤2.063\nILIM(nom)≅1.859A\n 3.9≤VIN≤14"
- moved on the sheet: C308, C309
Changed lines of the file:
@@
 L C C308
 U 1 1 5AE0040B
-P 7450 2800
-F 0 "C308" H 7475 2900 50  0000 L CNN
-F 1 "100nF" H 7475 2700 50  0000 L CNN
-F 2 "Capacitors_SMD:C_0603" H 7488 2650 50  0001 C CNN
-F 3 "" H 7450 2800 50  0001 C CNN
-	1    7450 2800
+P 7500 2800
+F 0 "C308" H 7525 2900 50  0000 L CNN
+F 1 "100nF" H 7500 2700 50  0000 L CNN
+F 2 "Capacitors_SMD:C_0603" H 7538 2650 50  0001 C CNN
+F 3 "" H 7500 2800 50  0001 C CNN
+	1    7500 2800
 	1    0    0    -1
 $EndComp
@@
 L C C309
 U 1 1 5AE01FE0
-P 7850 2800
-F 0 "C309" H 7875 2900 50  0000 L CNN
-F 1 "100nF" H 7875 2700 50  0000 L CNN
-F 2 "Capacitors_SMD:C_0603" H 7888 2650 50  0001 C CNN
-F 3 "" H 7850 2800 50  0001 C CNN
-	1    7850 2800
+P 7750 2800
+F 0 "C309" H 7775 2900 50  0000 L CNN
+F 1 "100nF" H 7775 2700 50  0000 L CNN
+F 2 "Capacitors_SMD:C_0603" H 7788 2650 50  0001 C CNN
+F 3 "" H 7750 2800 50  0001 C CNN
+	1    7750 2800
 	1    0    0    -1
 $EndComp
@@
 RGEN
 Text Notes 3800 2350 0    60   ~ 0
-1.658≤ILIM≤2.063\nILIM(nom)≅1.859A\n   3.9≤VIN≤14
+1.658≤ILIM≤2.063\nILIM(nom)≅1.859A\n    3.9≤VIN≤6
 Text HLabel 4500 4250 0    60   BiDi ~ 0
 I2C3_SDA
@@
 L GND #PWR060
 U 1 1 5AE86DE3
-P 7450 3050
-F 0 "#PWR060" H 7450 2800 50  0001 C CNN
-F 1 "GND" H 7450 2900 50  0000 C CNN
-F 2 "" H 7450 3050 50  0001 C CNN
-F 3 "" H 7450 3050 50  0001 C CNN
-	1    7450 3050
+P 7500 3050
+F 0 "#PWR060" H 7500 2800 50  0001 C CNN
+F 1 "GND" H 7500 2900 50  0000 C CNN
+F 2 "" H 7500 3050 50  0001 C CNN
+F 3 "" H 7500 3050 50  0001 C CNN
+	1    7500 3050
 	1    0    0    -1
 $EndComp
@@
 Text Notes 4300 5300 0    60   ~ 0
 BC1.2 is not mandated by PD spec\nICO used to determine max current\nAlso negotiated from CC pins (I2C)
-Text Notes 7225 2350 0    60   ~ 0
+Text Notes 7275 2350 0    60   ~ 0
 3.5~~4.25V
 Text Notes 5700 2400 0    60   ~ 0
@@
 L PWR_FLAG #FLG061
 U 1 1 5AF16085
-P 7450 2550
-F 0 "#FLG061" H 7450 2625 50  0001 C CNN
-F 1 "PWR_FLAG" H 7450 2700 50  0000 C CNN
-F 2 "" H 7450 2550 50  0001 C CNN
-F 3 "" H 7450 2550 50  0001 C CNN
-	1    7450 2550
+P 7500 2550
+F 0 "#FLG061" H 7500 2625 50  0001 C CNN
+F 1 "PWR_FLAG" H 7500 2700 50  0000 C CNN
+F 2 "" H 7500 2550 50  0001 C CNN
+F 3 "" H 7500 2550 50  0001 C CNN
+	1    7500 2550
 	1    0    0    -1
 $EndComp
@@
 $EndComp
 Wire Wire Line
-	4250 2550 4250 2650
+	4250 2550 4250 2600
+Wire Wire Line
+	4250 2600 4250 2650
 Connection ~ 4250 2600
 Wire Wire Line
 	4250 3000 4250 2950
 Wire Wire Line
-	5550 2600 5750 2600
+	5550 2600 5600 2600
+Wire Wire Line
+	5600 2600 5650 2600
+Wire Wire Line
+	5650 2600 5750 2600
 Wire Wire Line
 	5650 2650 5650 2600
@@
 	4450 3100 4450 3050
 Wire Wire Line
-	5550 3750 6100 3750
+	5550 3750 5600 3750
+Wire Wire Line
+	5600 3750 6100 3750
 Wire Wire Line
 	6100 3750 6100 2600
@@
 	6350 2950 6350 3000
 Wire Wire Line
-	6350 3000 6550 3000
+	6350 3000 6450 3000
+Wire Wire Line
+	6450 3000 6550 3000
 Wire Wire Line
 	6550 3000 6550 2950
@@
 Connection ~ 6100 5000
 Wire Wire Line
-	5550 4350 6300 4350
+	5550 4350 5900 4350
+Wire Wire Line
+	5900 4350 6300 4350
 Wire Wire Line
 	6300 4350 6300 4400
 Wire Wire Line
-	5900 4200 5900 4450
+	5900 4200 5900 4350
+Wire Wire Line
+	5900 4350 5900 4450
 Connection ~ 5900 4350
 Wire Wire Line
@@
 	4200 3300 4550 3300
 Wire Wire Line
-	6050 2600 6750 2600
-Wire Wire Line
-	7850 3000 7850 2950
-Wire Wire Line
-	7450 2950 7450 3050
+	6050 2600 6100 2600
+Wire Wire Line
+	6100 2600 6350 2600
+Wire Wire Line
+	6350 2600 6550 2600
+Wire Wire Line
+	6550 2600 6750 2600
+Wire Wire Line
+	7750 3000 7750 2950
+Wire Wire Line
+	7500 2950 7500 3000
+Wire Wire Line
+	7500 3000 7500 3050
 Wire Wire Line
 	7250 3000 7250 2950
 Wire Wire Line
-	7050 2600 9400 2600
-Connection ~ 7850 2600
-Wire Wire Line
-	7450 2550 7450 2650
-Connection ~ 7450 2600
+	7050 2600 7250 2600
+Wire Wire Line
+	7250 2600 7500 2600
+Wire Wire Line
+	7500 2600 7750 2600
+Wire Wire Line
+	7750 2600 8200 2600
+Wire Wire Line
+	8200 2600 8450 2600
+Wire Wire Line
+	8450 2600 8700 2600
+Wire Wire Line
+	8700 2600 8950 2600
+Wire Wire Line
+	8950 2600 9200 2600
+Wire Wire Line
+	9200 2600 9350 2600
+Wire Wire Line
+	9350 2600 9400 2600
+Connection ~ 7750 2600
+Wire Wire Line
+	7500 2550 7500 2600
+Wire Wire Line
+	7500 2600 7500 2650
+Connection ~ 7500 2600
 Wire Wire Line
 	7250 2650 7250 2600
@@
 	5600 4150 5550 4150
 Wire Wire Line
-	7250 3000 7850 3000
-Connection ~ 7450 3000
-Wire Wire Line
-	6700 4550 7500 4550
+	7250 3000 7500 3000
+Wire Wire Line
+	7500 3000 7750 3000
+Connection ~ 7500 3000
+Wire Wire Line
+	6700 4550 7100 4550
+Wire Wire Line
+	7100 4550 7500 4550
 Wire Wire Line
 	7500 4550 7500 4300
 Wire Wire Line
-	7100 4500 7100 4600
+	7100 4500 7100 4550
+Wire Wire Line
+	7100 4550 7100 4600
 Connection ~ 7100 4550
 Wire Wire Line
 	7500 3900 7500 4000
 Wire Wire Line
-	6700 3850 6700 4000
+	6700 3850 6700 3900
+Wire Wire Line
+	6700 3900 6700 4000
 Connection ~ 6700 3900
 Wire Wire Line
@@
 Connection ~ 5600 2600
 Wire Wire Line
-	3800 4400 3800 4700
+	3800 4400 3800 4650
+Wire Wire Line
+	3800 4650 3800 4700
 Wire Wire Line
 	3800 4100 3800 4050
@@
 	3850 3300 3900 3300
 Wire Wire Line
-	3400 4450 4550 4450
+	3400 4450 3450 4450
+Wire Wire Line
+	3450 4450 4550 4450
 Wire Wire Line
 	7250 3900 7500 3900
 Wire Wire Line
-	5550 3900 6950 3900
+	5550 3900 5600 3900
+Wire Wire Line
+	5600 3900 6400 3900
+Wire Wire Line
+	6400 3900 6700 3900
+Wire Wire Line
+	6700 3900 6950 3900
 Wire Wire Line
 	6400 3900 6400 3850
@@
 	3950 2500 4000 2500
 Wire Wire Line
-	4000 2500 4000 2700
+	4000 2500 4000 2600
+Wire Wire Line
+	4000 2600 4000 2700
 Wire Wire Line
 	4000 2700 3950 2700
 Connection ~ 4000 2600
 Wire Wire Line
-	4000 2600 4550 2600
+	4000 2600 4250 2600
+Wire Wire Line
+	4250 2600 4550 2600
 Wire Wire Line
 	10200 2500 10150 2500
 Wire Wire Line
-	10150 2500 10150 2700
+	10150 2500 10150 2600
+Wire Wire Line
+	10150 2600 10150 2700
 Wire Wire Line
 	10150 2700 10200 2700
@@
 	8200 2950 8200 3000
 Wire Wire Line
-	8200 3000 9200 3000
+	8200 3000 8450 3000
+Wire Wire Line
+	8450 3000 8700 3000
+Wire Wire Line
+	8700 3000 8950 3000
+Wire Wire Line
+	8950 3000 9200 3000
 Wire Wire Line
 	9200 3000 9200 2950
@@
 Connection ~ 8450 3000
 Wire Wire Line
-	8700 2950 8700 3050
+	8700 2950 8700 3000
+Wire Wire Line
+	8700 3000 8700 3050
 Wire Wire Line
 	8950 2950 8950 3000
@@
 	9500 2350 9500 2400
 Wire Wire Line
-	9350 2400 9750 2400
+	9350 2400 9500 2400
+Wire Wire Line
+	9500 2400 9600 2400
+Wire Wire Line
+	9600 2400 9750 2400
 Wire Wire Line
 	9350 2400 9350 2600
 Connection ~ 9350 2600
 Wire Wire Line
-	9700 2600 10150 2600
+	9700 2600 9750 2600
+Wire Wire Line
+	9750 2600 9950 2600
+Wire Wire Line
+	9950 2600 10150 2600
 Wire Wire Line
 	9600 2400 9600 2350
@@
 Connection ~ 9500 2400
 Wire Wire Line
-	7850 2650 7850 2600
+	7750 2650 7750 2600
 $Comp
 L C C310
@@
 Text Notes 10025 3075 0    60   ~ 0
 0.4mA~~2.4mA
-Text Notes 7500 3100 0    60   ~ 0
+Text Notes 7550 3100 0    60   ~ 0
 Vf(max)=1.1V
 Wire Wire Line
@@
 	5050 4950 5050 5000
 Wire Wire Line
-	5050 5000 6300 5000
-Wire Wire Line
-	5600 4550 5600 5000
+	5050 5000 5600 5000
+Wire Wire Line
+	5600 5000 5900 5000
+Wire Wire Line
+	5900 5000 6100 5000
+Wire Wire Line
+	6100 5000 6300 5000
+Wire Wire Line
+	5600 4550 5600 4650
+Wire Wire Line
+	5600 4650 5600 5000
 Connection ~ 5600 5000
 $Comp

Commit message: Move the charge controller, USB-C TCPC, and RTC to I2C1
Since each of these ICs will be powered at the same time as the SoM regardless of the PWR_EN state, they should share the same I2C bus as the PMIC.
Connections:
- net labels added: I2C1_SCL, I2C1_SDA
- net labels removed: I2C3_SCL, I2C3_SDA
- wire segments 157 -> 112
Other:
- moved on the sheet: Q301, R303, R304

Commit message: Replace the 103HT NTC thermistor with a ERTJ1VG103FA as found in TI's TIDA-01182 eval board which has a charge controller IC from the same family and uses an 18650 battery, change is due to it being smaller, cheaper, and has the same B value as the recommended thermistor in the charge controller IC's datasheet, comparing the thermistors' tables shows that they are nearly identical and that it should be a drop-in replacement
Parts:
- TH301: footprint dvk-mx8m-bsb:103HT -> Resistors_SMD:R_0603; Distrib Link https://www.mouser.com/ProductDetail/Semitec/103HT?qs=sGAEp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 -> https://www.arrow.com/en/products/ert-j1vg103fa/panasonic; Distrib PN 954-103HT -> ERT-J1VG103FA; MFG Name Semitec -> Panasonic; MFG Part Num 103HT -> ERTJ1VG103FA; Others https://octopart.com/search?q=semitec%20103ht&start=0 -> https://www.mouser.com/ProductDetail/Semitec/103HT?qs=sGAEp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; Tolerance 2% -> 1%
Changed lines of the file:
@@
 F 0 "TH301" H 6475 4650 50  0000 C CNN
 F 1 "10k" H 6450 4550 50  0000 C BNN
-F 2 "dvk-mx8m-bsb:103HT" H 6300 4600 50  0001 C CNN
-F 3 "http://www.semitec-usa.com/pdf/NTCThermistor_HT.pdf" H 6300 4600 50  0001 C CNN
-F 4 "Semitec" H 6300 4600 60  0001 C CNN "MFG Name"
-F 5 "103HT" H 6300 4600 60  0001 C CNN "MFG Part Num"
-F 6 "954-103HT" H 6300 4600 60  0001 C CNN "Distrib PN"
-F 7 "https://www.mouser.com/ProductDetail/Semitec/103HT?qs=sGAEpiMZZMuBd0%252bwiCVS2waoyKMmx3l3pnIFz88T2Ko%3d" H 6300 4600 60  0001 C CNN "Distrib Link"
-F 8 "2%" H 6300 4600 60  0001 C CNN "Tolerance"
-F 9 "https://octopart.com/search?q=semitec%20103ht&start=0" H 6300 4600 60  0001 C CNN "Others"
+F 2 "Resistors_SMD:R_0603" H 6300 4600 50  0001 C CNN
+F 3 "https://industrial.panasonic.com/cdbs/www-data/pdf2/AUA0000/AUA0000AE291.pdf" H 6300 4600 50  0001 C CNN
+F 4 "Panasonic" H 6300 4600 60  0001 C CNN "MFG Name"
+F 5 "ERTJ1VG103FA" H 6300 4600 60  0001 C CNN "MFG Part Num"
+F 6 "ERT-J1VG103FA" H 6300 4600 60  0001 C CNN "Distrib PN"
+F 7 "https://www.arrow.com/en/products/ert-j1vg103fa/panasonic" H 6300 4600 60  0001 C CNN "Distrib Link"
+F 8 "1%" H 6300 4600 60  0001 C CNN "Tolerance"
+F 9 "https://www.mouser.com/ProductDetail/Semitec/103HT?qs=sGAEpiMZZMuBd0%252bwiCVS2waoyKMmx3l3pnIFz88T2Ko%3d" H 6300 4600 60  0001 C CNN "Others"
 	1    6300 4600
 	1    0    0    -1

Commit message: Place and route the battery thermistor circuit, add covered B.Cu pads to the footprints which have thermal exposed pads
Other:
- note removed: "Battery holder gives ~~1mm clearance underneath the battery\nThermistor is 1.1±0.15mm thick, should fit fine with stack-up"
Changed lines of the file:
@@
 	-1   0    0    -1
 $EndComp
-Text Notes 6250 5250 0    60   ~ 0
-Battery holder gives ~~1mm clearance underneath the battery\nThermistor is 1.1±0.15mm thick, should fit fine with stack-up
-Text Notes 6250 5500 0    60   ~ 0
+Text Notes 6300 5400 0    60   ~ 0
 Battery holder seems to fit up to ~~68.88mm long batteries\nneed to test 18650 protected cells which are ~~69.35mm long
 $Comp

Commit message: Update project files to KiCad 5.0.0
Parts:
- BT301: symbol Battery_Cell -> dvk-mx8m-bsb-rescue:Battery_Cell
- C301, C302, C303, C304, C305, C306, C307, C308, C309, C310, C311, C312, C313, C314: symbol C -> dvk-mx8m-bsb-rescue:C
- D301, D302, D304: symbol LED_ALT -> dvk-mx8m-bsb-rescue:LED_ALT
- D303: symbol D_Zener_ALT -> dvk-mx8m-bsb-rescue:D_Zener_ALT
- F301: symbol Polyfuse -> dvk-mx8m-bsb-rescue:Polyfuse
- FB301: symbol Ferrite_Bead -> dvk-mx8m-bsb-rescue:Ferrite_Bead
- JP301: symbol Conn_01x02 -> dvk-mx8m-bsb-rescue:Conn_01x02
- L301: symbol L -> dvk-mx8m-bsb-rescue:L
- Q301: symbol Q_NMOS_GSD -> dvk-mx8m-bsb-rescue:Q_NMOS_GSD
- R301, R302, R303, R304, R305, R306, R307, R308, R309, R310: symbol R -> dvk-mx8m-bsb-rescue:R
- TH301: symbol Thermistor -> dvk-mx8m-bsb-rescue:Thermistor
- U301: symbol BQ25896 -> dvk-mx8m-bsb:BQ25896
Changed lines of the file:
@@
-EESchema Schematic File Version 2
-LIBS:power
-LIBS:device
-LIBS:switches
-LIBS:relays
-LIBS:motors
-LIBS:transistors
-LIBS:conn
-LIBS:linear
-LIBS:regul
-LIBS:74xx
-LIBS:cmos4000
-LIBS:adc-dac
-LIBS:memory
-LIBS:xilinx
-LIBS:microcontrollers
-LIBS:dsp
-LIBS:microchip
-LIBS:analog_switches
-LIBS:motorola
-LIBS:texas
-LIBS:intel
-LIBS:audio
-LIBS:interface
-LIBS:digital-audio
-LIBS:philips
-LIBS:display
-LIBS:cypress
-LIBS:siliconi
-LIBS:opto
-LIBS:atmel
-LIBS:contrib
-LIBS:valves
-LIBS:dvk-mx8m-bsb
+EESchema Schematic File Version 4
 LIBS:dvk-mx8m-bsb-cache
-EELAYER 25 0
+EELAYER 26 0
 EELAYER END
 $Descr A4 11693 8268
@@
 $EndDescr
 $Comp
-L PWR_FLAG #FLG051
+L power:PWR_FLAG #FLG051
 U 1 1 5ACBEC9D
 P 7100 4500
@@
 Vrwm(max)=5.0V\nVbr(min)=6.2V\nPd=150mW
 $Comp
-L Battery_Cell BT301
+L dvk-mx8m-bsb-rescue:Battery_Cell BT301
 U 1 1 5ADAE7AB
 P 7500 4200
@@
 $EndComp
 $Comp
-L C C301
+L dvk-mx8m-bsb-rescue:C C301
 U 1 1 5ADEA19F
 P 4250 2800
@@
 $EndComp
 $Comp
-L GND #PWR052
+L power:GND #PWR052
 U 1 1 5ADEA24E
 P 4250 3000
@@
 $EndComp
 $Comp
-L C C302
+L dvk-mx8m-bsb-rescue:C C302
 U 1 1 5ADEA322
 P 4450 2900
@@
 $EndComp
 $Comp
-L GND #PWR053
+L power:GND #PWR053
 U 1 1 5ADEA329
 P 4450 3100
@@
 $EndComp
 $Comp
-L C C303
+L dvk-mx8m-bsb-rescue:C C303
 U 1 1 5ADFB737
 P 5650 2800
@@
 $EndComp
 $Comp
-L L L301
+L dvk-mx8m-bsb-rescue:L L301
 U 1 1 5ADFB9AB
 P 5900 2600
@@
 $EndComp
 $Comp
-L C C304
+L dvk-mx8m-bsb-rescue:C C304
 U 1 1 5ADFC6C1
 P 5800 3350
@@
 $EndComp
 $Comp
-L GND #PWR054
+L power:GND #PWR054
 U 1 1 5ADFC71C
 P 5800 3550
@@
 $EndComp
 $Comp
-L R R306
+L dvk-mx8m-bsb-rescue:R R306
 U 1 1 5ADFDA10
 P 4350 3450
@@
 $EndComp
 $Comp
-L GND #PWR055
+L power:GND #PWR055
 U 1 1 5ADFDA73
 P 4150 3500
@@
 $EndComp
 $Comp
-L C C308
+L dvk-mx8m-bsb-rescue:C C308
 U 1 1 5AE0040B
 P 7500 2800
@@
 $EndComp
 $Comp
-L GND #PWR056
+L power:GND #PWR056
 U 1 1 5AE01F71
 P 6450 3050
@@
 $EndComp
 $Comp
-L C C309
+L dvk-mx8m-bsb-rescue:C C309
 U 1 1 5AE01FE0
 P 7750 2800
@@
 $EndComp
 $Comp
-L Polyfuse F301
+L dvk-mx8m-bsb-rescue:Polyfuse F301
 U 1 1 5AE34D8A
 P 7100 3900
@@
 $EndComp
 $Comp
-L R R308
+L dvk-mx8m-bsb-rescue:R R308
 U 1 1 5AE3641A
 P 6100 4200
@@
 $EndComp
 $Comp
-L R R307
+L dvk-mx8m-bsb-rescue:R R307
 U 1 1 5AE36487
 P 5900 4600
@@
 $EndComp
 $Comp
-L Thermistor TH301
+L dvk-mx8m-bsb-rescue:Thermistor TH301
 U 1 1 5AE369F4
 P 6300 4600
@@
 $EndComp
 $Comp
-L GND #PWR057
+L power:GND #PWR057
 U 1 1 5AE37872
 P 6100 5050
@@
 EN_SNK
 $Comp
-L VBAT_REG #PWR058
+L dvk-mx8m-bsb:VBAT_REG #PWR058
 U 1 1 5AE5FF35
 P 3400 2950
@@
 $EndComp
 $Comp
-L R R302
+L dvk-mx8m-bsb-rescue:R R302
 U 1 1 5AE61BA6
 P 3400 3500
@@
 $EndComp
 $Comp
-L R R301
+L dvk-mx8m-bsb-rescue:R R301
 U 1 1 5AE62134
 P 3000 3500
@@
 $EndComp
 $Comp
-L LED_ALT D301
+L dvk-mx8m-bsb-rescue:LED_ALT D301
 U 1 1 5AE62EC1
 P 3000 3150
@@
 $EndComp
 $Comp
-L VBAT_REG #PWR059
+L dvk-mx8m-bsb:VBAT_REG #PWR059
 U 1 1 5AE632B4
 P 3000 2950
@@
 $EndComp
 $Comp
-L GND #PWR060
+L power:GND #PWR060
 U 1 1 5AE67B37
 P 7100 4600
@@
 $EndComp
 $Comp
-L Ferrite_Bead FB301
+L dvk-mx8m-bsb-rescue:Ferrite_Bead FB301
 U 1 1 5AE846A8
 P 6900 2600
@@
 $EndComp
 $Comp
-L GND #PWR061
+L power:GND #PWR061
 U 1 1 5AE86DE3
 P 7500 3050
@@
 $EndComp
 $Comp
-L D_Zener_ALT D303
+L dvk-mx8m-bsb-rescue:D_Zener_ALT D303
 U 1 1 5AE86DF6
 P 7250 2800
@@
 reference design: http://www.ti.com/lit/ug/sluuba2b/sluuba2b.pdf
 $Comp
-L PWR_FLAG #FLG062
+L power:PWR_FLAG #FLG062
 U 1 1 5AF16085
 P 7500 2550
@@
 $EndComp
 $Comp
-L PWR_FLAG #FLG063
+L power:PWR_FLAG #FLG063
 U 1 1 5AF1CA20
 P 6400 3850
@@
 $EndComp
 $Comp
-L BQ25896 U301
+L dvk-mx8m-bsb:BQ25896 U301
 U 1 1 5AF31C9D
 P 5050 3600
@@
 $EndComp
 $Comp
-L GND #PWR064
+L power:GND #PWR064
 U 1 1 5AED22FA
 P 3900 5150
@@
  Default LOW:\nadapter source
 $Comp
-L GND #PWR065
+L power:GND #PWR065
 U 1 1 5AF3ADC2
 P 3850 3350
@@
 $EndComp
 $Comp
-L VBUS #PWR066
+L power:VBUS #PWR066
 U 1 1 5AF7190A
 P 4250 2550
@@
 VBAT(DPL)=2.15~~2.5V
 $Comp
-L VBAT #PWR067
+L dvk-mx8m-bsb:VBAT #PWR067
 U 1 1 5AE2587A
 P 6700 3850
@@
 Battery Charge Controller
 $Comp
-L GND #PWR068
+L power:GND #PWR068
 U 1 1 5B0600CE
 P 8700 3050
@@
 ~~110uF
 $Comp
-L R R309
+L dvk-mx8m-bsb-rescue:R R309
 U 1 1 5B0E4134
 P 9550 2600
@@
 $EndComp
 $Comp
-L Conn_01x02 JP301
+L dvk-mx8m-bsb-rescue:Conn_01x02 JP301
 U 1 1 5B0E413B
 P 9500 2150
@@
 	7750 2650 7750 2600
 $Comp
-L C C310
+L dvk-mx8m-bsb-rescue:C C310
 U 1 1 5B1BC001
 P 8200 2800
@@
 $EndComp
 $Comp
-L GND #PWR069
+L power:GND #PWR069
 U 1 1 5BA1BC16
 P 9950 3350
@@
 Connection ~ 9950 2600
 $Comp
-L R R305
+L dvk-mx8m-bsb-rescue:R R305
 U 1 1 5B302D80
 P 4050 3300
@@
 $EndComp
 $Comp
-L R R304
+L dvk-mx8m-bsb-rescue:R R304
 U 1 1 5B2F65C3
 P 3900 4250
@@
 Battery holder seems to fit up to ~~68.88mm long batteries\nneed to test 18650 protected cells which are ~~69.35mm long
 $Comp
-L C C305
+L dvk-mx8m-bsb-rescue:C C305
 U 1 1 5B0BB8A8
 P 6350 2800
@@
 $EndComp
 $Comp
-L C C306
+L dvk-mx8m-bsb-rescue:C C306
 U 1 1 5B0BBD65
 P 6550 2800
@@
 $EndComp
 $Comp
-L C C307
+L dvk-mx8m-bsb-rescue:C C307
 U 1 1 5B0BD3BE
 P 6700 4150
@@
 $EndComp
 $Comp
-L Q_NMOS_GSD Q301
+L dvk-mx8m-bsb-rescue:Q_NMOS_GSD Q301
 U 1 1 5B59770D
 P 3800 4900
@@
 ICHG(default)=REG[6:0]=2048mA (reduce to ~~1.6A [0011001])
 $Comp
-L R R303
+L dvk-mx8m-bsb-rescue:R R303
 U 1 1 5B2725A1
 P 3550 4250
@@
 	3550 4100 3550 4050
 $Comp
-L 3V3_OUT #PWR070
+L dvk-mx8m-bsb:3V3_OUT #PWR070
 U 1 1 5B2BB51D
 P 3550 4050
@@
 	3900 5150 3900 5100
 $Comp
-L 3V3_OUT #PWR071
+L dvk-mx8m-bsb:3V3_OUT #PWR071
 U 1 1 5B2C5C01
 P 3900 4050
@@
 sink current ~~5mA
 $Comp
-L LED_ALT D302
+L dvk-mx8m-bsb-rescue:LED_ALT D302
 U 1 1 5B304940
 P 3400 3150
@@
 $EndComp
 $Comp
-L LED_ALT D304
+L dvk-mx8m-bsb-rescue:LED_ALT D304
 U 1 1 5B3049D4
 P 9950 2800
@@
 $EndComp
 $Comp
-L R R310
+L dvk-mx8m-bsb-rescue:R R310
 U 1 1 5B30501E
 P 9950 3150
@@
 Connection ~ 5600 5000
 $Comp
-L C C311
+L dvk-mx8m-bsb-rescue:C C311
 U 1 1 5B3268DD
 P 8450 2800
@@
 $EndComp
 $Comp
-L C C312
+L dvk-mx8m-bsb-rescue:C C312
 U 1 1 5B326949
 P 8700 2800
@@
 $EndComp
 $Comp
-L C C313
+L dvk-mx8m-bsb-rescue:C C313
 U 1 1 5B3269CC
 P 8950 2800
@@
 $EndComp
 $Comp
-L C C314
+L dvk-mx8m-bsb-rescue:C C314
 U 1 1 5B326A44
 P 9200 2800

Commit message: Update the schematic symbols and footprints after upgrading to KiCad 5.0.0, fix all ERC and DRC violations after the new update/upgrade
Parts:
- BT301: symbol dvk-mx8m-bsb-rescue:Battery_Cell -> Device:Battery_Cell
- C301, C302, C303, C304, C305, C306, C307, C308, C309, C310, C311, C312, C313, C314: footprint Capacitors_SMD:C_0603 -> Capacitor_SMD:C_0603_1608Metric; symbol dvk-mx8m-bsb-rescue:C -> Device:C
- D301, D302, D304: symbol dvk-mx8m-bsb-rescue:LED_ALT -> Device:LED_ALT
- D303: symbol dvk-mx8m-bsb-rescue:D_Zener_ALT -> Device:D_Zener_ALT
- F301: symbol dvk-mx8m-bsb-rescue:Polyfuse -> Device:Polyfuse
- FB301: symbol dvk-mx8m-bsb-rescue:Ferrite_Bead -> Device:Ferrite_Bead
- JP301: footprint Pin_Headers:Pin_Header_Straight_1x02_Pitch2.54mm -> Connector_PinHeader_2.54mm:PinHeader_1x02_P2.54mm_Vertical; symbol dvk-mx8m-bsb-rescue:Conn_01x02 -> Connector_Generic:Conn_01x02
- L301: symbol dvk-mx8m-bsb-rescue:L -> Device:L
- Q301: symbol dvk-mx8m-bsb-rescue:Q_NMOS_GSD -> Device:Q_NMOS_GSD
- R301, R302, R303, R304, R305, R306, R307, R308, R310: footprint Resistors_SMD:R_0603 -> Resistor_SMD:R_0603_1608Metric; symbol dvk-mx8m-bsb-rescue:R -> Device:R
- R309: footprint Resistors_SMD:R_2512 -> Resistor_SMD:R_2512_6332Metric; symbol dvk-mx8m-bsb-rescue:R -> Device:R
- TH301: footprint Resistors_SMD:R_0603 -> Resistor_SMD:R_0603_1608Metric; symbol dvk-mx8m-bsb-rescue:Thermistor -> Device:Thermistor
Connections:
- wire segments 112 -> 157

Commit message: Reduce all 0603 resistor sizes to 0402
Parts:
- R301, R302, R303, R304, R305, R306, R307, R308, R310, TH301: footprint Resistor_SMD:R_0603_1608Metric -> Resistor_SMD:R_0402_1005Metric
Other:
- note added: "Proposed battery: NCR18650B"
- note removed: "NCR18650B meets requirements"
Changed lines of the file:
@@
 F 0 "R306" V 4430 3450 50  0000 C CNN
 F 1 "191" V 4250 3450 50  0000 C CNN
-F 2 "Resistor_SMD:R_0603_1608Metric" V 4280 3450 50  0001 C CNN
+F 2 "Resistor_SMD:R_0402_1005Metric" V 4280 3450 50  0001 C CNN
 F 3 "" H 4350 3450 50  0001 C CNN
 	1    4350 3450
@@
 F 0 "R308" V 6180 4200 50  0000 C CNN
 F 1 "5.23k" V 6000 4200 50  0000 C CNN
-F 2 "Resistor_SMD:R_0603_1608Metric" V 6030 4200 50  0001 C CNN
+F 2 "Resistor_SMD:R_0402_1005Metric" V 6030 4200 50  0001 C CNN
 F 3 "" H 6100 4200 50  0001 C CNN
 	1    6100 4200
@@
 F 0 "R307" H 6050 4650 50  0000 C CNN
 F 1 "30.1k" H 6050 4550 50  0000 C CNN
-F 2 "Resistor_SMD:R_0603_1608Metric" V 5830 4600 50  0001 C CNN
+F 2 "Resistor_SMD:R_0402_1005Metric" V 5830 4600 50  0001 C CNN
 F 3 "" H 5900 4600 50  0001 C CNN
 	1    5900 4600
@@
 F 0 "TH301" H 6475 4650 50  0000 C CNN
 F 1 "10k" H 6450 4550 50  0000 C BNN
-F 2 "Resistor_SMD:R_0603_1608Metric" H 6300 4600 50  0001 C CNN
+F 2 "Resistor_SMD:R_0402_1005Metric" H 6300 4600 50  0001 C CNN
 F 3 "https://industrial.panasonic.com/cdbs/www-data/pdf2/AUA0000/AUA0000AE291.pdf" H 6300 4600 50  0001 C CNN
 F 4 "Panasonic" H 6300 4600 60  0001 C CNN "MFG Name"
@@
 F 0 "R302" H 3550 3550 50  0000 C CNN
 F 1 "2.2k" H 3550 3450 50  0000 C CNN
-F 2 "Resistor_SMD:R_0603_1608Metric" V 3330 3500 50  0001 C CNN
+F 2 "Resistor_SMD:R_0402_1005Metric" V 3330 3500 50  0001 C CNN
 F 3 "" H 3400 3500 50  0001 C CNN
 	1    3400 3500
@@
 F 0 "R301" H 3150 3550 50  0000 C CNN
 F 1 "2.2k" H 3150 3450 50  0000 C CNN
-F 2 "Resistor_SMD:R_0603_1608Metric" V 2930 3500 50  0001 C CNN
+F 2 "Resistor_SMD:R_0402_1005Metric" V 2930 3500 50  0001 C CNN
 F 3 "" H 3000 3500 50  0001 C CNN
 	1    3000 3500
@@
 $EndBitmap
 Text Notes 7850 3475 0    60   ~ 0
-NCR18650B meets requirements
+Proposed battery: NCR18650B
 Text Notes 1300 2700 0    60   ~ 0
 (interpret RSOC% based on this plot)
@@
 F 0 "R305" V 4125 3300 50  0000 C CNN
 F 1 "10k" V 3950 3300 50  0000 C CNN
-F 2 "Resistor_SMD:R_0603_1608Metric" V 3980 3300 50  0001 C CNN
+F 2 "Resistor_SMD:R_0402_1005Metric" V 3980 3300 50  0001 C CNN
 F 3 "https://www.seielect.com/Catalog/SEI-RMCF_RMCP.pdf" H 4050 3300 50  0001 C CNN
 F 4 "Stackpole" H 4050 3300 60  0001 C CNN "MFG Name"
@@
 F 0 "R304" H 4050 4300 50  0000 C CNN
 F 1 "10k" H 4025 4200 50  0000 C CNN
-F 2 "Resistor_SMD:R_0603_1608Metric" V 3830 4250 50  0001 C CNN
+F 2 "Resistor_SMD:R_0402_1005Metric" V 3830 4250 50  0001 C CNN
 F 3 "https://www.seielect.com/Catalog/SEI-RMCF_RMCP.pdf" H 3900 4250 50  0001 C CNN
 F 4 "Stackpole" H 3900 4250 60  0001 C CNN "MFG Name"
@@
 F 0 "R303" H 3700 4300 50  0000 C CNN
 F 1 "10k" H 3675 4200 50  0000 C CNN
-F 2 "Resistor_SMD:R_0603_1608Metric" V 3480 4250 50  0001 C CNN
+F 2 "Resistor_SMD:R_0402_1005Metric" V 3480 4250 50  0001 C CNN
 F 3 "https://www.seielect.com/Catalog/SEI-RMCF_RMCP.pdf" H 3550 4250 50  0001 C CNN
 F 4 "Stackpole" H 3550 4250 60  0001 C CNN "MFG Name"
@@
 F 0 "R310" H 10100 3200 50  0000 C CNN
 F 1 "1.5k" H 10100 3100 50  0000 C CNN
-F 2 "Resistor_SMD:R_0603_1608Metric" V 9880 3150 50  0001 C CNN
+F 2 "Resistor_SMD:R_0402_1005Metric" V 9880 3150 50  0001 C CNN
 F 3 "" H 9950 3150 50  0001 C CNN
 	1    9950 3150
