File: battery.sch (KiCad schematic (older format))
At the start: 36 parts, among them Q301 FDV301N, U301 BQ25896

Commit message: Change all 0603 capacitors _EXCEPT_ the 2.2uF, 4.7uF, 8.2uF, 10uF, and 22uF caps to 0402
Parts:
- C301, C303, C308, C309: footprint Capacitor_SMD:C_0603_1608Metric -> Capacitor_SMD:C_0402_1005Metric
Changed lines of the file:
@@
 F 0 "C301" H 4275 2900 50  0000 L CNN
 F 1 "1uF" H 4275 2700 50  0000 L CNN
-F 2 "Capacitor_SMD:C_0603_1608Metric" H 4288 2650 50  0001 C CNN
+F 2 "Capacitor_SMD:C_0402_1005Metric" H 4288 2650 50  0001 C CNN
 F 3 "" H 4250 2800 50  0001 C CNN
 	1    4250 2800
@@
 F 0 "C303" H 5675 2900 50  0000 L CNN
 F 1 "47nF" H 5675 2700 50  0000 L CNN
-F 2 "Capacitor_SMD:C_0603_1608Metric" H 5688 2650 50  0001 C CNN
+F 2 "Capacitor_SMD:C_0402_1005Metric" H 5688 2650 50  0001 C CNN
 F 3 "" H 5650 2800 50  0001 C CNN
 	1    5650 2800
@@
 F 0 "C308" H 7525 2900 50  0000 L CNN
 F 1 "100nF" H 7500 2700 50  0000 L CNN
-F 2 "Capacitor_SMD:C_0603_1608Metric" H 7538 2650 50  0001 C CNN
+F 2 "Capacitor_SMD:C_0402_1005Metric" H 7538 2650 50  0001 C CNN
 F 3 "" H 7500 2800 50  0001 C CNN
 	1    7500 2800
@@
 F 0 "C309" H 7775 2900 50  0000 L CNN
 F 1 "100nF" H 7775 2700 50  0000 L CNN
-F 2 "Capacitor_SMD:C_0603_1608Metric" H 7788 2650 50  0001 C CNN
+F 2 "Capacitor_SMD:C_0402_1005Metric" H 7788 2650 50  0001 C CNN
 F 3 "" H 7750 2800 50  0001 C CNN
 	1    7750 2800
