File: power.sch (KiCad schematic (older format))
At the start: 94 parts, among them U401 RT8070, U402 MIC2876, U403 MIC5365-2.8, U404 AP22814, U405 AP22814, U406 FT440, U407 PAM2841

Commit message: Rename all diff pairs such that they end in _P/_N rather than just P/N (underscore needed for diff pair routing)
Parts:
- C408: Others https://www.mouser.com/productdetail/?qs=LlFn95tWfDgsujID1P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 -> https://www.mouser.com/productdetail/?qs=LlFn95tWfDgsujID1_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
- L401: Distrib Link https://www.mouser.com/ProductDetail/Coilcraft/XAL4020-102MEC?qs=zCSbvcPd3pbLq0M7ZKfPRA%3D%3D -> https://www.mouser.com/ProductDetail/Coilcraft/XAL4020-102MEC?qs=zCSbvcPD3_PbLq0M7ZKfPRA%3D%3D
Changed lines of the file:
@@
 F 5 "XAL4020-102MEC" V 2500 3600 60  0001 C CNN "MFG Part Num"
 F 6 "994-XAL4020-102MEC" V 2500 3600 60  0001 C CNN "Distrib PN"
-F 7 "https://www.mouser.com/ProductDetail/Coilcraft/XAL4020-102MEC?qs=zCSbvcPd3pbLq0M7ZKfPRA%3D%3D" V 2500 3600 60  0001 C CNN "Distrib Link"
+F 7 "https://www.mouser.com/ProductDetail/Coilcraft/XAL4020-102MEC?qs=zCSbvcPD3_PbLq0M7ZKfPRA%3D%3D" V 2500 3600 60  0001 C CNN "Distrib Link"
 F 8 "-" V 2500 3600 60  0001 C CNN "Tolerance"
 F 9 "https://www.mouser.com/ProductDetail/Coilcraft/XAL4020-102MEB?qs=sGAEpiMZZMsg%252by3WlYCkU2kWFds1hA9Dw%2fxz62COX58%3d" V 2500 3600 60  0001 C CNN "Others"
@@
 F 7 "https://www.digikey.com/product-detail/en/murata-electronics-north-america/GRM188R61A105KA61D/490-1543-1-ND/587782" H 1700 4150 60  0001 C CNN "Distrib Link"
 F 8 "-" H 1700 4150 60  0001 C CNN "Tolerance"
-F 9 "https://www.mouser.com/productdetail/?qs=LlFn95tWfDgsujID1PD8Jw%3D%3D" H 1700 4150 60  0001 C CNN "Others"
+F 9 "https://www.mouser.com/productdetail/?qs=LlFn95tWfDgsujID1_PD8Jw%3D%3D" H 1700 4150 60  0001 C CNN "Others"
 	1    1700 4150
 	-1   0    0    -1

Commit message: Re-route the differential tracks going from the USB-C switch IC to the EMI&TVS ICs along with some of the passives around the USB-C switch chip (similar placement to EmCraft's), add a 1uF cap to the EN pin of the 2.8V LDO in order to introduce a small (~10ms) delay between the 1.8V rail coming up and the 2.8V rail
Parts:
- added C447: 1uF, Capacitors_SMD:C_0603, symbol C
- renumbered C445 to C443, C443 to C444, C444 to C445, C447 to C448, C448 to C449, C449 to C450, C450 to C451, C451 to C452, C452 to C453, C453 to C454, C454 to C455, C455 to C456, C456 to C457, C457 to C458, C458 to C459, C459 to C460, C460 to C461, R413 to R412, R412 to R413
Connections:
- wire segments 242 -> 244
Other:
- moved on the sheet: C443, C451, R412

Commit message: Now using GPIO5_IO03 (P4.03) to put the class-D op-amp in shutdown and conserve energy when muted, make C1716 near the ETH PHY's DVDDL pin 47 220nF instead of 10uF (EmCraft suggested that this should be 100nF but their's is 220nF, asked why), added a 10k pull-down to PAM2841's ENA pin, added a 100nF cap to the smart card's C1 VCC pin, added a 1uF cap to the haptic motor circuit's 3V3_P rail
Still need to use I2C3 instead of I2C1 according to EmCraft's suggestions.
Parts:
- added R415: 10k, Resistors_SMD:R_0603, symbol R
- renumbered R415 to R416, R416 to R417, R417 to R418, R418 to R419
Connections:
- wire segments 244 -> 248
Other:
- moved on the sheet: C456, C457
Changed lines of the file:
@@
 $EndComp
 $Comp
-L R R418
+L R R419
 U 1 1 5B0C354D
 P 10300 1300
-F 0 "R418" V 10380 1300 50  0000 C CNN
+F 0 "R419" V 10380 1300 50  0000 C CNN
 F 1 "NC" V 10200 1300 50  0000 C CNN
 F 2 "Resistors_SMD:R_0805" V 10230 1300 50  0001 C CNN
@@
 L C C456
 U 1 1 5B19DCF4
-P 7750 3650
-F 0 "C456" H 7775 3750 50  0000 L CNN
-F 1 "10uF" H 7775 3550 50  0000 L CNN
-F 2 "Capacitors_SMD:C_0603" H 7788 3500 50  0001 C CNN
-F 3 "" H 7750 3650 50  0001 C CNN
-	1    7750 3650
+P 7700 3650
+F 0 "C456" H 7725 3750 50  0000 L CNN
+F 1 "10uF" H 7725 3550 50  0000 L CNN
+F 2 "Capacitors_SMD:C_0603" H 7738 3500 50  0001 C CNN
+F 3 "" H 7700 3650 50  0001 C CNN
+	1    7700 3650
 	1    0    0    -1
 $EndComp
@@
 L C C457
 U 1 1 5B19DE3D
-P 7750 4250
-F 0 "C457" H 7775 4350 50  0000 L CNN
-F 1 "1uF" H 7775 4150 50  0000 L CNN
-F 2 "Capacitors_SMD:C_0603" H 7788 4100 50  0001 C CNN
-F 3 "" H 7750 4250 50  0001 C CNN
-	1    7750 4250
+P 7700 4250
+F 0 "C457" H 7725 4350 50  0000 L CNN
+F 1 "1uF" H 7725 4150 50  0000 L CNN
+F 2 "Capacitors_SMD:C_0603" H 7738 4100 50  0001 C CNN
+F 3 "" H 7700 4250 50  0001 C CNN
+	1    7700 4250
 	1    0    0    -1
 $EndComp
@@
 L GND #PWR0102
 U 1 1 5B19DF14
-P 7750 3850
-F 0 "#PWR0102" H 7750 3600 50  0001 C CNN
-F 1 "GND" H 7750 3700 50  0000 C CNN
-F 2 "" H 7750 3850 50  0001 C CNN
-F 3 "" H 7750 3850 50  0001 C CNN
-	1    7750 3850
+P 7700 3850
+F 0 "#PWR0102" H 7700 3600 50  0001 C CNN
+F 1 "GND" H 7700 3700 50  0000 C CNN
+F 2 "" H 7700 3850 50  0001 C CNN
+F 3 "" H 7700 3850 50  0001 C CNN
+	1    7700 3850
 	1    0    0    -1
 $EndComp
@@
 L GND #PWR0103
 U 1 1 5B19FE2B
-P 7750 4450
-F 0 "#PWR0103" H 7750 4200 50  0001 C CNN
-F 1 "GND" H 7750 4300 50  0000 C CNN
-F 2 "" H 7750 4450 50  0001 C CNN
-F 3 "" H 7750 4450 50  0001 C CNN
-	1    7750 4450
+P 7700 4450
+F 0 "#PWR0103" H 7700 4200 50  0001 C CNN
+F 1 "GND" H 7700 4300 50  0000 C CNN
+F 2 "" H 7700 4450 50  0001 C CNN
+F 3 "" H 7700 4450 50  0001 C CNN
+	1    7700 4450
 	1    0    0    -1
 $EndComp
@@
 L VBAT_REG #PWR0104
 U 1 1 5B1A0ED2
-P 7750 3400
-F 0 "#PWR0104" H 7750 3250 50  0001 C CNN
-F 1 "VBAT_REG" H 7750 3540 50  0000 C CNN
-F 2 "" H 7750 3400 50  0001 C CNN
-F 3 "" H 7750 3400 50  0001 C CNN
-	1    7750 3400
+P 7700 3400
+F 0 "#PWR0104" H 7700 3250 50  0001 C CNN
+F 1 "VBAT_REG" H 7700 3540 50  0000 C CNN
+F 2 "" H 7700 3400 50  0001 C CNN
+F 3 "" H 7700 3400 50  0001 C CNN
+	1    7700 3400
 	1    0    0    -1
 $EndComp
@@
 $EndComp
 $Comp
-L R R416
+L R R417
 U 1 1 5B1A53A5
 P 10100 3750
-F 0 "R416" H 10250 3800 50  0000 C CNN
+F 0 "R417" H 10250 3800 50  0000 C CNN
 F 1 "910k" H 10250 3700 50  0000 C CNN
 F 2 "Resistors_SMD:R_0603" V 10030 3750 50  0001 C CNN
@@
 $EndComp
 $Comp
-L R R417
+L R R418
 U 1 1 5B1A5A2A
 P 10100 4400
-F 0 "R417" H 10250 4450 50  0000 C CNN
+F 0 "R418" H 10250 4450 50  0000 C CNN
 F 1 "30k" H 10225 4350 50  0000 C CNN
 F 2 "Resistors_SMD:R_0603" V 10030 4400 50  0001 C CNN
@@
 LEDK
 $Comp
-L R R415
+L R R416
 U 1 1 5B1AB6C8
 P 9600 4500
-F 0 "R415" H 9750 4550 50  0000 C CNN
+F 0 "R416" H 9750 4550 50  0000 C CNN
 F 1 "5.1" H 9725 4450 50  0000 C CNN
 F 2 "Resistors_SMD:R_0603" V 9530 4500 50  0001 C CNN
@@
 	1    0    0    -1
 $EndComp
-Text HLabel 8200 4300 0    60   Input ~ 0
+Text HLabel 8150 4300 0    60   Input ~ 0
 PWM
 $Comp
@@
 	1    0    0    -1
 $EndComp
-Text Notes 7650 5350 0    60   ~ 0
+Text Notes 7510 5350 0    60   ~ 0
 Optional:\nif PWR_EN == LOW\nset PWM = LOW (0% duty)
 Text Notes 9650 4700 0    39   ~ 0
@@
 	8200 3800 8250 3800
 Wire Wire Line
-	7750 3850 7750 3800
-Wire Wire Line
-	7750 4100 7750 4050
-Connection ~ 7750 4050
-Wire Wire Line
-	7750 4450 7750 4400
-Wire Wire Line
-	7750 3400 7750 3500
-Connection ~ 7750 3450
+	7700 3850 7700 3800
+Wire Wire Line
+	7700 4100 7700 4050
+Connection ~ 7700 4050
+Wire Wire Line
+	7700 4450 7700 4400
+Wire Wire Line
+	7700 3400 7700 3500
+Connection ~ 7700 3450
 Wire Wire Line
 	9000 3450 9650 3450
@@
 Connection ~ 9600 4300
 Wire Wire Line
-	7600 4050 8250 4050
-Wire Wire Line
-	7600 3450 8700 3450
-Wire Wire Line
-	7600 4050 7600 3450
-Wire Wire Line
-	8200 4300 8250 4300
+	7550 4050 8250 4050
+Wire Wire Line
+	7550 3450 8700 3450
+Wire Wire Line
+	7550 4050 7550 3450
+Wire Wire Line
+	8150 4300 8250 4300
 Connection ~ 10500 3450
 Wire Notes Line
@@
 	5200 6250 5200 6200
 Connection ~ 5200 6200
+$Comp
+L R R415
+U 1 1 5B406431
+P 8000 4750
+F 0 "R415" H 8150 4800 50  0000 C CNN
+F 1 "10k" H 8125 4700 50  0000 C CNN
+F 2 "Resistors_SMD:R_0603" V 7930 4750 50  0001 C CNN
+F 3 "https://www.seielect.com/Catalog/SEI-RMCF_RMCP.pdf" H 8000 4750 50  0001 C CNN
+F 4 "Stackpole" H 8000 4750 60  0001 C CNN "MFG Name"
+F 5 "RMCF0603JG10K0" H 8000 4750 60  0001 C CNN "MFG Part Num"
+F 6 "RMCF0603JG10K0CT-ND" H 8000 4750 60  0001 C CNN "Distrib PN"
+F 7 "https://www.digikey.com/product-detail/en/stackpole-electronics-inc/RMCF0603JG10K0/RMCF0603JG10K0CT-ND/4425128" H 8000 4750 60  0001 C CNN "Distrib Link"
+F 8 "5%" H 8000 4750 60  0001 C CNN "Tolerance"
+F 9 "https://www.digikey.com/products/en/resistors/chip-resistor-surface-mount/52?FV=ffe00034%2C400005%2C1f140000%2Cmu10+kOhms%7C2085&quantity=&ColumnSort=1000011&page=1&pageSize=500" H 8000 4750 60  0001 C CNN "Others"
+	1    8000 4750
+	-1   0    0    -1
+$EndComp
+$Comp
+L GND #PWR0126
+U 1 1 5B40856E
+P 8000 4950
+F 0 "#PWR0126" H 8000 4700 50  0001 C CNN
+F 1 "GND" H 8000 4800 50  0000 C CNN
+F 2 "" H 8000 4950 50  0001 C CNN
+F 3 "" H 8000 4950 50  0001 C CNN
+	1    8000 4950
+	1    0    0    -1
+$EndComp
+Wire Wire Line
+	8000 4600 8000 4400
+Wire Wire Line
+	8000 4400 8200 4400
+Wire Wire Line
+	8200 4400 8200 4300
+Connection ~ 8200 4300
+Wire Wire Line
+	8000 4900 8000 4950
 $EndSCHEMATC

Commit message: Update project files to KiCad 5.0.0
Parts:
- C401, C402, C403, C404, C405, C406, C407, C408, C409, C410, C411, C412, C413, C414, C415, C416, C417, C418, C419, C420, C421, C422, C423, C424, C425, C426, C427, C428, C429, C430, C431, C432, C433, C434, C435, C436, C437, C438, C439, C440, C441, C442, C443, C444, C445, C446, C447, C448, C449, C450, C451, C452, C453, C456, C457, C458, C459, C460, C461: symbol C -> dvk-mx8m-bsb-rescue:C
- C454, C455: symbol CP1 -> dvk-mx8m-bsb-rescue:CP1
- D401: symbol D_Schottky_ALT -> dvk-mx8m-bsb-rescue:D_Schottky_ALT
- JP401, JP402, JP403, JP404: symbol Conn_01x02 -> dvk-mx8m-bsb-rescue:Conn_01x02
- L401, L402, L403, L404: symbol L -> dvk-mx8m-bsb-rescue:L
- R401, R402, R403, R404, R405, R406, R407, R408, R409, R410, R411, R412, R413, R414, R415, R416, R417, R418, R419: symbol R -> dvk-mx8m-bsb-rescue:R
- U401: symbol RT8070 -> dvk-mx8m-bsb:RT8070
- U402: symbol MIC2876 -> dvk-mx8m-bsb:MIC2876
- U403: symbol MIC5365-2.8 -> dvk-mx8m-bsb:MIC5365-2.8
- U404, U405: symbol AP22814 -> dvk-mx8m-bsb:AP22814
- U406: symbol FT440 -> dvk-mx8m-bsb:FT440
- U407: symbol PAM2841 -> dvk-mx8m-bsb:PAM2841

Commit message: Update the schematic symbols and footprints after upgrading to KiCad 5.0.0, fix all ERC and DRC violations after the new update/upgrade
Parts:
- removed C460: 22uF, Capacitors_SMD:C_0805, symbol dvk-mx8m-bsb-rescue:C
- added C460: 22uF, Capacitor_SMD:C_0603_1608Metric, symbol Device:C
- C401, C402, C403, C404, C405, C406, C407, C408, C409, C410, C411, C412, C413, C414, C415, C416, C417, C418, C419, C420, C421, C422, C423, C424, C425, C426, C427, C428, C429, C430, C431, C432, C433, C434, C435, C436, C437, C438, C439, C440, C441, C442, C443, C444, C445, C446, C447, C448, C449, C450, C451, C452, C453, C456, C457, C458, C459, C461: footprint Capacitors_SMD:C_0603 -> Capacitor_SMD:C_0603_1608Metric; symbol dvk-mx8m-bsb-rescue:C -> Device:C
- C454, C455: footprint Capacitors_Tantalum_SMD:CP_Tantalum_Case-D_EIA-7343-31_Reflow -> Capacitor_Tantalum_SMD:CP_EIA-7343-31_Kemet-D; symbol dvk-mx8m-bsb-rescue:CP1 -> Device:CP1
- D401: symbol dvk-mx8m-bsb-rescue:D_Schottky_ALT -> Device:D_Schottky_ALT
- JP401, JP402, JP403, JP404: footprint Pin_Headers:Pin_Header_Straight_1x02_Pitch2.00mm -> Connector_PinHeader_2.00mm:PinHeader_1x02_P2.00mm_Vertical; symbol dvk-mx8m-bsb-rescue:Conn_01x02 -> Connector_Generic:Conn_01x02
- L401, L402, L403, L404: symbol dvk-mx8m-bsb-rescue:L -> Device:L
- R401, R402, R403, R404, R405, R406, R407, R408, R409, R410, R412, R415, R416, R417, R418: footprint Resistors_SMD:R_0603 -> Resistor_SMD:R_0603_1608Metric; symbol dvk-mx8m-bsb-rescue:R -> Device:R
- R411, R413, R414: footprint Resistors_SMD:R_1206 -> Resistor_SMD:R_1206_3216Metric; symbol dvk-mx8m-bsb-rescue:R -> Device:R
- R419: footprint Resistors_SMD:R_0805 -> Resistor_SMD:R_0805_2012Metric; symbol dvk-mx8m-bsb-rescue:R -> Device:R
Connections:
- wire segments 248 -> 380

Commit message: Reduce all 0603 resistor sizes to 0402
Parts:
- R401, R402, R403, R404, R405, R406, R407, R408, R409, R410, R412, R415, R416, R417, R418: footprint Resistor_SMD:R_0603_1608Metric -> Resistor_SMD:R_0402_1005Metric
Changed lines of the file:
@@
 F 0 "R406" H 3600 1550 50  0000 C CNN
 F 1 "75k" H 3600 1450 50  0000 C CNN
-F 2 "Resistor_SMD:R_0603_1608Metric" V 3380 1500 50  0001 C CNN
+F 2 "Resistor_SMD:R_0402_1005Metric" V 3380 1500 50  0001 C CNN
 F 3 "" H 3450 1500 50  0001 C CNN
 	1    3450 1500
@@
 F 0 "R407" H 3600 1950 50  0000 C CNN
 F 1 "24k" H 3600 1850 50  0000 C CNN
-F 2 "Resistor_SMD:R_0603_1608Metric" V 3380 1900 50  0001 C CNN
+F 2 "Resistor_SMD:R_0402_1005Metric" V 3380 1900 50  0001 C CNN
 F 3 "" H 3450 1900 50  0001 C CNN
 	1    3450 1900
@@
 F 0 "R405" V 2980 1800 50  0000 C CNN
 F 1 "33k" V 2900 1800 50  0000 C CNN
-F 2 "Resistor_SMD:R_0603_1608Metric" V 2830 1800 50  0001 C CNN
+F 2 "Resistor_SMD:R_0402_1005Metric" V 2830 1800 50  0001 C CNN
 F 3 "" H 2900 1800 50  0001 C CNN
 	1    2900 1800
@@
 F 0 "R403" V 1580 2000 50  0000 C CNN
 F 1 "300k" V 1500 2000 50  0000 C CNN
-F 2 "Resistor_SMD:R_0603_1608Metric" V 1430 2000 50  0001 C CNN
+F 2 "Resistor_SMD:R_0402_1005Metric" V 1430 2000 50  0001 C CNN
 F 3 "" H 1500 2000 50  0001 C CNN
 	1    1500 2000
@@
 F 0 "R401" H 1000 1750 50  0000 C CNN
 F 1 "1M" H 1050 1850 50  0000 C CNN
-F 2 "Resistor_SMD:R_0603_1608Metric" V 1080 1800 50  0001 C CNN
+F 2 "Resistor_SMD:R_0402_1005Metric" V 1080 1800 50  0001 C CNN
 F 3 "" H 1150 1800 50  0001 C CNN
 	1    1150 1800
@@
 F 0 "R409" H 4050 4200 50  0000 C CNN
 F 1 "910k" H 4050 4100 50  0000 C CNN
-F 2 "Resistor_SMD:R_0603_1608Metric" V 3830 4150 50  0001 C CNN
+F 2 "Resistor_SMD:R_0402_1005Metric" V 3830 4150 50  0001 C CNN
 F 3 "" H 3900 4150 50  0001 C CNN
 	1    3900 4150
@@
 F 0 "R410" H 4050 4600 50  0000 C CNN
 F 1 "200k" H 4050 4500 50  0000 C CNN
-F 2 "Resistor_SMD:R_0603_1608Metric" V 3830 4550 50  0001 C CNN
+F 2 "Resistor_SMD:R_0402_1005Metric" V 3830 4550 50  0001 C CNN
 F 3 "" H 3900 4550 50  0001 C CNN
 	1    3900 4550
@@
 F 0 "R408" V 3580 4200 50  0000 C CNN
 F 1 "1M" V 3500 4200 50  0000 C CNN
-F 2 "Resistor_SMD:R_0603_1608Metric" V 3430 4200 50  0001 C CNN
+F 2 "Resistor_SMD:R_0402_1005Metric" V 3430 4200 50  0001 C CNN
 F 3 "" H 3500 4200 50  0001 C CNN
 	1    3500 4200
@@
 F 0 "R404" H 2350 4200 50  0000 C CNN
 F 1 "1M" H 2300 4100 50  0000 C CNN
-F 2 "Resistor_SMD:R_0603_1608Metric" V 2130 4150 50  0001 C CNN
+F 2 "Resistor_SMD:R_0402_1005Metric" V 2130 4150 50  0001 C CNN
 F 3 "" H 2200 4150 50  0001 C CNN
 	1    2200 4150
@@
 F 0 "R402" H 1600 1500 50  0000 C CNN
 F 1 "NC" H 1550 1600 50  0000 C CNN
-F 2 "Resistor_SMD:R_0603_1608Metric" V 1380 1550 50  0001 C CNN
+F 2 "Resistor_SMD:R_0402_1005Metric" V 1380 1550 50  0001 C CNN
 F 3 "" H 1450 1550 50  0001 C CNN
 	1    1450 1550
@@
 F 0 "R417" H 10250 3800 50  0000 C CNN
 F 1 "910k" H 10250 3700 50  0000 C CNN
-F 2 "Resistor_SMD:R_0603_1608Metric" V 10030 3750 50  0001 C CNN
+F 2 "Resistor_SMD:R_0402_1005Metric" V 10030 3750 50  0001 C CNN
 F 3 "" H 10100 3750 50  0001 C CNN
 	1    10100 3750
@@
 F 0 "R418" H 10250 4450 50  0000 C CNN
 F 1 "30k" H 10225 4350 50  0000 C CNN
-F 2 "Resistor_SMD:R_0603_1608Metric" V 10030 4400 50  0001 C CNN
+F 2 "Resistor_SMD:R_0402_1005Metric" V 10030 4400 50  0001 C CNN
 F 3 "" H 10100 4400 50  0001 C CNN
 	1    10100 4400
@@
 F 0 "R416" H 9750 4550 50  0000 C CNN
 F 1 "5.1" H 9725 4450 50  0000 C CNN
-F 2 "Resistor_SMD:R_0603_1608Metric" V 9530 4500 50  0001 C CNN
+F 2 "Resistor_SMD:R_0402_1005Metric" V 9530 4500 50  0001 C CNN
 F 3 "http://www.yageo.com/documents/recent/PYu-RT_1-to-0.01_RoHS_L_9.pdf" H 9600 4500 50  0001 C CNN
 F 4 "Yageo" H 9600 4500 60  0001 C CNN "MFG Name"
@@
 F 0 "R412" V 5100 6200 50  0000 C CNN
 F 1 "10k" V 5000 6200 50  0000 C CNN
-F 2 "Resistor_SMD:R_0603_1608Metric" V 4930 6200 50  0001 C CNN
+F 2 "Resistor_SMD:R_0402_1005Metric" V 4930 6200 50  0001 C CNN
 F 3 "https://www.seielect.com/Catalog/SEI-RMCF_RMCP.pdf" H 5000 6200 50  0001 C CNN
 F 4 "Stackpole" H 5000 6200 60  0001 C CNN "MFG Name"
@@
 F 0 "R415" H 8150 4800 50  0000 C CNN
 F 1 "10k" H 8125 4700 50  0000 C CNN
-F 2 "Resistor_SMD:R_0603_1608Metric" V 7930 4750 50  0001 C CNN
+F 2 "Resistor_SMD:R_0402_1005Metric" V 7930 4750 50  0001 C CNN
 F 3 "https://www.seielect.com/Catalog/SEI-RMCF_RMCP.pdf" H 8000 4750 50  0001 C CNN
 F 4 "Stackpole" H 8000 4750 60  0001 C CNN "MFG Name"

Commit message: Change all 0603 capacitors _EXCEPT_ the 2.2uF, 4.7uF, 8.2uF, 10uF, and 22uF caps to 0402
Parts:
- C401, C402, C403, C404, C405, C406, C408, C409, C410, C411, C413, C414, C415, C416, C417, C418, C419, C420, C421, C422, C423, C424, C425, C426, C427, C428, C429, C430, C431, C432, C433, C434, C435, C436, C438, C440, C443, C447, C449, C450, C451, C452, C453, C457, C459, C461: footprint Capacitor_SMD:C_0603_1608Metric -> Capacitor_SMD:C_0402_1005Metric
