File: gnss.sch (KiCad schematic (older format))
At the start: 13 parts, among them U2301 MAX-M8Q

Commit message: Update project files to KiCad 5.0.0
Parts:
- AE2301: symbol Antenna_Chip -> dvk-mx8m-bsb:Antenna_Chip
- C2301, C2302, C2303, C2304, C2305, C2306, C2307: symbol C -> dvk-mx8m-bsb-rescue:C
- FB2301: symbol Ferrite_Bead -> dvk-mx8m-bsb-rescue:Ferrite_Bead
- L2301, L2302: symbol L -> dvk-mx8m-bsb-rescue:L
- R2301: symbol R -> dvk-mx8m-bsb-rescue:R
- U2301: symbol MAX-M8 -> dvk-mx8m-bsb:MAX-M8
Changed lines of the file:
@@
-EESchema Schematic File Version 2
-LIBS:power
-LIBS:device
-LIBS:switches
-LIBS:relays
-LIBS:motors
-LIBS:transistors
-LIBS:conn
-LIBS:linear
-LIBS:regul
-LIBS:74xx
-LIBS:cmos4000
-LIBS:adc-dac
-LIBS:memory
-LIBS:xilinx
-LIBS:microcontrollers
-LIBS:dsp
-LIBS:microchip
-LIBS:analog_switches
-LIBS:motorola
-LIBS:texas
-LIBS:intel
-LIBS:audio
-LIBS:interface
-LIBS:digital-audio
-LIBS:philips
-LIBS:display
-LIBS:cypress
-LIBS:siliconi
-LIBS:opto
-LIBS:atmel
-LIBS:contrib
-LIBS:valves
-LIBS:dvk-mx8m-bsb
+EESchema Schematic File Version 4
 LIBS:dvk-mx8m-bsb-cache
-EELAYER 25 0
+EELAYER 26 0
 EELAYER END
 $Descr A4 11693 8268
@@
 $EndDescr
 $Comp
-L GND #PWR0389
+L power:GND #PWR0389
 U 1 1 5B0E0D78
 P 4800 4700
@@
 NoConn ~ 6150 4450
 $Comp
-L C C2301
+L dvk-mx8m-bsb-rescue:C C2301
 U 1 1 5B0ED9E5
 P 3900 3750
@@
 $EndComp
 $Comp
-L GND #PWR0390
+L power:GND #PWR0390
 U 1 1 5B0EDAF7
 P 3900 4000
@@
 Connection ~ 4800 3550
 $Comp
-L C C2302
+L dvk-mx8m-bsb-rescue:C C2302
 U 1 1 5B1028D6
 P 4150 3750
@@
 $EndComp
 $Comp
-L C C2303
+L dvk-mx8m-bsb-rescue:C C2303
 U 1 1 5B102929
 P 4400 3750
@@
 $EndComp
 $Comp
-L C C2304
+L dvk-mx8m-bsb-rescue:C C2304
 U 1 1 5B1029AE
 P 4650 3750
@@
 UART3_TXD
 $Comp
-L Antenna_Chip AE2301
+L dvk-mx8m-bsb:Antenna_Chip AE2301
 U 1 1 5B123EED
 P 7900 2100
@@
 $EndComp
 $Comp
-L GND #PWR0391
+L power:GND #PWR0391
 U 1 1 5B12431F
 P 8000 2350
@@
 	7350 3450 7300 3450
 $Comp
-L L L2301
+L dvk-mx8m-bsb-rescue:L L2301
 U 1 1 5B103CD2
 P 7150 3450
@@
 	6950 3850 6950 3800
 $Comp
-L GND #PWR0392
+L power:GND #PWR0392
 U 1 1 5B103EA0
 P 6950 3850
@@
 	6900 3450 7000 3450
 $Comp
-L C C2305
+L dvk-mx8m-bsb-rescue:C C2305
 U 1 1 5B103D07
 P 6950 3650
@@
 $EndComp
 $Comp
-L R R2301
+L dvk-mx8m-bsb-rescue:R R2301
 U 1 1 5B103CA5
 P 6750 3450
@@
 33nH\n22pF\n10Ω
 $Comp
-L L L2302
+L dvk-mx8m-bsb-rescue:L L2302
 U 1 1 5B2088FC
 P 7700 2800
@@
 	7500 3200 7500 3150
 $Comp
-L GND #PWR0393
+L power:GND #PWR0393
 U 1 1 5B208BC0
 P 7500 3200
@@
 $EndComp
 $Comp
-L C C2306
+L dvk-mx8m-bsb-rescue:C C2306
 U 1 1 5B208BC6
 P 7500 3000
@@
 	7900 3200 7900 3150
 $Comp
-L GND #PWR0394
+L power:GND #PWR0394
 U 1 1 5B208DA1
 P 7900 3200
@@
 $EndComp
 $Comp
-L C C2307
+L dvk-mx8m-bsb-rescue:C C2307
 U 1 1 5B208DA7
 P 7900 3000
@@
 GNSS
 $Comp
-L MAX-M8 U2301
+L dvk-mx8m-bsb:MAX-M8 U2301
 U 1 1 5B0DFDBF
 P 5500 3950
@@
 $EndComp
 $Comp
-L 3V3_P #PWR0395
+L dvk-mx8m-bsb:3V3_P #PWR0395
 U 1 1 5B259E98
 P 3900 2850
@@
 $EndComp
 $Comp
-L Ferrite_Bead FB2301
+L dvk-mx8m-bsb-rescue:Ferrite_Bead FB2301
 U 1 1 5B2B7A3D
 P 3900 3050
@@
 	3900 2900 3900 2850
 $Comp
-L PWR_FLAG #FLG0396
+L power:PWR_FLAG #FLG0396
 U 1 1 5B2B7FC5
 P 4800 3100

Commit message: Update the schematic symbols and footprints after upgrading to KiCad 5.0.0, fix all ERC and DRC violations after the new update/upgrade
Parts:
- C2301, C2302, C2303, C2304, C2305, C2306, C2307: footprint Capacitors_SMD:C_0603 -> Capacitor_SMD:C_0603_1608Metric; symbol dvk-mx8m-bsb-rescue:C -> Device:C
- FB2301: symbol dvk-mx8m-bsb-rescue:Ferrite_Bead -> Device:Ferrite_Bead
- L2301, L2302: footprint Inductors_SMD:L_0603 -> Inductor_SMD:L_0603_1608Metric; symbol dvk-mx8m-bsb-rescue:L -> Device:L
- R2301: footprint Resistors_SMD:R_0603 -> Resistor_SMD:R_0603_1608Metric; symbol dvk-mx8m-bsb-rescue:R -> Device:R
Changed lines of the file:
@@
 Sheet 23 24
 Title "GNSS"
-Date "2018-06-18"
+Date "2018-07-17"
 Rev "v0.1.0"
 Comp "Copyright 2018 GNU GPLv3"
@@
 NoConn ~ 6150 4450
 $Comp
-L dvk-mx8m-bsb-rescue:C C2301
+L Device:C C2301
 U 1 1 5B0ED9E5
 P 3900 3750
 F 0 "C2301" H 3925 3850 50  0000 L CNN
 F 1 "100nF" H 3925 3650 50  0000 L CNN
-F 2 "Capacitors_SMD:C_0603" H 3938 3600 50  0001 C CNN
+F 2 "Capacitor_SMD:C_0603_1608Metric" H 3938 3600 50  0001 C CNN
 F 3 "" H 3900 3750 50  0001 C CNN
 	1    3900 3750
@@
 Connection ~ 4800 3550
 $Comp
-L dvk-mx8m-bsb-rescue:C C2302
+L Device:C C2302
 U 1 1 5B1028D6
 P 4150 3750
 F 0 "C2302" H 4150 3850 50  0000 L CNN
 F 1 "10nF" H 4175 3650 50  0000 L CNN
-F 2 "Capacitors_SMD:C_0603" H 4188 3600 50  0001 C CNN
+F 2 "Capacitor_SMD:C_0603_1608Metric" H 4188 3600 50  0001 C CNN
 F 3 "" H 4150 3750 50  0001 C CNN
 	1    4150 3750
@@
 $EndComp
 $Comp
-L dvk-mx8m-bsb-rescue:C C2303
+L Device:C C2303
 U 1 1 5B102929
 P 4400 3750
 F 0 "C2303" H 4400 3850 50  0000 L CNN
 F 1 "1nF" H 4425 3650 50  0000 L CNN
-F 2 "Capacitors_SMD:C_0603" H 4438 3600 50  0001 C CNN
+F 2 "Capacitor_SMD:C_0603_1608Metric" H 4438 3600 50  0001 C CNN
 F 3 "" H 4400 3750 50  0001 C CNN
 	1    4400 3750
@@
 $EndComp
 $Comp
-L dvk-mx8m-bsb-rescue:C C2304
+L Device:C C2304
 U 1 1 5B1029AE
 P 4650 3750
 F 0 "C2304" H 4650 3850 50  0000 L CNN
 F 1 "100pF" H 4650 3650 50  0000 L CNN
-F 2 "Capacitors_SMD:C_0603" H 4688 3600 50  0001 C CNN
+F 2 "Capacitor_SMD:C_0603_1608Metric" H 4688 3600 50  0001 C CNN
 F 3 "" H 4650 3750 50  0001 C CNN
 	1    4650 3750
@@
 	7350 3450 7300 3450
 $Comp
-L dvk-mx8m-bsb-rescue:L L2301
+L Device:L L2301
 U 1 1 5B103CD2
 P 7150 3450
 F 0 "L2301" V 7225 3450 50  0000 C CNN
 F 1 "NC" V 7105 3450 50  0000 C CNN
-F 2 "Inductors_SMD:L_0603" H 7150 3450 50  0001 C CNN
+F 2 "Inductor_SMD:L_0603_1608Metric" H 7150 3450 50  0001 C CNN
 F 3 "" H 7150 3450 50  0001 C CNN
 	1    7150 3450
@@
 	6900 3450 7000 3450
 $Comp
-L dvk-mx8m-bsb-rescue:C C2305
+L Device:C C2305
 U 1 1 5B103D07
 P 6950 3650
 F 0 "C2305" H 6975 3735 50  0000 L CNN
 F 1 "NC" H 6975 3550 50  0000 L CNN
-F 2 "Capacitors_SMD:C_0603" H 6988 3500 50  0001 C CNN
+F 2 "Capacitor_SMD:C_0603_1608Metric" H 6988 3500 50  0001 C CNN
 F 3 "" H 6950 3650 50  0001 C CNN
 	1    6950 3650
@@
 $EndComp
 $Comp
-L dvk-mx8m-bsb-rescue:R R2301
+L Device:R R2301
 U 1 1 5B103CA5
 P 6750 3450
 F 0 "R2301" V 6830 3450 50  0000 C CNN
 F 1 "NC" V 6650 3450 50  0000 C CNN
-F 2 "Resistors_SMD:R_0603" V 6680 3450 50  0001 C CNN
+F 2 "Resistor_SMD:R_0603_1608Metric" V 6680 3450 50  0001 C CNN
 F 3 "" H 6750 3450 50  0001 C CNN
 	1    6750 3450
@@
 33nH\n22pF\n10Ω
 $Comp
-L dvk-mx8m-bsb-rescue:L L2302
+L Device:L L2302
 U 1 1 5B2088FC
 P 7700 2800
 F 0 "L2302" V 7775 2800 50  0000 C CNN
 F 1 "NC" V 7655 2800 50  0000 C CNN
-F 2 "Inductors_SMD:L_0603" H 7700 2800 50  0001 C CNN
+F 2 "Inductor_SMD:L_0603_1608Metric" H 7700 2800 50  0001 C CNN
 F 3 "" H 7700 2800 50  0001 C CNN
 	1    7700 2800
@@
 $EndComp
 $Comp
-L dvk-mx8m-bsb-rescue:C C2306
+L Device:C C2306
 U 1 1 5B208BC6
 P 7500 3000
 F 0 "C2306" H 7525 3085 50  0000 L CNN
 F 1 "NC" H 7525 2900 50  0000 L CNN
-F 2 "Capacitors_SMD:C_0603" H 7538 2850 50  0001 C CNN
+F 2 "Capacitor_SMD:C_0603_1608Metric" H 7538 2850 50  0001 C CNN
 F 3 "" H 7500 3000 50  0001 C CNN
 	1    7500 3000
@@
 $EndComp
 $Comp
-L dvk-mx8m-bsb-rescue:C C2307
+L Device:C C2307
 U 1 1 5B208DA7
 P 7900 3000
 F 0 "C2307" H 7925 3085 50  0000 L CNN
 F 1 "NC" H 7925 2900 50  0000 L CNN
-F 2 "Capacitors_SMD:C_0603" H 7938 2850 50  0001 C CNN
+F 2 "Capacitor_SMD:C_0603_1608Metric" H 7938 2850 50  0001 C CNN
 F 3 "" H 7900 3000 50  0001 C CNN
 	1    7900 3000
@@
 $EndComp
 $Comp
-L dvk-mx8m-bsb-rescue:Ferrite_Bead FB2301
+L Device:Ferrite_Bead FB2301
 U 1 1 5B2B7A3D
 P 3900 3050

Commit message: Reduce all 0603 resistor sizes to 0402
Parts:
- R2301: footprint Resistor_SMD:R_0603_1608Metric -> Resistor_SMD:R_0402_1005Metric
Changed lines of the file:
@@
 F 0 "R2301" V 6830 3450 50  0000 C CNN
 F 1 "NC" V 6650 3450 50  0000 C CNN
-F 2 "Resistor_SMD:R_0603_1608Metric" V 6680 3450 50  0001 C CNN
+F 2 "Resistor_SMD:R_0402_1005Metric" V 6680 3450 50  0001 C CNN
 F 3 "" H 6750 3450 50  0001 C CNN
 	1    6750 3450

Commit message: Change all 0603 capacitors _EXCEPT_ the 2.2uF, 4.7uF, 8.2uF, 10uF, and 22uF caps to 0402
Parts:
- C2301, C2302, C2303, C2304, C2305, C2306, C2307: footprint Capacitor_SMD:C_0603_1608Metric -> Capacitor_SMD:C_0402_1005Metric
Changed lines of the file:
@@
 F 0 "C2301" H 3925 3850 50  0000 L CNN
 F 1 "100nF" H 3925 3650 50  0000 L CNN
-F 2 "Capacitor_SMD:C_0603_1608Metric" H 3938 3600 50  0001 C CNN
+F 2 "Capacitor_SMD:C_0402_1005Metric" H 3938 3600 50  0001 C CNN
 F 3 "" H 3900 3750 50  0001 C CNN
 	1    3900 3750
@@
 F 0 "C2302" H 4150 3850 50  0000 L CNN
 F 1 "10nF" H 4175 3650 50  0000 L CNN
-F 2 "Capacitor_SMD:C_0603_1608Metric" H 4188 3600 50  0001 C CNN
+F 2 "Capacitor_SMD:C_0402_1005Metric" H 4188 3600 50  0001 C CNN
 F 3 "" H 4150 3750 50  0001 C CNN
 	1    4150 3750
@@
 F 0 "C2303" H 4400 3850 50  0000 L CNN
 F 1 "1nF" H 4425 3650 50  0000 L CNN
-F 2 "Capacitor_SMD:C_0603_1608Metric" H 4438 3600 50  0001 C CNN
+F 2 "Capacitor_SMD:C_0402_1005Metric" H 4438 3600 50  0001 C CNN
 F 3 "" H 4400 3750 50  0001 C CNN
 	1    4400 3750
@@
 F 0 "C2304" H 4650 3850 50  0000 L CNN
 F 1 "100pF" H 4650 3650 50  0000 L CNN
-F 2 "Capacitor_SMD:C_0603_1608Metric" H 4688 3600 50  0001 C CNN
+F 2 "Capacitor_SMD:C_0402_1005Metric" H 4688 3600 50  0001 C CNN
 F 3 "" H 4650 3750 50  0001 C CNN
 	1    4650 3750
@@
 F 0 "C2305" H 6975 3735 50  0000 L CNN
 F 1 "NC" H 6975 3550 50  0000 L CNN
-F 2 "Capacitor_SMD:C_0603_1608Metric" H 6988 3500 50  0001 C CNN
+F 2 "Capacitor_SMD:C_0402_1005Metric" H 6988 3500 50  0001 C CNN
 F 3 "" H 6950 3650 50  0001 C CNN
 	1    6950 3650
@@
 F 0 "C2306" H 7525 3085 50  0000 L CNN
 F 1 "NC" H 7525 2900 50  0000 L CNN
-F 2 "Capacitor_SMD:C_0603_1608Metric" H 7538 2850 50  0001 C CNN
+F 2 "Capacitor_SMD:C_0402_1005Metric" H 7538 2850 50  0001 C CNN
 F 3 "" H 7500 3000 50  0001 C CNN
 	1    7500 3000
@@
 F 0 "C2307" H 7925 3085 50  0000 L CNN
 F 1 "NC" H 7925 2900 50  0000 L CNN
-F 2 "Capacitor_SMD:C_0603_1608Metric" H 7938 2850 50  0001 C CNN
+F 2 "Capacitor_SMD:C_0402_1005Metric" H 7938 2850 50  0001 C CNN
 F 3 "" H 7900 3000 50  0001 C CNN
 	1    7900 3000

Commit message: Place and route the GNSS antenna and its feedline, re-calculate the coplanar waveguide to 50Ohms using EmCraft's baseboard parameters (include new calculations), make the M.2 mounting hole connect to GND and use the recommended size for the hole's dimensions
Parts:
- L2301, L2302: footprint Inductor_SMD:L_0603_1608Metric -> Inductor_SMD:L_0402_1005Metric
Connections:
- wire segments 37 -> 55
Changed lines of the file:
@@
 3.4dBic
 Wire Wire Line
-	3900 3550 4850 3550
-Wire Wire Line
-	3900 3250 4850 3250
+	3900 3550 4150 3550
+Wire Wire Line
+	3900 3250 4800 3250
 Connection ~ 3900 3250
 Wire Wire Line
@@
 Connection ~ 3900 3550
 Wire Wire Line
-	3900 3900 3900 4000
+	3900 3900 3900 3950
 NoConn ~ 6150 3950
 NoConn ~ 6150 4050
@@
 $EndComp
 Wire Wire Line
-	3900 3950 4650 3950
+	3900 3950 4150 3950
 Wire Wire Line
 	4650 3950 4650 3900
@@
 	6150 3750 6200 3750
 Wire Wire Line
-	4800 4450 4800 4700
+	4800 4450 4800 4550
 NoConn ~ 6150 4550
 Text HLabel 6200 3650 2    60   Output ~ 0
@@
 	8000 2350 8000 2300
 Wire Wire Line
-	7900 2300 7900 2850
+	7900 2300 7900 2650
 NoConn ~ 7350 3450
 Wire Wire Line
@@
 F 0 "L2301" V 7225 3450 50  0000 C CNN
 F 1 "NC" V 7105 3450 50  0000 C CNN
-F 2 "Inductor_SMD:L_0603_1608Metric" H 7150 3450 50  0001 C CNN
+F 2 "Inductor_SMD:L_0402_1005Metric" H 7150 3450 50  0001 C CNN
 F 3 "" H 7150 3450 50  0001 C CNN
 	1    7150 3450
@@
 $EndComp
 Wire Wire Line
-	6900 3450 7000 3450
+	6900 3450 6950 3450
 $Comp
 L Device:C C2305
@@
 F 0 "L2302" V 7775 2800 50  0000 C CNN
 F 1 "NC" V 7655 2800 50  0000 C CNN
-F 2 "Inductor_SMD:L_0603_1608Metric" H 7700 2800 50  0001 C CNN
+F 2 "Inductor_SMD:L_0402_1005Metric" H 7700 2800 50  0001 C CNN
 F 3 "" H 7700 2800 50  0001 C CNN
 	1    7700 2800
@@
 	7350 3250 7350 2800
 Wire Wire Line
-	7350 2800 7550 2800
-Wire Wire Line
-	7500 2650 7500 2850
+	7350 2800 7500 2800
+Wire Wire Line
+	7500 2650 7500 2800
 Connection ~ 7500 2800
 Wire Wire Line
@@
 $EndComp
 Wire Wire Line
-	3900 3200 3900 3600
+	3900 3200 3900 3250
 Wire Wire Line
 	3900 2900 3900 2850
@@
 	4800 3100 4800 3250
 Connection ~ 4800 3250
+Wire Wire Line
+	4800 4550 4800 4650
+Wire Wire Line
+	4800 4650 4800 4700
+Wire Wire Line
+	3900 3250 3900 3350
+Wire Wire Line
+	3900 3350 3900 3550
+Wire Wire Line
+	3900 3550 3900 3600
+Wire Wire Line
+	4800 3550 4850 3550
+Wire Wire Line
+	3900 3950 3900 4000
+Wire Wire Line
+	4400 3950 4650 3950
+Wire Wire Line
+	4150 3950 4400 3950
+Wire Wire Line
+	4150 3550 4400 3550
+Wire Wire Line
+	4400 3550 4650 3550
+Wire Wire Line
+	4650 3550 4800 3550
+Wire Wire Line
+	6950 3450 7000 3450
+Wire Wire Line
+	7500 2800 7550 2800
+Wire Wire Line
+	7500 2800 7500 2850
+Wire Wire Line
+	7900 2800 7900 2850
+Wire Wire Line
+	7900 2650 7900 2800
+Wire Wire Line
+	4800 3250 4850 3250
 $EndSCHEMATC
