File: dsi.sch (KiCad schematic (older format))
At the start: 20 parts, among them J1201 Touch, J1202 LCD, Q1201 FDV301N, Q1202 FDV301N

Commit message: Use I2C3 bus instead of I2C1 bus based on EmCraft's feedback
Connections:
- net labels added: I2C3_SCL_1V8, I2C3_SDA_1V8
- net labels removed: I2C1_SCL_1V8, I2C1_SDA_1V8
Changed lines of the file:
@@
 D3_N
 Text HLabel 5500 3500 0    60   BiDi ~ 0
-I2C1_SDA_1V8
+I2C3_SDA_1V8
 Text HLabel 5500 3400 0    60   Input ~ 0
-I2C1_SCL_1V8
+I2C3_SCL_1V8
 Text HLabel 3550 3600 0    60   Output ~ 0
 CAPTOUCH_~INT

Commit message: Update project files to KiCad 5.0.0
Parts:
- C1201, C1202, C1203, C1204, C1205, C1206, C1207, C1208, C1209, C1210: symbol C -> dvk-mx8m-bsb-rescue:C
- DISP1201: symbol Display_JH057N00900 -> dvk-mx8m-bsb:Display_JH057N00900
- J1201: symbol Conn_01x06 -> dvk-mx8m-bsb-rescue:Conn_01x06
- J1202: symbol Conn_01x39 -> dvk-mx8m-bsb-rescue:Conn_01x39
- Q1201, Q1202: symbol Q_NMOS_GSD -> dvk-mx8m-bsb-rescue:Q_NMOS_GSD
- R1201, R1202, R1203, R1204, R1205: symbol R -> dvk-mx8m-bsb-rescue:R
Changed lines of the file:
@@
-EESchema Schematic File Version 2
-LIBS:power
-LIBS:device
-LIBS:switches
-LIBS:relays
-LIBS:motors
-LIBS:transistors
-LIBS:conn
-LIBS:linear
-LIBS:regul
-LIBS:74xx
-LIBS:cmos4000
-LIBS:adc-dac
-LIBS:memory
-LIBS:xilinx
-LIBS:microcontrollers
-LIBS:dsp
-LIBS:microchip
-LIBS:analog_switches
-LIBS:motorola
-LIBS:texas
-LIBS:intel
-LIBS:audio
-LIBS:interface
-LIBS:digital-audio
-LIBS:philips
-LIBS:display
-LIBS:cypress
-LIBS:siliconi
-LIBS:opto
-LIBS:atmel
-LIBS:contrib
-LIBS:valves
-LIBS:dvk-mx8m-bsb
+EESchema Schematic File Version 4
 LIBS:dvk-mx8m-bsb-cache
-EELAYER 25 0
+EELAYER 26 0
 EELAYER END
 $Descr A4 11693 8268
@@
 Note:\nNo power-up sequence is\ngiven in the spec sheet
 $Comp
-L 3V3_P #PWR0186
+L dvk-mx8m-bsb:3V3_P #PWR0186
 U 1 1 5AEA3227
 P 3600 3150
@@
 $EndComp
 $Comp
-L 3V3_P #PWR0187
+L dvk-mx8m-bsb:3V3_P #PWR0187
 U 1 1 5AEA329B
 P 1700 3250
@@
 $EndComp
 $Comp
-L 1V8_P #PWR0188
+L dvk-mx8m-bsb:1V8_P #PWR0188
 U 1 1 5AEDE2F3
 P 2300 3250
@@
 $EndComp
 $Comp
-L R R1202
+L dvk-mx8m-bsb-rescue:R R1202
 U 1 1 5B323584
 P 2550 3500
@@
 $EndComp
 $Comp
-L R R1201
+L dvk-mx8m-bsb-rescue:R R1201
 U 1 1 5B3235E0
 P 1700 3500
@@
 $EndComp
 $Comp
-L R R1203
+L dvk-mx8m-bsb-rescue:R R1203
 U 1 1 5B32362A
 P 3600 3400
@@
 $EndComp
 $Comp
-L R R1204
+L dvk-mx8m-bsb-rescue:R R1204
 U 1 1 5B3236A9
 P 4450 3400
@@
 $EndComp
 $Comp
-L 1V8_P #PWR0189
+L dvk-mx8m-bsb:1V8_P #PWR0189
 U 1 1 5B300B10
 P 4450 3150
@@
 $EndComp
 $Comp
-L Conn_01x39 J1202
+L dvk-mx8m-bsb-rescue:Conn_01x39 J1202
 U 1 1 5B314440
 P 8950 3150
@@
 $EndComp
 $Comp
-L GND #PWR0190
+L power:GND #PWR0190
 U 1 1 5B314AC6
 P 8700 5100
@@
 NoConn ~ 8750 4850
 $Comp
-L 22V4_P #PWR0191
+L dvk-mx8m-bsb:22V4_P #PWR0191
 U 1 1 5B3239F0
 P 8000 5000
@@
 NoConn ~ 8750 2950
 $Comp
-L 1V8_P #PWR0192
+L dvk-mx8m-bsb:1V8_P #PWR0192
 U 1 1 5B328FC1
 P 6750 2400
@@
 $EndComp
 $Comp
-L C C1202
+L dvk-mx8m-bsb-rescue:C C1202
 U 1 1 5B32A2B5
 P 6300 2750
@@
 $EndComp
 $Comp
-L GND #PWR0193
+L power:GND #PWR0193
 U 1 1 5B32A2F2
 P 6750 3000
@@
 	8650 4550 8750 4550
 $Comp
-L 2V8_P #PWR0194
+L dvk-mx8m-bsb:2V8_P #PWR0194
 U 1 1 5B3FFD6E
 P 7500 2400
@@
 $EndComp
 $Comp
-L C C1206
+L dvk-mx8m-bsb-rescue:C C1206
 U 1 1 5B3FFDB6
 P 7500 2750
@@
 $EndComp
 $Comp
-L GND #PWR0195
+L power:GND #PWR0195
 U 1 1 5B3FFE19
 P 7500 2950
@@
 Connection ~ 7500 2550
 $Comp
-L Conn_01x06 J1201
+L dvk-mx8m-bsb-rescue:Conn_01x06 J1201
 U 1 1 5B445B35
 P 5800 3600
@@
 	5500 3500 5600 3500
 $Comp
-L GND #PWR0196
+L power:GND #PWR0196
 U 1 1 5B449295
 P 5550 3950
@@
 	5550 2700 5550 3800
 $Comp
-L 2V8_P #PWR0197
+L dvk-mx8m-bsb:2V8_P #PWR0197
 U 1 1 5B449772
 P 5550 2700
@@
 $EndComp
 $Comp
-L C C1201
+L dvk-mx8m-bsb-rescue:C C1201
 U 1 1 5B44A018
 P 5400 2950
@@
 $EndComp
 $Comp
-L GND #PWR0198
+L power:GND #PWR0198
 U 1 1 5B44A063
 P 5400 3150
@@
 	5400 3150 5400 3100
 $Comp
-L C C1205
+L dvk-mx8m-bsb-rescue:C C1205
 U 1 1 5B44F3BF
 P 7200 2750
@@
 $EndComp
 $Comp
-L C C1204
+L dvk-mx8m-bsb-rescue:C C1204
 U 1 1 5B44F3C6
 P 6900 2750
@@
 $EndComp
 $Comp
-L C C1203
+L dvk-mx8m-bsb-rescue:C C1203
 U 1 1 5B44F3CD
 P 6600 2750
@@
 Connection ~ 6750 2450
 $Comp
-L C C1207
+L dvk-mx8m-bsb-rescue:C C1207
 U 1 1 5B452925
 P 7550 5350
@@
 $EndComp
 $Comp
-L GND #PWR0199
+L power:GND #PWR0199
 U 1 1 5B45292C
 P 8000 5600
@@
 $EndComp
 $Comp
-L C C1210
+L dvk-mx8m-bsb-rescue:C C1210
 U 1 1 5B452932
 P 8450 5350
@@
 $EndComp
 $Comp
-L C C1209
+L dvk-mx8m-bsb-rescue:C C1209
 U 1 1 5B452939
 P 8150 5350
@@
 $EndComp
 $Comp
-L C C1208
+L dvk-mx8m-bsb-rescue:C C1208
 U 1 1 5B452940
 P 7850 5350
@@
 Display & Touch Controller
 $Comp
-L Q_NMOS_GSD Q1202
+L dvk-mx8m-bsb-rescue:Q_NMOS_GSD Q1202
 U 1 1 5B2E270A
 P 4200 3500
@@
 $EndComp
 $Comp
-L Q_NMOS_GSD Q1201
+L dvk-mx8m-bsb-rescue:Q_NMOS_GSD Q1201
 U 1 1 5B2E3533
 P 2300 3600
@@
 $EndComp
 $Comp
-L Display_JH057N00900 DISP1201
+L dvk-mx8m-bsb:Display_JH057N00900 DISP1201
 U 1 1 5B2C05F7
 P 10300 2500
@@
 $EndComp
 $Comp
-L GND #PWR0200
+L power:GND #PWR0200
 U 1 1 5B477319
 P 8200 3250
@@
 	8200 3250 8200 3200
 $Comp
-L R R1205
+L dvk-mx8m-bsb-rescue:R R1205
 U 1 1 5B477A28
 P 8200 3050

Commit message: Update the schematic symbols and footprints after upgrading to KiCad 5.0.0, fix all ERC and DRC violations after the new update/upgrade
Parts:
- C1201, C1202, C1203, C1204, C1205, C1206, C1207, C1208, C1209, C1210: footprint Capacitors_SMD:C_0603 -> Capacitor_SMD:C_0603_1608Metric; symbol dvk-mx8m-bsb-rescue:C -> Device:C
- J1201: symbol dvk-mx8m-bsb-rescue:Conn_01x06 -> Connector_Generic:Conn_01x06
- J1202: symbol dvk-mx8m-bsb-rescue:Conn_01x39 -> Connector_Generic:Conn_01x39
- Q1201, Q1202: symbol dvk-mx8m-bsb-rescue:Q_NMOS_GSD -> Device:Q_NMOS_GSD
- R1201, R1202, R1203, R1204, R1205: footprint Resistors_SMD:R_0603 -> Resistor_SMD:R_0603_1608Metric; symbol dvk-mx8m-bsb-rescue:R -> Device:R
Connections:
- wire segments 74 -> 103
Changed lines of the file:
@@
 Sheet 12 24
 Title "MIPI DSI"
-Date "2018-06-18"
+Date "2018-07-17"
 Rev "v0.1.0"
 Comp "Copyright 2018 GNU GPLv3"
@@
 CAPTOUCH_~RST
 Wire Wire Line
-	4400 3600 5600 3600
+	4400 3600 4450 3600
 Wire Wire Line
-	2500 3700 5600 3700
+	2500 3700 2550 3700
 Wire Wire Line
 	2550 3700 2550 3650
 Connection ~ 2550 3700
 Wire Wire Line
-	2300 3250 2300 3400
+	2300 3250 2300 3300
 Wire Wire Line
 	2550 3350 2550 3300
@@
 Connection ~ 2300 3300
 Wire Wire Line
-	1650 3700 2100 3700
+	1650 3700 1700 3700
 Wire Wire Line
 	1700 3700 1700 3650
@@
 Connection ~ 4450 3600
 Wire Wire Line
-	4450 3150 4450 3250
+	4450 3150 4450 3200
 Wire Wire Line
 	4450 3200 4200 3200
@@
 Connection ~ 4450 3200
 Wire Wire Line
-	3550 3600 4000 3600
+	3550 3600 3600 3600
 Wire Wire Line
 	3600 3600 3600 3550
@@
 $EndComp
 $Comp
-L dvk-mx8m-bsb-rescue:R R1202
+L Device:R R1202
 U 1 1 5B323584
 P 2550 3500
 F 0 "R1202" H 2725 3550 50  0000 C CNN
 F 1 "10k" H 2675 3450 50  0000 C CNN
-F 2 "Resistors_SMD:R_0603" V 2480 3500 50  0001 C CNN
+F 2 "Resistor_SMD:R_0603_1608Metric" V 2480 3500 50  0001 C CNN
 F 3 "https://www.seielect.com/Catalog/SEI-RMCF_RMCP.pdf" H 2550 3500 50  0001 C CNN
 F 4 "Stackpole" H 2550 3500 60  0001 C CNN "MFG Name"
@@
 $EndComp
 $Comp
-L dvk-mx8m-bsb-rescue:R R1201
+L Device:R R1201
 U 1 1 5B3235E0
 P 1700 3500
 F 0 "R1201" H 1875 3550 50  0000 C CNN
 F 1 "10k" H 1825 3450 50  0000 C CNN
-F 2 "Resistors_SMD:R_0603" V 1630 3500 50  0001 C CNN
+F 2 "Resistor_SMD:R_0603_1608Metric" V 1630 3500 50  0001 C CNN
 F 3 "https://www.seielect.com/Catalog/SEI-RMCF_RMCP.pdf" H 1700 3500 50  0001 C CNN
 F 4 "Stackpole" H 1700 3500 60  0001 C CNN "MFG Name"
@@
 $EndComp
 $Comp
-L dvk-mx8m-bsb-rescue:R R1203
+L Device:R R1203
 U 1 1 5B32362A
 P 3600 3400
 F 0 "R1203" H 3775 3450 50  0000 C CNN
 F 1 "10k" H 3725 3350 50  0000 C CNN
-F 2 "Resistors_SMD:R_0603" V 3530 3400 50  0001 C CNN
+F 2 "Resistor_SMD:R_0603_1608Metric" V 3530 3400 50  0001 C CNN
 F 3 "https://www.seielect.com/Catalog/SEI-RMCF_RMCP.pdf" H 3600 3400 50  0001 C CNN
 F 4 "Stackpole" H 3600 3400 60  0001 C CNN "MFG Name"
@@
 $EndComp
 $Comp
-L dvk-mx8m-bsb-rescue:R R1204
+L Device:R R1204
 U 1 1 5B3236A9
 P 4450 3400
 F 0 "R1204" H 4625 3450 50  0000 C CNN
 F 1 "10k" H 4575 3350 50  0000 C CNN
-F 2 "Resistors_SMD:R_0603" V 4380 3400 50  0001 C CNN
+F 2 "Resistor_SMD:R_0603_1608Metric" V 4380 3400 50  0001 C CNN
 F 3 "https://www.seielect.com/Catalog/SEI-RMCF_RMCP.pdf" H 4450 3400 50  0001 C CNN
 F 4 "Stackpole" H 4450 3400 60  0001 C CNN "MFG Name"
@@
 $EndComp
 $Comp
-L dvk-mx8m-bsb-rescue:Conn_01x39 J1202
+L Connector_Generic:Conn_01x39 J1202
 U 1 1 5B314440
 P 8950 3150
@@
 	8750 2050 8700 2050
 Wire Wire Line
-	8700 2050 8700 5100
+	8700 2050 8700 3150
 Wire Wire Line
 	8750 3150 8700 3150
@@
 LCD_LEDK
 Wire Wire Line
-	7550 5050 8750 5050
+	7550 5050 7850 5050
 Wire Wire Line
 	8650 4950 8750 4950
@@
 $EndComp
 $Comp
-L dvk-mx8m-bsb-rescue:C C1202
+L Device:C C1202
 U 1 1 5B32A2B5
 P 6300 2750
 F 0 "C1202" H 6325 2850 50  0000 L CNN
 F 1 "100nF" H 6325 2650 50  0000 L CNN
-F 2 "Capacitors_SMD:C_0603" H 6338 2600 50  0001 C CNN
+F 2 "Capacitor_SMD:C_0603_1608Metric" H 6338 2600 50  0001 C CNN
 F 3 "" H 6300 2750 50  0001 C CNN
 	1    6300 2750
@@
 LCD_~RESET
 Wire Wire Line
-	8150 2850 8750 2850
+	8150 2850 8200 2850
 Wire Wire Line
 	8650 3250 8750 3250
@@
 $EndComp
 $Comp
-L dvk-mx8m-bsb-rescue:C C1206
+L Device:C C1206
 U 1 1 5B3FFDB6
 P 7500 2750
 F 0 "C1206" H 7525 2850 50  0000 L CNN
 F 1 "100nF" H 7525 2650 50  0000 L CNN
-F 2 "Capacitors_SMD:C_0603" H 7538 2600 50  0001 C CNN
+F 2 "Capacitor_SMD:C_0603_1608Metric" H 7538 2600 50  0001 C CNN
 F 3 "" H 7500 2750 50  0001 C CNN
 	1    7500 2750
@@
 	7500 2950 7500 2900
 Wire Wire Line
-	7500 2400 7500 2600
+	7500 2400 7500 2550
 Wire Wire Line
 	8750 2550 7500 2550
 Connection ~ 7500 2550
 $Comp
-L dvk-mx8m-bsb-rescue:Conn_01x06 J1201
+L Connector_Generic:Conn_01x06 J1201
 U 1 1 5B445B35
 P 5800 3600
@@
 	5550 3800 5600 3800
 Wire Wire Line
-	5550 2700 5550 3800
+	5550 2700 5550 2750
 $Comp
 L dvk-mx8m-bsb:2V8_P #PWR0197
@@
 $EndComp
 $Comp
-L dvk-mx8m-bsb-rescue:C C1201
+L Device:C C1201
 U 1 1 5B44A018
 P 5400 2950
 F 0 "C1201" H 5425 3050 50  0000 L CNN
 F 1 "100nF" H 5425 2850 50  0000 L CNN
-F 2 "Capacitors_SMD:C_0603" H 5438 2800 50  0001 C CNN
+F 2 "Capacitor_SMD:C_0603_1608Metric" H 5438 2800 50  0001 C CNN
 F 3 "" H 5400 2950 50  0001 C CNN
 	1    5400 2950
@@
 	5400 3150 5400 3100
 $Comp
-L dvk-mx8m-bsb-rescue:C C1205
+L Device:C C1205
 U 1 1 5B44F3BF
 P 7200 2750
 F 0 "C1205" H 7225 2850 50  0000 L CNN
 F 1 "100pF" H 7225 2650 50  0000 L CNN
-F 2 "Capacitors_SMD:C_0603" H 7238 2600 50  0001 C CNN
+F 2 "Capacitor_SMD:C_0603_1608Metric" H 7238 2600 50  0001 C CNN
 F 3 "" H 7200 2750 50  0001 C CNN
 	1    7200 2750
@@
 $EndComp
 $Comp
-L dvk-mx8m-bsb-rescue:C C1204
+L Device:C C1204
 U 1 1 5B44F3C6
 P 6900 2750
 F 0 "C1204" H 6925 2850 50  0000 L CNN
 F 1 "1nF" H 6925 2650 50  0000 L CNN
-F 2 "Capacitors_SMD:C_0603" H 6938 2600 50  0001 C CNN
+F 2 "Capacitor_SMD:C_0603_1608Metric" H 6938 2600 50  0001 C CNN
 F 3 "" H 6900 2750 50  0001 C CNN
 	1    6900 2750
@@
 $EndComp
 $Comp
-L dvk-mx8m-bsb-rescue:C C1203
+L Device:C C1203
 U 1 1 5B44F3CD
 P 6600 2750
 F 0 "C1203" H 6625 2850 50  0000 L CNN
 F 1 "10nF" H 6625 2650 50  0000 L CNN
-F 2 "Capacitors_SMD:C_0603" H 6638 2600 50  0001 C CNN
+F 2 "Capacitor_SMD:C_0603_1608Metric" H 6638 2600 50  0001 C CNN
 F 3 "" H 6600 2750 50  0001 C CNN
 	1    6600 2750
@@
 $EndComp
 Wire Wire Line
-	6300 2450 8750 2450
+	6300 2450 6600 2450
 Wire Wire Line
 	6300 2450 6300 2600
@@
 	6300 2900 6300 2950
 Wire Wire Line
-	6300 2950 7200 2950
+	6300 2950 6600 2950
 Wire Wire Line
 	7200 2950 7200 2900
@@
 Connection ~ 6750 2450
 $Comp
-L dvk-mx8m-bsb-rescue:C C1207
+L Device:C C1207
 U 1 1 5B452925
 P 7550 5350
 F 0 "C1207" H 7575 5450 50  0000 L CNN
 F 1 "100nF" H 7575 5250 50  0000 L CNN
-F 2 "Capacitors_SMD:C_0603" H 7588 5200 50  0001 C CNN
+F 2 "Capacitor_SMD:C_0603_1608Metric" H 7588 5200 50  0001 C CNN
 F 3 "" H 7550 5350 50  0001 C CNN
 	1    7550 5350
@@
 $EndComp
 $Comp
-L dvk-mx8m-bsb-rescue:C C1210
+L Device:C C1210
 U 1 1 5B452932
 P 8450 5350
 F 0 "C1210" H 8475 5450 50  0000 L CNN
 F 1 "100pF" H 8475 5250 50  0000 L CNN
-F 2 "Capacitors_SMD:C_0603" H 8488 5200 50  0001 C CNN
+F 2 "Capacitor_SMD:C_0603_1608Metric" H 8488 5200 50  0001 C CNN
 F 3 "" H 8450 5350 50  0001 C CNN
 	1    8450 5350
@@
 $EndComp
 $Comp
-L dvk-mx8m-bsb-rescue:C C1209
+L Device:C C1209
 U 1 1 5B452939
 P 8150 5350
 F 0 "C1209" H 8175 5450 50  0000 L CNN
 F 1 "1nF" H 8175 5250 50  0000 L CNN
-F 2 "Capacitors_SMD:C_0603" H 8188 5200 50  0001 C CNN
+F 2 "Capacitor_SMD:C_0603_1608Metric" H 8188 5200 50  0001 C CNN
 F 3 "" H 8150 5350 50  0001 C CNN
 	1    8150 5350
@@
 $EndComp
 $Comp
-L dvk-mx8m-bsb-rescue:C C1208
+L Device:C C1208
 U 1 1 5B452940
 P 7850 5350
 F 0 "C1208" H 7875 5450 50  0000 L CNN
 F 1 "10nF" H 7875 5250 50  0000 L CNN
-F 2 "Capacitors_SMD:C_0603" H 7888 5200 50  0001 C CNN
+F 2 "Capacitor_SMD:C_0603_1608Metric" H 7888 5200 50  0001 C CNN
 F 3 "" H 7850 5350 50  0001 C CNN
 	1    7850 5350
@@
 	7550 5500 7550 5550
 Wire Wire Line
-	7550 5550 8450 5550
+	7550 5550 7850 5550
 Wire Wire Line
 	8450 5550 8450 5500
@@
 Display & Touch Controller
 $Comp
-L dvk-mx8m-bsb-rescue:Q_NMOS_GSD Q1202
+L Device:Q_NMOS_GSD Q1202
 U 1 1 5B2E270A
 P 4200 3500
@@
 $EndComp
 $Comp
-L dvk-mx8m-bsb-rescue:Q_NMOS_GSD Q1201
+L Device:Q_NMOS_GSD Q1201
 U 1 1 5B2E3533
 P 2300 3600
@@
 	8200 3250 8200 3200
 $Comp
-L dvk-mx8m-bsb-rescue:R R1205
+L Device:R R1205
 U 1 1 5B477A28
 P 8200 3050
 F 0 "R1205" H 8375 3100 50  0000 C CNN
 F 1 "10k" H 8325 3000 50  0000 C CNN
-F 2 "Resistors_SMD:R_0603" V 8130 3050 50  0001 C CNN
+F 2 "Resistor_SMD:R_0603_1608Metric" V 8130 3050 50  0001 C CNN
 F 3 "https://www.seielect.com/Catalog/SEI-RMCF_RMCP.pdf" H 8200 3050 50  0001 C CNN
 F 4 "Stackpole" H 8200 3050 60  0001 C CNN "MFG Name"
@@
 	-1   0    0    -1
 $EndComp
+Wire Wire Line
+	2550 3700 5600 3700
+Wire Wire Line
+	2300 3300 2300 3400
+Wire Wire Line
+	4450 3600 5600 3600
+Wire Wire Line
+	4450 3200 4450 3250
+Wire Wire Line
+	3600 3600 4000 3600
+Wire Wire Line
+	1700 3700 2100 3700
+Wire Wire Line
+	8700 3150 8700 3450
+Wire Wire Line
+	8700 3450 8700 3750
+Wire Wire Line
+	8700 3750 8700 4050
+Wire Wire Line
+	8700 4050 8700 4350
+Wire Wire Line
+	8700 4350 8700 4650
+Wire Wire Line
+	8700 4650 8700 5100
+Wire Wire Line
+	7500 2550 7500 2600
+Wire Wire Line
+	5550 2750 5550 3800
+Wire Wire Line
+	6600 2450 6750 2450
+Wire Wire Line
+	6900 2450 7200 2450
+Wire Wire Line
+	7200 2450 8750 2450
+Wire Wire Line
+	6600 2950 6750 2950
+Wire Wire Line
+	6900 2950 7200 2950
+Wire Wire Line
+	6750 2950 6900 2950
+Wire Wire Line
+	6750 2450 6900 2450
+Wire Wire Line
+	7850 5550 8000 5550
+Wire Wire Line
+	8150 5550 8450 5550
+Wire Wire Line
+	8000 5550 8150 5550
+Wire Wire Line
+	7850 5050 8000 5050
+Wire Wire Line
+	8150 5050 8450 5050
+Wire Wire Line
+	8450 5050 8750 5050
+Wire Wire Line
+	8000 5050 8150 5050
+Wire Wire Line
+	8200 2850 8750 2850
 $EndSCHEMATC

Commit message: Reduce all 0603 resistor sizes to 0402
Parts:
- R1201, R1202, R1203, R1204, R1205: footprint Resistor_SMD:R_0603_1608Metric -> Resistor_SMD:R_0402_1005Metric
Changed lines of the file:
@@
 F 0 "R1202" H 2725 3550 50  0000 C CNN
 F 1 "10k" H 2675 3450 50  0000 C CNN
-F 2 "Resistor_SMD:R_0603_1608Metric" V 2480 3500 50  0001 C CNN
+F 2 "Resistor_SMD:R_0402_1005Metric" V 2480 3500 50  0001 C CNN
 F 3 "https://www.seielect.com/Catalog/SEI-RMCF_RMCP.pdf" H 2550 3500 50  0001 C CNN
 F 4 "Stackpole" H 2550 3500 60  0001 C CNN "MFG Name"
@@
 F 0 "R1201" H 1875 3550 50  0000 C CNN
 F 1 "10k" H 1825 3450 50  0000 C CNN
-F 2 "Resistor_SMD:R_0603_1608Metric" V 1630 3500 50  0001 C CNN
+F 2 "Resistor_SMD:R_0402_1005Metric" V 1630 3500 50  0001 C CNN
 F 3 "https://www.seielect.com/Catalog/SEI-RMCF_RMCP.pdf" H 1700 3500 50  0001 C CNN
 F 4 "Stackpole" H 1700 3500 60  0001 C CNN "MFG Name"
@@
 F 0 "R1203" H 3775 3450 50  0000 C CNN
 F 1 "10k" H 3725 3350 50  0000 C CNN
-F 2 "Resistor_SMD:R_0603_1608Metric" V 3530 3400 50  0001 C CNN
+F 2 "Resistor_SMD:R_0402_1005Metric" V 3530 3400 50  0001 C CNN
 F 3 "https://www.seielect.com/Catalog/SEI-RMCF_RMCP.pdf" H 3600 3400 50  0001 C CNN
 F 4 "Stackpole" H 3600 3400 60  0001 C CNN "MFG Name"
@@
 F 0 "R1204" H 4625 3450 50  0000 C CNN
 F 1 "10k" H 4575 3350 50  0000 C CNN
-F 2 "Resistor_SMD:R_0603_1608Metric" V 4380 3400 50  0001 C CNN
+F 2 "Resistor_SMD:R_0402_1005Metric" V 4380 3400 50  0001 C CNN
 F 3 "https://www.seielect.com/Catalog/SEI-RMCF_RMCP.pdf" H 4450 3400 50  0001 C CNN
 F 4 "Stackpole" H 4450 3400 60  0001 C CNN "MFG Name"
@@
 F 0 "R1205" H 8375 3100 50  0000 C CNN
 F 1 "10k" H 8325 3000 50  0000 C CNN
-F 2 "Resistor_SMD:R_0603_1608Metric" V 8130 3050 50  0001 C CNN
+F 2 "Resistor_SMD:R_0402_1005Metric" V 8130 3050 50  0001 C CNN
 F 3 "https://www.seielect.com/Catalog/SEI-RMCF_RMCP.pdf" H 8200 3050 50  0001 C CNN
 F 4 "Stackpole" H 8200 3050 60  0001 C CNN "MFG Name"

Commit message: Change all 0603 capacitors _EXCEPT_ the 2.2uF, 4.7uF, 8.2uF, 10uF, and 22uF caps to 0402
Parts:
- C1201, C1202, C1203, C1204, C1205, C1206, C1207, C1208, C1209, C1210: footprint Capacitor_SMD:C_0603_1608Metric -> Capacitor_SMD:C_0402_1005Metric
Changed lines of the file:
@@
 F 0 "C1202" H 6325 2850 50  0000 L CNN
 F 1 "100nF" H 6325 2650 50  0000 L CNN
-F 2 "Capacitor_SMD:C_0603_1608Metric" H 6338 2600 50  0001 C CNN
+F 2 "Capacitor_SMD:C_0402_1005Metric" H 6338 2600 50  0001 C CNN
 F 3 "" H 6300 2750 50  0001 C CNN
 	1    6300 2750
@@
 F 0 "C1206" H 7525 2850 50  0000 L CNN
 F 1 "100nF" H 7525 2650 50  0000 L CNN
-F 2 "Capacitor_SMD:C_0603_1608Metric" H 7538 2600 50  0001 C CNN
+F 2 "Capacitor_SMD:C_0402_1005Metric" H 7538 2600 50  0001 C CNN
 F 3 "" H 7500 2750 50  0001 C CNN
 	1    7500 2750
@@
 F 0 "C1201" H 5425 3050 50  0000 L CNN
 F 1 "100nF" H 5425 2850 50  0000 L CNN
-F 2 "Capacitor_SMD:C_0603_1608Metric" H 5438 2800 50  0001 C CNN
+F 2 "Capacitor_SMD:C_0402_1005Metric" H 5438 2800 50  0001 C CNN
 F 3 "" H 5400 2950 50  0001 C CNN
 	1    5400 2950
@@
 F 0 "C1205" H 7225 2850 50  0000 L CNN
 F 1 "100pF" H 7225 2650 50  0000 L CNN
-F 2 "Capacitor_SMD:C_0603_1608Metric" H 7238 2600 50  0001 C CNN
+F 2 "Capacitor_SMD:C_0402_1005Metric" H 7238 2600 50  0001 C CNN
 F 3 "" H 7200 2750 50  0001 C CNN
 	1    7200 2750
@@
 F 0 "C1204" H 6925 2850 50  0000 L CNN
 F 1 "1nF" H 6925 2650 50  0000 L CNN
-F 2 "Capacitor_SMD:C_0603_1608Metric" H 6938 2600 50  0001 C CNN
+F 2 "Capacitor_SMD:C_0402_1005Metric" H 6938 2600 50  0001 C CNN
 F 3 "" H 6900 2750 50  0001 C CNN
 	1    6900 2750
@@
 F 0 "C1203" H 6625 2850 50  0000 L CNN
 F 1 "10nF" H 6625 2650 50  0000 L CNN
-F 2 "Capacitor_SMD:C_0603_1608Metric" H 6638 2600 50  0001 C CNN
+F 2 "Capacitor_SMD:C_0402_1005Metric" H 6638 2600 50  0001 C CNN
 F 3 "" H 6600 2750 50  0001 C CNN
 	1    6600 2750
@@
 F 0 "C1207" H 7575 5450 50  0000 L CNN
 F 1 "100nF" H 7575 5250 50  0000 L CNN
-F 2 "Capacitor_SMD:C_0603_1608Metric" H 7588 5200 50  0001 C CNN
+F 2 "Capacitor_SMD:C_0402_1005Metric" H 7588 5200 50  0001 C CNN
 F 3 "" H 7550 5350 50  0001 C CNN
 	1    7550 5350
@@
 F 0 "C1210" H 8475 5450 50  0000 L CNN
 F 1 "100pF" H 8475 5250 50  0000 L CNN
-F 2 "Capacitor_SMD:C_0603_1608Metric" H 8488 5200 50  0001 C CNN
+F 2 "Capacitor_SMD:C_0402_1005Metric" H 8488 5200 50  0001 C CNN
 F 3 "" H 8450 5350 50  0001 C CNN
 	1    8450 5350
@@
 F 0 "C1209" H 8175 5450 50  0000 L CNN
 F 1 "1nF" H 8175 5250 50  0000 L CNN
-F 2 "Capacitor_SMD:C_0603_1608Metric" H 8188 5200 50  0001 C CNN
+F 2 "Capacitor_SMD:C_0402_1005Metric" H 8188 5200 50  0001 C CNN
 F 3 "" H 8150 5350 50  0001 C CNN
 	1    8150 5350
@@
 F 0 "C1208" H 7875 5450 50  0000 L CNN
 F 1 "10nF" H 7875 5250 50  0000 L CNN
-F 2 "Capacitor_SMD:C_0603_1608Metric" H 7888 5200 50  0001 C CNN
+F 2 "Capacitor_SMD:C_0402_1005Metric" H 7888 5200 50  0001 C CNN
 F 3 "" H 7850 5350 50  0001 C CNN
 	1    7850 5350
