File: haptic.sch (KiCad schematic (older format))
At the start: 7 parts, among them J2401 Conn_01x02, M2401 Motor, Q2401 DMG2301L

Commit message: Now using GPIO5_IO03 (P4.03) to put the class-D op-amp in shutdown and conserve energy when muted, make C1716 near the ETH PHY's DVDDL pin 47 220nF instead of 10uF (EmCraft suggested that this should be 100nF but their's is 220nF, asked why), added a 10k pull-down to PAM2841's ENA pin, added a 100nF cap to the smart card's C1 VCC pin, added a 1uF cap to the haptic motor circuit's 3V3_P rail
Still need to use I2C3 instead of I2C1 according to EmCraft's suggestions.
Parts:
- added C2402: 1uF, Capacitors_SMD:C_0603, symbol C
Connections:
- wire segments 16 -> 18
Changed lines of the file:
@@
 $EndDescr
 $Comp
-L GND #PWR0393
+L GND #PWR0395
 U 1 1 5AFCF90B
 P 6050 4700
-F 0 "#PWR0393" H 6050 4450 50  0001 C CNN
+F 0 "#PWR0395" H 6050 4450 50  0001 C CNN
 F 1 "GND" H 6050 4550 50  0000 C CNN
 F 2 "" H 6050 4700 50  0001 C CNN
@@
 $EndComp
 $Comp
-L 3V3_P #PWR0394
+L 3V3_P #PWR0396
 U 1 1 5AFD13E2
 P 6050 3350
-F 0 "#PWR0394" H 6050 3200 50  0001 C CNN
+F 0 "#PWR0396" H 6050 3200 50  0001 C CNN
 F 1 "3V3_P" H 6050 3490 50  0000 C CNN
 F 2 "" H 6050 3350 50  0001 C CNN
@@
 Wire Wire Line
 	5350 3450 5350 3400
-Wire Wire Line
-	5350 3400 6050 3400
 Connection ~ 6050 3400
 Wire Wire Line
@@
 	1    0    0    -1
 $EndComp
+$Comp
+L C C2402
+U 1 1 5B428193
+P 6650 3600
+F 0 "C2402" H 6675 3700 50  0000 L CNN
+F 1 "1uF" H 6675 3500 50  0000 L CNN
+F 2 "Capacitors_SMD:C_0603" H 6688 3450 50  0001 C CNN
+F 3 "" H 6650 3600 50  0001 C CNN
+	1    6650 3600
+	1    0    0    -1
+$EndComp
+$Comp
+L GND #PWR0397
+U 1 1 5B428255
+P 6650 3800
+F 0 "#PWR0397" H 6650 3550 50  0001 C CNN
+F 1 "GND" H 6650 3650 50  0000 C CNN
+F 2 "" H 6650 3800 50  0001 C CNN
+F 3 "" H 6650 3800 50  0001 C CNN
+	1    6650 3800
+	1    0    0    -1
+$EndComp
+Wire Wire Line
+	6650 3800 6650 3750
+Wire Wire Line
+	5350 3400 6650 3400
+Wire Wire Line
+	6650 3400 6650 3450
 $EndSCHEMATC

Commit message: Update project files to KiCad 5.0.0
Parts:
- C2401, C2402: symbol C -> dvk-mx8m-bsb-rescue:C
- D2401: symbol D_Schottky_ALT -> dvk-mx8m-bsb-rescue:D_Schottky_ALT
- J2401: symbol Conn_01x02 -> dvk-mx8m-bsb-rescue:Conn_01x02
- M2401: symbol Motor_Haptic -> dvk-mx8m-bsb:Motor_Haptic
- Q2401: symbol Q_PMOS_GSD -> dvk-mx8m-bsb-rescue:Q_PMOS_GSD
- R2401, R2402: symbol R -> dvk-mx8m-bsb-rescue:R
Changed lines of the file:
@@
-EESchema Schematic File Version 2
-LIBS:power
-LIBS:device
-LIBS:switches
-LIBS:relays
-LIBS:motors
-LIBS:transistors
-LIBS:conn
-LIBS:linear
-LIBS:regul
-LIBS:74xx
-LIBS:cmos4000
-LIBS:adc-dac
-LIBS:memory
-LIBS:xilinx
-LIBS:microcontrollers
-LIBS:dsp
-LIBS:microchip
-LIBS:analog_switches
-LIBS:motorola
-LIBS:texas
-LIBS:intel
-LIBS:audio
-LIBS:interface
-LIBS:digital-audio
-LIBS:philips
-LIBS:display
-LIBS:cypress
-LIBS:siliconi
-LIBS:opto
-LIBS:atmel
-LIBS:contrib
-LIBS:valves
-LIBS:dvk-mx8m-bsb
+EESchema Schematic File Version 4
 LIBS:dvk-mx8m-bsb-cache
-EELAYER 25 0
+EELAYER 26 0
 EELAYER END
 $Descr A4 11693 8268
@@
 $EndDescr
 $Comp
-L GND #PWR0397
+L power:GND #PWR0397
 U 1 1 5AFCF90B
 P 6050 4700
@@
 When the motor is off\nboth terminals are at GND
 $Comp
-L Q_PMOS_GSD Q2401
+L dvk-mx8m-bsb-rescue:Q_PMOS_GSD Q2401
 U 1 1 5AFD137F
 P 5950 3800
@@
 $EndComp
 $Comp
-L 3V3_P #PWR0398
+L dvk-mx8m-bsb:3V3_P #PWR0398
 U 1 1 5AFD13E2
 P 6050 3350
@@
 $EndComp
 $Comp
-L R R2401
+L dvk-mx8m-bsb-rescue:R R2401
 U 1 1 5AFD2E14
 P 5350 3600
@@
 HAPTIC
 $Comp
-L D_Schottky_ALT D2401
+L dvk-mx8m-bsb-rescue:D_Schottky_ALT D2401
 U 1 1 5AFD563E
 P 5250 4350
@@
 $EndComp
 $Comp
-L R R2402
+L dvk-mx8m-bsb-rescue:R R2402
 U 1 1 5AFFD30C
 P 5550 3800
@@
 $EndComp
 $Comp
-L C C2401
+L dvk-mx8m-bsb-rescue:C C2401
 U 1 1 5B0285ED
 P 5650 4350
@@
 Haptic Motor
 $Comp
-L Conn_01x02 J2401
+L dvk-mx8m-bsb-rescue:Conn_01x02 J2401
 U 1 1 5B316276
 P 6300 4400
@@
 	6050 4300 6100 4300
 $Comp
-L Motor_Haptic M2401
+L dvk-mx8m-bsb:Motor_Haptic M2401
 U 1 1 5B316C25
 P 6600 4350
@@
 $EndComp
 $Comp
-L C C2402
+L dvk-mx8m-bsb-rescue:C C2402
 U 1 1 5B428193
 P 6650 3600
@@
 $EndComp
 $Comp
-L GND #PWR0399
+L power:GND #PWR0399
 U 1 1 5B428255
 P 6650 3800

Commit message: Update the schematic symbols and footprints after upgrading to KiCad 5.0.0, fix all ERC and DRC violations after the new update/upgrade
Parts:
- C2401, C2402: footprint Capacitors_SMD:C_0603 -> Capacitor_SMD:C_0603_1608Metric; symbol dvk-mx8m-bsb-rescue:C -> Device:C
- D2401: symbol dvk-mx8m-bsb-rescue:D_Schottky_ALT -> Device:D_Schottky_ALT
- J2401: symbol dvk-mx8m-bsb-rescue:Conn_01x02 -> Connector_Generic:Conn_01x02
- Q2401: footprint TO_SOT_Packages_SMD:SOT-23 -> Package_TO_SOT_SMD:SOT-23; symbol dvk-mx8m-bsb-rescue:Q_PMOS_GSD -> Device:Q_PMOS_GSD
- R2401, R2402: footprint Resistors_SMD:R_0603 -> Resistor_SMD:R_0603_1608Metric; symbol dvk-mx8m-bsb-rescue:R -> Device:R
Changed lines of the file:
@@
 Sheet 24 24
 Title "Haptic/Vibration Motor"
-Date "2018-06-18"
+Date "2018-07-17"
 Rev "v0.1.0"
 Comp "Copyright 2018 GNU GPLv3"
@@
 When the motor is off\nboth terminals are at GND
 $Comp
-L dvk-mx8m-bsb-rescue:Q_PMOS_GSD Q2401
+L Device:Q_PMOS_GSD Q2401
 U 1 1 5AFD137F
 P 5950 3800
 F 0 "Q2401" H 6150 3750 50  0000 L CNN
 F 1 "DMG2301L" H 6150 3850 50  0000 L CNN
-F 2 "TO_SOT_Packages_SMD:SOT-23" H 6150 3900 50  0001 C CNN
+F 2 "Package_TO_SOT_SMD:SOT-23" H 6150 3900 50  0001 C CNN
 F 3 "https://www.diodes.com/assets/Datasheets/DMG2301L.pdf" H 5950 3800 50  0001 C CNN
 F 4 "Diodes Inc" H 5950 3800 60  0001 C CNN "MFG Name"
@@
 $EndComp
 $Comp
-L dvk-mx8m-bsb-rescue:R R2401
+L Device:R R2401
 U 1 1 5AFD2E14
 P 5350 3600
 F 0 "R2401" H 5525 3650 50  0000 C CNN
 F 1 "100k" H 5500 3550 50  0000 C CNN
-F 2 "Resistors_SMD:R_0603" V 5280 3600 50  0001 C CNN
+F 2 "Resistor_SMD:R_0603_1608Metric" V 5280 3600 50  0001 C CNN
 F 3 "" H 5350 3600 50  0001 C CNN
 	1    5350 3600
@@
 HAPTIC
 $Comp
-L dvk-mx8m-bsb-rescue:D_Schottky_ALT D2401
+L Device:D_Schottky_ALT D2401
 U 1 1 5AFD563E
 P 5250 4350
@@
 $EndComp
 $Comp
-L dvk-mx8m-bsb-rescue:R R2402
+L Device:R R2402
 U 1 1 5AFFD30C
 P 5550 3800
 F 0 "R2402" V 5450 3800 50  0000 C CNN
 F 1 "100" V 5650 3800 50  0000 C CNN
-F 2 "Resistors_SMD:R_0603" V 5480 3800 50  0001 C CNN
+F 2 "Resistor_SMD:R_0603_1608Metric" V 5480 3800 50  0001 C CNN
 F 3 "" H 5550 3800 50  0001 C CNN
 	1    5550 3800
@@
 $EndComp
 $Comp
-L dvk-mx8m-bsb-rescue:C C2401
+L Device:C C2401
 U 1 1 5B0285ED
 P 5650 4350
 F 0 "C2401" H 5675 4450 50  0000 L CNN
 F 1 "100nF" H 5675 4250 50  0000 L CNN
-F 2 "Capacitors_SMD:C_0603" H 5688 4200 50  0001 C CNN
+F 2 "Capacitor_SMD:C_0603_1608Metric" H 5688 4200 50  0001 C CNN
 F 3 "" H 5650 4350 50  0001 C CNN
 	1    5650 4350
@@
 Haptic Motor
 $Comp
-L dvk-mx8m-bsb-rescue:Conn_01x02 J2401
+L Connector_Generic:Conn_01x02 J2401
 U 1 1 5B316276
 P 6300 4400
@@
 $EndComp
 $Comp
-L dvk-mx8m-bsb-rescue:C C2402
+L Device:C C2402
 U 1 1 5B428193
 P 6650 3600
 F 0 "C2402" H 6675 3700 50  0000 L CNN
 F 1 "1uF" H 6675 3500 50  0000 L CNN
-F 2 "Capacitors_SMD:C_0603" H 6688 3450 50  0001 C CNN
+F 2 "Capacitor_SMD:C_0603_1608Metric" H 6688 3450 50  0001 C CNN
 F 3 "" H 6650 3600 50  0001 C CNN
 	1    6650 3600

Commit message: Reduce all 0603 resistor sizes to 0402
Parts:
- R2401, R2402: footprint Resistor_SMD:R_0603_1608Metric -> Resistor_SMD:R_0402_1005Metric
Changed lines of the file:
@@
 F 0 "R2401" H 5525 3650 50  0000 C CNN
 F 1 "100k" H 5500 3550 50  0000 C CNN
-F 2 "Resistor_SMD:R_0603_1608Metric" V 5280 3600 50  0001 C CNN
+F 2 "Resistor_SMD:R_0402_1005Metric" V 5280 3600 50  0001 C CNN
 F 3 "" H 5350 3600 50  0001 C CNN
 	1    5350 3600
@@
 F 0 "R2402" V 5450 3800 50  0000 C CNN
 F 1 "100" V 5650 3800 50  0000 C CNN
-F 2 "Resistor_SMD:R_0603_1608Metric" V 5480 3800 50  0001 C CNN
+F 2 "Resistor_SMD:R_0402_1005Metric" V 5480 3800 50  0001 C CNN
 F 3 "" H 5550 3800 50  0001 C CNN
 	1    5550 3800

Commit message: Change all 0603 capacitors _EXCEPT_ the 2.2uF, 4.7uF, 8.2uF, 10uF, and 22uF caps to 0402
Parts:
- C2401, C2402: footprint Capacitor_SMD:C_0603_1608Metric -> Capacitor_SMD:C_0402_1005Metric
Changed lines of the file:
@@
 F 0 "C2401" H 5675 4450 50  0000 L CNN
 F 1 "100nF" H 5675 4250 50  0000 L CNN
-F 2 "Capacitor_SMD:C_0603_1608Metric" H 5688 4200 50  0001 C CNN
+F 2 "Capacitor_SMD:C_0402_1005Metric" H 5688 4200 50  0001 C CNN
 F 3 "" H 5650 4350 50  0001 C CNN
 	1    5650 4350
@@
 F 0 "C2402" H 6675 3700 50  0000 L CNN
 F 1 "1uF" H 6675 3500 50  0000 L CNN
-F 2 "Capacitor_SMD:C_0603_1608Metric" H 6688 3450 50  0001 C CNN
+F 2 "Capacitor_SMD:C_0402_1005Metric" H 6688 3450 50  0001 C CNN
 F 3 "" H 6650 3600 50  0001 C CNN
 	1    6650 3600
