File: sd.sch (KiCad schematic (older format))
At the start: 9 parts, among them J1001 Micro_SD

Commit message: Change GRM219R61C226ME15L X5R 0805 22uF capacitor to being a CL10A226MP8NUNE X5R 0603 22uF capacitor
Parts:
- C1002, C1003: footprint Capacitors_SMD:C_0805 -> Capacitors_SMD:C_0603; Distrib Link https://www.digikey.com/product-detail/en/murata-electronic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 -> https://lcsc.com/product-detail/Multilayer-Ceramic-Capacito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; Distrib PN 490-9952-1-ND -> C86295; MFG Name Murata -> Samsung; MFG Part Num GRM219R61C226ME15L -> CL10A226MP8NUNE; Others https://www.digikey.com/products/en/capacitors/ceramic-capa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 -> https://lcsc.com/product-detail/Multilayer-Ceramic-Capacito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
Changed lines of the file:
@@
 Wire Wire Line
 	4250 3450 5650 3450
+Text Notes 5800 1900 0    236  ~ 47
+μSD
 $Comp
 L C C1002
-U 1 1 5B1961D2
+U 1 1 5B3619B2
 P 5800 2550
 F 0 "C1002" H 5825 2650 50  0000 L CNN
 F 1 "22uF" H 5825 2450 50  0000 L CNN
-F 2 "Capacitors_SMD:C_0805" H 5838 2400 50  0001 C CNN
-F 3 "https://search.murata.co.jp/Ceramy/image/img/A01X/G101/ENG/GRM219R61C226ME15-01.pdf" H 5800 2550 50  0001 C CNN
-F 4 "Murata" H 5800 2550 60  0001 C CNN "MFG Name"
-F 5 "GRM219R61C226ME15L" H 5800 2550 60  0001 C CNN "MFG Part Num"
-F 6 "490-9952-1-ND" H 5800 2550 60  0001 C CNN "Distrib PN"
-F 7 "https://www.digikey.com/product-detail/en/murata-electronics-north-america/GRM219R61C226ME15L/490-9952-1-ND/5026415" H 5800 2550 60  0001 C CNN "Distrib Link"
+F 2 "Capacitors_SMD:C_0603" H 5838 2400 50  0001 C CNN
+F 3 "http://www.samsungsem.com/kr/support/product-search/mlcc/__icsFiles/afieldfile/2018/06/21/CL10A226MP8NUNE.pdf" H 5800 2550 50  0001 C CNN
+F 4 "Samsung" H 5800 2550 60  0001 C CNN "MFG Name"
+F 5 "CL10A226MP8NUNE" H 5800 2550 60  0001 C CNN "MFG Part Num"
+F 6 "C86295" H 5800 2550 60  0001 C CNN "Distrib PN"
+F 7 "https://lcsc.com/product-detail/Multilayer-Ceramic-Capacitors-MLCC-SMD-SMT_SAMSUNG_CL10A226MP8NUNE_22uF-226-20-10V_C86295.html" H 5800 2550 60  0001 C CNN "Distrib Link"
 F 8 "20%" H 5800 2550 60  0001 C CNN "Tolerance"
-F 9 "https://www.digikey.com/products/en/capacitors/ceramic-capacitors/60?k=&pkeyword=&pv1989=0&FV=380014%2C380016%2C380004%2C380009%2C400006%2C440013%2Cmu22%C2%B5F%7C2049%2Cffe0003c&quantity=0&ColumnSort=1000011&page=1&pageSize=500" H 5800 2550 60  0001 C CNN "Others"
+F 9 "https://lcsc.com/product-detail/Multilayer-Ceramic-Capacitors-MLCC-SMD-SMT_MuRata_ZRB18AR61A226ME01L_22uF-226-20-10V_C162690.html" H 5800 2550 60  0001 C CNN "Others"
 	1    5800 2550
 	1    0    0    -1
@@
 $Comp
 L C C1003
-U 1 1 5B1961EF
+U 1 1 5B3619FD
 P 6100 2550
 F 0 "C1003" H 6125 2650 50  0000 L CNN
 F 1 "22uF" H 6125 2450 50  0000 L CNN
-F 2 "Capacitors_SMD:C_0805" H 6138 2400 50  0001 C CNN
-F 3 "https://search.murata.co.jp/Ceramy/image/img/A01X/G101/ENG/GRM219R61C226ME15-01.pdf" H 6100 2550 50  0001 C CNN
-F 4 "Murata" H 6100 2550 60  0001 C CNN "MFG Name"
-F 5 "GRM219R61C226ME15L" H 6100 2550 60  0001 C CNN "MFG Part Num"
-F 6 "490-9952-1-ND" H 6100 2550 60  0001 C CNN "Distrib PN"
-F 7 "https://www.digikey.com/product-detail/en/murata-electronics-north-america/GRM219R61C226ME15L/490-9952-1-ND/5026415" H 6100 2550 60  0001 C CNN "Distrib Link"
+F 2 "Capacitors_SMD:C_0603" H 6138 2400 50  0001 C CNN
+F 3 "http://www.samsungsem.com/kr/support/product-search/mlcc/__icsFiles/afieldfile/2018/06/21/CL10A226MP8NUNE.pdf" H 6100 2550 50  0001 C CNN
+F 4 "Samsung" H 6100 2550 60  0001 C CNN "MFG Name"
+F 5 "CL10A226MP8NUNE" H 6100 2550 60  0001 C CNN "MFG Part Num"
+F 6 "C86295" H 6100 2550 60  0001 C CNN "Distrib PN"
+F 7 "https://lcsc.com/product-detail/Multilayer-Ceramic-Capacitors-MLCC-SMD-SMT_SAMSUNG_CL10A226MP8NUNE_22uF-226-20-10V_C86295.html" H 6100 2550 60  0001 C CNN "Distrib Link"
 F 8 "20%" H 6100 2550 60  0001 C CNN "Tolerance"
-F 9 "https://www.digikey.com/products/en/capacitors/ceramic-capacitors/60?k=&pkeyword=&pv1989=0&FV=380014%2C380016%2C380004%2C380009%2C400006%2C440013%2Cmu22%C2%B5F%7C2049%2Cffe0003c&quantity=0&ColumnSort=1000011&page=1&pageSize=500" H 6100 2550 60  0001 C CNN "Others"
+F 9 "https://lcsc.com/product-detail/Multilayer-Ceramic-Capacitors-MLCC-SMD-SMT_MuRata_ZRB18AR61A226ME01L_22uF-226-20-10V_C162690.html" H 6100 2550 60  0001 C CNN "Others"
 	1    6100 2550
 	1    0    0    -1
 $EndComp
-Text Notes 5800 1900 0    236  ~ 47
-μSD
 $EndSCHEMATC

Commit message: Update project files to KiCad 5.0.0
Parts:
- C1001, C1002, C1003, C1004: symbol C -> dvk-mx8m-bsb-rescue:C
- J1001: symbol Micro_SD_Card_Det_ALPS_SCHA -> dvk-mx8m-bsb:Micro_SD_Card_Det_ALPS_SCHA
- R1001, R1002, R1003, R1004: symbol R -> dvk-mx8m-bsb-rescue:R
Changed lines of the file:
@@
-EESchema Schematic File Version 2
-LIBS:power
-LIBS:device
-LIBS:switches
-LIBS:relays
-LIBS:motors
-LIBS:transistors
-LIBS:conn
-LIBS:linear
-LIBS:regul
-LIBS:74xx
-LIBS:cmos4000
-LIBS:adc-dac
-LIBS:memory
-LIBS:xilinx
-LIBS:microcontrollers
-LIBS:dsp
-LIBS:microchip
-LIBS:analog_switches
-LIBS:motorola
-LIBS:texas
-LIBS:intel
-LIBS:audio
-LIBS:interface
-LIBS:digital-audio
-LIBS:philips
-LIBS:display
-LIBS:cypress
-LIBS:siliconi
-LIBS:opto
-LIBS:atmel
-LIBS:contrib
-LIBS:valves
-LIBS:dvk-mx8m-bsb
+EESchema Schematic File Version 4
 LIBS:dvk-mx8m-bsb-cache
-EELAYER 25 0
+EELAYER 26 0
 EELAYER END
 $Descr A4 11693 8268
@@
 CONN_SD2_CD_B
 $Comp
-L GND #PWR0178
+L power:GND #PWR0178
 U 1 1 5AC9FCAE
 P 7400 4300
@@
 $EndComp
 $Comp
-L GND #PWR0179
+L power:GND #PWR0179
 U 1 1 5ACA0128
 P 5600 4300
@@
 $EndComp
 $Comp
-L GND #PWR0180
+L power:GND #PWR0180
 U 1 1 5ACA12D0
 P 6100 2800
@@
 $EndComp
 $Comp
-L 3V3_SD #PWR0181
+L dvk-mx8m-bsb:3V3_SD #PWR0181
 U 1 1 5AE8C9A8
 P 6100 2300
@@
 $EndComp
 $Comp
-L C C1004
+L dvk-mx8m-bsb-rescue:C C1004
 U 1 1 5AE8CA13
 P 6400 2550
@@
 	4250 3350 5650 3350
 $Comp
-L Micro_SD_Card_Det_ALPS_SCHA J1001
+L dvk-mx8m-bsb:Micro_SD_Card_Det_ALPS_SCHA J1001
 U 1 1 5AFA0CE0
 P 6550 3750
@@
 Connection ~ 5100 3550
 $Comp
-L R R1004
+L dvk-mx8m-bsb-rescue:R R1004
 U 1 1 5B32051A
 P 5450 3150
@@
 $EndComp
 $Comp
-L R R1003
+L dvk-mx8m-bsb-rescue:R R1003
 U 1 1 5B3204AF
 P 5100 3150
@@
 $EndComp
 $Comp
-L R R1002
+L dvk-mx8m-bsb-rescue:R R1002
 U 1 1 5B32045F
 P 4750 3150
@@
 	5450 3300 5450 3950
 $Comp
-L 3V3_SD #PWR0182
+L dvk-mx8m-bsb:3V3_SD #PWR0182
 U 1 1 5B09DC2A
 P 5100 2900
@@
 $EndComp
 $Comp
-L R R1001
+L dvk-mx8m-bsb-rescue:R R1001
 U 1 1 5B0D207F
 P 4450 3750
@@
 	4250 3750 4300 3750
 $Comp
-L C C1001
+L dvk-mx8m-bsb-rescue:C C1001
 U 1 1 5B0D22C2
 P 4650 4450
@@
 $EndComp
 $Comp
-L GND #PWR0183
+L power:GND #PWR0183
 U 1 1 5B0D2F89
 P 4650 4650
@@
 μSD
 $Comp
-L C C1002
+L dvk-mx8m-bsb-rescue:C C1002
 U 1 1 5B3619B2
 P 5800 2550
@@
 $EndComp
 $Comp
-L C C1003
+L dvk-mx8m-bsb-rescue:C C1003
 U 1 1 5B3619FD
 P 6100 2550

Commit message: Update the schematic symbols and footprints after upgrading to KiCad 5.0.0, fix all ERC and DRC violations after the new update/upgrade
Parts:
- C1001, C1002, C1003, C1004: footprint Capacitors_SMD:C_0603 -> Capacitor_SMD:C_0603_1608Metric; symbol dvk-mx8m-bsb-rescue:C -> Device:C
- R1001, R1002, R1003, R1004: footprint Resistors_SMD:R_0603 -> Resistor_SMD:R_0603_1608Metric; symbol dvk-mx8m-bsb-rescue:R -> Device:R
Changed lines of the file:
@@
 Sheet 10 24
 Title "uSD Card"
-Date "2018-06-18"
+Date "2018-07-17"
 Rev "v0.1.0"
 Comp "Copyright 2018 GNU GPLv3"
@@
 $EndComp
 $Comp
-L dvk-mx8m-bsb-rescue:C C1004
+L Device:C C1004
 U 1 1 5AE8CA13
 P 6400 2550
 F 0 "C1004" H 6425 2650 50  0000 L CNN
 F 1 "100nF" H 6425 2450 50  0000 L CNN
-F 2 "Capacitors_SMD:C_0603" H 6438 2400 50  0001 C CNN
+F 2 "Capacitor_SMD:C_0603_1608Metric" H 6438 2400 50  0001 C CNN
 F 3 "" H 6400 2550 50  0001 C CNN
 	1    6400 2550
@@
 Connection ~ 5100 3550
 $Comp
-L dvk-mx8m-bsb-rescue:R R1004
+L Device:R R1004
 U 1 1 5B32051A
 P 5450 3150
 F 0 "R1004" H 5625 3200 50  0000 C CNN
 F 1 "NC" H 5575 3100 50  0000 C CNN
-F 2 "Resistors_SMD:R_0603" V 5380 3150 50  0001 C CNN
+F 2 "Resistor_SMD:R_0603_1608Metric" V 5380 3150 50  0001 C CNN
 F 3 "https://www.seielect.com/Catalog/SEI-RMCF_RMCP.pdf" H 5450 3150 50  0001 C CNN
 F 4 "Stackpole" H 5450 3150 60  0001 C CNN "MFG Name"
@@
 $EndComp
 $Comp
-L dvk-mx8m-bsb-rescue:R R1003
+L Device:R R1003
 U 1 1 5B3204AF
 P 5100 3150
 F 0 "R1003" H 5275 3200 50  0000 C CNN
 F 1 "NC" H 5225 3100 50  0000 C CNN
-F 2 "Resistors_SMD:R_0603" V 5030 3150 50  0001 C CNN
+F 2 "Resistor_SMD:R_0603_1608Metric" V 5030 3150 50  0001 C CNN
 F 3 "https://www.seielect.com/Catalog/SEI-RMCF_RMCP.pdf" H 5100 3150 50  0001 C CNN
 F 4 "Stackpole" H 5100 3150 60  0001 C CNN "MFG Name"
@@
 $EndComp
 $Comp
-L dvk-mx8m-bsb-rescue:R R1002
+L Device:R R1002
 U 1 1 5B32045F
 P 4750 3150
 F 0 "R1002" H 4925 3200 50  0000 C CNN
 F 1 "NC" H 4875 3100 50  0000 C CNN
-F 2 "Resistors_SMD:R_0603" V 4680 3150 50  0001 C CNN
+F 2 "Resistor_SMD:R_0603_1608Metric" V 4680 3150 50  0001 C CNN
 F 3 "https://www.seielect.com/Catalog/SEI-RMCF_RMCP.pdf" H 4750 3150 50  0001 C CNN
 F 4 "Stackpole" H 4750 3150 60  0001 C CNN "MFG Name"
@@
 $EndComp
 $Comp
-L dvk-mx8m-bsb-rescue:R R1001
+L Device:R R1001
 U 1 1 5B0D207F
 P 4450 3750
 F 0 "R1001" V 4530 3750 50  0000 C CNN
 F 1 "0" V 4450 3750 50  0000 C CNN
-F 2 "Resistors_SMD:R_0603" V 4380 3750 50  0001 C CNN
+F 2 "Resistor_SMD:R_0603_1608Metric" V 4380 3750 50  0001 C CNN
 F 3 "" H 4450 3750 50  0001 C CNN
 	1    4450 3750
@@
 	4250 3750 4300 3750
 $Comp
-L dvk-mx8m-bsb-rescue:C C1001
+L Device:C C1001
 U 1 1 5B0D22C2
 P 4650 4450
 F 0 "C1001" H 4675 4550 50  0000 L CNN
 F 1 "NC" H 4675 4350 50  0000 L CNN
-F 2 "Capacitors_SMD:C_0603" H 4688 4300 50  0001 C CNN
+F 2 "Capacitor_SMD:C_0603_1608Metric" H 4688 4300 50  0001 C CNN
 F 3 "" H 4650 4450 50  0001 C CNN
 	1    4650 4450
@@
 μSD
 $Comp
-L dvk-mx8m-bsb-rescue:C C1002
+L Device:C C1002
 U 1 1 5B3619B2
 P 5800 2550
 F 0 "C1002" H 5825 2650 50  0000 L CNN
 F 1 "22uF" H 5825 2450 50  0000 L CNN
-F 2 "Capacitors_SMD:C_0603" H 5838 2400 50  0001 C CNN
+F 2 "Capacitor_SMD:C_0603_1608Metric" H 5838 2400 50  0001 C CNN
 F 3 "http://www.samsungsem.com/kr/support/product-search/mlcc/__icsFiles/afieldfile/2018/06/21/CL10A226MP8NUNE.pdf" H 5800 2550 50  0001 C CNN
 F 4 "Samsung" H 5800 2550 60  0001 C CNN "MFG Name"
@@
 $EndComp
 $Comp
-L dvk-mx8m-bsb-rescue:C C1003
+L Device:C C1003
 U 1 1 5B3619FD
 P 6100 2550
 F 0 "C1003" H 6125 2650 50  0000 L CNN
 F 1 "22uF" H 6125 2450 50  0000 L CNN
-F 2 "Capacitors_SMD:C_0603" H 6138 2400 50  0001 C CNN
+F 2 "Capacitor_SMD:C_0603_1608Metric" H 6138 2400 50  0001 C CNN
 F 3 "http://www.samsungsem.com/kr/support/product-search/mlcc/__icsFiles/afieldfile/2018/06/21/CL10A226MP8NUNE.pdf" H 6100 2550 50  0001 C CNN
 F 4 "Samsung" H 6100 2550 60  0001 C CNN "MFG Name"

Commit message: Reduce all 0603 resistor sizes to 0402
Parts:
- R1001, R1002, R1003, R1004: footprint Resistor_SMD:R_0603_1608Metric -> Resistor_SMD:R_0402_1005Metric
Changed lines of the file:
@@
 F 0 "R1004" H 5625 3200 50  0000 C CNN
 F 1 "NC" H 5575 3100 50  0000 C CNN
-F 2 "Resistor_SMD:R_0603_1608Metric" V 5380 3150 50  0001 C CNN
+F 2 "Resistor_SMD:R_0402_1005Metric" V 5380 3150 50  0001 C CNN
 F 3 "https://www.seielect.com/Catalog/SEI-RMCF_RMCP.pdf" H 5450 3150 50  0001 C CNN
 F 4 "Stackpole" H 5450 3150 60  0001 C CNN "MFG Name"
@@
 F 0 "R1003" H 5275 3200 50  0000 C CNN
 F 1 "NC" H 5225 3100 50  0000 C CNN
-F 2 "Resistor_SMD:R_0603_1608Metric" V 5030 3150 50  0001 C CNN
+F 2 "Resistor_SMD:R_0402_1005Metric" V 5030 3150 50  0001 C CNN
 F 3 "https://www.seielect.com/Catalog/SEI-RMCF_RMCP.pdf" H 5100 3150 50  0001 C CNN
 F 4 "Stackpole" H 5100 3150 60  0001 C CNN "MFG Name"
@@
 F 0 "R1002" H 4925 3200 50  0000 C CNN
 F 1 "NC" H 4875 3100 50  0000 C CNN
-F 2 "Resistor_SMD:R_0603_1608Metric" V 4680 3150 50  0001 C CNN
+F 2 "Resistor_SMD:R_0402_1005Metric" V 4680 3150 50  0001 C CNN
 F 3 "https://www.seielect.com/Catalog/SEI-RMCF_RMCP.pdf" H 4750 3150 50  0001 C CNN
 F 4 "Stackpole" H 4750 3150 60  0001 C CNN "MFG Name"
@@
 F 0 "R1001" V 4530 3750 50  0000 C CNN
 F 1 "0" V 4450 3750 50  0000 C CNN
-F 2 "Resistor_SMD:R_0603_1608Metric" V 4380 3750 50  0001 C CNN
+F 2 "Resistor_SMD:R_0402_1005Metric" V 4380 3750 50  0001 C CNN
 F 3 "" H 4450 3750 50  0001 C CNN
 	1    4450 3750

Commit message: Change all 0603 capacitors _EXCEPT_ the 2.2uF, 4.7uF, 8.2uF, 10uF, and 22uF caps to 0402
Parts:
- C1001, C1004: footprint Capacitor_SMD:C_0603_1608Metric -> Capacitor_SMD:C_0402_1005Metric
Changed lines of the file:
@@
 F 0 "C1004" H 6425 2650 50  0000 L CNN
 F 1 "100nF" H 6425 2450 50  0000 L CNN
-F 2 "Capacitor_SMD:C_0603_1608Metric" H 6438 2400 50  0001 C CNN
+F 2 "Capacitor_SMD:C_0402_1005Metric" H 6438 2400 50  0001 C CNN
 F 3 "" H 6400 2550 50  0001 C CNN
 	1    6400 2550
@@
 F 0 "C1001" H 4675 4550 50  0000 L CNN
 F 1 "NC" H 4675 4350 50  0000 L CNN
-F 2 "Capacitor_SMD:C_0603_1608Metric" H 4688 4300 50  0001 C CNN
+F 2 "Capacitor_SMD:C_0402_1005Metric" H 4688 4300 50  0001 C CNN
 F 3 "" H 4650 4450 50  0001 C CNN
 	1    4650 4450
