File: smartcard.sch (KiCad schematic (older format))
At the start: 10 parts, among them J2201 Smart_Card, U2201 SEC1110

Commit message: Update project files to KiCad 5.0.0
Parts:
- C2201, C2202, C2203, C2204, C2205: symbol C -> dvk-mx8m-bsb-rescue:C
- J2201: symbol SMART_CARD -> dvk-mx8m-bsb:SMART_CARD
- R2201, R2202, R2203: symbol R -> dvk-mx8m-bsb-rescue:R
- U2201: symbol SEC1110 -> dvk-mx8m-bsb:SEC1110
Changed lines of the file:
@@
-EESchema Schematic File Version 2
-LIBS:power
-LIBS:device
-LIBS:switches
-LIBS:relays
-LIBS:motors
-LIBS:transistors
-LIBS:conn
-LIBS:linear
-LIBS:regul
-LIBS:74xx
-LIBS:cmos4000
-LIBS:adc-dac
-LIBS:memory
-LIBS:xilinx
-LIBS:microcontrollers
-LIBS:dsp
-LIBS:microchip
-LIBS:analog_switches
-LIBS:motorola
-LIBS:texas
-LIBS:intel
-LIBS:audio
-LIBS:interface
-LIBS:digital-audio
-LIBS:philips
-LIBS:display
-LIBS:cypress
-LIBS:siliconi
-LIBS:opto
-LIBS:atmel
-LIBS:contrib
-LIBS:valves
-LIBS:dvk-mx8m-bsb
+EESchema Schematic File Version 4
 LIBS:dvk-mx8m-bsb-cache
-EELAYER 25 0
+EELAYER 26 0
 EELAYER END
 $Descr A4 11693 8268
@@
 SMARTCARD_D_N
 $Comp
-L 5V_P #PWR0378
+L dvk-mx8m-bsb:5V_P #PWR0378
 U 1 1 5B1F0A54
 P 6700 2450
@@
 $EndComp
 $Comp
-L C C2202
+L dvk-mx8m-bsb-rescue:C C2202
 U 1 1 5B1F1971
 P 6300 2800
@@
 $EndComp
 $Comp
-L GND #PWR0379
+L power:GND #PWR0379
 U 1 1 5B1F199A
 P 6300 3000
@@
 $EndComp
 $Comp
-L C C2204
+L dvk-mx8m-bsb-rescue:C C2204
 U 1 1 5B1F1CFA
 P 6700 2700
@@
 $EndComp
 $Comp
-L GND #PWR0380
+L power:GND #PWR0380
 U 1 1 5B1F1D4E
 P 6700 2900
@@
 $EndComp
 $Comp
-L R R2202
+L dvk-mx8m-bsb-rescue:R R2202
 U 1 1 5B1F2A2C
 P 6600 3600
@@
 $EndComp
 $Comp
-L R R2203
+L dvk-mx8m-bsb-rescue:R R2203
 U 1 1 5B1F2AD0
 P 6600 3700
@@
 NoConn ~ 6250 4550
 $Comp
-L R R2201
+L dvk-mx8m-bsb-rescue:R R2201
 U 1 1 5B20FE9D
 P 4500 4100
@@
 $EndComp
 $Comp
-L 5V_P #PWR0381
+L dvk-mx8m-bsb:5V_P #PWR0381
 U 1 1 5B20FF3B
 P 4500 3900
@@
 $EndComp
 $Comp
-L C C2201
+L dvk-mx8m-bsb-rescue:C C2201
 U 1 1 5B20FF65
 P 4500 4500
@@
 $EndComp
 $Comp
-L GND #PWR0382
+L power:GND #PWR0382
 U 1 1 5B20FFAF
 P 4500 4700
@@
 $EndComp
 $Comp
-L C C2203
+L dvk-mx8m-bsb-rescue:C C2203
 U 1 1 5B210DE6
 P 6500 3350
@@
 $EndComp
 $Comp
-L GND #PWR0383
+L power:GND #PWR0383
 U 1 1 5B210E33
 P 6300 3400
@@
 $EndComp
 $Comp
-L GND #PWR0384
+L power:GND #PWR0384
 U 1 1 5B21589D
 P 6300 4750
@@
 ISO/IEC 7816
 $Comp
-L SEC1110 U2201
+L dvk-mx8m-bsb:SEC1110 U2201
 U 1 1 5B265531
 P 5450 3600
@@
 $EndComp
 $Comp
-L SMART_CARD J2201
+L dvk-mx8m-bsb:SMART_CARD J2201
 U 1 1 5B26711A
 P 7650 3500
@@
 NoConn ~ 7150 3600
 $Comp
-L GND #PWR0385
+L power:GND #PWR0385
 U 1 1 5B27C54B
 P 7000 4150
@@
 Normally\nOpen
 $Comp
-L GND #PWR0386
+L power:GND #PWR0386
 U 1 1 5B296537
 P 8500 3600
@@
 	8650 3450 8450 3450
 $Comp
-L GND #PWR0387
+L power:GND #PWR0387
 U 1 1 5B29449E
 P 7700 4050
@@
 	7750 4000 7750 3950
 $Comp
-L GND #PWR0388
+L power:GND #PWR0388
 U 1 1 5B41E04B
 P 7250 2850
@@
 $EndComp
 $Comp
-L C C2205
+L dvk-mx8m-bsb-rescue:C C2205
 U 1 1 5B41E11A
 P 7250 2650

Commit message: Update the schematic symbols and footprints after upgrading to KiCad 5.0.0, fix all ERC and DRC violations after the new update/upgrade
Parts:
- C2201, C2202, C2203, C2204, C2205: footprint Capacitors_SMD:C_0603 -> Capacitor_SMD:C_0603_1608Metric; symbol dvk-mx8m-bsb-rescue:C -> Device:C
- R2201, R2202, R2203: footprint Resistors_SMD:R_0603 -> Resistor_SMD:R_0603_1608Metric; symbol dvk-mx8m-bsb-rescue:R -> Device:R
Changed lines of the file:
@@
 Sheet 22 24
 Title "Smart Card"
-Date "2018-06-18"
+Date "2018-07-17"
 Rev "v0.1.0"
 Comp "Copyright 2018 GNU GPLv3"
@@
 $EndComp
 $Comp
-L dvk-mx8m-bsb-rescue:C C2202
+L Device:C C2202
 U 1 1 5B1F1971
 P 6300 2800
 F 0 "C2202" H 6325 2900 50  0000 L CNN
 F 1 "1uF" H 6325 2700 50  0000 L CNN
-F 2 "Capacitors_SMD:C_0603" H 6338 2650 50  0001 C CNN
+F 2 "Capacitor_SMD:C_0603_1608Metric" H 6338 2650 50  0001 C CNN
 F 3 "" H 6300 2800 50  0001 C CNN
 	1    6300 2800
@@
 $EndComp
 $Comp
-L dvk-mx8m-bsb-rescue:C C2204
+L Device:C C2204
 U 1 1 5B1F1CFA
 P 6700 2700
 F 0 "C2204" H 6725 2800 50  0000 L CNN
 F 1 "1uF" H 6725 2600 50  0000 L CNN
-F 2 "Capacitors_SMD:C_0603" H 6738 2550 50  0001 C CNN
+F 2 "Capacitor_SMD:C_0603_1608Metric" H 6738 2550 50  0001 C CNN
 F 3 "" H 6700 2700 50  0001 C CNN
 	1    6700 2700
@@
 $EndComp
 $Comp
-L dvk-mx8m-bsb-rescue:R R2202
+L Device:R R2202
 U 1 1 5B1F2A2C
 P 6600 3600
 F 0 "R2202" V 6680 3600 50  0000 C CNN
 F 1 "0" V 6600 3600 50  0000 C CNN
-F 2 "Resistors_SMD:R_0603" V 6530 3600 50  0001 C CNN
+F 2 "Resistor_SMD:R_0603_1608Metric" V 6530 3600 50  0001 C CNN
 F 3 "" H 6600 3600 50  0001 C CNN
 	1    6600 3600
@@
 $EndComp
 $Comp
-L dvk-mx8m-bsb-rescue:R R2203
+L Device:R R2203
 U 1 1 5B1F2AD0
 P 6600 3700
 F 0 "R2203" V 6630 3930 50  0000 C CNN
 F 1 "33" V 6600 3700 50  0000 C CNN
-F 2 "Resistors_SMD:R_0603" V 6530 3700 50  0001 C CNN
+F 2 "Resistor_SMD:R_0603_1608Metric" V 6530 3700 50  0001 C CNN
 F 3 "" H 6600 3700 50  0001 C CNN
 	1    6600 3700
@@
 NoConn ~ 6250 4550
 $Comp
-L dvk-mx8m-bsb-rescue:R R2201
+L Device:R R2201
 U 1 1 5B20FE9D
 P 4500 4100
 F 0 "R2201" H 4675 4150 50  0000 C CNN
 F 1 "100k" H 4650 4050 50  0000 C CNN
-F 2 "Resistors_SMD:R_0603" V 4430 4100 50  0001 C CNN
+F 2 "Resistor_SMD:R_0603_1608Metric" V 4430 4100 50  0001 C CNN
 F 3 "" H 4500 4100 50  0001 C CNN
 	1    4500 4100
@@
 $EndComp
 $Comp
-L dvk-mx8m-bsb-rescue:C C2201
+L Device:C C2201
 U 1 1 5B20FF65
 P 4500 4500
 F 0 "C2201" H 4525 4600 50  0000 L CNN
 F 1 "100nF" H 4525 4400 50  0000 L CNN
-F 2 "Capacitors_SMD:C_0603" H 4538 4350 50  0001 C CNN
+F 2 "Capacitor_SMD:C_0603_1608Metric" H 4538 4350 50  0001 C CNN
 F 3 "" H 4500 4500 50  0001 C CNN
 	1    4500 4500
@@
 $EndComp
 $Comp
-L dvk-mx8m-bsb-rescue:C C2203
+L Device:C C2203
 U 1 1 5B210DE6
 P 6500 3350
 F 0 "C2203" V 6550 3400 50  0000 L CNN
 F 1 "1uF" V 6540 3170 50  0000 L CNN
-F 2 "Capacitors_SMD:C_0603" H 6538 3200 50  0001 C CNN
+F 2 "Capacitor_SMD:C_0603_1608Metric" H 6538 3200 50  0001 C CNN
 F 3 "" H 6500 3350 50  0001 C CNN
 	1    6500 3350
@@
 $EndComp
 $Comp
-L dvk-mx8m-bsb-rescue:C C2205
+L Device:C C2205
 U 1 1 5B41E11A
 P 7250 2650
 F 0 "C2205" H 7275 2750 50  0000 L CNN
 F 1 "100nF" H 7275 2550 50  0000 L CNN
-F 2 "Capacitors_SMD:C_0603" H 7288 2500 50  0001 C CNN
+F 2 "Capacitor_SMD:C_0603_1608Metric" H 7288 2500 50  0001 C CNN
 F 3 "" H 7250 2650 50  0001 C CNN
 	1    7250 2650

Commit message: Reduce all 0603 resistor sizes to 0402
Parts:
- R2201, R2202, R2203: footprint Resistor_SMD:R_0603_1608Metric -> Resistor_SMD:R_0402_1005Metric
Changed lines of the file:
@@
 F 0 "R2202" V 6680 3600 50  0000 C CNN
 F 1 "0" V 6600 3600 50  0000 C CNN
-F 2 "Resistor_SMD:R_0603_1608Metric" V 6530 3600 50  0001 C CNN
+F 2 "Resistor_SMD:R_0402_1005Metric" V 6530 3600 50  0001 C CNN
 F 3 "" H 6600 3600 50  0001 C CNN
 	1    6600 3600
@@
 F 0 "R2203" V 6630 3930 50  0000 C CNN
 F 1 "33" V 6600 3700 50  0000 C CNN
-F 2 "Resistor_SMD:R_0603_1608Metric" V 6530 3700 50  0001 C CNN
+F 2 "Resistor_SMD:R_0402_1005Metric" V 6530 3700 50  0001 C CNN
 F 3 "" H 6600 3700 50  0001 C CNN
 	1    6600 3700
@@
 F 0 "R2201" H 4675 4150 50  0000 C CNN
 F 1 "100k" H 4650 4050 50  0000 C CNN
-F 2 "Resistor_SMD:R_0603_1608Metric" V 4430 4100 50  0001 C CNN
+F 2 "Resistor_SMD:R_0402_1005Metric" V 4430 4100 50  0001 C CNN
 F 3 "" H 4500 4100 50  0001 C CNN
 	1    4500 4100

Commit message: Change all 0603 capacitors _EXCEPT_ the 2.2uF, 4.7uF, 8.2uF, 10uF, and 22uF caps to 0402
Parts:
- C2201, C2202, C2203, C2204, C2205: footprint Capacitor_SMD:C_0603_1608Metric -> Capacitor_SMD:C_0402_1005Metric
Changed lines of the file:
@@
 F 0 "C2202" H 6325 2900 50  0000 L CNN
 F 1 "1uF" H 6325 2700 50  0000 L CNN
-F 2 "Capacitor_SMD:C_0603_1608Metric" H 6338 2650 50  0001 C CNN
+F 2 "Capacitor_SMD:C_0402_1005Metric" H 6338 2650 50  0001 C CNN
 F 3 "" H 6300 2800 50  0001 C CNN
 	1    6300 2800
@@
 F 0 "C2204" H 6725 2800 50  0000 L CNN
 F 1 "1uF" H 6725 2600 50  0000 L CNN
-F 2 "Capacitor_SMD:C_0603_1608Metric" H 6738 2550 50  0001 C CNN
+F 2 "Capacitor_SMD:C_0402_1005Metric" H 6738 2550 50  0001 C CNN
 F 3 "" H 6700 2700 50  0001 C CNN
 	1    6700 2700
@@
 F 0 "C2201" H 4525 4600 50  0000 L CNN
 F 1 "100nF" H 4525 4400 50  0000 L CNN
-F 2 "Capacitor_SMD:C_0603_1608Metric" H 4538 4350 50  0001 C CNN
+F 2 "Capacitor_SMD:C_0402_1005Metric" H 4538 4350 50  0001 C CNN
 F 3 "" H 4500 4500 50  0001 C CNN
 	1    4500 4500
@@
 F 0 "C2203" V 6550 3400 50  0000 L CNN
 F 1 "1uF" V 6540 3170 50  0000 L CNN
-F 2 "Capacitor_SMD:C_0603_1608Metric" H 6538 3200 50  0001 C CNN
+F 2 "Capacitor_SMD:C_0402_1005Metric" H 6538 3200 50  0001 C CNN
 F 3 "" H 6500 3350 50  0001 C CNN
 	1    6500 3350
@@
 F 0 "C2205" H 7275 2750 50  0000 L CNN
 F 1 "100nF" H 7275 2550 50  0000 L CNN
-F 2 "Capacitor_SMD:C_0603_1608Metric" H 7288 2500 50  0001 C CNN
+F 2 "Capacitor_SMD:C_0402_1005Metric" H 7288 2500 50  0001 C CNN
 F 3 "" H 7250 2650 50  0001 C CNN
 	1    7250 2650

Commit message: Route USB2 to the hub chip's upstream port and re-order & route each of the downstream ports to their respective locations (smartcard, mPCIe, & M.2), place and route the HDMI fuse, schottky diodes, TVS diodes, capacitors, and pull-up resistors, route the rest of the HDMI's interface to the SoM (HPD & I2C), adjust the GNSS antenna's CPW width using the PCB manufacturer's recommendation from their calculations
The HDMI circuit should be complete now. The GNSS & WiFi+BT antennae should also be complete. The GNSS module's RX & TX lines need to be routed next.
Connections:
- wire segments 57 -> 61
Changed lines of the file:
@@
 	7000 4150 7000 3500
-Wire Wire Line
-	7150 3700 7150 3700
 Wire Wire Line
 	6900 3400 7150 3400
@@
 	6650 3350 6700 3350
 Wire Wire Line
-	6250 3200 7150 3200
+	6250 3200 6700 3200
 Wire Wire Line
 	4500 3950 4500 3900
@@
 	4500 4700 4500 4650
 Wire Wire Line
-	4500 4250 4500 4350
+	4500 4250 4500 4300
 Wire Wire Line
 	6450 3700 6250 3700
@@
 	6250 2500 6700 2500
 Wire Wire Line
-	6700 2450 6700 2550
+	6700 2450 6700 2500
 Wire Wire Line
 	6300 3000 6300 2950
@@
 	7650 3950 7650 4000
 Wire Wire Line
-	7650 4000 7750 4000
+	7650 4000 7700 4000
 Wire Wire Line
 	7750 4000 7750 3950
@@
 Wire Wire Line
 	8500 3550 8500 3600
+Wire Wire Line
+	6700 3200 7100 3200
+Wire Wire Line
+	4500 4300 4500 4350
+Wire Wire Line
+	6700 2500 6700 2550
+Wire Wire Line
+	7100 3200 7150 3200
+Wire Wire Line
+	7700 4000 7750 4000
 $EndSCHEMATC
