File: wwan_mpcie.sch (KiCad schematic (older format))
At the start: 53 parts, among them J1501 u.FL, J1502 u.FL, J1503 mPCIe, J1504 Micro_SIM_Card, Q1501 FDV301N, Q1502 MMBT2222A, SW1501 WWAN_HKS, U1501 NTB0104GU12, U1502 NUP5120, U1503 74LVC1G86, U1504 74LVC1G08

Commit message: Update the schematic symbols and footprints after upgrading to KiCad 5.0.0, fix all ERC and DRC violations after the new update/upgrade
Parts:
- AE1501, AE1502: symbol dvk-mx8m-bsb-rescue:Antenna_Shield -> Device:Antenna_Shield
- C1501, C1502, C1503: footprint Capacitors_Tantalum_SMD:CP_Tantalum_Case-D_EIA-7343-31_Reflow -> Capacitor_Tantalum_SMD:CP_EIA-7343-31_Kemet-D; symbol dvk-mx8m-bsb-rescue:CP1 -> Device:CP1
- C1504, C1505, C1506, C1507, C1508, C1509, C1510, C1511, C1512, C1513, C1514, C1515, C1516, C1517, C1518, C1519, C1520, C1521, C1522, C1523, C1524: footprint Capacitors_SMD:C_0603 -> Capacitor_SMD:C_0603_1608Metric; symbol dvk-mx8m-bsb-rescue:C -> Device:C
- D1501: symbol dvk-mx8m-bsb-rescue:D_TVS_ALT -> Device:D_TVS_ALT
- D1502: symbol dvk-mx8m-bsb-rescue:D_Schottky_ALT -> Device:D_Schottky_ALT
- J1501, J1502: symbol dvk-mx8m-bsb-rescue:Conn_Coaxial -> Connector:Conn_Coaxial
- Q1501: symbol dvk-mx8m-bsb-rescue:Q_NMOS_GSD -> Device:Q_NMOS_GSD
- Q1502: footprint TO_SOT_Packages_SMD:SOT-23 -> Package_TO_SOT_SMD:SOT-23; symbol dvk-mx8m-bsb-rescue:Q_NPN_BEC -> Device:Q_NPN_BEC
- R1501, R1502, R1503, R1504, R1505, R1506, R1507, R1508, R1509, R1510, R1511: footprint Resistors_SMD:R_0603 -> Resistor_SMD:R_0603_1608Metric; symbol dvk-mx8m-bsb-rescue:R -> Device:R
- SW1501: symbol dvk-mx8m-bsb-rescue:SW_DPDT_x2 -> Switch:SW_DPDT_x2
- U1501: symbol dvk-mx8m-bsb-rescue:TXB0104RUT -> Logic_LevelTranslator:TXB0104RUT
Connections:
- wire segments 198 -> 279

Commit message: Reduce all 0603 resistor sizes to 0402
Parts:
- R1501, R1502, R1503, R1504, R1505, R1506, R1507, R1508, R1509, R1510, R1511: footprint Resistor_SMD:R_0603_1608Metric -> Resistor_SMD:R_0402_1005Metric
Changed lines of the file:
@@
 F 0 "R1506" H 7275 4550 50  0000 C CNN
 F 1 "15k" H 7225 4450 50  0000 C CNN
-F 2 "Resistor_SMD:R_0603_1608Metric" V 7030 4500 50  0001 C CNN
+F 2 "Resistor_SMD:R_0402_1005Metric" V 7030 4500 50  0001 C CNN
 F 3 "" H 7100 4500 50  0001 C CNN
 	1    7100 4500
@@
 F 0 "R1501" H 1925 6700 50  0000 C CNN
 F 1 "10k" H 1875 6600 50  0000 C CNN
-F 2 "Resistor_SMD:R_0603_1608Metric" V 1680 6650 50  0001 C CNN
+F 2 "Resistor_SMD:R_0402_1005Metric" V 1680 6650 50  0001 C CNN
 F 3 "https://www.seielect.com/Catalog/SEI-RMCF_RMCP.pdf" H 1750 6650 50  0001 C CNN
 F 4 "Stackpole" H 1750 6650 60  0001 C CNN "MFG Name"
@@
 F 0 "R1502" H 2425 6700 50  0000 C CNN
 F 1 "10k" H 2375 6600 50  0000 C CNN
-F 2 "Resistor_SMD:R_0603_1608Metric" V 2180 6650 50  0001 C CNN
+F 2 "Resistor_SMD:R_0402_1005Metric" V 2180 6650 50  0001 C CNN
 F 3 "https://www.seielect.com/Catalog/SEI-RMCF_RMCP.pdf" H 2250 6650 50  0001 C CNN
 F 4 "Stackpole" H 2250 6650 60  0001 C CNN "MFG Name"
@@
 F 0 "R1511" H 10375 1650 50  0000 C CNN
 F 1 "100k" H 10350 1550 50  0000 C CNN
-F 2 "Resistor_SMD:R_0603_1608Metric" V 10130 1600 50  0001 C CNN
+F 2 "Resistor_SMD:R_0402_1005Metric" V 10130 1600 50  0001 C CNN
 F 3 "" H 10200 1600 50  0001 C CNN
 	1    10200 1600
@@
 F 0 "R1509" V 9925 1800 50  0000 C CNN
 F 1 "100k" V 9750 1800 50  0000 C CNN
-F 2 "Resistor_SMD:R_0603_1608Metric" V 9780 1800 50  0001 C CNN
+F 2 "Resistor_SMD:R_0402_1005Metric" V 9780 1800 50  0001 C CNN
 F 3 "" H 9850 1800 50  0001 C CNN
 	1    9850 1800
@@
 F 0 "R1510" H 10275 3700 50  0000 C CNN
 F 1 "10k" H 10225 3600 50  0000 C CNN
-F 2 "Resistor_SMD:R_0603_1608Metric" V 10030 3650 50  0001 C CNN
+F 2 "Resistor_SMD:R_0402_1005Metric" V 10030 3650 50  0001 C CNN
 F 3 "https://www.seielect.com/Catalog/SEI-RMCF_RMCP.pdf" H 10100 3650 50  0001 C CNN
 F 4 "Stackpole" H 10100 3650 60  0001 C CNN "MFG Name"
@@
 F 0 "R1507" H 8525 3500 50  0000 C CNN
 F 1 "10k" H 8475 3400 50  0000 C CNN
-F 2 "Resistor_SMD:R_0603_1608Metric" V 8280 3450 50  0001 C CNN
+F 2 "Resistor_SMD:R_0402_1005Metric" V 8280 3450 50  0001 C CNN
 F 3 "https://www.seielect.com/Catalog/SEI-RMCF_RMCP.pdf" H 8350 3450 50  0001 C CNN
 F 4 "Stackpole" H 8350 3450 60  0001 C CNN "MFG Name"
@@
 F 0 "R1508" V 8630 3650 50  0000 C CNN
 F 1 "NC" V 8450 3650 50  0000 C CNN
-F 2 "Resistor_SMD:R_0603_1608Metric" V 8480 3650 50  0001 C CNN
+F 2 "Resistor_SMD:R_0402_1005Metric" V 8480 3650 50  0001 C CNN
 F 3 "" H 8550 3650 50  0001 C CNN
 	1    8550 3650
@@
 F 0 "R1504" V 6925 4050 50  0000 C CNN
 F 1 "4.7k" V 6850 4050 50  0000 C CNN
-F 2 "Resistor_SMD:R_0603_1608Metric" V 6780 4050 50  0001 C CNN
+F 2 "Resistor_SMD:R_0402_1005Metric" V 6780 4050 50  0001 C CNN
 F 3 "" H 6850 4050 50  0001 C CNN
 	1    6850 4050
@@
 F 0 "R1505" V 7075 3450 50  0000 C CNN
 F 1 "4.7k" V 7000 3450 50  0000 C CNN
-F 2 "Resistor_SMD:R_0603_1608Metric" V 6930 3450 50  0001 C CNN
+F 2 "Resistor_SMD:R_0402_1005Metric" V 6930 3450 50  0001 C CNN
 F 3 "" H 7000 3450 50  0001 C CNN
 	1    7000 3450
@@
 F 0 "R1503" V 6675 3700 50  0000 C CNN
 F 1 "47k" V 6600 3700 50  0000 C CNN
-F 2 "Resistor_SMD:R_0603_1608Metric" V 6530 3700 50  0001 C CNN
+F 2 "Resistor_SMD:R_0402_1005Metric" V 6530 3700 50  0001 C CNN
 F 3 "" H 6600 3700 50  0001 C CNN
 	1    6600 3700

Commit message: Change all 0603 capacitors _EXCEPT_ the 2.2uF, 4.7uF, 8.2uF, 10uF, and 22uF caps to 0402
Parts:
- C1504, C1505, C1506, C1507, C1508, C1509, C1510, C1511, C1512, C1513, C1514, C1515, C1516, C1517, C1518, C1519, C1520, C1521, C1522, C1523, C1524: footprint Capacitor_SMD:C_0603_1608Metric -> Capacitor_SMD:C_0402_1005Metric
Changed lines of the file:
@@
 F 0 "C1510" H 3600 1800 50  0000 L CNN
 F 1 "6.8pF" H 3625 1600 50  0000 L CNN
-F 2 "Capacitor_SMD:C_0603_1608Metric" H 3638 1550 50  0001 C CNN
+F 2 "Capacitor_SMD:C_0402_1005Metric" H 3638 1550 50  0001 C CNN
 F 3 "" H 3600 1700 50  0001 C CNN
 	1    3600 1700
@@
 F 0 "C1509" H 3350 1800 50  0000 L CNN
 F 1 "8.2pF" H 3375 1600 50  0000 L CNN
-F 2 "Capacitor_SMD:C_0603_1608Metric" H 3388 1550 50  0001 C CNN
+F 2 "Capacitor_SMD:C_0402_1005Metric" H 3388 1550 50  0001 C CNN
 F 3 "" H 3350 1700 50  0001 C CNN
 	1    3350 1700
@@
 F 0 "C1520" H 7125 5000 50  0000 L CNN
 F 1 "22pF" H 7125 4800 50  0000 L CNN
-F 2 "Capacitor_SMD:C_0603_1608Metric" H 7138 4750 50  0001 C CNN
+F 2 "Capacitor_SMD:C_0402_1005Metric" H 7138 4750 50  0001 C CNN
 F 3 "" H 7100 4900 50  0001 C CNN
 	1    7100 4900
@@
 F 0 "C1524" H 9975 4750 50  0000 L CNN
 F 1 "NC" H 9975 4550 50  0000 L CNN
-F 2 "Capacitor_SMD:C_0603_1608Metric" H 9988 4500 50  0001 C CNN
+F 2 "Capacitor_SMD:C_0402_1005Metric" H 9988 4500 50  0001 C CNN
 F 3 "" H 9950 4650 50  0001 C CNN
 	1    9950 4650
@@
 F 0 "C1519" H 6825 5000 50  0000 L CNN
 F 1 "NC" H 6825 4800 50  0000 L CNN
-F 2 "Capacitor_SMD:C_0603_1608Metric" H 6838 4750 50  0001 C CNN
+F 2 "Capacitor_SMD:C_0402_1005Metric" H 6838 4750 50  0001 C CNN
 F 3 "" H 6800 4900 50  0001 C CNN
 	1    6800 4900
@@
 F 0 "C1518" H 6525 5000 50  0000 L CNN
 F 1 "NC" H 6525 4800 50  0000 L CNN
-F 2 "Capacitor_SMD:C_0603_1608Metric" H 6538 4750 50  0001 C CNN
+F 2 "Capacitor_SMD:C_0402_1005Metric" H 6538 4750 50  0001 C CNN
 F 3 "" H 6500 4900 50  0001 C CNN
 	1    6500 4900
@@
 F 0 "C1517" H 6225 5000 50  0000 L CNN
 F 1 "1uF" H 6225 4800 50  0000 L CNN
-F 2 "Capacitor_SMD:C_0603_1608Metric" H 6238 4750 50  0001 C CNN
+F 2 "Capacitor_SMD:C_0402_1005Metric" H 6238 4750 50  0001 C CNN
 F 3 "" H 6200 4900 50  0001 C CNN
 	1    6200 4900
@@
 F 0 "C1514" H 5825 5000 50  0000 L CNN
 F 1 "33pF" H 5825 4800 50  0000 L CNN
-F 2 "Capacitor_SMD:C_0603_1608Metric" H 5838 4750 50  0001 C CNN
+F 2 "Capacitor_SMD:C_0402_1005Metric" H 5838 4750 50  0001 C CNN
 F 3 "" H 5800 4900 50  0001 C CNN
 	1    5800 4900
@@
 F 0 "C1513" H 5525 5950 50  0000 L CNN
 F 1 "10nF" H 5525 5750 50  0000 L CNN
-F 2 "Capacitor_SMD:C_0603_1608Metric" H 5538 5700 50  0001 C CNN
+F 2 "Capacitor_SMD:C_0402_1005Metric" H 5538 5700 50  0001 C CNN
 F 3 "" H 5500 5850 50  0001 C CNN
 	1    5500 5850
@@
 F 0 "C1515" H 5825 5950 50  0000 L CNN
 F 1 "1uF" H 5825 5750 50  0000 L CNN
-F 2 "Capacitor_SMD:C_0603_1608Metric" H 5838 5700 50  0001 C CNN
+F 2 "Capacitor_SMD:C_0402_1005Metric" H 5838 5700 50  0001 C CNN
 F 3 "" H 5800 5850 50  0001 C CNN
 	1    5800 5850
@@
 F 0 "C1512" H 4075 5950 50  0000 L CNN
 F 1 "10nF" H 4075 5750 50  0000 L CNN
-F 2 "Capacitor_SMD:C_0603_1608Metric" H 4088 5700 50  0001 C CNN
+F 2 "Capacitor_SMD:C_0402_1005Metric" H 4088 5700 50  0001 C CNN
 F 3 "" H 4050 5850 50  0001 C CNN
 	1    4050 5850
@@
 F 0 "C1511" H 3775 5950 50  0000 L CNN
 F 1 "1uF" H 3775 5750 50  0000 L CNN
-F 2 "Capacitor_SMD:C_0603_1608Metric" H 3788 5700 50  0001 C CNN
+F 2 "Capacitor_SMD:C_0402_1005Metric" H 3788 5700 50  0001 C CNN
 F 3 "" H 3750 5850 50  0001 C CNN
 	1    3750 5850
@@
 F 0 "C1507" H 2850 1800 50  0000 L CNN
 F 1 "33pF" H 2875 1600 50  0000 L CNN
-F 2 "Capacitor_SMD:C_0603_1608Metric" H 2888 1550 50  0001 C CNN
+F 2 "Capacitor_SMD:C_0402_1005Metric" H 2888 1550 50  0001 C CNN
 F 3 "" H 2850 1700 50  0001 C CNN
 	1    2850 1700
@@
 F 0 "C1506" H 2600 1800 50  0000 L CNN
 F 1 "39pF" H 2625 1600 50  0000 L CNN
-F 2 "Capacitor_SMD:C_0603_1608Metric" H 2638 1550 50  0001 C CNN
+F 2 "Capacitor_SMD:C_0402_1005Metric" H 2638 1550 50  0001 C CNN
 F 3 "" H 2600 1700 50  0001 C CNN
 	1    2600 1700
@@
 F 0 "C1505" H 2350 1800 50  0000 L CNN
 F 1 "100nF" H 2350 1600 50  0000 L CNN
-F 2 "Capacitor_SMD:C_0603_1608Metric" H 2388 1550 50  0001 C CNN
+F 2 "Capacitor_SMD:C_0402_1005Metric" H 2388 1550 50  0001 C CNN
 F 3 "" H 2350 1700 50  0001 C CNN
 	1    2350 1700
@@
 F 0 "C1504" H 2100 1850 50  0000 L CNN
 F 1 "1uF" H 2125 1600 50  0000 L CNN
-F 2 "Capacitor_SMD:C_0603_1608Metric" H 2138 1550 50  0001 C CNN
+F 2 "Capacitor_SMD:C_0402_1005Metric" H 2138 1550 50  0001 C CNN
 F 3 "" H 2100 1700 50  0001 C CNN
 	1    2100 1700
@@
 F 0 "C1522" H 8725 1650 50  0000 L CNN
 F 1 "100nF" H 8725 1450 50  0000 L CNN
-F 2 "Capacitor_SMD:C_0603_1608Metric" H 8738 1400 50  0001 C CNN
+F 2 "Capacitor_SMD:C_0402_1005Metric" H 8738 1400 50  0001 C CNN
 F 3 "" H 8700 1550 50  0001 C CNN
 	1    8700 1550
@@
 F 0 "C1523" H 9625 2100 50  0000 L CNN
 F 1 "1uF" H 9625 1900 50  0000 L CNN
-F 2 "Capacitor_SMD:C_0603_1608Metric" H 9638 1850 50  0001 C CNN
+F 2 "Capacitor_SMD:C_0402_1005Metric" H 9638 1850 50  0001 C CNN
 F 3 "" H 9600 2000 50  0001 C CNN
 	1    9600 2000
@@
 F 0 "C1521" H 7975 3200 50  0000 L CNN
 F 1 "100nF" H 8000 3000 50  0000 L CNN
-F 2 "Capacitor_SMD:C_0603_1608Metric" H 7988 2950 50  0001 C CNN
+F 2 "Capacitor_SMD:C_0402_1005Metric" H 7988 2950 50  0001 C CNN
 F 3 "" H 7950 3100 50  0001 C CNN
 	1    7950 3100
@@
 F 0 "C1508" H 3100 1800 50  0000 L CNN
 F 1 "18pF" H 3125 1600 50  0000 L CNN
-F 2 "Capacitor_SMD:C_0603_1608Metric" H 3138 1550 50  0001 C CNN
+F 2 "Capacitor_SMD:C_0402_1005Metric" H 3138 1550 50  0001 C CNN
 F 3 "" H 3100 1700 50  0001 C CNN
 	1    3100 1700
@@
 F 0 "C1516" H 6200 3525 50  0000 L CNN
 F 1 "100nF" H 6200 3375 50  0000 L CNN
-F 2 "Capacitor_SMD:C_0603_1608Metric" H 6238 3300 50  0001 C CNN
+F 2 "Capacitor_SMD:C_0402_1005Metric" H 6238 3300 50  0001 C CNN
 F 3 "" H 6200 3450 50  0001 C CNN
 	1    6200 3450

Commit message: Add WiFi+BT antenna footprint, add pi matching circuit to the WiFi+BT antennas' feedlines, increment the capacitor part numbers on page 18 after adding the new (NC) feedline caps and make the respective changes to the reference designators in the BoM
Parts:
- AE1501, AE1502: footprint dvk-mx8m-bsb:placeholder_WLAN+BT_antenna -> dvk-mx8m-bsb:placeholder_WWAN_antenna
Changed lines of the file:
@@
 F 0 "AE1501" H 1300 2625 50  0000 R CNN
 F 1 "Antenna" H 1300 2550 50  0000 R CNN
-F 2 "dvk-mx8m-bsb:placeholder_WLAN+BT_antenna" H 950 2600 50  0001 C CNN
+F 2 "dvk-mx8m-bsb:placeholder_WWAN_antenna" H 950 2600 50  0001 C CNN
 F 3 "https://www.fractusantennas.com/files/UM_FR05_S1_NO_1_004.pdf" H 950 2600 50  0001 C CNN
 	1    950  2500
@@
 F 0 "AE1502" H 1300 4775 50  0000 R CNN
 F 1 "Antenna" H 1300 4700 50  0000 R CNN
-F 2 "dvk-mx8m-bsb:placeholder_WLAN+BT_antenna" H 950 4750 50  0001 C CNN
+F 2 "dvk-mx8m-bsb:placeholder_WWAN_antenna" H 950 4750 50  0001 C CNN
 F 3 "https://www.fractusantennas.com/files/UM_FR05_S1_NO_1_004.pdf" H 950 4750 50  0001 C CNN
 	1    950  4650

Commit message: Use MHF4 instead of U.FL connectors on the WiFi+BT antennae
Parts:
- J1501, J1502: value u.FL -> U.FL
Changed lines of the file:
@@
 P 1300 2850
 F 0 "J1501" H 1310 2970 50  0000 C CNN
-F 1 "u.FL" H 1500 2850 50  0000 C CNN
+F 1 "U.FL" H 1500 2850 50  0000 C CNN
 F 2 "dvk-mx8m-bsb:U.FL_Hirose_U.FL-R-SMT-1_Vertical" H 1300 2850 50  0001 C CNN
 F 3 "https://linxtechnologies.com/wp/wp-content/uploads/conufl001-smd.pdf" H 1300 2850 50  0001 C CNN
@@
 P 1300 5000
 F 0 "J1502" H 1310 5120 50  0000 C CNN
-F 1 "u.FL" H 1500 5000 50  0000 C CNN
+F 1 "U.FL" H 1500 5000 50  0000 C CNN
 F 2 "dvk-mx8m-bsb:U.FL_Hirose_U.FL-R-SMT-1_Vertical" H 1300 5000 50  0001 C CNN
 F 3 "https://linxtechnologies.com/wp/wp-content/uploads/conufl001-smd.pdf" H 1300 5000 50  0001 C CNN

Commit message: Add ANT-LTE-CER-T as the baseband modem antenna into the schematic and BoM, update the layout accordingly
Parts:
- removed AE1502: Antenna, dvk-mx8m-bsb:placeholder_WWAN_antenna, symbol Device:Antenna_Shield
- removed CBL1502: Coax_cable_ufl_ufl, dvk-mx8m-bsb:Coax_Cable_Straight_4cm, symbol dvk-mx8m-bsb:Coax_cable_ufl_ufl
- removed J1502: U.FL, dvk-mx8m-bsb:U.FL_Hirose_U.FL-R-SMT-1_Vertical, symbol Connector:Conn_Coaxial
- AE1501: value Antenna -> ANT-LTE-CER-T; Distrib Link (none) -> https://www.mouser.com/ProductDetail/Linx-Technologies/ANT-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; Distrib PN (none) -> 712-ANT-LTE-CER-T; MFG Name (none) -> Linx; MFG Part Num (none) -> ANT-LTE-CER-T; Others (none) -> https://www.mouser.com/Passive-Components/Antennas/_/N-8w0f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; Tolerance (none) -> -
- renumbered J1503 to J1502, J1504 to J1503
Connections:
- wire segments 279 -> 275
Other:
- note removed: "TODO:\nAssign antennae\nfootprints"

Commit message: Update the WWAN/BB antenna to use the Antenova SR4L034-R antenna
Parts:
- AE1501: value ANT-LTE-CER-T -> SR4L034-R; footprint dvk-mx8m-bsb:placeholder_WWAN_antenna -> dvk-mx8m-bsb:SR4L034-R; Distrib Link https://www.mouser.com/ProductDetail/Linx-Technologies/ANT-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 -> https://www.arrow.com/en/products/sr4l034-r/antenova; Distrib PN 712-ANT-LTE-CER-T -> SR4L034-R; MFG Name Linx -> Antenova; MFG Part Num ANT-LTE-CER-T -> SR4L034-R; Others https://www.mouser.com/Passive-Components/Antennas/_/N-8w0f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 -> https://octopart.com/search?q=SR4L034-R&start=0
Changed lines of the file:
@@
 L power:GND #PWR01503
 U 1 1 5B118C1F
-P 1550 3050
-F 0 "#PWR01503" H 1550 2800 50  0001 C CNN
-F 1 "GND" H 1550 2900 50  0000 C CNN
-F 2 "" H 1550 3050 50  0001 C CNN
-F 3 "" H 1550 3050 50  0001 C CNN
-	1    1550 3050
+P 1400 3100
+F 0 "#PWR01503" H 1400 2850 50  0001 C CNN
+F 1 "GND" H 1400 2950 50  0000 C CNN
+F 2 "" H 1400 3100 50  0001 C CNN
+F 3 "" H 1400 3100 50  0001 C CNN
+	1    1400 3100
 	1    0    0    -1
 $EndComp
@@
 L Connector:Conn_Coaxial J1501
 U 1 1 5B3301D0
-P 1550 2800
-F 0 "J1501" H 1560 2920 50  0000 C CNN
-F 1 "U.FL" H 1750 2800 50  0000 C CNN
-F 2 "dvk-mx8m-bsb:U.FL_Hirose_U.FL-R-SMT-1_Vertical" H 1550 2800 50  0001 C CNN
-F 3 "https://linxtechnologies.com/wp/wp-content/uploads/conufl001-smd.pdf" H 1550 2800 50  0001 C CNN
-F 4 "Linx" H 1550 2800 60  0001 C CNN "MFG Name"
-F 5 "CONUFL001-SMD-T" H 1550 2800 60  0001 C CNN "MFG Part Num"
-F 6 "712-CONUFL001-SMD-T" H 1550 2800 60  0001 C CNN "Distrib PN"
-F 7 "https://www.mouser.com/ProductDetail/Linx-Technologies/CONUFL001-SMD-T?qs=%2fha2pyFaduivK93xHKUivxg4VjfDQlObuMZMwyaL26SpKX%252bySjigOg%3d%3d" H 1550 2800 60  0001 C CNN "Distrib Link"
-F 8 "-" H 1550 2800 60  0001 C CNN "Tolerance"
-F 9 "https://octopart.com/search?q=CONUFL001-SMD-T&oq=CONUFL001-SMD-T&start=0" H 1550 2800 60  0001 C CNN "Others"
-	1    1550 2800
+P 1400 2850
+F 0 "J1501" H 1410 2970 50  0000 C CNN
+F 1 "U.FL" H 1600 2850 50  0000 C CNN
+F 2 "dvk-mx8m-bsb:U.FL_Hirose_U.FL-R-SMT-1_Vertical" H 1400 2850 50  0001 C CNN
+F 3 "https://linxtechnologies.com/wp/wp-content/uploads/conufl001-smd.pdf" H 1400 2850 50  0001 C CNN
+F 4 "Linx" H 1400 2850 60  0001 C CNN "MFG Name"
+F 5 "CONUFL001-SMD-T" H 1400 2850 60  0001 C CNN "MFG Part Num"
+F 6 "712-CONUFL001-SMD-T" H 1400 2850 60  0001 C CNN "Distrib PN"
+F 7 "https://www.mouser.com/ProductDetail/Linx-Technologies/CONUFL001-SMD-T?qs=%2fha2pyFaduivK93xHKUivxg4VjfDQlObuMZMwyaL26SpKX%252bySjigOg%3d%3d" H 1400 2850 60  0001 C CNN "Distrib Link"
+F 8 "-" H 1400 2850 60  0001 C CNN "Tolerance"
+F 9 "https://octopart.com/search?q=CONUFL001-SMD-T&oq=CONUFL001-SMD-T&start=0" H 1400 2850 60  0001 C CNN "Others"
+	1    1400 2850
 	1    0    0    -1
 $EndComp
@@
 L dvk-mx8m-bsb:ModemCard MOD1501
 U 1 1 5B2C06BF
-P 2800 3200
-F 0 "MOD1501" H 2625 3600 60  0000 C CNN
-F 1 "ModemCard" H 2625 3475 60  0000 C CNN
-F 2 "dvk-mx8m-bsb:mpcie-outline" H 3375 3450 60  0001 C CNN
-F 3 "https://cloud.puri.sm/s/iSg345Zb5Fyd354" H 3375 3450 60  0001 C CNN
-	1    2800 3200
+P 2650 3250
+F 0 "MOD1501" H 2475 3650 60  0000 C CNN
+F 1 "ModemCard" H 2475 3525 60  0000 C CNN
+F 2 "dvk-mx8m-bsb:mpcie-outline" H 3225 3500 60  0001 C CNN
+F 3 "https://cloud.puri.sm/s/iSg345Zb5Fyd354" H 3225 3500 60  0001 C CNN
+	1    2650 3250
 	1    0    0    -1
 $EndComp
@@
 	1600 1500 1600 1550
 Wire Wire Line
-	1550 3000 1550 3050
+	1400 3050 1400 3100
 Wire Wire Line
 	4600 5650 4600 6000
@@
 L dvk-mx8m-bsb:Coax_cable_ufl_ufl CBL1501
 U 1 1 5B2DDE6A
-P 2300 2550
-F 0 "CBL1501" H 1825 2675 60  0000 C CNN
-F 1 "Coax_cable_ufl_ufl" H 2500 2675 60  0000 C CNN
-F 2 "dvk-mx8m-bsb:Coax_Cable_Straight_4cm" H 2500 2550 60  0001 C CNN
-F 3 "" H 2500 2550 60  0001 C CNN
-	1    2300 2550
+P 2150 2600
+F 0 "CBL1501" H 1675 2725 60  0000 C CNN
+F 1 "Coax_cable_ufl_ufl" H 2350 2725 60  0000 C CNN
+F 2 "dvk-mx8m-bsb:Coax_Cable_Straight_4cm" H 2350 2600 60  0001 C CNN
+F 3 "" H 2350 2600 60  0001 C CNN
+	1    2150 2600
 	1    0    0    -1
 $EndComp
@@
 L Device:Antenna_Shield AE1501
 U 1 1 5B383934
-P 1200 2450
-F 0 "AE1501" H 1550 2550 50  0000 R CNN
-F 1 "ANT-LTE-CER-T" H 1900 2450 50  0000 R CNN
-F 2 "dvk-mx8m-bsb:placeholder_WWAN_antenna" H 1200 2550 50  0001 C CNN
-F 3 "https://linxtechnologies.com/wp/wp-content/uploads/ant-lte-cer.pdf" H 1200 2550 50  0001 C CNN
-F 4 "Linx" H 1200 2450 50  0001 C CNN "MFG Name"
-F 5 "ANT-LTE-CER-T" H 1200 2450 50  0001 C CNN "MFG Part Num"
-F 6 "712-ANT-LTE-CER-T" H 1200 2450 50  0001 C CNN "Distrib PN"
-F 7 "https://www.mouser.com/ProductDetail/Linx-Technologies/ANT-LTE-CER-T?qs=F5EMLAvA7IB7cQaKyhfEiQ%3d%3d" H 1200 2450 50  0001 C CNN "Distrib Link"
-F 8 "-" H 1200 2450 50  0001 C CNN "Tolerance"
-F 9 "https://www.mouser.com/Passive-Components/Antennas/_/N-8w0fa?P=1y94rceZ1yr2ofqZ1yuqgh4Z1y92y2dZ1yzxtllZ1yzv8z0Z1y94rlyZ1yzu5bhZ1yzxtl9Z1yzxpklZ1yyabshZ1yzxqw6Z1y94rh6Z1y9iqlfZ1y94rr8Z1yyabcjZ1y9guvjZ1y94rgvZ1y94rhdZ1yzu5bwZ1y9guvlZ1yzxq81Z1z0x1exZ1z0x0msZ1z0x1eqZ1z0x0wrZ1z0x1fdZ1yzxdv5&Rl=8w0faZgjdhamZ1y94rd6Z1y93y46SGT&Ns=Pricing|0" H 1200 2450 50  0001 C CNN "Others"
-	1    1200 2450
+P 1050 2500
+F 0 "AE1501" H 1400 2600 50  0000 R CNN
+F 1 "SR4L034-R" H 1550 2500 50  0000 R CNN
+F 2 "dvk-mx8m-bsb:SR4L034-R" H 1050 2600 50  0001 C CNN
+F 3 "http://www.antenova-m2m.com/wp-content/uploads/2018/04/Inversa-SR4L034-PS-1.0.pdf?hsCtaTracking=a9dc692e-b13d-47be-9833-dc5991ce0b63%7Cad2a757a-c239-4a11-84f9-686c9a9d57a6" H 1050 2600 50  0001 C CNN
+F 4 "Antenova" H 1050 2500 50  0001 C CNN "MFG Name"
+F 5 "SR4L034-R" H 1050 2500 50  0001 C CNN "MFG Part Num"
+F 6 "SR4L034-R" H 1050 2500 50  0001 C CNN "Distrib PN"
+F 7 "https://www.arrow.com/en/products/sr4l034-r/antenova" H 1050 2500 50  0001 C CNN "Distrib Link"
+F 8 "-" H 1050 2500 50  0001 C CNN "Tolerance"
+F 9 "https://octopart.com/search?q=SR4L034-R&start=0" H 1050 2500 50  0001 C CNN "Others"
+	1    1050 2500
 	-1   0    0    -1
 $EndComp
@@
 L power:GND #PWR01501
 U 1 1 5B3865C4
-P 1100 2700
-F 0 "#PWR01501" H 1100 2450 50  0001 C CNN
-F 1 "GND" H 1100 2550 50  0000 C CNN
-F 2 "" H 1100 2700 50  0001 C CNN
-F 3 "" H 1100 2700 50  0001 C CNN
-	1    1100 2700
-	1    0    0    -1
-$EndComp
-Wire Wire Line
-	1100 2700 1100 2650
+P 950 2750
+F 0 "#PWR01501" H 950 2500 50  0001 C CNN
+F 1 "GND" H 950 2600 50  0000 C CNN
+F 2 "" H 950 2750 50  0001 C CNN
+F 3 "" H 950 2750 50  0001 C CNN
+	1    950  2750
+	1    0    0    -1
+$EndComp
+Wire Wire Line
+	950  2750 950  2700
 Wire Wire Line
 	3800 2650 3800 2750
@@
 	6400 3700 6450 3700
 Wire Wire Line
-	1200 2650 1200 2800
-Wire Wire Line
-	1200 2800 1350 2800
+	1050 2700 1050 2850
+Wire Wire Line
+	1050 2850 1200 2850
 $EndSCHEMATC

Commit message: Add pi-matching circuit to the baseband modem antenna's feedline
The return path for the antenna may have to have a 6.8nH Murata LQG15HN inductor installed on it (cutting the ground trace shorting the pads). The BoM was updated with the new components and everything was reannotated and updated (page 2's caps were out of order).
Parts:
- added C1501, C1504: NC, Capacitor_SMD:C_0402_1005Metric, symbol Device:C
- added L1501, L1502: NC, Inductor_SMD:L_0402_1005Metric, symbol Device:L
- renumbered C1501 to C1502, C1502 to C1503, C1503 to C1505, C1504 to C1506, C1505 to C1507, C1506 to C1508, C1507 to C1509, C1508 to C1510, C1509 to C1511, C1510 to C1512, C1511 to C1513, C1512 to C1514, C1513 to C1515, C1514 to C1516, C1515 to C1517, C1516 to C1518, C1517 to C1519, C1518 to C1520, C1519 to C1521, C1520 to C1522, C1521 to C1523, C1522 to C1524, C1523 to C1525, C1524 to C1526
Connections:
- wire segments 275 -> 294
